File: 555_toggle-switch/_autosave-555_toggle-switch.kicad_sch (KiCad schematic)
At the start: 10 parts, among them J1 3V3, J2 OUT, SW1 SW_Push, SW2 SW_SPDT, U1 NE555D

Commit message: .
Parts:
- C2: footprint Capacitor_THT:C_Radial_D5.0mm_H7.0mm_P2.00mm -> Capacitor_THT:CP_Radial_D5.0mm_P2.50mm
Changed lines of the file:
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@@
       (effects (font (size 1.27 1.27)) (justify left))
     )
-    (property "Footprint" "Capacitor_THT:C_Radial_D5.0mm_H7.0mm_P2.00mm" (at 177.4952 124.46 0)
+    (property "Footprint" "Capacitor_THT:CP_Radial_D5.0mm_P2.50mm" (at 177.4952 124.46 0)
       (effects (font (size 1.27 1.27)) hide)
     )
