File: esp32-wroom-adapter/esp32-wroom-adapter/esp32-wroom-adapter.kicad_pcb (KiCad board)
At the start: 2 copper layers, 97.5 x 97.5 mm, 14 parts, among them J1 PWR, J2 I2C, J3 I2C, J4 e-Paper, J6 UART, U1 ESP32-WROOM-32D, U2 LM78M05, U3 LM78M33

Commit message: .
Parts:
- removed U3: LM78M33, Package_TO_SOT_THT:TO-220-3_Vertical
- added H1: MountingHole, MountingHole:MountingHole_3mm_Pad_TopBottom, F.Cu at (114.9, 38.0)
- added H2: MountingHole, MountingHole:MountingHole_3mm_Pad_TopBottom, F.Cu at (114.9, 45.5)
- added H3: MountingHole, MountingHole:MountingHole_3mm_Pad_TopBottom, F.Cu at (114.9, 53.0)
- added H4: MountingHole, MountingHole:MountingHole_3mm_Pad_TopBottom, F.Cu at (114.9, 60.6)
- added U4: LD1117_TO220, Alexander Footprints Library:LD1117, F.Cu at (152.5, 47.5)
- moved C3 0.80 mm to (140.5, 50.2)
Routing:
- net +3V3: track 425.9 -> 422.3 mm
- net Net-(J1-Pin_1): track 20.8 -> 21.5 mm
Other:
- board text added: "GND"
