File: esp32-wroom-socket-v2/esp32-wroom-socket-v2.kicad_pcb (KiCad board)
At the start: 2 copper layers, 41.7 x 41.7 mm, 7 parts, among them U1 ESP32-WROOM-32D

Commit message: .
Parts:
- added D2: LED, Alexander Footprints Library:LED_2.5mm, F.Cu at (177.8, 99.1)
Connections:
- U1 pad 25: unconnected-(U1-IO0-Pad25) -> Net-(D2-A)
Routing:
- net unconnected-(U1-IO0-Pad25): track 7.28 -> 0.00 mm
- net Net-(D2-A): track 0.00 -> 7.28 mm
Other:
- board text added: "PRG"

Commit message: .
Routing:
- net GND: track 61.7 -> 65.2 mm
- net Net-(D1-K): track 2.54 -> 0.00 mm
- net Net-(D2-A): track 7.28 -> 9.07 mm
- net unconnected-(U1-SWP/SD3-Pad18): track 6.84 -> 6.00 mm
Changed lines of the file:
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@@
     (effects (font (size 0.5 0.5) (thickness 0.125)))
   )
+  (segment (start 153.924 80.65) (end 154.94 80.65) (width 0.25) (layer "F.Cu") (net 1))
   (segment (start 148.847251 80.01) (end 144.78 80.01) (width 0.25) (layer "F.Cu") (net 1))
-  (segment (start 156.85 80.65) (end 158.52 82.32) (width 0.25) (layer "F.Cu") (net 1))
-  (segment (start 158.52 92.94) (end 158.52 88.37) (width 0.25) (layer "F.Cu") (net 1))
+  (segment (start 151.27 80.65) (end 153.924 80.65) (width 0.25) (layer "F.Cu") (net 1))
   (segment (start 153.416 100.584) (end 152.146 101.854) (width 0.25) (layer "F.Cu") (net 1))
   (segment (start 149.487251 80.65) (end 148.847251 80.01) (width 0.25) (layer "F.Cu") (net 1))
+  (segment (start 155.05 88.37) (end 154.31 87.63) (width 0.25) (layer "F.Cu") (net 1))
   (segment (start 151.27 80.65) (end 149.487251 80.65) (width 0.25) (layer "F.Cu") (net 1))
-  (segment (start 158.52 82.32) (end 158.52 88.37) (width 0.25) (layer "F.Cu") (net 1))
-  (segment (start 154.31 98.41) (end 154.31 97.15) (width 0.25) (layer "F.Cu") (net 1))
   (segment (start 147.32 103.505) (end 147.955 104.14) (width 0.25) (layer "F.Cu") (net 1))
+  (segment (start 154.686 80.65) (end 168.77 80.65) (width 0.25) (layer "F.Cu") (net 1))
+  (segment (start 154.31 81.036) (end 153.924 80.65) (width 0.25) (layer "F.Cu") (net 1))
   (segment (start 154.31 100.452) (end 154.178 100.584) (width 0.25) (layer "F.Cu") (net 1))
-  (segment (start 154.31 97.15) (end 158.52 92.94) (width 0.25) (layer "F.Cu") (net 1))
+  (segment (start 154.31 98.41) (end 154.31 87.63) (width 0.25) (layer "F.Cu") (net 1))
+  (segment (start 158.52 88.37) (end 155.05 88.37) (width 0.25) (layer "F.Cu") (net 1))
   (segment (start 152.146 101.854) (end 149.86 104.14) (width 0.25) (layer "F.Cu") (net 1))
   (segment (start 147.32 101.6) (end 147.32 103.505) (width 0.25) (layer "F.Cu") (net 1))
   (segment (start 171.45 81.28) (end 172.72 81.28) (width 0.25) (layer "F.Cu") (net 1))
-  (segment (start 168.77 80.65) (end 160.19 80.65) (width 0.25) (layer "F.Cu") (net 1))
   (segment (start 147.955 104.14) (end 149.86 104.14) (width 0.25) (layer "F.Cu") (net 1))
-  (segment (start 160.19 80.65) (end 158.52 82.32) (width 0.25) (layer "F.Cu") (net 1))
-  (segment (start 151.27 80.65) (end 156.85 80.65) (width 0.25) (layer "F.Cu") (net 1))
   (segment (start 154.31 98.41) (end 154.31 100.452) (width 0.25) (layer "F.Cu") (net 1))
   (segment (start 170.82 80.65) (end 171.45 81.28) (width 0.25) (layer "F.Cu") (net 1))
   (segment (start 144.78 80.01) (end 144.78 81.28) (width 0.25) (layer "F.Cu") (net 1))
   (segment (start 154.178 100.584) (end 153.416 100.584) (width 0.25) (layer "F.Cu") (net 1))
+  (segment (start 154.31 87.63) (end 154.31 81.036) (width 0.25) (layer "F.Cu") (net 1))
   (segment (start 168.77 80.65) (end 170.82 80.65) (width 0.25) (layer "F.Cu") (net 1))
   (segment (start 147.32 99.06) (end 151.892 99.06) (width 0.25) (layer "F.Cu") (net 2))
@@
   (segment (start 156.85 100.326396) (end 154.94 102.236396) (width 0.25) (layer "F.Cu") (net 16))
   (segment (start 154.94 102.236396) (end 154.94 104.14) (width 0.25) (layer "F.Cu") (net 16))
-  (segment (start 158.12 98.41) (end 158.12 101.468) (width 0.25) (layer "F.Cu") (net 17))
-  (segment (start 156.464 103.124) (end 157.48 104.14) (width 0.25) (layer "F.Cu") (net 17))
-  (segment (start 158.12 101.468) (end 156.464 103.124) (width 0.25) (layer "F.Cu") (net 17))
+  (segment (start 158.12 98.41) (end 158.12 101.722) (width 0.25) (layer "F.Cu") (net 17))
+  (segment (start 157.48 102.362) (end 157.48 104.14) (width 0.25) (layer "F.Cu") (net 17))
+  (segment (start 158.12 101.722) (end 157.48 102.362) (width 0.25) (layer "F.Cu") (net 17))
   (segment (start 159.39 101.986) (end 160.02 102.616) (width 0.25) (layer "F.Cu") (net 18))
   (segment (start 159.39 98.41) (end 159.39 101.986) (width 0.25) (layer "F.Cu") (net 18))
@@
   (segment (start 170.82 81.92) (end 171.45 82.55) (width 0.25) (layer "F.Cu") (net 35))
   (segment (start 171.45 82.55) (end 173.99 82.55) (width 0.25) (layer "F.Cu") (net 35))
-  (segment (start 144.78 99.06) (end 144.78 101.6) (width 0.25) (layer "F.Cu") (net 36))
   (segment (start 168.77 97.16) (end 169.926 97.16) (width 0.25) (layer "F.Cu") (net 37))
   (segment (start 170.556 97.79) (end 173.99 97.79) (width 0.25) (layer "F.Cu") (net 37))
   (segment (start 169.926 97.16) (end 170.556 97.79) (width 0.25) (layer "F.Cu") (net 37))
   (segment (start 173.99 97.79) (end 175.26 96.52) (width 0.25) (layer "F.Cu") (net 37))
+  (segment (start 175.26 99.06) (end 173.99 97.79) (width 0.25) (layer "F.Cu") (net 37))
 )

Commit message: .
Routing:
- net Net-(D1-K): track 0.00 -> 40.6 mm
- net unconnected-(U1-IO15-Pad23): track 9.58 -> 10.8 mm
- net unconnected-(U1-SDI/SD1-Pad22): track 8.68 -> 9.57 mm
- net unconnected-(U1-IO35-Pad7): track 7.13 -> 7.88 mm
- net unconnected-(U1-SENSOR_VN-Pad5): track 7.13 -> 7.88 mm
- net unconnected-(U1-IO26-Pad11): track 7.28 -> 7.88 mm
- net unconnected-(U1-IO13-Pad16): track 7.64 -> 8.24 mm
- net GND: track 65.2 -> 65.7 mm
- net unconnected-(U1-IO33-Pad9): track 7.28 -> 7.88 mm
- net unconnected-(U1-IO14-Pad13): track 7.28 -> 7.88 mm
- net unconnected-(U1-SDO/SD0-Pad21): track 7.04 -> 7.64 mm

Commit message: GND
Routing:
- net GND: track 65.7 -> 40.6 mm, vias 0 -> 4
- net unconnected-(U1-SDI/SD1-Pad22): track 9.57 -> 0.00 mm
- net unconnected-(U1-SDO/SD0-Pad21): track 7.64 -> 0.00 mm
- net unconnected-(U1-SHD/SD2-Pad17): track 6.52 -> 0.00 mm
- net unconnected-(U1-SCK/CLK-Pad20): track 6.52 -> 0.00 mm
- net unconnected-(U1-SWP/SD3-Pad18): track 6.00 -> 0.00 mm
- net unconnected-(U1-SCS/CMD-Pad19): track 5.99 -> 0.00 mm
- net Net-(D1-K): track 40.6 -> 41.4 mm
- net unconnected-(U1-SENSOR_VN-Pad5): track 7.88 -> 7.15 mm
- net unconnected-(U1-IO35-Pad7): track 7.88 -> 7.18 mm
- net unconnected-(U1-IO26-Pad11): track 7.88 -> 7.28 mm
- net unconnected-(U1-IO33-Pad9): track 7.88 -> 7.28 mm
- net unconnected-(U1-IO14-Pad13): track 7.88 -> 7.28 mm
- added copper zone on B.Cu, net GND

Commit message: .
Parts:
- added SW1: PRG, Button_Switch_SMD:SW_SPST_EVQPE1, F.Cu at (170.0, 109.5)
Connections:
- U1 pad 25: Net-(D2-A) -> Net-(U1-IO0)
Routing:
- net Net-(U1-IO0): track 0.00 -> 25.0 mm
- net Net-(D2-A): track 9.07 -> 20.0 mm
Changed lines of the file:
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@@
   (net 36 "Net-(D1-K)")
   (net 37 "Net-(D2-A)")
+  (net 38 "Net-(U1-IO0)")
   (footprint "Alexander Footprints Library:R_2.5mm" (layer "F.Cu")
     (at 147.32 104.14)
@@
       (net 23 "unconnected-(U1-IO2-Pad24)") (pinfunction "IO2") (pintype "bidirectional"))
     (pad "25" smd rect (at 8.75 8.26) (size 1.5 0.9) (layers "F.Cu" "F.Paste" "F.Mask")
-      (net 37 "Net-(D2-A)") (pinfunction "IO0") (pintype "bidirectional"))
+      (net 38 "Net-(U1-IO0)") (pinfunction "IO0") (pintype "bidirectional"))
     (pad "25" thru_hole circle (at 15.24 7.62) (size 1.524 1.524) (drill 0.762) (layers "*.Cu" "*.Mask")
-      (net 37 "Net-(D2-A)") (pinfunction "IO0") (pintype "bidirectional"))
+      (net 38 "Net-(U1-IO0)") (pinfunction "IO0") (pintype "bidirectional"))
     (pad "26" smd rect (at 8.75 6.99) (size 1.5 0.9) (layers "F.Cu" "F.Paste" "F.Mask")
       (net 24 "unconnected-(U1-IO4-Pad26)") (pinfunction "IO4") (pintype "bidirectional"))
@@
     )
   )
+  (footprint "Button_Switch_SMD:SW_SPST_EVQPE1" (layer "F.Cu")
+    (at 170 109.5 180)
+    (descr "Light Touch Switch, https://industrial.panasonic.com/cdbs/www-data/pdf/ATK0000/ATK0000CE7.pdf")
+    (property "Sheetfile" "esp32-wroom-socket-v2.kicad_sch")
+    (property "Sheetname" "")
+    (property "ki_description" "Push button switch, generic, two pins")
+    (property "ki_keywords" "switch normally-open pushbutton push-button")
+    (attr smd)
+    (fp_text reference "SW1" (at 0 -2.65) (layer "F.SilkS")
+        (effects (font (size 1 1) (thickness 0.15)))
+    )
+    (fp_text value "PRG" (at 0 3) (layer "F.Fab")
+        (effects (font (size 1 1) (thickness 0.15)))
+    )
+    (fp_text user "${REFERENCE}" (at 0 -2.65) (layer "F.Fab")
+        (effects (font (size 1 1) (thickness 0.15)))
+    )
+    (fp_line (start -3.1 -1.85) (end -3.1 -1.2)
+      (stroke (width 0.12) (type solid)) (layer "F.SilkS"))
+    (fp_line (start -3.1 1.2) (end -3.1 1.85)
+      (stroke (width 0.12) (type solid)) (layer "F.SilkS"))
+    (fp_line (start -3.1 1.85) (end 3.1 1.85)
+      (stroke (width 0.12) (type solid)) (layer "F.SilkS"))
+    (fp_line (start 3.1 -1.85) (end -3.1 -1.85)
+      (stroke (width 0.12) (type solid)) (layer "F.SilkS"))
+    (fp_line (start 3.1 -1.85) (end 3.1 -1.2)
+      (stroke (width 0.12) (type solid)) (layer "F.SilkS"))
+    (fp_line (start 3.1 1.85) (end 3.1 1.2)
+      (stroke (width 0.12) (type solid)) (layer "F.SilkS"))
+    (fp_line (start -3.95 -2) (end 3.95 -2)
+      (stroke (width 0.05) (type solid)) (layer "F.CrtYd"))
+    (fp_line (start -3.95 2) (end -3.95 -2)
+      (stroke (width 0.05) (type solid)) (layer "F.CrtYd"))
+    (fp_line (start 3.95 -2) (end 3.95 2)
+      (stroke (width 0.05) (type solid)) (layer "F.CrtYd"))
+    (fp_line (start 3.95 2) (end -3.95 2)
+      (stroke (width 0.05) (type solid)) (layer "F.CrtYd"))
+    (fp_line (start -3 -1.75) (end 3 -1.75)
+      (stroke (width 0.1) (type solid)) (layer "F.Fab"))
+    (fp_line (start -3 1.75) (end -3 -1.75)
+      (stroke (width 0.1) (type solid)) (layer "F.Fab"))
+    (fp_line (start -1.4 -0.7) (end 1.4 -0.7)
+      (stroke (width 0.1) (type solid)) (layer "F.Fab"))
+    (fp_line (start -1.4 0.7) (end -1.4 -0.7)
+      (stroke (width 0.1) (type solid)) (layer "F.Fab"))
+    (fp_line (start 1.4 -0.7) (end 1.4 0.7)
+      (stroke (width 0.1) (type solid)) (layer "F.Fab"))
+    (fp_line (start 1.4 0.7) (end -1.4 0.7)
+      (stroke (width 0.1) (type solid)) (layer "F.Fab"))
+    (fp_line (start 3 -1.75) (end 3 1.75)
+      (stroke (width 0.1) (type solid)) (layer "F.Fab"))
+    (fp_line (start 3 1.75) (end -3 1.75)
+      (stroke (width 0.1) (type solid)) (layer "F.Fab"))
+    (pad "1" smd rect (at -2.7 0 180) (size 2 1.6) (layers "F.Cu" "F.Paste" "F.Mask")
+      (net 38 "Net-(U1-IO0)") (pinfunction "1") (pintype "passive"))
+    (pad "2" smd rect (at 2.7 0 180) (size 2 1.6) (layers "F.Cu" "F.Paste" "F.Mask")
+      (net 37 "Net-(D2-A)") (pinfunction "2") (pintype "passive"))
+    (model "${KICAD6_3DMODEL_DIR}/Button_Switch_SMD.3dshapes/SW_SPST_EVQPE1.wrl"
+      (offset (xyz 0 0 0))
+      (scale (xyz 1 1 1))
+      (rotate (xyz 0 0 0))
+    )
+  )
   (gr_line (start 177.8 113.538) (end 142.24 113.538)
     (stroke (width 0.1) (type default)) (layer "Edge.Cuts"))
@@
     (effects (font (size 0.5 0.5) (thickness 0.125)))
   )
-  (gr_text "PRG" (at 177.7746 102.0064 90) (layer "F.SilkS" knockout)
+  (gr_text "PRG" (at 165.1 111.76 90) (layer "F.SilkS" knockout)
     (effects (font (size 1 1) (thickness 0.2) bold) (justify left bottom))
   )
@@
   (segment (start 170.82 81.92) (end 171.45 82.55) (width 0.25) (layer "F.Cu") (net 35))
   (segment (start 171.45 82.55) (end 173.99 82.55) (width 0.25) (layer "F.Cu") (net 35))
-  (segment (start 144.78 99.06) (end 144.78 101.6) (width 0.25) (layer "F.Cu") (net 36))
+  (segment (start 144.78 101.6) (end 144.78 99.06) (width 0.25) (layer "F.Cu") (net 36))
   (segment (start 174 106.5) (end 146 106.5) (width 0.25) (layer "B.Cu") (net 36))
   (segment (start 144.78 105.28) (end 144.78 101.6) (width 0.25) (layer "B.Cu") (net 36))
@@
   (segment (start 175.26 101.6) (end 175.26 105.24) (width 0.25) (layer "B.Cu") (net 36))
   (segment (start 146 106.5) (end 144.78 105.28) (width 0.25) (layer "B.Cu") (net 36))
-  (segment (start 168.77 97.16) (end 169.926 97.16) (width 0.25) (layer "F.Cu") (net 37))
-  (segment (start 173.99 97.79) (end 175.26 99.06) (width 0.25) (layer "F.Cu") (net 37))
-  (segment (start 170.556 97.79) (end 173.99 97.79) (width 0.25) (layer "F.Cu") (net 37))
-  (segment (start 169.926 97.16) (end 170.556 97.79) (width 0.25) (layer "F.Cu") (net 37))
-  (segment (start 173.99 97.79) (end 175.26 96.52) (width 0.25) (layer "F.Cu") (net 37))
+  (segment (start 175.25 107.75) (end 177 106) (width 0.25) (layer "F.Cu") (net 37))
+  (segment (start 177 106) (end 177 100) (width 0.25) (layer "F.Cu") (net 37))
+  (segment (start 167.3 109.5) (end 167.3 108.2) (width 0.25) (layer "F.Cu") (net 37))
+  (segment (start 167.3 108.2) (end 167.75 107.75) (width 0.25) (layer "F.Cu") (net 37))
+  (segment (start 167.75 107.75) (end 175.25 107.75) (width 0.25) (layer "F.Cu") (net 37))
+  (segment (start 177 100) (end 176.06 99.06) (width 0.25) (layer "F.Cu") (net 37))
+  (segment (start 176.06 99.06) (end 175.26 99.06) (width 0.25) (layer "F.Cu") (net 37))
+  (segment (start 168.77 97.16) (end 169.926 97.16) (width 0.25) (layer "F.Cu") (net 38))
+  (segment (start 170.556 97.79) (end 173.99 97.79) (width 0.25) (layer "F.Cu") (net 38))
+  (segment (start 174.25 109.5) (end 177.5 106.25) (width 0.25) (layer "F.Cu") (net 38))
+  (segment (start 169.926 97.16) (end 170.556 97.79) (width 0.25) (layer "F.Cu") (net 38))
+  (segment (start 177.5 106.25) (end 177.5 97.25) (width 0.25) (layer "F.Cu") (net 38))
+  (segment (start 176.77 96.52) (end 175.26 96.52) (width 0.25) (layer "F.Cu") (net 38))
+  (segment (start 173.99 97.79) (end 175.26 96.52) (width 0.25) (layer "F.Cu") (net 38))
+  (segment (start 172.7 109.5) (end 174.25 109.5) (width 0.25) (layer "F.Cu") (net 38))
+  (segment (start 177.5 97.25) (end 176.77 96.52) (width 0.25) (layer "F.Cu") (net 38))
   (zone (net 1) (net_name "GND") (layer "B.Cu") (name "GND") (hatch edge 0.5)
     (connect_pads (clearance 0.5))
