File: esp32-node-box-40x65/esp32-node-board-40x65/_autosave-esp32-node-board-40x65.kicad_pcb (KiCad board)
At the start: 2 copper layers, 65.2 x 40 mm, 20 parts, among them J10 Conn_01x02_Socket, J2 PWD, J3 UART, J4 I2C, J5 DAC_Socket, J6 ADC, J7 GPIO, J8 Conn_01x02_Socket, J9 Conn_01x02_Socket, U1 MAX1726EUK33, U3 ULN2003, U4 L7805

Commit message: .
Routing:
- net /OUT1: track 58.5 -> 42.9 mm
Changed lines of the file:
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@@
 	)
 	(segment
-		(start 135.25 78.5)
-		(end 100 78.5)
+		(start 133.16 63.25)
+		(end 115 63.25)
 		(width 0.25)
 		(layer "F.Cu")
@@
 	)
 	(segment
-		(start 100 78.5)
-		(end 99.06 77.56)
+		(start 134.54 61.87)
+		(end 133.16 63.25)
 		(width 0.25)
 		(layer "F.Cu")
@@
 	)
 	(segment
-		(start 136.5 63.7)
-		(end 136.5 77.25)
+		(start 115 63.25)
+		(end 104.59 73.66)
 		(width 0.25)
 		(layer "F.Cu")
@@
 	)
 	(segment
-		(start 99.06 77.56)
-		(end 99.06 76.2)
+		(start 104.59 73.66)
+		(end 99.06 73.66)
 		(width 0.25)
 		(layer "F.Cu")
@@
 	)
 	(segment
-		(start 136.5 77.25)
-		(end 135.25 78.5)
-		(width 0.25)
-		(layer "F.Cu")
-		(net 35)
-	)
-	(segment
-		(start 134.62 61.82)
-		(end 136.5 63.7)
-		(width 0.25)
-		(layer "F.Cu")
-		(net 35)
-	)
-	(segment
-		(start 112.9284 51.75)
-		(end 111.6784 50.5)
+		(start 110.0892 50.5)
+		(end 105.3 50.5)
 		(width 0.25)
 		(layer "F.Cu")
@@
 	)
 	(segment
-		(start 111.6784 50.5)
-		(end 105.3 50.5)
+		(start 112.9284 51.75)
+		(end 111.3392 51.75)
 		(width 0.25)
 		(layer "F.Cu")
+		(net 36)
+	)
+	(segment
+		(start 111.3392 51.75)
+		(end 110.0892 50.5)
+		(width 0.25)
+		(layer "F.Cu")
