File: esp32-node-box-40x65/esp32-node-board-40x65/_autosave-esp32-node-board-40x65.kicad_sch (KiCad schematic)
At the start: 29 parts, among them J10 Conn_01x02_Socket, J12 Conn_01x02_Socket, J13 Conn_01x06_Socket, J2 PWD, J3 UART, J4 I2C, J5 DAC_Socket, J6 ADC, J7 GPIO, J8 Conn_01x02_Socket, J9 Conn_01x02_Socket, Q1 NPN, Q2 NPN, SW1 SW_Push, U1 MAX1726EUK33, U2 4N35, U3 ULN2003, U4 L7805

Commit message: .
Parts:
- Q1, Q2: footprint Package_TO_SOT_THT:TO-3 -> Package_TO_SOT_THT:TO-92
Changed lines of the file:
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@@
 			)
 		)
-		(property "Footprint" "Package_TO_SOT_THT:TO-3"
+		(property "Footprint" "Package_TO_SOT_THT:TO-92"
 			(at 215.9 160.02 0)
 			(effects
@@
 			)
 		)
-		(property "Footprint" "Package_TO_SOT_THT:TO-3"
+		(property "Footprint" "Package_TO_SOT_THT:TO-92"
 			(at 69.85 172.72 0)
 			(effects
