File: esp32-node-box-40x65/esp32-node-board-40x65/esp32-node-board-40x65.kicad_pcb (KiCad board)
At the start: 2 copper layers, 65.2 x 40 mm, 23 parts, among them J10 Conn_01x02_Socket, J12 Conn_01x02_Socket, J2 PWD, J3 UART, J4 I2C, J5 DAC_Socket, J6 ADC, J7 GPIO, J8 Conn_01x02_Socket, J9 Conn_01x02_Socket, U1 MAX1726EUK33, U2 4N35, U3 ULN2003, U4 L7805

Commit message: .
Parts:
- added J13: Conn_01x06_Socket, Connector_PinSocket_2.54mm:PinSocket_1x06_P2.54mm_Vertical, F.Cu at (128.3, 49.5)
- added Q1: NPN, Package_TO_SOT_THT:TO-92, F.Cu at (120.8, 54.6)
- added Q2: NPN, Package_TO_SOT_THT:TO-92, F.Cu at (133.4, 68.2)
- added R3: 10K, Resistor_SMD:R_1210_3225Metric_Pad1.30x2.65mm_HandSolder, F.Cu at (123.8, 49.4)
- added R4: 10K, Resistor_SMD:R_1210_3225Metric_Pad1.30x2.65mm_HandSolder, F.Cu at (116.8, 54.0)
- moved C2 7.25 mm to (132.0, 43.6)
- moved R1 0.65 mm to (111.6, 52.8)
Routing:
- net /DTR: track 0.00 -> 17.0 mm
- net /TXD: track 6.00 -> 13.5 mm
- net /RXD: track 9.41 -> 14.3 mm
- net /ADC2_CH0: track 12.6 -> 15.4 mm
- net /OUT1: track 48.1 -> 45.4 mm

Commit message: .
Parts:
- removed J10: Conn_01x02_Socket, Alexander Footprints Library:Conn_Terminal_5mm
- moved C2 31.9 mm to (100.2, 46.0), turned to 90 degrees
- moved R4 17.0 mm to (131.1, 44.9)
- moved R3 11.9 mm to (134.8, 44.9), turned to 90 degrees
- moved Q1 11.8 mm to (124.7, 43.5), turned to -90 degrees
- moved U4 11.0 mm to (82.9, 50.1), turned to -90 degrees
- moved J2 2.50 mm to (88.5, 43.2), turned to 0 degrees
- moved C3 2.07 mm to (89.8, 54.6), turned to 90 degrees
Routing:
- net Net-(Q2-B): track 0.00 -> 38.1 mm, vias 0 -> 1
- net /RTS: track 0.00 -> 30.5 mm
- net /DTR: track 17.0 -> 7.57 mm
- net /VDC: track 30.7 -> 39.4 mm
- net Net-(Q1-B): track 0.00 -> 5.72 mm
- net +3V3: track 66.3 -> 71.8 mm
- net +5V: track 18.1 -> 13.5 mm
- net /BOOT: track 0.00 -> 4.26 mm

Commit message: .
Parts:
- moved C3 9.95 mm to (94.8, 46.0)
- moved R2 0.65 mm to (111.6, 60.2)
Connections:
- J13 pad 1: GND -> +3V3
- J13 pad 2: +3V3 -> GND
Routing:
- net /EN: track 9.26 -> 33.3 mm
- net /DTR: track 7.57 -> 27.4 mm, vias 0 -> 1
- net +5V: track 13.5 -> 30.5 mm
- net +3V3: track 71.8 -> 86.3 mm
- net /OUT1: track 45.4 -> 47.6 mm
- net /V1+: track 29.6 -> 28.7 mm
- net /ADC2_CH0: track 15.4 -> 14.8 mm
- net Net-(Q2-B): track 38.1 -> 38.6 mm
- net /VDC: track 39.4 -> 38.9 mm

Commit message: .
Parts:
- Q1, Q2: footprint Package_TO_SOT_THT:TO-92 -> Package_TO_SOT_THT:TO-92_Inline_W4.0mm_Horizontal_FlatSideDown
- moved Q1 2.24 mm to (122.4, 43.6), turned to 0 degrees
- moved Q2 1.19 mm to (133.7, 67.0), turned to -90 degrees
Routing:
- net /DTR: track 27.4 -> 31.1 mm, vias 1 -> 3
- net Net-(Q1-B): track 5.72 -> 8.65 mm
- net /EN: track 33.3 -> 30.7 mm
- net Net-(Q2-B): track 38.6 -> 39.6 mm
- net /BOOT: track 4.26 -> 3.37 mm

Commit message: .
Parts:
- moved U1 1.40 mm to (115.0, 45.5)
- moved J5 1.26 mm to (100.3, 50.8)
- moved R2 1.12 mm to (110.5, 60.2)
- moved U4 0.54 mm to (82.9, 49.5)
- moved Q1 0.52 mm to (121.9, 43.6)
Routing:
- net Net-(R2-Pad2): track 4.96 -> 6.75 mm
- net /GPIO27: track 5.68 -> 3.93 mm
- net /DAC1: track 13.8 -> 12.2 mm
- net /VDC: track 38.9 -> 37.5 mm
- net /DAC2: track 11.6 -> 11.0 mm

Commit message: traces
Parts:
- moved C2 0.12 mm to (100.3, 46.0)
Routing:
- net +3V3: track 85.8 -> 130.8 mm
- net /VDC: track 37.5 -> 67.9 mm
- net +5V: track 30.5 -> 49.7 mm
- net /V1-: track 27.6 -> 31.4 mm
- net /V1+: track 28.7 -> 32.0 mm
- net /DTR: track 31.1 -> 31.8 mm
- net /DAC1: track 12.2 -> 12.9 mm

Commit message: traces
Routing:
- net +3V3: track 130.8 -> 141.1 mm
- net Net-(Q2-B): track 39.6 -> 38.9 mm

Commit message: .
Parts:
- J6: value ADC -> SOURCE
- moved J6 23.6 mm to (102.9, 76.1)
- moved J12 8.85 mm to (115.6, 76.5)
Connections:
- J1 pad 7: /GPIO35 -> /OUT5
- J1 pad 9: /GPIO33 -> /OUT4
- J6 pad 1: /ADC2_CH3 -> /SOURCE3
- J6 pad 2: /ADC2_CH0 -> /SOURCE4
- J6 pad 3: /ADC2_CH2 -> /SOURCE5
- J6 pad 4: unconnected-(J6-Pin_4-Pad4) -> GND
- J9 pad 2: /SOURCE3 -> GND
- U3 pad 10: /SOURCE3 -> /SOURCE5
- U3 pad 11: /SOURCE3 -> /SOURCE4
- U3 pad 6: /OUT3 -> /OUT4
- U3 pad 7: /OUT3 -> /OUT5
Routing:
- net /V1-: track 31.4 -> 2.72 mm
- net /V1+: track 32.0 -> 5.30 mm
- net /SOURCE3: track 16.3 -> 0.00 mm
- net /OUT4: track 0.00 -> 8.65 mm
- net /OUT5: track 0.00 -> 8.37 mm
- net /OUT3: track 10.9 -> 5.78 mm
- net /DAC1: track 12.9 -> 15.1 mm
- net /DAC2: track 11.0 -> 12.4 mm
- net Net-(Q1-B): track 8.86 -> 9.43 mm
- net GND: track 0.00 -> 0.55 mm
