File: esp32-node-box-40x65/esp32-node-board-40x65/esp32-node-board-40x65.kicad_sch (KiCad schematic)
At the start: 29 parts, among them J10 ADC, J12 Conn_01x02_Socket, J13 Conn_01x06_Socket, J2 PWD, J3 UART, J4 I2C, J5 DAC_Socket, J6 SOURCE, J7 GPIO, J8 Conn_01x02_Socket, J9 Conn_01x02_Socket, Q1 NPN, Q2 NPN, SW1 SW_Push, U1 MAX1726EUK33, U2 4N35, U3 ULN2003, U4 L7805

Commit message: 595
Parts:
- added D1, D2: LED, LED_SMD:LED_1210_3225Metric_Pad1.42x2.65mm_HandSolder, symbol Device:LED
- added U5: 74LS595, Package_DIP:DIP-16_W7.62mm, symbol 74xx:74LS595
Connections:
- net +3V3: now also D1.2 (A)
- net +5V: now also U5.16 (VCC)
- net GND: now also D1.1 (K), D2.1 (K), U5.8 (GND)
- net GPIO34: now also D2.2 (A)

Commit message: .
Parts:
- added D3: 1N4007, symbol Device:D
- added J11: Conn_01x02_Socket, Connector_PinSocket_2.54mm:PinSocket_1x02_P2.54mm_Vertical, symbol Connector:Conn_01x02_Socket
- added Q3: 2N3904, Package_TO_SOT_THT:TO-92, symbol Simulation_SPICE:NPN
- added R5: 470, Resistor_SMD:R_1210_3225Metric_Pad1.30x2.65mm_HandSolder, symbol Device:R
- added R6: 120, Resistor_SMD:R_1210_3225Metric_Pad1.30x2.65mm_HandSolder, symbol Device:R
- added U6: PC817, Package_DIP:DIP-4_W7.62mm, symbol Isolator:PC817
Connections:
- net +5V: now also D3.1 (K), J11.1 (Pin_1), U6.4
- net GND: now also Q3.3 (E), U6.2
- net GPIO13: now also R5.2
- new net: D3.2 (A), J11.2 (Pin_2), Q3.1 (C)
- new net: R5.1, U6.1
- new net: Q3.2 (B), R6.1
- new net: R6.2, U6.3
Other:
- moved on the sheet: H1, H2, H4

Commit message: .
Connections:
- net OUT1: no longer U3.1 (I1), U3.2 (I2)
- net OUT2: no longer U3.3 (I3), U3.4 (I4)
- net OUT3: no longer U3.5 (I5)
- net OUT4: no longer U3.6 (I6)
- net OUT5: no longer U3.7 (I7)
- net SOURCE1: now also U3.12 (O5), U3.13 (O4); no longer U3.15 (O2), U3.16 (O1)
- net SOURCE2: now also U3.10 (O7), U3.11 (O6); no longer U3.13 (O4), U3.14 (O3)
- net SOURCE3: now also J6.1 (Pin_1); no longer J6.3 (Pin_3), U3.12 (O5)
- net SOURCE4: no longer U3.11 (O6)
- net SOURCE5: now also J6.3 (Pin_3); no longer J6.1 (Pin_1), U3.10 (O7)
- net I7: now reaches U5.1 (QB)
- net I7: now also U3.6 (I6), U3.7 (I7), U5.2 (QC)
- net I6: now reaches U5.3 (QD)
- net I5: now reaches U5.4 (QE)
- net I5: now also U3.4 (I4), U3.5 (I5), U5.5 (QF)
- net I3: now reaches U5.6 (QG)
- net I3: now also U3.3 (I3)
- net I1: now reaches U5.7 (QH)
- net I1: now also U3.2 (I2)
Other:
- moved on the sheet: U3

Commit message: .
Parts:
- R1, R5, R6: footprint Resistor_SMD:R_1210_3225Metric_Pad1.30x2.65mm_HandSolder -> Resistor_SMD:R_1206_3216Metric_Pad1.30x1.75mm_HandSolder
Changed lines of the file:
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@@
 			)
 		)
-		(property "Footprint" "Resistor_SMD:R_1210_3225Metric_Pad1.30x2.65mm_HandSolder"
+		(property "Footprint" "Resistor_SMD:R_1206_3216Metric_Pad1.30x1.75mm_HandSolder"
 			(at 201.93 32.512 90)
 			(effects
@@
 			)
 		)
-		(property "Footprint" "Resistor_SMD:R_1210_3225Metric_Pad1.30x2.65mm_HandSolder"
+		(property "Footprint" "Resistor_SMD:R_1206_3216Metric_Pad1.30x1.75mm_HandSolder"
 			(at 229.87 37.592 90)
 			(effects
@@
 			)
 		)
-		(property "Footprint" "Resistor_SMD:R_1210_3225Metric_Pad1.30x2.65mm_HandSolder"
+		(property "Footprint" "Resistor_SMD:R_1206_3216Metric_Pad1.30x1.75mm_HandSolder"
 			(at 144.272 45.72 90)
 			(effects

Commit message: smd
Other:
- added sheet Extras (untitled.kicad_sch)
- moved on the sheet: J12, J13, Q1, Q2, R2, R3, R4, SW1, U2

Commit message: sensor
Parts:
- added U7: BME(P)280, Alexander Footprint Library:BME280_BMP280_I2C, symbol Alexander Symbol Library:BME(P)280
Connections:
- net +3V3: now also U7.1 (VDD)
- net GND: now also U7.2 (GND)
Changed lines of the file:
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@@
 	(wire
 		(pts
+			(xy 256.54 67.31) (xy 256.54 72.39)
+		)
+		(stroke
+			(width 0)
+			(type default)
+		)
+	)
+	(wire
+		(pts
 			(xy 220.98 129.54) (xy 223.52 129.54)
 		)
@@
 	(wire
 		(pts
+			(xy 256.54 87.63) (xy 256.54 91.44)
+		)
+		(stroke
+			(width 0)
+			(type default)
+		)
+	)
+	(wire
+		(pts
 			(xy 58.42 100.33) (xy 50.8 100.33)
 		)
@@
 	(symbol
 		(lib_id "power:+3V3")
+		(at 256.54 67.31 0)
+		(unit 1)
+		(exclude_from_sim no)
+		(in_bom yes)
+		(on_board yes)
+		(dnp no)
+		(fields_autoplaced yes)
+		(property "Reference" "#PWR022"
+			(at 256.54 71.12 0)
+			(effects
+				(font
+					(size 1.27 1.27)
+				)
+				(hide yes)
+			)
+		)
+		(property "Value" "+3V3"
+			(at 256.54 62.23 0)
+			(effects
+				(font
+					(size 1.27 1.27)
+				)
+			)
+		)
+		(property "Footprint" ""
+			(at 256.54 67.31 0)
+			(effects
+				(font
+					(size 1.27 1.27)
+				)
+				(hide yes)
+			)
+		)
+		(property "Datasheet" ""
+			(at 256.54 67.31 0)
+			(effects
+				(font
+					(size 1.27 1.27)
+				)
+				(hide yes)
+			)
+		)
+		(property "Description" ""
+			(at 256.54 67.31 0)
+			(effects
+				(font
+					(size 1.27 1.27)
+				)
+				(hide yes)
+			)
+		)
+		(pin "1"
+		)
+		(instances
+			(project "esp32-node-board-40x65"
+				(path "/5f5eb0ac-ab9b-41ab-8d2f-875870c41abc"
+					(reference "#PWR022")
+					(unit 1)
+				)
+			)
+		)
+	)
+	(symbol
+		(lib_id "power:+3V3")
 		(at 34.29 152.4 90)
 		(unit 1)
@@
 	)
 	(symbol
+		(lib_id "Alexander Symbol Library:BME(P)280")
+		(at 257.81 82.55 0)
+		(unit 1)
+		(exclude_from_sim no)
+		(in_bom yes)
+		(on_board yes)
+		(dnp no)
+		(fields_autoplaced yes)
+		(property "Reference" "U7"
+			(at 264.16 78.7399 0)
+			(effects
+				(font
+					(size 1.27 1.27)
+				)
+				(justify left)
+			)
+		)
+		(property "Value" "BME(P)280"
+			(at 264.16 81.2799 0)
+			(effects
+				(font
+					(size 1.27 1.27)
+				)
+				(justify left)
+			)
+		)
+		(property "Footprint" "Alexander Footprint Library:BME280_BMP280_I2C"
+			(at 257.81 100.33 0)
+			(effects
+				(font
+					(size 1.27 1.27)
+				)
+				(hide yes)
+			)
+		)
+		(property "Datasheet" ""
+			(at 257.81 82.55 0)
+			(effects
+				(font
+					(size 1.27 1.27)
+				)
+				(hide yes)
+			)
+		)
+		(property "Description" "Absolute Barometric Pressure Sensor"
+			(at 257.81 103.632 0)
+			(effects
+				(font
+					(size 1.27 1.27)
+				)
+				(hide yes)
+			)
+		)
+		(pin "1"
+		)
+		(pin "3"
+		)
+		(pin "4"
+		)
+		(pin "2"
+		)
+		(instances
+			(project "esp32-node-board-40x65"
+				(path "/5f5eb0ac-ab9b-41ab-8d2f-875870c41abc"
+					(reference "U7")
+					(unit 1)
+				)
+			)
+		)
+	)
+	(symbol
 		(lib_id "Device:LED")
 		(at 114.3 46.99 90)
@@
 		(exclude_from_sim no)
 		(in_bom yes)
-		(on_board yes)
+		(on_board no)
 		(dnp no)
 		(fields_autoplaced yes)
@@
 		(exclude_from_sim no)
 		(in_bom yes)
-		(on_board yes)
+		(on_board no)
 		(dnp no)
 		(fields_autoplaced yes)
@@
 		(exclude_from_sim no)
 		(in_bom yes)
-		(on_board yes)
+		(on_board no)
 		(dnp no)
 		(fields_autoplaced yes)
@@
 		(exclude_from_sim no)
 		(in_bom yes)
-		(on_board yes)
+		(on_board no)
 		(dnp no)
 		(fields_autoplaced yes)
@@
 		(exclude_from_sim no)
 		(in_bom yes)
-		(on_board yes)
+		(on_board no)
 		(dnp no)
 		(fields_autoplaced yes)
@@
 					(unit 1)
 				)
+			)
+		)
+	)
+	(symbol
+		(lib_name "GND_5")
+		(lib_id "power:GND")
+		(at 256.54 91.44 0)
+		(unit 1)
+		(exclude_from_sim no)
+		(in_bom yes)
+		(on_board yes)
+		(dnp no)
+		(fields_autoplaced yes)
+		(property "Reference" "#PWR021"
+			(at 256.54 97.79 0)
+			(effects
+				(font
+					(size 1.27 1.27)
+				)
+				(hide yes)
+			)
+		)
+		(property "Value" "GND"
+			(at 256.54 96.52 0)
+			(effects
+				(font
+					(size 1.27 1.27)
+				)
+			)
+		)
+		(property "Footprint" ""
+			(at 256.54 91.44 0)
+			(effects
+				(font
+					(size 1.27 1.27)
+				)
+				(hide yes)
+			)
+		)
+		(property "Datasheet" ""
+			(at 256.54 91.44 0)
+			(effects
+				(font
+					(size 1.27 1.27)
+				)
+				(hide yes)
+			)
+		)
+		(property "Description" "Power symbol creates a global label with name \"GND\" , ground"
+			(at 256.54 91.44 0)
+			(effects
+				(font
+					(size 1.27 1.27)
+				)
+				(hide yes)
+			)
+		)
+		(pin "1"
+		)
+		(instances
+			(project "esp32-node-board-40x65"
+				(path "/5f5eb0ac-ab9b-41ab-8d2f-875870c41abc"
+					(reference "#PWR021")
+					(unit 1)
+				)

Commit message: BMP280
Connections:
- net SCL: now also U7.3 (SCL)
- net SDA: now also U7.4 (SDA)
Changed lines of the file:
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@@
 	(wire
 		(pts
+			(xy 241.3 81.28) (xy 247.65 81.28)
+		)
+		(stroke
+			(width 0)
+			(type default)
+		)
+	)
+	(wire
+		(pts
 			(xy 261.62 129.54) (xy 264.16 129.54)
 		)
@@
 	(wire
 		(pts
+			(xy 241.3 78.74) (xy 247.65 78.74)
+		)
+		(stroke
+			(width 0)
+			(type default)
+		)
+	)
+	(wire
+		(pts
 			(xy 180.34 62.23) (xy 185.42 62.23)
 		)
@@
 		)
 	)
+	(label "SCL"
+		(at 241.3 78.74 0)
+		(fields_autoplaced yes)
+		(effects
+			(font
+				(size 1.27 1.27)
+			)
+			(justify left bottom)
+		)
+	)
 	(label "SD_CLK"
 		(at 146.05 102.87 0)
@@
 		)
 	)
+	(label "SDA"
+		(at 241.3 81.28 0)
+		(fields_autoplaced yes)
+		(effects
+			(font
+				(size 1.27 1.27)
+			)
+			(justify left bottom)
+		)
+	)
 	(label "DAC1"
 		(at 185.42 97.79 0)
@@
 				(font
 					(size 1.27 1.27)
+					(bold yes)
 				)
 			)
@@
 		(exclude_from_sim no)
 		(in_bom yes)
-		(on_board yes)
+		(on_board no)
 		(dnp no)
 		(property "Reference" "J13"

Commit message: gpio
Parts:
- removed J7: GPIO, Connector_PinSocket_2.54mm:PinSocket_1x05_P2.54mm_Vertical, symbol Connector:Conn_01x05_Pin
- added J14: GPIO, Alexander Footprint Library:CONN_2x3, symbol Alexander_Library_Symbols:Conn_2x3
Connections:
- net GPIO17: now also J14.6
- net GPIO18: now also J14.2
- net GPIO19: now also J14.5
- net GPIO23: now also J14.4
- net GPIO5: now also J14.1
- net I1: now also U5.1 (QB); no longer U5.7 (QH)
- net I6: now also U3.1 (I1), U5.7 (QH); no longer U5.3 (QD)
- net I7: now also U5.3 (QD); no longer U5.1 (QB)
- net SOURCE3: now also U3.16 (O1)
- net SOURCE4: now also U3.15 (O2)
- net SOURCE5: now also U3.14 (O3)
Other:
- moved on the sheet: U7
