File: esp32-wroom-board/esp32-wroom-board/esp32-wroom-board.kicad_sch (KiCad schematic)
At the start: 75 parts, among them J10 Conn_01x04_Socket, J11 Conn_01x04_Socket, J12 Conn_01x04_Socket, J13 Conn_01x04_Socket, J14 I1, J15 I2, J16 I3, J17 I3, J18 I3, J19 I3, J2 I2C, J20 I3, J21 I3, J22 USB-C, J3 I2C, J4 e-Paper, J6 UART, J9 Conn_01x04_Socket, K1 Relay_DPDT, K2 Relay_DPDT, K3 Relay_DPDT, K4 Relay_DPDT, K5 Relay_DPDT, SW1 SW_SPDT_321, SW2 SW_SPDT_321, SW3 SW_SPDT_321, SW4 SW_SPDT_321, SW5 PWR, U1 ULN2003, U10 4N35, U11 4N35, U12 4N35, U13 74HC165, U14 4N35, U15 4N35, U16 4N35, U17 4N35, U18 4N35, U2 MAX1726EUK50, U3 MAX1726EUK33, U4 4N35, U5 4N35, U6 4N35, U7 74LS595, U8 CH343G, U9 74HC165

Commit message: .
Other:
- added sheet mounting-board-devkit-32U (mounting-board-devkit-32U.kicad_sch)
Changed lines of the file:
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@@
+		)
+	)
+	(sheet
+		(at 508 307.34)
+		(size 68.58 11.43)
+		(fields_autoplaced yes)
+		(stroke
+			(width 0.1524)
+			(type solid)
+		)
+		(fill
+			(color 0 0 0 0.0000)
+		)
+		(property "Sheetname" "mounting-board-devkit-32U"
+			(at 508 306.6284 0)
+			(effects
+				(font
+					(size 1.27 1.27)
+				)
+				(justify left bottom)
+			)
+		)
+		(property "Sheetfile" "mounting-board-devkit-32U.kicad_sch"
+			(at 508 319.3546 0)
+			(effects
+				(font
+					(size 1.27 1.27)
+				)
+				(justify left top)
+			)
+		)
+		(instances
+			(project "esp32-wroom-board"
+				(path "/4a90ead8-6e51-429d-a467-47fbf8655e89"
+					(page "4")
+				)
+			)
 		)
 	)

Commit message: .
Parts:
- SW5: footprint Connector_PinHeader_2.54mm:PinHeader_1x03_P2.54mm_Vertical -> Connector_PinHeader_2.54mm:PinHeader_1x02_P2.54mm_Vertical
Changed lines of the file:
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@@
 			)
 		)
-		(property "Footprint" "Connector_PinHeader_2.54mm:PinHeader_1x03_P2.54mm_Vertical"
+		(property "Footprint" "Connector_PinHeader_2.54mm:PinHeader_1x02_P2.54mm_Vertical"
 			(at 66.04 50.8 0)
 			(effects
