File: esp32-wroom-socket-v3/esp32-wroom-socket-v3/esp32-wroom-socket-v3.kicad_pcb (KiCad board)
At the start: 2 copper layers, 99.1 x 96.5 mm, 39 parts, among them J1 PWR, J10 Conn_01x04_Socket, J11 Conn_01x04_Socket, J12 Conn_01x04_Socket, J13 Conn_01x04_Socket, J2 I2C, J3 I2C, J4 e-Paper, J6 UART, J9 Conn_01x04_Socket, K1 Relay_DPDT, K2 Relay_DPDT, K3 Relay_DPDT, K4 Relay_DPDT, K5 Relay_DPDT, U1 ULN2003, U2 MAX1726EUK50, U3 MAX1726EUK33, U4 4N35, U5 4N35, U6 4N35

Commit message: ePaper
Parts:
- removed H2: MountingHole, MountingHole:MountingHole_3mm_Pad_TopBottom
- removed J10, J11: Conn_01x04_Socket, Connector_PinHeader_2.54mm:PinHeader_1x04_P2.54mm_Vertical
- removed K2, K3: Relay_DPDT, Relay_THT:Relay_DPDT_Finder_30.22
- removed R2: 4k7, Resistor_SMD:R_1812_4532Metric
- removed U1: ULN2003, Package_DIP:DIP-16_W7.62mm
Connections:
- U4 pad 4: Net-(D2-A) -> GND
- U5 pad 4: Net-(D3-A) -> GND
- U6 pad 4: Net-(D1-A) -> GND
Routing:
- net +3V3: track 266.8 -> 333.8 mm
- net +5V: track 198.5 -> 160.7 mm
- net VDC: track 224.2 -> 204.7 mm
- net Net-(U1-O2): track 14.6 -> 0.00 mm
- net Net-(U1-O1): track 7.62 -> 0.00 mm
- net unconnected-(U1-O3-Pad14): track 4.82 -> 0.00 mm
- net Net-(J5-IO16): track 32.7 -> 37.2 mm
- net Net-(J5-IO4): track 28.4 -> 32.7 mm
- net Net-(J5-IO17): track 35.8 -> 38.7 mm
- net Net-(J5-IO5): track 41.9 -> 44.3 mm
- net Net-(J5-IO18): track 46.9 -> 48.9 mm
- net Net-(J5-IO21): track 157.9 -> 156.3 mm
- net Net-(J5-TXD0): track 19.2 -> 20.6 mm
- net Net-(J5-RXD0): track 23.6 -> 24.8 mm
- net Net-(J5-IO22): track 160.4 -> 159.7 mm

Commit message: .
Parts:
- removed D3: LED, LED_SMD:LED_2010_5025Metric_Pad1.52x2.65mm_HandSolder
- removed J12: Conn_01x04_Socket, Connector_PinHeader_2.54mm:PinHeader_1x04_P2.54mm_Vertical
- removed K4: Relay_DPDT, Relay_THT:Relay_DPDT_Finder_30.22
- removed U5: 4N35, Package_DIP:DIP-6_W7.62mm
- added J10: IO34, Connector_PinHeader_2.54mm:PinHeader_1x01_P2.54mm_Vertical, F.Cu at (66.0, 63.5)
- added J11: IO27, Connector_PinHeader_2.54mm:PinHeader_1x01_P2.54mm_Vertical, F.Cu at (71.1, 73.7)
- added J14: IO12, Connector_PinHeader_2.54mm:PinHeader_1x01_P2.54mm_Vertical, F.Cu at (71.1, 78.7)
- added J15: IO14, Connector_PinHeader_2.54mm:PinHeader_1x01_P2.54mm_Vertical, F.Cu at (66.0, 78.7)
- added J16: IO26, Connector_PinHeader_2.54mm:PinHeader_1x01_P2.54mm_Vertical, F.Cu at (66.0, 73.7)
- added J17: IO25, Connector_PinHeader_2.54mm:PinHeader_1x01_P2.54mm_Vertical, F.Cu at (60.8, 73.5)
- added J18: IO33, Connector_PinHeader_2.54mm:PinHeader_1x01_P2.54mm_Vertical, F.Cu at (71.1, 68.6)
- added J19: IO32, Connector_PinHeader_2.54mm:PinHeader_1x01_P2.54mm_Vertical, F.Cu at (66.0, 68.6)
- added J5: IO35, Connector_PinHeader_2.54mm:PinHeader_1x01_P2.54mm_Vertical, F.Cu at (71.1, 63.5)
- J13, J9: footprint Connector_PinHeader_2.54mm:PinHeader_1x04_P2.54mm_Vertical -> Alexander Footprints Library:Conn_Terminal_4_Large
- moved J7 21.6 mm to (57.2, 52.6)
- moved J13 15.8 mm to (62.4, 142.2)
- moved J9 5.99 mm to (84.0, 142.2)
- moved D1 2.51 mm to (82.2, 100.0), turned to 180 degrees
- moved D2 2.25 mm to (94.0, 99.8), turned to 180 degrees
Connections:
- J8 pad 25: Net-(J5-IO0) -> unconnected-(J8-IO0-Pad25)
- J8 pad 31: Net-(J5-IO19) -> unconnected-(J8-IO19-Pad31)
- K1 pad 14: Net-(J9-Pin_2) -> Net-(J9-Pin_3)
- K1 pad 22: Net-(J9-Pin_3) -> Net-(J9-Pin_2)
- K5 pad 14: Net-(J13-Pin_2) -> Net-(J13-Pin_3)
- K5 pad 22: Net-(J13-Pin_3) -> Net-(J13-Pin_2)
Routing:
- net Net-(J17-Pin_1): track 0.00 -> 22.7 mm
- net GND: track 33.4 -> 13.4 mm, vias 5 -> 6
- net Net-(J15-Pin_1): track 0.00 -> 16.6 mm
- net Net-(J19-Pin_1): track 0.00 -> 16.5 mm
- net Net-(J10-Pin_1): track 0.00 -> 15.4 mm
- net Net-(J14-Pin_1): track 0.00 -> 14.1 mm
- net Net-(J16-Pin_1): track 0.00 -> 13.9 mm
- net +5V: track 160.7 -> 147.0 mm
- net VDC: track 204.7 -> 191.3 mm
- net Net-(J13-Pin_2): track 7.97 -> 20.9 mm
- net Net-(J12-Pin_3): track 12.5 -> 0.00 mm
- net Net-(J12-Pin_1): track 12.2 -> 0.00 mm
- net Net-(J11-Pin_1): track 0.00 -> 10.5 mm
- net Net-(J12-Pin_2): track 8.06 -> 0.00 mm
- net Net-(J9-Pin_4): track 6.46 -> 13.3 mm
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
Commit message: .
Routing:
- net +3V3: track 340.5 -> 369.5 mm
- net GND: track 13.4 -> 10.1 mm
- net VDC: track 191.3 -> 193.8 mm
