File: esp32-wroom-socket-v3/esp32-wroom-socket-v3/esp32-wroom-socket-v3.kicad_sch (KiCad schematic)
At the start: 39 parts, among them J1 PWR, J10 Conn_01x04_Socket, J11 Conn_01x04_Socket, J12 Conn_01x04_Socket, J13 Conn_01x04_Socket, J2 I2C, J3 I2C, J4 e-Paper, J6 UART, J9 Conn_01x04_Socket, K1 Relay_DPDT, K2 Relay_DPDT, K3 Relay_DPDT, K4 Relay_DPDT, K5 Relay_DPDT, U1 ULN2003, U2 MAX1726EUK50, U3 MAX1726EUK33, U4 4N35, U5 4N35, U6 4N35

Commit message: ePaper
Connections:
- net GND: now also U4.4, U5.4, U6.4
- net at D3.2 (A), U5.2: no longer U5.4
- net at D2.2 (A), U4.2: no longer U4.4
- net at D1.2 (A), U6.2: no longer U6.4
Other:
- moved on the sheet: BRD_15x1, D1, D2, D3

Commit message: .
Parts:
- removed D3: LED, LED_SMD:LED_2010_5025Metric_Pad1.52x2.65mm_HandSolder, symbol Device:LED
- removed H2: MountingHole, MountingHole:MountingHole_3mm_Pad_TopBottom, symbol Mechanical:MountingHole
- removed J10, J11, J12: Conn_01x04_Socket, Connector_PinHeader_2.54mm:PinHeader_1x04_P2.54mm_Vertical, symbol Connector:Conn_01x04_Socket
- removed J5: ~, Alexander Footprints Library:ESP32-WROOM-32D-Interface_2, symbol Alexander_Library_Symbols:ESP32-WROOM-32D
- removed K2, K3, K4: Relay_DPDT, Relay_THT:Relay_DPDT_Finder_30.22, symbol Relay:Relay_DPDT
- removed R2: 4k7, Resistor_SMD:R_1812_4532Metric, symbol Device:R
- removed U1: ULN2003, Package_DIP:DIP-16_W7.62mm, symbol Transistor_Array:ULN2003
- removed U5: 4N35, Package_DIP:DIP-6_W7.62mm, symbol Isolator:4N35
- added J10: IO34, Connector_PinHeader_2.54mm:PinHeader_1x01_P2.54mm_Vertical, symbol Connector:Conn_01x01_Socket
- added J11: IO27, Connector_PinHeader_2.54mm:PinHeader_1x01_P2.54mm_Vertical, symbol Connector:Conn_01x01_Socket
- added J14: IO12, Connector_PinHeader_2.54mm:PinHeader_1x01_P2.54mm_Vertical, symbol Connector:Conn_01x01_Socket
- added J15: IO14, Connector_PinHeader_2.54mm:PinHeader_1x01_P2.54mm_Vertical, symbol Connector:Conn_01x01_Socket
- added J16: IO26, Connector_PinHeader_2.54mm:PinHeader_1x01_P2.54mm_Vertical, symbol Connector:Conn_01x01_Socket
- added J17: IO25, Connector_PinHeader_2.54mm:PinHeader_1x01_P2.54mm_Vertical, symbol Connector:Conn_01x01_Socket
- added J18: IO33, Connector_PinHeader_2.54mm:PinHeader_1x01_P2.54mm_Vertical, symbol Connector:Conn_01x01_Socket
- added J19: IO32, Connector_PinHeader_2.54mm:PinHeader_1x01_P2.54mm_Vertical, symbol Connector:Conn_01x01_Socket
- added J5: IO35, Connector_PinHeader_2.54mm:PinHeader_1x01_P2.54mm_Vertical, symbol Connector:Conn_01x01_Socket
- J13, J9: footprint Connector_PinHeader_2.54mm:PinHeader_1x04_P2.54mm_Vertical -> Alexander Footprints Library:Conn_Terminal_4_Large
Connections:
- net at K5.14: now also J13.3 (Pin_3); no longer J13.2 (Pin_2)
- net at K5.22: now also J13.2 (Pin_2); no longer J13.3 (Pin_3)
- net at J9.2 (Pin_2): now also K1.22; no longer K1.14
- net at J9.3 (Pin_3): now also K1.14; no longer K1.22
- net at J8.10 (IO25): now also J17.1 (Pin_1)
- net at J8.11 (IO26): now also J16.1 (Pin_1)
- net at J8.12 (IO27): now also J11.1 (Pin_1)
- net at J8.13 (IO14): now also J15.1 (Pin_1)
- net at J8.14 (IO12): now also J14.1 (Pin_1)
- net at J8.6 (IO34): now also J10.1 (Pin_1)
- net at J8.7 (IO35): now also J5.1 (Pin_1)
- net at J8.8 (IO32): now also J19.1 (Pin_1)
- net at J8.9 (IO33): now also J18.1 (Pin_1)
Other:
- moved on the sheet: D2, J9, K1, U4
