File: rp2040w-zero/rp2040w-zero/rp2040w-zero.kicad_sch (KiCad schematic)
At the start: 1 part

Commit message: .
Parts:
- removed U1: ~, Alexander Footprint Library:RP2040-Zero, symbol Alexander Symbol Library:rp2040w-zero
- added U1: ~, Alexander Footprint Library:RP2040-Zero, symbol Alexander_Library_Symbols:rp2040w-zero
Connections:
- net +5V: now also U1.1 (5V)
- net GND: now also U1.2 (GND)
Changed lines of the file:
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@@
 	(wire
 		(pts
-			(xy 125.73 60.96) (xy 130.81 60.96)
+			(xy 147.32 45.72) (xy 147.32 49.53)
 		)
 		(stroke
@@
 	(wire
 		(pts
-			(xy 107.95 55.88) (xy 107.95 59.69)
+			(xy 148.59 100.33) (xy 148.59 105.41)
 		)
 		(stroke
@@
 	(wire
 		(pts
-			(xy 125.73 58.42) (xy 130.81 58.42)
+			(xy 107.95 55.88) (xy 107.95 59.69)
 		)
 		(stroke
@@
 	)
 	(label "GND"
-		(at 125.73 60.96 0)
+		(at 148.59 105.41 90)
 		(fields_autoplaced yes)
 		(effects
@@
 	)
 	(label "5V"
-		(at 125.73 58.42 0)
-		(fields_autoplaced yes)
-		(effects
-			(font
-				(size 1.27 1.27)
-			)
-			(justify left bottom)
-		)
-	)
-	(symbol
-		(lib_id "Alexander Symbol Library:rp2040w-zero")
-		(at 143.51 100.33 0)
-		(unit 1)
-		(exclude_from_sim no)
-		(in_bom yes)
-		(on_board yes)
-		(dnp no)
-		(fields_autoplaced yes)
-		(property "Reference" "U1"
-			(at 143.51 52.07 0)
-			(effects
-				(font
-					(size 1.27 1.27)
-				)
-			)
-		)
-		(property "Value" "~"
-			(at 143.51 54.61 0)
-			(effects
-				(font
-					(size 1.27 1.27)
-				)
-			)
-		)
-		(property "Footprint" "Alexander Footprint Library:RP2040-Zero"
-			(at 143.51 100.33 0)
-			(effects
-				(font
-					(size 1.27 1.27)
-				)
-				(hide yes)
-			)
-		)
-		(property "Datasheet" ""
-			(at 143.51 100.33 0)
-			(effects
-				(font
-					(size 1.27 1.27)
-				)
-				(hide yes)
-			)
-		)
-		(property "Description" ""
-			(at 143.51 100.33 0)
-			(effects
-				(font
-					(size 1.27 1.27)
-				)
-				(hide yes)
-			)
-		)
-		(pin "16"
-		)
-		(pin "6"
-		)
-		(pin "15"
-		)
-		(pin "4"
-		)
-		(pin "21"
-		)
-		(pin "1"
-		)
-		(pin "9"
-		)
-		(pin "12"
-		)
-		(pin "13"
-		)
-		(pin "5"
-		)
-		(pin "8"
-		)
-		(pin "18"
-		)
-		(pin "10"
-		)
-		(pin "20"
-		)
-		(pin "22"
-		)
-		(pin "17"
-		)
-		(pin "2"
-		)
-		(pin "14"
-		)
-		(pin "11"
-		)
-		(pin "7"
-		)
-		(pin "23"
-		)
-		(pin "3"
-		)
-		(pin "19"
-		)
-		(instances
-			(project "rp2040w-zero"
-				(path "/f77e979b-3f34-49b3-9cbf-ac4fd50744f2"
-					(reference "U1")
-					(unit 1)
-				)
-			)
+		(at 147.32 48.26 90)
+		(fields_autoplaced yes)
+		(effects
+			(font
+				(size 1.27 1.27)
+			)
+			(justify left bottom)
 		)
 	)
@@
 					(unit 1)
 				)
+			)
+		)
+	)
+	(symbol
+		(lib_id "Alexander_Library_Symbols:rp2040w-zero")
+		(at 148.59 101.6 0)
+		(unit 1)
+		(exclude_from_sim no)
+		(in_bom yes)
+		(on_board yes)
+		(dnp no)
+		(fields_autoplaced yes)
+		(property "Reference" "U1"
+			(at 150.7841 100.33 0)
+			(effects
+				(font
+					(size 1.27 1.27)
+				)
+				(justify left)
+			)
+		)
+		(property "Value" "~"
+			(at 150.7841 101.6 0)
+			(effects
+				(font
+					(size 1.27 1.27)
+				)
+				(justify left)
+			)
+		)
+		(property "Footprint" "Alexander Footprint Library:RP2040-Zero"
+			(at 148.336 99.822 0)
+			(effects
+				(font
+					(size 1.27 1.27)
+				)
+				(hide yes)
+			)
+		)
+		(property "Datasheet" ""
+			(at 148.59 101.6 0)
+			(effects
+				(font
+					(size 1.27 1.27)
+				)
+				(hide yes)
+			)
+		)
+		(property "Description" "RP2040W-Zero"
+			(at 148.082 75.692 90)
+			(effects
+				(font
+					(size 1.27 1.27)
+					(bold yes)
+				)
+				(hide yes)
+			)
+		)
+		(pin "21"
+		)
+		(pin "10"
+		)
+		(pin "19"
+		)
+		(pin "13"
+		)
+		(pin "15"
+		)
+		(pin "16"
+		)
+		(pin "20"
+		)
+		(pin "22"
+		)
+		(pin "7"
+		)
+		(pin "4"
+		)
+		(pin "5"
+		)
+		(pin "11"
+		)
+		(pin "3"
+		)
+		(pin "14"
+		)
+		(pin "9"
+		)
+		(pin "8"
+		)
+		(pin "1"
+		)
+		(pin "2"
+		)
+		(pin "17"
+		)
+		(pin "18"
+		)
+		(pin "12"
+		)
+		(pin "23"
+		)
+		(pin "6"
+		)
+		(instances
+			(project "rp2040w-zero"
+				(path "/f77e979b-3f34-49b3-9cbf-ac4fd50744f2"
+					(reference "U1")
+					(unit 1)
+				)

Commit message: .
Parts:
- U1: footprint Alexander Footprint Library:RP2040-Zero -> Alexander Footprint Library:RP2040-Zero-constellation
Changed lines of the file:
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@@
 			)
 		)
-		(property "Footprint" "Alexander Footprint Library:RP2040-Zero"
+		(property "Footprint" "Alexander Footprint Library:RP2040-Zero-constellation"
 			(at 148.336 99.822 0)
 			(effects

Commit message: .
Parts:
- added BRD1: ~, Alexander Footprint Library:Board_65-40, symbol Alexander Symbol Library:Board-65-40
- added J1: PWR, Connector_Wire:SolderWire-0.75sqmm_1x02_P4.8mm_D1.25mm_OD2.3mm, symbol Connector:Conn_01x02_Socket
- added U2: LM78M05_TO252, Package_TO_SOT_SMD:TO-252-2, symbol Regulator_Linear:LM78M05_TO252
Connections:
- net +5V: now also U2.3 (VO)
- net GND: now also BRD1.1 (GND), J1.2 (Pin_2), U2.2 (GND)
- new net VCC: J1.1 (Pin_1), U2.1 (VI)
