File: rp2040w-zero/rp2040w-zero/rp2040w-zero.kicad_pcb (KiCad board)
At the start: 2 copper layers, 65 x 40 mm, 4 parts, among them J1 PWR, U2 LM78M05_TO252

Commit message: .
Parts:
- added J2: I2C, Alexanddr Footprints Library:Conn_I2C, F.Cu at (144.8, 46.0)
- moved J1 21.3 mm to (144.5, 74.8), turned to 90 degrees
- moved U2 19.4 mm to (134.9, 69.8), turned to 90 degrees
- moved U1 18.5 mm to (108.5, 49.4), turned to 180 degrees
Connections:
- U1 pad 3: unconnected-(U1-3V3-Pad3) -> /3V3
- U1 pad 6: unconnected-(U1-ADC1/SCL1-Pad6) -> /SCL
- U1 pad 7: unconnected-(U1-ADC0/SDA1-Pad7) -> /SDA
Routing:
- net /3V3: track 0.00 -> 40.1 mm
- net /SCL: track 0.00 -> 29.1 mm
- net /SDA: track 0.00 -> 29.1 mm
- net +5V: track 7.68 -> 16.5 mm
- net /VCC: track 11.0 -> 7.38 mm

Commit message: .
Parts:
- U2: moved to F.Cu
- moved J1 59.8 mm to (86.9, 59.0)
- moved U2 41.5 mm to (96.5, 54.0)
- moved U1 26.6 mm to (118.9, 73.9), turned to 0 degrees
- moved J2 1.52 mm to (143.3, 46.0)
Connections:
- U1 pad 18: unconnected-(U1-SCL0-Pad18) -> /SCL
- U1 pad 19: unconnected-(U1-SDA0-Pad19) -> /SDA
- U1 pad 6: /SCL -> unconnected-(U1-ADC1/SCL1-Pad6)
- U1 pad 7: /SDA -> unconnected-(U1-ADC0/SDA1-Pad7)
Routing:
- net /3V3: track 40.1 -> 0.00 mm
- net /SCL: track 29.1 -> 0.00 mm
- net /SDA: track 29.1 -> 0.00 mm
- net +5V: track 16.5 -> 0.00 mm
- net /VCC: track 7.38 -> 0.00 mm

Commit message: .
Parts:
- U2: moved to B.Cu
- moved J1 5.31 mm to (86.9, 53.7), turned to -90 degrees
- moved U1 0.57 mm to (118.4, 74.2)
- turned U2 to -90 degrees
Routing:
- net /VCC: track 0.00 -> 11.0 mm
