File: esp32-node-box-40x65_telemetry/esp32-node-board-40x65_telemetry/esp32-node-board-40x65_telemetry.kicad_pcb (KiCad board)
At the start: 2 copper layers, 65.3 x 80.9 mm, 65 parts, among them J10 ADC, J14 GPIO, J15 LED_PWR, J16 GND, J17 GND, J18 LED_PWR, J19 LED_PWR, J2 PWR, J21 PWR, J22 Conn_01x04_Pin, J23 I2C, J25 PWR_SATA_Conn_01x04, J3 UART, J4 I2C, J5 DAC, J6 SOURCE, J7 LED_PWR, J8 Conn_01x02_Socket, J9 Conn_01x02_Socket, SW1 SW_Push, U1 MAX1726EUK33, U10 BME(P)280, U4 L7805, U7 BME(P)280, U8 BME(P)280, U9 L7805

Commit message: .
Parts:
- moved J5 20.5 mm to (111.8, 45.9), turned to 90 degrees
Routing:
- net /DAC1: track 0.00 -> 19.4 mm
- net /DAC2: track 0.00 -> 11.1 mm
Changed lines of the file:
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@@
 	(footprint "Connector_PinSocket_2.54mm:PinSocket_1x02_P2.54mm_Vertical"
 		(layer "F.Cu")
-		(at 99.2 62.15 180)
+		(at 111.75 45.925 90)
 		(descr "Through hole straight socket strip, 1x02, 2.54mm pitch, single row (from Kicad 4.0.7), script generated")
 		(tags "Through hole socket strip THT 1x02 2.54mm single row")
 		(property "Reference" "J5"
-			(at 0.075 -2.15 0)
+			(at 0.075 -2.15 90)
 			(layer "F.SilkS")
 			(effects
@@
 		)
 		(property "Value" "DAC"
-			(at 0 5.31 0)
+			(at 2.775 1.25 0)
 			(layer "F.Fab")
 			(effects
@@
 		)
 		(property "Footprint" "Connector_PinSocket_2.54mm:PinSocket_1x02_P2.54mm_Vertical"
-			(at 0 0 180)
+			(at 0 0 90)
 			(unlocked yes)
 			(layer "F.Fab")
@@
 		)
 		(property "Datasheet" ""
-			(at 0 0 180)
+			(at 0 0 90)
 			(unlocked yes)
 			(layer "F.Fab")
@@
 		)
 		(property "Description" ""
-			(at 0 0 180)
+			(at 0 0 90)
 			(unlocked yes)
 			(layer "F.Fab")
@@
 		(attr through_hole)
 		(fp_line
-			(start 1.33 1.27)
-			(end 1.33 3.87)
-			(stroke
-				(width 0.12)
-				(type solid)
-			)
-			(layer "F.SilkS")
-		)
-		(fp_line
 			(start 1.33 -1.33)
 			(end 1.33 0)
@@
 		)
 		(fp_line
-			(start -1.33 3.87)
+			(start 1.33 1.27)
 			(end 1.33 3.87)
 			(stroke
@@
 		)
 		(fp_line
-			(start 1.75 4.3)
-			(end -1.8 4.3)
+			(start -1.33 3.87)
+			(end 1.33 3.87)
 			(stroke
-				(width 0.05)
+				(width 0.12)
 				(type solid)
 			)
-			(layer "F.CrtYd")
+			(layer "F.SilkS")
 		)
 		(fp_line
@@
 		)
 		(fp_line
-			(start -1.8 4.3)
-			(end -1.8 -1.8)
+			(start -1.8 -1.8)
+			(end 1.75 -1.8)
 			(stroke
 				(width 0.05)
@@
 		)
 		(fp_line
-			(start -1.8 -1.8)
-			(end 1.75 -1.8)
+			(start 1.75 4.3)
+			(end -1.8 4.3)
 			(stroke
 				(width 0.05)
@@
 		)
 		(fp_line
-			(start 1.27 3.81)
-			(end -1.27 3.81)
+			(start -1.8 4.3)
+			(end -1.8 -1.8)
+			(stroke
+				(width 0.05)
+				(type solid)
+			)
+			(layer "F.CrtYd")
+		)
+		(fp_line
+			(start 0.635 -1.27)
+			(end 1.27 -0.635)
 			(stroke
 				(width 0.1)
@@
 		)
 		(fp_line
-			(start 1.27 -0.635)
-			(end 1.27 3.81)
+			(start -1.27 -1.27)
+			(end 0.635 -1.27)
 			(stroke
 				(width 0.1)
@@
 		)
 		(fp_line
-			(start 0.635 -1.27)
-			(end 1.27 -0.635)
+			(start 1.27 -0.635)
+			(end 1.27 3.81)
 			(stroke
 				(width 0.1)
@@
 		)
 		(fp_line
-			(start -1.27 3.81)
-			(end -1.27 -1.27)
+			(start 1.27 3.81)
+			(end -1.27 3.81)
 			(stroke
 				(width 0.1)
@@
 		)
 		(fp_line
-			(start -1.27 -1.27)
-			(end 0.635 -1.27)
+			(start -1.27 3.81)
+			(end -1.27 -1.27)
 			(stroke
 				(width 0.1)
@@
 		)
 		(fp_text user "${REFERENCE}"
-			(at 0 1.27 90)
+			(at 0 1.27 0)
 			(layer "F.Fab")
 			(effects
@@
 		)
 		(pad "1" thru_hole rect
-			(at 0 0 180)
+			(at 0 0 90)
 			(size 1.7 1.7)
 			(drill 1)
@@
 		)
 		(pad "2" thru_hole oval
-			(at 0 2.54 180)
+			(at 0 2.54 90)
 			(size 1.7 1.7)
 			(drill 1)
@@
 	)
 	(segment
+		(start 123.8 43.65)
+		(end 123.15 43)
+		(width 0.25)
+		(layer "F.Cu")
+		(net 15)
+	)
+	(segment
+		(start 111.75 43.5)
+		(end 111.75 45.925)
+		(width 0.25)
+		(layer "F.Cu")
+		(net 15)
+	)
+	(segment
+		(start 123.8 46.29)
+		(end 123.8 43.65)
+		(width 0.25)
+		(layer "F.Cu")
+		(net 15)
+	)
+	(segment
+		(start 112.25 43)
+		(end 111.75 43.5)
+		(width 0.25)
+		(layer "F.Cu")
+		(net 15)
+	)
+	(segment
+		(start 123.15 43)
+		(end 112.25 43)
+		(width 0.25)
+		(layer "F.Cu")
+		(net 15)
+	)
+	(segment
+		(start 125.06 47.55)
+		(end 123.8 46.29)
+		(width 0.25)
+		(layer "F.Cu")
+		(net 15)
+	)
+	(segment
+		(start 114.8 43.45)
+		(end 120.96 43.45)
+		(width 0.25)
+		(layer "F.Cu")
+		(net 16)
+	)
+	(segment
+		(start 114.29 45.925)
+		(end 114.29 43.96)
+		(width 0.25)
+		(layer "F.Cu")
+		(net 16)
+	)
+	(segment
+		(start 120.96 43.45)
+		(end 122.52 45.01)
+		(width 0.25)
+		(layer "F.Cu")
+		(net 16)
+	)
+	(segment
+		(start 114.29 43.96)
+		(end 114.8 43.45)
+		(width 0.25)
+		(layer "F.Cu")
+		(net 16)
+	)
+	(segment

Commit message: .
Routing:
- net /EN: track 17.5 -> 51.7 mm
- net /DAC2: track 11.1 -> 11.8 mm
Changed lines of the file:
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@@
 	)
 	(segment
-		(start 100 51.8)
-		(end 103.9 51.8)
+		(start 130.62 42.95)
+		(end 117.962749 42.95)
+		(width 0.25)
+		(layer "B.Cu")
+		(net 10)
+	)
+	(segment
+		(start 113.462749 48.487251)
+		(end 103.012749 48.487251)
+		(width 0.25)
+		(layer "B.Cu")
+		(net 10)
+	)
+	(segment
+		(start 115.5 45.412749)
+		(end 115.5 46.45)
+		(width 0.25)
+		(layer "B.Cu")
+		(net 10)
+	)
+	(segment
+		(start 117.962749 42.95)
+		(end 115.5 45.412749)
+		(width 0.25)
+		(layer "B.Cu")
+		(net 10)
+	)
+	(segment
+		(start 103.012749 48.487251)
+		(end 99.7 51.8)
+		(width 0.25)
+		(layer "B.Cu")
+		(net 10)
+	)
+	(segment
+		(start 115.5 46.45)
+		(end 113.462749 48.487251)
+		(width 0.25)
+		(layer "B.Cu")
+		(net 10)
+	)
+	(segment
+		(start 132.68 45.01)
+		(end 130.62 42.95)
 		(width 0.25)
 		(layer "B.Cu")
@@
 	)
 	(segment
-		(start 123.8 43.65)
-		(end 123.15 43)
+		(start 112.25 43)
+		(end 111.75 43.5)
+		(width 0.25)
+		(layer "F.Cu")
+		(net 15)
+	)
+	(segment
+		(start 123.8 43.35)
+		(end 123.45 43)
+		(width 0.25)
+		(layer "F.Cu")
+		(net 15)
+	)
+	(segment
+		(start 125.06 47.55)
+		(end 123.8 46.29)
+		(width 0.25)
+		(layer "F.Cu")
+		(net 15)
+	)
+	(segment
+		(start 123.8 46.29)
+		(end 123.8 43.35)
 		(width 0.25)
 		(layer "F.Cu")
@@
 	)
 	(segment
-		(start 123.8 46.29)
-		(end 123.8 43.65)
-		(width 0.25)
-		(layer "F.Cu")
-		(net 15)
-	)
-	(segment
-		(start 112.25 43)
-		(end 111.75 43.5)
-		(width 0.25)
-		(layer "F.Cu")
-		(net 15)
-	)
-	(segment
-		(start 123.15 43)
+		(start 123.45 43)
 		(end 112.25 43)
 		(width 0.25)
@@
 	)
 	(segment
-		(start 125.06 47.55)
-		(end 123.8 46.29)
-		(width 0.25)
-		(layer "F.Cu")
-		(net 15)
-	)
-	(segment
 		(start 114.8 43.45)
-		(end 120.96 43.45)
+		(end 122.2 43.45)
 		(width 0.25)
 		(layer "F.Cu")
@@
 	)
 	(segment
-		(start 120.96 43.45)
+		(start 122.52 43.77)
 		(end 122.52 45.01)
 		(width 0.25)
@@
 		(width 0.25)
 		(layer "F.Cu")
+		(net 16)
+	)
+	(segment
+		(start 122.2 43.45)
+		(end 122.52 43.77)
+		(width 0.25)
+		(layer "F.Cu")

Commit message: .
Routing:
- net /EN: track 51.7 -> 49.0 mm
Changed lines of the file:
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@@
 	)
 	(segment
-		(start 130.62 42.95)
-		(end 117.962749 42.95)
+		(start 116.3 42.95)
+		(end 115.9 43.35)
 		(width 0.25)
 		(layer "B.Cu")
@@
 	)
 	(segment
-		(start 113.462749 48.487251)
-		(end 103.012749 48.487251)
+		(start 115.262749 48.487251)
+		(end 104.762749 48.487251)
 		(width 0.25)
 		(layer "B.Cu")
@@
 	)
 	(segment
-		(start 115.5 45.412749)
-		(end 115.5 46.45)
+		(start 115.9 43.35)
+		(end 115.9 47.85)
 		(width 0.25)
 		(layer "B.Cu")
@@
 	)
 	(segment
-		(start 117.962749 42.95)
-		(end 115.5 45.412749)
+		(start 115.9 47.85)
+		(end 115.262749 48.487251)
 		(width 0.25)
 		(layer "B.Cu")
@@
 	)
 	(segment
-		(start 103.012749 48.487251)
+		(start 101.45 51.8)
 		(end 99.7 51.8)
 		(width 0.25)
@@
 	)
 	(segment
-		(start 115.5 46.45)
-		(end 113.462749 48.487251)
+		(start 130.62 42.95)
+		(end 116.3 42.95)
 		(width 0.25)
 		(layer "B.Cu")

Commit message: .
Routing:
- net /EN: track 49.0 -> 55.0 mm
Changed lines of the file:
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@@
+	)
+	(segment
+		(start 115.9 43.35)
+		(end 116.3 42.95)
+		(width 0.25)
+		(layer "B.Cu")
+		(net 10)
 	)
 	(segment
 		(start 116.3 42.95)
+		(end 130.62 42.95)
+		(width 0.25)
+		(layer "B.Cu")
+		(net 10)
+	)
+	(segment
+		(start 115.9 47.85)
 		(end 115.9 43.35)
 		(width 0.25)
@@
 	)
 	(segment
-		(start 115.262749 48.487251)
-		(end 104.762749 48.487251)
+		(start 102 49.05)
+		(end 102.562749 48.487251)
 		(width 0.25)
 		(layer "B.Cu")
@@
 	)
 	(segment
-		(start 115.9 43.35)
+		(start 115.262749 48.487251)
 		(end 115.9 47.85)
 		(width 0.25)
@@
 	)
 	(segment
-		(start 115.9 47.85)
+		(start 130.62 42.95)
+		(end 132.68 45.01)
+		(width 0.25)
+		(layer "B.Cu")
+		(net 10)
+	)
+	(segment
+		(start 102 51.25)
+		(end 102 49.05)
+		(width 0.25)
+		(layer "B.Cu")
+		(net 10)
+	)
+	(segment
+		(start 101.45 51.8)
+		(end 102 51.25)
+		(width 0.25)
+		(layer "B.Cu")
+		(net 10)
+	)
+	(segment
+		(start 102.562749 48.487251)
 		(end 115.262749 48.487251)
 		(width 0.25)
@@
 	)
 	(segment
-		(start 101.45 51.8)
-		(end 99.7 51.8)
+		(start 99.7 51.8)
+		(end 101.45 51.8)
 		(width 0.25)
 		(layer "B.Cu")
-		(net 10)
-	)
-	(segment
-		(start 130.62 42.95)
-		(end 116.3 42.95)
-		(width 0.25)
-		(layer "B.Cu")
-		(net 10)
-	)
-	(segment
-		(start 132.68 45.01)
-		(end 130.62 42.95)
-		(width 0.25)
-		(layer "B.Cu")

Commit message: .
Routing:
- net /EN: track 55.0 -> 51.8 mm, vias 0 -> 1
Changed lines of the file:
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@@
 	(segment
 		(start 92.3 52.75)
-		(end 103.27 52.75)
+		(end 96.9 52.75)
+		(width 0.25)
+		(layer "F.Cu")
+		(net 10)
+	)
+	(segment
+		(start 96.9 52.75)
+		(end 97.2 52.45)
 		(width 0.25)
 		(layer "F.Cu")
@@
 		(width 0.25)
 		(layer "F.Cu")
+		(net 10)
+	)
+	(via
+		(at 97.2 52.45)
+		(size 0.8)
+		(drill 0.4)
+		(layers "F.Cu" "B.Cu")
 		(net 10)
 	)
@@
 	)
 	(segment
+		(start 97.2 52.45)
+		(end 97.85 51.8)
+		(width 0.25)
+		(layer "B.Cu")
+		(net 10)
+	)
+	(segment
 		(start 102 49.05)
 		(end 102.562749 48.487251)
 		(width 0.25)
 		(layer "B.Cu")
+		(net 10)
+	)
+	(segment
+		(start 97.85 51.8)
+		(end 99.7 51.8)
+		(width 0.25)
+		(layer "B.Cu")

Commit message: .
Parts:
- moved J14 59.9 mm to (162.9, 41.0)
- moved C8 17.0 mm to (99.9, 33.9)
- moved J5 12.3 mm to (112.2, 33.6)
- moved J1 7.31 mm to (121.1, 56.9), turned to 0 degrees
Routing:
- net /EN: track 51.8 -> 16.6 mm
- net /DAC1: track 19.5 -> 0.00 mm
- net /DAC2: track 11.8 -> 0.00 mm
- net /SCL: track 96.7 -> 90.0 mm
- net /RXD: track 36.9 -> 31.6 mm
- net /TXD: track 34.9 -> 30.1 mm
- net +3V3: track 169.6 -> 165.0 mm
- net /SDA: track 72.1 -> 69.5 mm

Commit message: .
Parts:
- moved C5 20.4 mm to (140.6, 67.8), turned to -90 degrees
- moved J18 4.57 mm to (101.2, 61.5)

Commit message: .
Parts:
- moved C8 36.7 mm to (135.2, 44.0), turned to 180 degrees
Changed lines of the file:
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@@
 	(footprint "Capacitor_SMD:CP_Elec_3x5.3"
 		(layer "F.Cu")
-		(at 99.9 33.85 -90)
+		(at 135.2 43.95 180)
 		(descr "SMT capacitor, aluminium electrolytic, 3x5.3, Cornell Dubilier Electronics ")
 		(tags "Capacitor Electrolytic")
 		(property "Reference" "C8"
-			(at 0 -2.7 90)
+			(at 0 -2.7 0)
 			(layer "F.SilkS")
 			(effects
@@
 		)
 		(property "Value" "10uF"
-			(at 0 2.7 90)
+			(at 0 2.7 0)
 			(layer "F.Fab")
 			(effects
@@
 		)
 		(property "Footprint" "Capacitor_SMD:CP_Elec_3x5.3"
-			(at 0 0 -90)
+			(at 0 0 180)
 			(unlocked yes)
 			(layer "F.Fab")
@@
 		)
 		(property "Datasheet" ""
-			(at 0 0 -90)
+			(at 0 0 180)
 			(unlocked yes)
 			(layer "F.Fab")
@@
 		)
 		(property "Description" ""
-			(at 0 0 -90)
+			(at 0 0 180)
 			(unlocked yes)
 			(layer "F.Fab")
@@
 		(attr smd)
 		(fp_line
+			(start 1.76 1.76)
+			(end 1.76 1.06)
+			(stroke
+				(width 0.12)
+				(type solid)
+			)
+			(layer "F.SilkS")
+		)
+		(fp_line
+			(start 1.76 -1.76)
+			(end 1.76 -1.06)
+			(stroke
+				(width 0.12)
+				(type solid)
+			)
+			(layer "F.SilkS")
+		)
+		(fp_line
 			(start -0.870563 1.76)
 			(end 1.76 1.76)
@@
 		)
 		(fp_line
-			(start 1.76 1.76)
-			(end 1.76 1.06)
+			(start -0.870563 -1.76)
+			(end 1.76 -1.76)
 			(stroke
 				(width 0.12)
@@
 		)
 		(fp_line
+			(start -2.1875 -1.6225)
+			(end -2.1875 -1.2475)
+			(stroke
+				(width 0.12)
+				(type solid)
+			)
+			(layer "F.SilkS")
+		)
+		(fp_line
 			(start -2.375 -1.435)
 			(end -2 -1.435)
@@
 		)
 		(fp_line
-			(start -2.1875 -1.6225)
-			(end -2.1875 -1.2475)
-			(stroke
-				(width 0.12)
-				(type solid)
-			)
-			(layer "F.SilkS")
-		)
-		(fp_line
-			(start -0.870563 -1.76)
-			(end 1.76 -1.76)
-			(stroke
-				(width 0.12)
-				(type solid)
-			)
-			(layer "F.SilkS")
-		)
-		(fp_line
-			(start 1.76 -1.76)
-			(end 1.76 -1.06)
-			(stroke
-				(width 0.12)
-				(type solid)
-			)
-			(layer "F.SilkS")
+			(start 2.85 1.05)
+			(end 1.9 1.05)
+			(stroke
+				(width 0.05)
+				(type solid)
+			)
+			(layer "F.CrtYd")
+		)
+		(fp_line
+			(start 2.85 -1.05)
+			(end 2.85 1.05)
+			(stroke
+				(width 0.05)
+				(type solid)
+			)
+			(layer "F.CrtYd")
+		)
+		(fp_line
+			(start 1.9 1.05)
+			(end 1.9 1.9)
+			(stroke
+				(width 0.05)
+				(type solid)
+			)
+			(layer "F.CrtYd")
+		)
+		(fp_line
+			(start 1.9 -1.05)
+			(end 2.85 -1.05)
+			(stroke
+				(width 0.05)
+				(type solid)
+			)
+			(layer "F.CrtYd")
+		)
+		(fp_line
+			(start 1.9 -1.9)
+			(end 1.9 -1.05)
+			(stroke
+				(width 0.05)
+				(type solid)
+			)
+			(layer "F.CrtYd")
 		)
 		(fp_line
@@
 		)
 		(fp_line
+			(start -0.93 -1.9)
+			(end 1.9 -1.9)
+			(stroke
+				(width 0.05)
+				(type solid)
+			)
+			(layer "F.CrtYd")
+		)
+		(fp_line
+			(start -1.78 1.05)
+			(end -0.93 1.9)
+			(stroke
+				(width 0.05)
+				(type solid)
+			)
+			(layer "F.CrtYd")
+		)
+		(fp_line
+			(start -1.78 -1.05)
+			(end -0.93 -1.9)
+			(stroke
+				(width 0.05)
+				(type solid)
+			)
+			(layer "F.CrtYd")
+		)
+		(fp_line
+			(start -1.78 -1.05)
+			(end -2.85 -1.05)
+			(stroke
+				(width 0.05)
+				(type solid)
+			)
+			(layer "F.CrtYd")
+		)
+		(fp_line
 			(start -2.85 1.05)
 			(end -1.78 1.05)
@@
 		)
 		(fp_line
-			(start -1.78 1.05)
-			(end -0.93 1.9)
-			(stroke
-				(width 0.05)
-				(type solid)
-			)
-			(layer "F.CrtYd")
-		)
-		(fp_line
-			(start 1.9 1.05)
-			(end 1.9 1.9)
-			(stroke
-				(width 0.05)
-				(type solid)
-			)
-			(layer "F.CrtYd")
-		)
-		(fp_line
-			(start 2.85 1.05)
-			(end 1.9 1.05)
-			(stroke
-				(width 0.05)
-				(type solid)
-			)
-			(layer "F.CrtYd")
-		)
-		(fp_line
 			(start -2.85 -1.05)
 			(end -2.85 1.05)
@@
 		)
 		(fp_line
-			(start -1.78 -1.05)
-			(end -2.85 -1.05)
-			(stroke
-				(width 0.05)
-				(type solid)
-			)
-			(layer "F.CrtYd")
-		)
-		(fp_line
-			(start -1.78 -1.05)
-			(end -0.93 -1.9)
-			(stroke
-				(width 0.05)
-				(type solid)
-			)
-			(layer "F.CrtYd")
-		)
-		(fp_line
-			(start 1.9 -1.05)
-			(end 2.85 -1.05)
-			(stroke
-				(width 0.05)
-				(type solid)
-			)
-			(layer "F.CrtYd")
-		)
-		(fp_line
-			(start 2.85 -1.05)
-			(end 2.85 1.05)
-			(stroke
-				(width 0.05)
-				(type solid)
-			)
-			(layer "F.CrtYd")
-		)
-		(fp_line
-			(start -0.93 -1.9)
-			(end 1.9 -1.9)
-			(stroke
-				(width 0.05)
-				(type solid)
-			)
-			(layer "F.CrtYd")
-		)
-		(fp_line
-			(start 1.9 -1.9)
-			(end 1.9 -1.05)
-			(stroke
-				(width 0.05)
-				(type solid)
-			)
-			(layer "F.CrtYd")
+			(start 1.65 -1.65)
+			(end 1.65 1.65)
+			(stroke
+				(width 0.1)
+				(type solid)
+			)
+			(layer "F.Fab")
 		)
 		(fp_line
@@
 		)
 		(fp_line
+			(start -0.825 -1.65)
+			(end 1.65 -1.65)
+			(stroke
+				(width 0.1)
+				(type solid)
+			)
+			(layer "F.Fab")
+		)
+		(fp_line
+			(start -0.960469 -0.95)
+			(end -0.960469 -0.65)
+			(stroke
+				(width 0.1)
+				(type solid)
+			)
+			(layer "F.Fab")
+		)
+		(fp_line
+			(start -1.110469 -0.8)
+			(end -0.810469 -0.8)
+			(stroke
+				(width 0.1)
+				(type solid)
+			)
+			(layer "F.Fab")
+		)
+		(fp_line
 			(start -1.65 0.825)
 			(end -0.825 1.65)
@@
 		)
 		(fp_line
-			(start -1.110469 -0.8)
-			(end -0.810469 -0.8)
+			(start -1.65 -0.825)
+			(end -0.825 -1.65)
 			(stroke
 				(width 0.1)
@@
 			(start -1.65 -0.825)
 			(end -1.65 0.825)
-			(stroke
-				(width 0.1)
-				(type solid)
-			)
-			(layer "F.Fab")
-		)
-		(fp_line
-			(start -1.65 -0.825)
-			(end -0.825 -1.65)
-			(stroke
-				(width 0.1)
-				(type solid)
-			)
-			(layer "F.Fab")
-		)
-		(fp_line
-			(start -0.960469 -0.95)
-			(end -0.960469 -0.65)
-			(stroke
-				(width 0.1)
-				(type solid)
-			)
-			(layer "F.Fab")
-		)
-		(fp_line
-			(start -0.825 -1.65)
-			(end 1.65 -1.65)
-			(stroke
-				(width 0.1)
-				(type solid)
-			)
-			(layer "F.Fab")
-		)
-		(fp_line
-			(start 1.65 -1.65)
-			(end 1.65 1.65)
 			(stroke
 				(width 0.1)
@@
 		)
 		(fp_text user "${REFERENCE}"
-			(at 0 0 90)
+			(at 0 0 0)
 			(layer "F.Fab")
 			(effects
@@
 		)
 		(pad "1" smd rect
-			(at -1.5 0 270)
+			(at -1.5 0 180)
 			(size 2.2 1.6)
 			(layers "F.Cu" "F.Paste" "F.Mask")
@@
 		)
 		(pad "2" smd rect
-			(at 1.5 0 270)
+			(at 1.5 0 180)
 			(size 2.2 1.6)
 			(layers "F.Cu" "F.Paste" "F.Mask")
