File: esp32-node-box-40x65_telemetry/esp32-node-board-40x65_telemetry/node-esp32-wroom-32u.kicad_sch (KiCad schematic)
At the start: 24 parts, among them J21 PWR, J22 PWR_SATA_Conn_01x04, J23 I2C, J25 Conn_01x04_Pin, J27 Power_Jack, SW1 SW_SPDT, U10 BME(P)280, U8 BME(P)280, U9 L7805

Commit message: .
Parts:
- removed SW1: SW_SPDT, Button_Switch_THT:SW_Slide-03_Wuerth-WS-SLTV_10x2.5x6.4_P2.54mm, symbol Switch:SW_SPDT
- added SW1: SW_SPDT, symbol Alexander_Library_Symbols:SW_SPDT
Changed lines of the file:
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@@
 	)
 	(junction
-		(at 60.96 25.4)
-		(diameter 0)
-		(color 0 0 0 0)
-	)
-	(junction
 		(at 135.89 105.41)
 		(diameter 0)
@@
 	(wire
 		(pts
-			(xy 40.64 27.94) (xy 44.45 27.94)
-		)
-		(stroke
-			(width 0)
-			(type default)
-		)
-	)
-	(wire
-		(pts
 			(xy 87.63 181.61) (xy 95.25 181.61)
 		)
@@
 	(wire
 		(pts
-			(xy 54.61 25.4) (xy 60.96 25.4)
-		)
-		(stroke
-			(width 0)
-			(type default)
-		)
-	)
-	(wire
-		(pts
 			(xy 29.21 44.45) (xy 31.75 44.45)
 		)
@@
 	)
 	(symbol
+		(lib_id "Alexander_Library_Symbols:SW_SPDT")
+		(at 49.53 27.94 0)
+		(unit 1)
+		(exclude_from_sim no)
+		(in_bom yes)
+		(on_board yes)
+		(dnp no)
+		(fields_autoplaced yes)
+		(property "Reference" "SW1"
+			(at 49.53 19.05 0)
+			(effects
+				(font
+					(size 1.27 1.27)
+				)
+			)
+		)
+		(property "Value" "SW_SPDT"
+			(at 49.53 21.59 0)
+			(effects
+				(font
+					(size 1.27 1.27)
+				)
+			)
+		)
+		(property "Footprint" ""
+			(at 49.53 27.94 0)
+			(effects
+				(font
+					(size 1.27 1.27)
+				)
+				(hide yes)
+			)
+		)
+		(property "Datasheet" "~"
+			(at 49.53 35.56 0)
+			(effects
+				(font
+					(size 1.27 1.27)
+				)
+				(hide yes)
+			)
+		)
+		(property "Description" "Switch, single pole double throw"
+			(at 49.53 27.94 0)
+			(effects
+				(font
+					(size 1.27 1.27)
+				)
+				(hide yes)
+			)
+		)
+		(pin "1"
+		)
+		(pin "2"
+		)
+		(pin "3"
+		)
+		(instances
+			(project ""
+				(path "/5f5eb0ac-ab9b-41ab-8d2f-875870c41abc/dab1a116-6bbe-49e5-a398-9f75bdcbe4bf"
+					(reference "SW1")
+					(unit 1)
+				)
+			)
+		)
+	)
+	(symbol
 		(lib_name "+5V_2")
 		(lib_id "power:+5V")
@@
 					(unit 1)
 				)
-			)
-		)
-	)
-	(symbol
-		(lib_id "Switch:SW_SPDT")
-		(at 49.53 25.4 180)
-		(unit 1)
-		(exclude_from_sim no)
-		(in_bom yes)
-		(on_board yes)
-		(dnp no)
-		(fields_autoplaced yes)
-		(property "Reference" "SW1"
-			(at 49.53 16.51 0)
-			(effects
-				(font
-					(size 1.27 1.27)
-				)
-			)
-		)
-		(property "Value" "SW_SPDT"
-			(at 49.53 19.05 0)
-			(effects
-				(font
-					(size 1.27 1.27)
-				)
-			)
-		)
-		(property "Footprint" "Button_Switch_THT:SW_Slide-03_Wuerth-WS-SLTV_10x2.5x6.4_P2.54mm"
-			(at 49.53 25.4 0)
-			(effects
-				(font
-					(size 1.27 1.27)
-				)
-				(hide yes)
-			)
-		)
-		(property "Datasheet" "~"
-			(at 49.53 17.78 0)
-			(effects
-				(font
-					(size 1.27 1.27)
-				)
-				(hide yes)
-			)
-		)
-		(property "Description" "Switch, single pole double throw"
-			(at 49.53 25.4 0)
-			(effects
-				(font
-					(size 1.27 1.27)
-				)
-				(hide yes)
-			)
-		)
-		(pin "1"
-		)
-		(pin "3"
-		)
-		(pin "2"
-		)
-		(instances
-			(project "esp32-node-board-40x65_telemetry"
-				(path "/5f5eb0ac-ab9b-41ab-8d2f-875870c41abc/dab1a116-6bbe-49e5-a398-9f75bdcbe4bf"
-					(reference "SW1")
-					(unit 1)
-				)

Commit message: .
Connections:
- net VDC: now also SW1.1 (COM)
- net VIN: now also SW1.2 (A)
Changed lines of the file:
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@@
+	)
+	(junction
+		(at 60.96 25.4)
+		(diameter 0)
+		(color 0 0 0 0)
 	)
 	(junction
@@
 	(wire
 		(pts
+			(xy 54.61 25.4) (xy 60.96 25.4)
+		)
+		(stroke
+			(width 0)
+			(type default)
+		)
+	)
+	(wire
+		(pts
 			(xy 134.62 34.29) (xy 134.62 38.1)
 		)
@@
 		(pts
 			(xy 120.65 64.77) (xy 124.46 64.77)
+		)
+		(stroke
+			(width 0)
+			(type default)
+		)
+	)
+	(wire
+		(pts
+			(xy 40.64 27.94) (xy 44.45 27.94)
 		)
 		(stroke
@@
 	)
 	(label "VIN"
-		(at 60.96 25.4 0)
-		(fields_autoplaced yes)
-		(effects
+		(at 57.15 25.4 0)
+		(fields_autoplaced yes)
+		(effects

Commit message: .
Parts:
- J21: footprint Connector_PinSocket_2.54mm:PinSocket_1x02_P2.54mm_Vertical -> Alexander Footprint Library:SW_Slide-03_7.3x2.5x2.5_P2.54mm
- SW1: footprint (none) -> Button_Switch_THT:SW_Slide-03_Wuerth-WS-SLTV_10x2.5x6.4_P2.54mm
Connections:
- net VDC: now also SW1.3 (B); no longer SW1.1 (COM)
- net VIN: now also SW1.1 (COM); no longer SW1.2 (A)
Other:
- moved on the sheet: SW1
Changed lines of the file:
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@@
 	)
 	(junction
-		(at 60.96 25.4)
+		(at 246.38 35.56)
 		(diameter 0)
 		(color 0 0 0 0)
 	)
 	(junction
-		(at 246.38 35.56)
+		(at 60.96 25.4)
 		(diameter 0)
 		(color 0 0 0 0)
@@
 	(wire
 		(pts
-			(xy 54.61 25.4) (xy 60.96 25.4)
-		)
-		(stroke
-			(width 0)
-			(type default)
-		)
-	)
-	(wire
-		(pts
 			(xy 134.62 34.29) (xy 134.62 38.1)
 		)
@@
 	(wire
 		(pts
-			(xy 40.64 27.94) (xy 44.45 27.94)
-		)
-		(stroke
-			(width 0)
-			(type default)
-		)
-	)
-	(wire
-		(pts
 			(xy 147.32 76.2) (xy 152.4 76.2)
 		)
@@
 	(wire
 		(pts
+			(xy 54.61 25.4) (xy 60.96 25.4)
+		)
+		(stroke
+			(width 0)
+			(type default)
+		)
+	)
+	(wire
+		(pts
+			(xy 40.64 27.94) (xy 44.45 27.94)
+		)
+		(stroke
+			(width 0)
+			(type default)
+		)
+	)
+	(wire
+		(pts
 			(xy 73.66 33.02) (xy 73.66 36.83)
 		)
@@
 	)
 	(label "VIN"
-		(at 57.15 25.4 0)
+		(at 60.96 25.4 0)
 		(fields_autoplaced yes)
 		(effects
@@
 			)
 		)
-		(property "Footprint" "Connector_PinSocket_2.54mm:PinSocket_1x02_P2.54mm_Vertical"
+		(property "Footprint" "Alexander Footprint Library:SW_Slide-03_7.3x2.5x2.5_P2.54mm"
 			(at 16.51 33.02 0)
 			(effects
@@
 	(symbol
 		(lib_id "Alexander_Library_Symbols:SW_SPDT")
-		(at 49.53 27.94 0)
+		(at 49.53 25.4 0)
+		(mirror y)
 		(unit 1)
 		(exclude_from_sim no)
@@
 		(on_board yes)
 		(dnp no)
-		(fields_autoplaced yes)
 		(property "Reference" "SW1"
-			(at 49.53 19.05 0)
+			(at 49.53 16.51 0)
 			(effects
 				(font
@@
 		)
 		(property "Value" "SW_SPDT"
-			(at 49.53 21.59 0)
+			(at 49.53 19.05 0)
 			(effects
 				(font
@@
 			)
 		)
-		(property "Footprint" ""
-			(at 49.53 27.94 0)
+		(property "Footprint" "Button_Switch_THT:SW_Slide-03_Wuerth-WS-SLTV_10x2.5x6.4_P2.54mm"
+			(at 49.53 25.4 0)
 			(effects
 				(font
@@
 		)
 		(property "Datasheet" "~"
-			(at 49.53 35.56 0)
+			(at 49.53 33.02 0)
 			(effects
 				(font
@@
 		)
 		(property "Description" "Switch, single pole double throw"
-			(at 49.53 27.94 0)
+			(at 49.53 25.4 0)
 			(effects
 				(font

Commit message: .
Parts:
- J21: footprint Alexander Footprint Library:SW_Slide-03_7.3x2.5x2.5_P2.54mm -> Alexander Footprint Library:PinSocket_1x02_P2.54
Changed lines of the file:
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@@
 			)
 		)
-		(property "Footprint" "Alexander Footprint Library:SW_Slide-03_7.3x2.5x2.5_P2.54mm"
+		(property "Footprint" "Alexander Footprint Library:PinSocket_1x02_P2.54"
 			(at 16.51 33.02 0)
 			(effects

Commit message: .
Parts:
- SW1: footprint Button_Switch_THT:SW_Slide-03_Wuerth-WS-SLTV_10x2.5x6.4_P2.54mm -> Alexander Footprint Library:SW_Slide-03_7.3x2.5x2.5_P2.54mm
Changed lines of the file:
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@@
 			)
 		)
-		(property "Footprint" "Button_Switch_THT:SW_Slide-03_Wuerth-WS-SLTV_10x2.5x6.4_P2.54mm"
+		(property "Footprint" "Alexander Footprint Library:SW_Slide-03_7.3x2.5x2.5_P2.54mm"
 			(at 49.53 25.4 0)
 			(effects

Commit message: .
Parts:
- added U11: AMS1117-5.0, Package_TO_SOT_SMD:SOT-223-3_TabPin2, symbol Regulator_Linear:AMS1117-5.0
Connections:
- net +5V: now also U11.2 (VO); no longer U9.3 (OUT)
- net GND: now also U11.1 (GND); no longer U9.2 (GND)
- net VIN: now also U11.3 (VI); no longer U9.1 (IN)
Changed lines of the file:
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@@
 	)
 	(junction
-		(at 60.96 33.02)
-		(diameter 0)
-		(color 0 0 0 0)
-	)
-	(junction
 		(at 242.57 35.56)
 		(diameter 0)
@@
 	)
 	(junction
-		(at 73.66 33.02)
+		(at 60.96 49.53)
+		(diameter 0)
+		(color 0 0 0 0)
+	)
+	(junction
+		(at 73.66 49.53)
 		(diameter 0)
 		(color 0 0 0 0)
@@
 	(wire
 		(pts
+			(xy 73.66 49.53) (xy 73.66 33.02)
+		)
+		(stroke
+			(width 0)
+			(type default)
+		)
+	)
+	(wire
+		(pts
 			(xy 200.66 83.82) (xy 207.01 83.82)
 		)
@@
 	(wire
 		(pts
-			(xy 87.63 33.02) (xy 73.66 33.02)
+			(xy 87.63 49.53) (xy 73.66 49.53)
 		)
 		(stroke
@@
 	(wire
 		(pts
+			(xy 60.96 52.07) (xy 60.96 49.53)
+		)
+		(stroke
+			(width 0)
+			(type default)
+		)
+	)
+	(wire
+		(pts
 			(xy 60.96 26.67) (xy 60.96 25.4)
 		)
@@
 	(wire
 		(pts
-			(xy 87.63 31.75) (xy 87.63 33.02)
+			(xy 87.63 31.75) (xy 87.63 49.53)
 		)
 		(stroke
@@
 	(wire
 		(pts
-			(xy 87.63 25.4) (xy 99.06 25.4)
+			(xy 60.96 49.53) (xy 73.66 49.53)
 		)
 		(stroke
 			(width 0)
 			(type default)
-			(color 255 0 0 1)
 		)
 	)
 	(wire
 		(pts
-			(xy 149.86 133.35) (xy 156.21 133.35)
+			(xy 87.63 25.4) (xy 99.06 25.4)
 		)
 		(stroke
 			(width 0)
 			(type default)
+			(color 255 0 0 1)
 		)
 	)
 	(wire
 		(pts
-			(xy 95.25 166.37) (xy 95.25 170.18)
+			(xy 149.86 133.35) (xy 156.21 133.35)
 		)
 		(stroke
@@
 	(wire
 		(pts
-			(xy 29.21 139.7) (xy 40.64 139.7)
+			(xy 95.25 166.37) (xy 95.25 170.18)
 		)
 		(stroke
@@
 	(wire
 		(pts
-			(xy 31.75 97.79) (xy 39.37 97.79)
+			(xy 29.21 139.7) (xy 40.64 139.7)
 		)
 		(stroke
@@
 	(wire
 		(pts
-			(xy 60.96 33.02) (xy 73.66 33.02)
+			(xy 31.75 97.79) (xy 39.37 97.79)
 		)
 		(stroke
@@
 	(wire
 		(pts
-			(xy 73.66 33.02) (xy 73.66 36.83)
-		)
-		(stroke
-			(width 0)
-			(type default)
-		)
-	)
-	(wire
-		(pts
-			(xy 60.96 49.53) (xy 60.96 33.02)
-		)
-		(stroke
-			(width 0)
-			(type default)
-		)
-	)
-	(wire
-		(pts
 			(xy 147.32 71.12) (xy 152.4 71.12)
 		)
@@
 	(wire
 		(pts
-			(xy 80.01 154.94) (xy 72.39 154.94)
+			(xy 60.96 31.75) (xy 60.96 49.53)
 		)
 		(stroke
@@
 	(wire
 		(pts
-			(xy 60.96 31.75) (xy 60.96 33.02)
+			(xy 80.01 154.94) (xy 72.39 154.94)
 		)
 		(stroke
@@
 	)
 	(symbol
+		(lib_id "Regulator_Linear:AMS1117-5.0")
+		(at 73.66 25.4 0)
+		(unit 1)
+		(exclude_from_sim no)
+		(in_bom yes)
+		(on_board yes)
+		(dnp no)
+		(fields_autoplaced yes)
+		(property "Reference" "U11"
+			(at 73.66 19.05 0)
+			(effects
+				(font
+					(size 1.27 1.27)
+				)
+			)
+		)
+		(property "Value" "AMS1117-5.0"
+			(at 73.66 21.59 0)
+			(effects
+				(font
+					(size 1.27 1.27)
+				)
+			)
+		)
+		(property "Footprint" "Package_TO_SOT_SMD:SOT-223-3_TabPin2"
+			(at 73.66 20.32 0)
+			(effects
+				(font
+					(size 1.27 1.27)
+				)
+				(hide yes)
+			)
+		)
+		(property "Datasheet" "http://www.advanced-monolithic.com/pdf/ds1117.pdf"
+			(at 76.2 31.75 0)
+			(effects
+				(font
+					(size 1.27 1.27)
+				)
+				(hide yes)
+			)
+		)
+		(property "Description" "1A Low Dropout regulator, positive, 5.0V fixed output, SOT-223"
+			(at 73.66 25.4 0)
+			(effects
+				(font
+					(size 1.27 1.27)
+				)
+				(hide yes)
+			)
+		)
+		(pin "1"
+		)
+		(pin "2"
+		)
+		(pin "3"
+		)
+		(instances
+			(project ""
+				(path "/5f5eb0ac-ab9b-41ab-8d2f-875870c41abc/dab1a116-6bbe-49e5-a398-9f75bdcbe4bf"
+					(reference "U11")
+					(unit 1)
+				)
+			)
+		)
+	)
+	(symbol
 		(lib_id "power:GND")
 		(at 29.21 76.2 270)
@@
 	)
 	(symbol
+		(lib_id "Regulator_Linear:L7805")
+		(at 118.11 22.86 0)
+		(unit 1)
+		(exclude_from_sim no)
+		(in_bom yes)
+		(on_board yes)
+		(dnp no)
+		(fields_autoplaced yes)
+		(property "Reference" "U9"
+			(at 118.11 16.51 0)
+			(effects
+				(font
+					(size 1.27 1.27)
+				)
+			)
+		)
+		(property "Value" "L7805"
+			(at 118.11 19.05 0)
+			(effects
+				(font
+					(size 1.27 1.27)
+				)
+			)
+		)
+		(property "Footprint" "Alexander Footprint Library:LD1117"
+			(at 118.745 26.67 0)
+			(effects
+				(font
+					(size 1.27 1.27)
+					(italic yes)
+				)
+				(justify left)
+				(hide yes)
+			)
+		)
+		(property "Datasheet" "datasheets/Voltage-Regulator_L7805.pdf"
+			(at 118.11 24.13 0)
+			(effects
+				(font
+					(size 1.27 1.27)
+				)
+				(hide yes)
+			)
+		)
+		(property "Description" "Voltage Regulator 1.5A Positive"
+			(at 118.11 22.86 0)
+			(effects
+				(font
+					(size 1.27 1.27)
+				)
+				(hide yes)
+			)
+		)
+		(pin "2"
+		)
+		(pin "1"
+		)
+		(pin "3"
+		)
+		(instances
+			(project "esp32-node-board-40x65_telemetry"
+				(path "/5f5eb0ac-ab9b-41ab-8d2f-875870c41abc/dab1a116-6bbe-49e5-a398-9f75bdcbe4bf"
+					(reference "U9")
+					(unit 1)
+				)
+			)
+		)
+	)
+	(symbol
 		(lib_id "PCM_arduino-library:Arduino_Micro_Socket")
 		(at 86.36 105.41 0)
@@
 		(lib_name "GND_7")
 		(lib_id "power:GND")
-		(at 73.66 36.83 0)
+		(at 60.96 52.07 0)
 		(unit 1)
 		(exclude_from_sim no)
@@
 		(fields_autoplaced yes)
 		(property "Reference" "#PWR035"
-			(at 73.66 43.18 0)
+			(at 60.96 58.42 0)
 			(effects
 				(font
@@
 		)
 		(property "Value" "GND"
-			(at 73.66 41.91 0)
+			(at 60.96 57.15 0)
 			(effects
 				(font
@@
 		)
 		(property "Footprint" ""
-			(at 73.66 36.83 0)
+			(at 60.96 52.07 0)
 			(effects
 				(font
@@
 		)
 		(property "Datasheet" ""
-			(at 73.66 36.83 0)
+			(at 60.96 52.07 0)
 			(effects
 				(font
@@
 		)
 		(property "Description" "Power symbol creates a global label with name \"GND\" , ground"
-			(at 73.66 36.83 0)
+			(at 60.96 52.07 0)
 			(effects
 				(font
@@
 					(unit 1)
 				)
-			)
-		)
-	)
-	(symbol
-		(lib_id "Regulator_Linear:L7805")
-		(at 73.66 25.4 0)
-		(unit 1)
-		(exclude_from_sim no)
-		(in_bom yes)
-		(on_board yes)
-		(dnp no)
-		(fields_autoplaced yes)
-		(property "Reference" "U9"
-			(at 73.66 19.05 0)
-			(effects
-				(font
-					(size 1.27 1.27)
-				)
-			)
-		)
-		(property "Value" "L7805"
-			(at 73.66 21.59 0)
-			(effects
-				(font
-					(size 1.27 1.27)
-				)
-			)
-		)
-		(property "Footprint" "Alexander Footprint Library:LD1117"
-			(at 74.295 29.21 0)
-			(effects
-				(font
-					(size 1.27 1.27)
-					(italic yes)
-				)
-				(justify left)
-				(hide yes)
-			)
-		)
-		(property "Datasheet" "datasheets/Voltage-Regulator_L7805.pdf"
-			(at 73.66 26.67 0)
-			(effects
-				(font
-					(size 1.27 1.27)
-				)
-				(hide yes)
-			)
-		)
-		(property "Description" "Voltage Regulator 1.5A Positive"
-			(at 73.66 25.4 0)
-			(effects
-				(font
-					(size 1.27 1.27)
-				)
-				(hide yes)
-			)
-		)
-		(pin "2"
-		)
-		(pin "1"
-		)
-		(pin "3"
-		)
-		(instances
-			(project "esp32-node-board-40x65_telemetry"
-				(path "/5f5eb0ac-ab9b-41ab-8d2f-875870c41abc/dab1a116-6bbe-49e5-a398-9f75bdcbe4bf"
-					(reference "U9")
-					(unit 1)
-				)

Commit message: .
Connections:
- net 3V3 is gone; now on net +3V3: J20.20 (3V3)
Changed lines of the file:
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@@
 	(wire
 		(pts
-			(xy 134.62 34.29) (xy 134.62 38.1)
+			(xy 134.62 31.75) (xy 134.62 38.1)
 		)
 		(stroke
@@
 	(wire
 		(pts
+			(xy 137.16 31.75) (xy 137.16 38.1)
+		)
+		(stroke
+			(width 0)
+			(type default)
+		)
+	)
+	(wire
+		(pts
 			(xy 133.35 101.6) (xy 133.35 105.41)
 		)
@@
 	(wire
 		(pts
-			(xy 137.16 34.29) (xy 137.16 38.1)
-		)
-		(stroke
-			(width 0)
-			(type default)
-		)
-	)
-	(wire
-		(pts
 			(xy 72.39 162.56) (xy 80.01 162.56)
 		)
@@
 	)
 	(label "3V3"
-		(at 137.16 34.29 0)
+		(at 137.16 35.56 0)
 		(fields_autoplaced yes)
 		(effects
@@
 		(dnp no)
 		(property "Reference" "J20"
-			(at 139.3541 36.83 0)
+			(at 144.018 38.354 0)
 			(effects
 				(font
@@
 	)
 	(symbol
+		(lib_name "+3V3_2")
+		(lib_id "power:+3V3")
+		(at 137.16 31.75 0)
+		(unit 1)
+		(exclude_from_sim no)
+		(in_bom yes)
+		(on_board yes)
+		(dnp no)
+		(property "Reference" "#PWR046"
+			(at 137.16 35.56 0)
+			(effects
+				(font
+					(size 1.27 1.27)
+				)
+				(hide yes)
+			)
+		)
+		(property "Value" "+3V3"
+			(at 137.16 26.162 90)
+			(effects
+				(font
+					(size 1.27 1.27)
+				)
+			)
+		)
+		(property "Footprint" ""
+			(at 137.16 31.75 0)
+			(effects
+				(font
+					(size 1.27 1.27)
+				)
+				(hide yes)
+			)
+		)
+		(property "Datasheet" ""
+			(at 137.16 31.75 0)
+			(effects
+				(font
+					(size 1.27 1.27)
+				)
+				(hide yes)
+			)
+		)
+		(property "Description" "Power symbol creates a global label with name \"+3V3\""
+			(at 137.16 31.75 0)
+			(effects
+				(font
+					(size 1.27 1.27)
+				)
+				(hide yes)
+			)
+		)
+		(pin "1"
+		)
+		(instances
+			(project "esp32-node-board-40x65_telemetry"
+				(path "/5f5eb0ac-ab9b-41ab-8d2f-875870c41abc/dab1a116-6bbe-49e5-a398-9f75bdcbe4bf"
+					(reference "#PWR046")
+					(unit 1)
+				)
+			)
+		)
+	)
+	(symbol
 		(lib_id "power:GND")
 		(at 29.21 76.2 270)
@@
 		(lib_name "+5V_2")
 		(lib_id "power:+5V")
-		(at 134.62 34.29 0)
+		(at 134.62 31.75 0)
 		(unit 1)
 		(exclude_from_sim no)
@@
 		(on_board yes)
 		(dnp no)
-		(fields_autoplaced yes)
 		(property "Reference" "#PWR029"
-			(at 134.62 38.1 0)
+			(at 134.62 35.56 0)
 			(effects
 				(font
@@
 		)
 		(property "Value" "+5V"
-			(at 134.62 29.21 0)
+			(at 134.62 26.67 90)
 			(effects
 				(font
@@
 		)
 		(property "Footprint" ""
-			(at 134.62 34.29 0)
+			(at 134.62 31.75 0)
 			(effects
 				(font
@@
 		)
 		(property "Datasheet" ""
-			(at 134.62 34.29 0)
+			(at 134.62 31.75 0)
 			(effects
 				(font
@@
 		)
 		(property "Description" "Power symbol creates a global label with name \"+5V\""
-			(at 134.62 34.29 0)
+			(at 134.62 31.75 0)
 			(effects
 				(font
