File: esp32-node-box-40x65_telemetry/esp32-node-board-40x65_telemetry/schematics-snips.kicad_sch (KiCad schematic)
At the start: 11 parts, among them J11 Conn_01x06_Socket, J13 Conn_01x02_Socket, Q1 NPN, Q2 NPN, Q3 2N3904, U6 PC817

Commit message: .
Parts:
- added J12: Conn_01x02_Socket, Connector_PinSocket_2.54mm:PinSocket_1x02_P2.54mm_Vertical, symbol Connector:Conn_01x02_Socket
- added R2: 1K, Resistor_SMD:R_1210_3225Metric_Pad1.30x2.65mm_HandSolder, symbol Device:R
- added U2: 4N35, Package_DIP:DIP-6_W7.62mm, symbol Isolator:4N35
Connections:
- net GND: now also U2.2
- new net: R2.2, U2.1
- new net GPIO27: R2.1
- new net V1+: J12.1 (Pin_1), U2.5
- new net V1-: J12.2 (Pin_2), U2.4
- no-connect marks 0 -> 1

Commit message: .
Parts:
- added A1: Arduino_Micro_Socket, PCM_arduino-library:Arduino_Micro_Socket, symbol PCM_arduino-library:Arduino_Micro_Socket
Changed lines of the file:
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@@
+	)
+	(symbol
+		(lib_id "PCM_arduino-library:Arduino_Micro_Socket")
+		(at 157.48 74.93 0)
+		(unit 1)
+		(exclude_from_sim no)
+		(in_bom yes)
+		(on_board no)
+		(dnp no)
+		(fields_autoplaced yes)
+		(property "Reference" "A1"
+			(at 157.48 43.18 0)
+			(effects
+				(font
+					(size 1.524 1.524)
+				)
+			)
+		)
+		(property "Value" "Arduino_Micro_Socket"
+			(at 157.48 45.72 0)
+			(effects
+				(font
+					(size 1.524 1.524)
+				)
+			)
+		)
+		(property "Footprint" "PCM_arduino-library:Arduino_Micro_Socket"
+			(at 157.48 109.22 0)
+			(effects
+				(font
+					(size 1.524 1.524)
+				)
+				(hide yes)
+			)
+		)
+		(property "Datasheet" "https://docs.arduino.cc/hardware/micro"
+			(at 157.48 105.41 0)
+			(effects
+				(font
+					(size 1.524 1.524)
+				)
+				(hide yes)
+			)
+		)
+		(property "Description" "Socket for Arduino Micro"
+			(at 157.48 74.93 0)
+			(effects
+				(font
+					(size 1.27 1.27)
+				)
+				(hide yes)
+			)
+		)
+		(pin "D9"
+		)
+		(pin "SCK"
+		)
+		(pin "D4"
+		)
+		(pin "RST2"
+		)
+		(pin "A4"
+		)
+		(pin "D1"
+		)
+		(pin "D7"
+		)
+		(pin "MISO"
+		)
+		(pin "RST1"
+		)
+		(pin "VIN"
+		)
+		(pin "GND1"
+		)
+		(pin "D6"
+		)
+		(pin "AREF"
+		)
+		(pin "GND2"
+		)
+		(pin "MOSI"
+		)
+		(pin "D8"
+		)
+		(pin "D13"
+		)
+		(pin "D2"
+		)
+		(pin "D3"
+		)
+		(pin "D5"
+		)
+		(pin "3V3"
+		)
+		(pin "A2"
+		)
+		(pin "5V"
+		)
+		(pin "A1"
+		)
+		(pin "D10"
+		)
+		(pin "SS"
+		)
+		(pin "D11"
+		)
+		(pin "D0"
+		)
+		(pin "D12"
+		)
+		(pin "A3"
+		)
+		(pin "A0"
+		)
+		(pin "A5"
+		)
+		(instances
+			(project "esp32-node-board-40x65_telemetry"
+				(path "/5f5eb0ac-ab9b-41ab-8d2f-875870c41abc/4d11314b-2f19-4ab5-8867-985fed32d05b"
+					(reference "A1")
+					(unit 1)
+				)
+			)
+		)
 	)
 	(symbol
