File: esp32-node-box-40x65_telemetry/esp32-node-board-40x65_telemetry/esp32-node-board-40x65_telemetry.kicad_sch (KiCad schematic)
At the start: 43 parts, among them J10 ADC, J14 GPIO, J15 LED_PWR, J16 GND, J17 GND, J18 LED_PWR, J19 LED_PWR, J2 PWR, J26 Conn_UFL-R-SMT, J3 UART, J4 I2C, J5 DAC, J6 SOURCE, J7 LED_PWR, J8 Conn_01x02_Socket, J9 Conn_01x02_Socket, U1 AMS1117-3V3, U3 ULN2003, U4 L7805, U5 74LS595, U7 BME(P)280

Commit message: .
Connections:
- net I1: no longer U3.7 (I7)
- net I5: no longer U3.3 (I3), U3.4 (I4)
- net I7: no longer U3.5 (I5), U3.6 (I6)
- new net: U3.4 (I4), U3.5 (I5)
- new net: U3.6 (I6), U3.7 (I7)

Commit message: .
Connections:
- net I1: now also U3.4 (I4), U3.5 (I5)
- net I3: now also U3.1 (I1); no longer U3.2 (I2)
- net I5: now also U3.3 (I3)
- net I6: no longer U3.1 (I1)
- net I2: now reaches U3.6 (I6), U3.7 (I7)
- new net I4: U3.2 (I2)

Commit message: .
Connections:
- net GPIO17: no longer J1.28 (IO17)
- net I3: now also J1.28 (IO17)
Changed lines of the file:
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@@
 		)
 	)
-	(label "GPIO17"
+	(label "I3"
 		(at 254 67.31 0)
 		(fields_autoplaced yes)

Commit message: .
Connections:
- net I4 is gone; now on net GPIO18: U3.2 (I2)
- net GPIO17: now also J1.28 (IO17), U3.1 (I1)
- net I3: no longer J1.28 (IO17), U3.1 (I1)

Commit message: .
Connections:
- net GPIO18: now also U3.3 (I3); no longer U3.2 (I2)
- net GPIO5: now also U3.2 (I2)
- net I5: no longer U3.3 (I3)
- net SIPO_CLK: no longer J1.12 (IO27)
- net SIPO_DATA: no longer J1.6 (IO34)
- net SIPO_LATCH: no longer J1.8 (IO32)
- new net GPIO27: J1.12 (IO27)
- new net GPIO32: J1.8 (IO32)
- new net GPIO34: J1.6 (IO34)

Commit message: .
Parts:
- J1: footprint Alexander Footprints Library:ESP32-WROOM-Adapter-Socket-2 -> Alexander Footprint Library:ESP32-WROOM-Adapter-Socket-2
Connections:
- net I2 is gone; now on net GPIO23: U3.6 (I6), U3.7 (I7)
- net GPIO19: now also U3.4 (I4), U3.5 (I5)
- net I1: no longer U3.4 (I4), U3.5 (I5)
- net GPIO_33 renamed GPIO33
Changed lines of the file:
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@@
 	)
 	(junction
+		(at 175.26 107.95)
+		(diameter 0)
+		(color 0 0 0 0)
+	)
+	(junction
 		(at 198.12 107.95)
 		(diameter 0)
@@
 	)
 	(junction
-		(at 236.22 105.41)
+		(at 175.26 102.87)
 		(diameter 0)
 		(color 0 0 0 0)
 	)
 	(junction
-		(at 158.75 99.06)
+		(at 236.22 105.41)
 		(diameter 0)
 		(color 0 0 0 0)
 	)
 	(junction
-		(at 175.26 105.41)
+		(at 158.75 99.06)
 		(diameter 0)
 		(color 0 0 0 0)
@@
 	)
 	(junction
-		(at 175.26 100.33)
-		(diameter 0)
-		(color 0 0 0 0)
-	)
-	(junction
 		(at 76.2 26.67)
 		(diameter 0)
@@
 	(wire
 		(pts
-			(xy 170.18 105.41) (xy 175.26 105.41)
-		)
-		(stroke
-			(width 0)
-			(type default)
-		)
-	)
-	(wire
-		(pts
 			(xy 158.75 99.06) (xy 158.75 101.6)
 		)
@@
 	(wire
 		(pts
+			(xy 167.64 102.87) (xy 175.26 102.87)
+		)
+		(stroke
+			(width 0)
+			(type default)
+		)
+	)
+	(wire
+		(pts
 			(xy 35.56 179.07) (xy 34.29 179.07)
 		)
@@
 	(wire
 		(pts
+			(xy 167.64 107.95) (xy 175.26 107.95)
+		)
+		(stroke
+			(width 0)
+			(type default)
+		)
+	)
+	(wire
+		(pts
 			(xy 95.25 76.2) (xy 95.25 77.47)
 		)
@@
 	(wire
 		(pts
-			(xy 170.18 100.33) (xy 175.26 100.33)
-		)
-		(stroke
-			(width 0)
-			(type default)
-		)
-	)
-	(wire
-		(pts
 			(xy 248.92 52.07) (xy 254 52.07)
 		)
@@
 		)
 	)
-	(label "I2"
-		(at 170.18 105.41 0)
-		(fields_autoplaced yes)
-		(effects
-			(font
-				(size 1.27 1.27)
-			)
-			(justify left bottom)
-		)
-	)
 	(label "SOURCE3"
 		(at 19.05 73.66 0)
@@
 		)
 	)
-	(label "GPIO_33"
+	(label "GPIO33"
 		(at 254 92.71 0)
 		(fields_autoplaced yes)
@@
 		)
 	)
+	(label "GPIO23"
+		(at 167.64 107.95 0)
+		(fields_autoplaced yes)
+		(effects
+			(font
+				(size 1.27 1.27)
+			)
+			(justify left bottom)
+		)
+	)
 	(label "I3"
 		(at 160.02 104.14 0)
@@
 		)
 	)
+	(label "GPIO19"
+		(at 167.64 102.87 0)
+		(fields_autoplaced yes)
+		(effects
+			(font
+				(size 1.27 1.27)
+			)
+			(justify left bottom)
+		)
+	)
 	(label "SIPO_CLK"
 		(at 127 93.98 0)
@@
 		)
 	)
-	(label "I1"
-		(at 170.18 100.33 0)
-		(fields_autoplaced yes)
-		(effects
-			(font
-				(size 1.27 1.27)
-			)
-			(justify left bottom)
-		)
-	)
 	(label "BOOT"
 		(at 223.52 127 0)
@@
 			)
 		)
-		(property "Footprint" "Alexander Footprints Library:ESP32-WROOM-Adapter-Socket-2"
+		(property "Footprint" "Alexander Footprint Library:ESP32-WROOM-Adapter-Socket-2"
 			(at 227.33 33.02 0)
 			(effects

Commit message: .
Connections:
- net GPIO17: now also J14.1; no longer J14.6
- net GPIO23: now also J14.6; no longer J14.1
Changed lines of the file:
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@@
+	(wire
+		(pts
+			(xy 49.53 73.66) (xy 58.42 73.66)
+		)
+		(stroke
+			(width 0)
+			(type default)
+		)
+	)
 	(wire
 		(pts
@@
 	(wire
 		(pts
-			(xy 49.53 73.66) (xy 58.42 73.66)
-		)
-		(stroke
-			(width 0)
-			(type default)
-		)
-	)
-	(wire
-		(pts
 			(xy 147.32 82.55) (xy 147.32 83.82)
 		)
@@
 	(wire
 		(pts
+			(xy 236.22 105.41) (xy 236.22 107.95)
+		)
+		(stroke
+			(width 0)
+			(type default)
+		)
+	)
+	(wire
+		(pts
+			(xy 248.92 54.61) (xy 254 54.61)
+		)
+		(stroke
+			(width 0)
+			(type default)
+		)
+	)
+	(wire
+		(pts
+			(xy 248.92 82.55) (xy 254 82.55)
+		)
+		(stroke
+			(width 0)
+			(type default)
+		)
+	)
+	(wire
+		(pts
+			(xy 248.92 97.79) (xy 254 97.79)
+		)
+		(stroke
+			(width 0)
+			(type default)
+		)
+	)
+	(wire
+		(pts
+			(xy 76.2 44.45) (xy 76.2 46.99)
+		)
+		(stroke
+			(width 0)
+			(type default)
+		)
+	)
+	(wire
+		(pts
+			(xy 127 101.6) (xy 137.16 101.6)
+		)
+		(stroke
+			(width 0)
+			(type default)
+		)
+	)
+	(wire
+		(pts
+			(xy 223.52 127) (xy 223.52 147.32)
+		)
+		(stroke
+			(width 0)
+			(type default)
+		)
+	)
+	(wire
+		(pts
+			(xy 24.13 135.89) (xy 34.29 135.89)
+		)
+		(stroke
+			(width 0)
+			(type default)
+		)
+	)
+	(wire
+		(pts
+			(xy 167.64 97.79) (xy 175.26 97.79)
+		)
+		(stroke
+			(width 0)
+			(type default)
+		)
+	)
+	(wire
+		(pts
+			(xy 184.15 53.34) (xy 184.15 55.88)
+		)
+		(stroke
+			(width 0)
+			(type default)
+		)
+	)
+	(wire
+		(pts
+			(xy 24.13 138.43) (xy 34.29 138.43)
+		)
+		(stroke
+			(width 0)
+			(type default)
+		)
+	)
+	(wire
+		(pts
+			(xy 69.85 46.99) (xy 76.2 46.99)
+		)
+		(stroke
+			(width 0)
+			(type default)
+		)
+	)
+	(wire
+		(pts
+			(xy 69.85 26.67) (xy 76.2 26.67)
+		)
+		(stroke
+			(width 0)
+			(type default)
+		)
+	)
+	(wire
+		(pts
 			(xy 49.53 86.36) (xy 58.42 86.36)
-		)
-		(stroke
-			(width 0)
-			(type default)
-		)
-	)
-	(wire
-		(pts
-			(xy 236.22 105.41) (xy 236.22 107.95)
-		)
-		(stroke
-			(width 0)
-			(type default)
-		)
-	)
-	(wire
-		(pts
-			(xy 248.92 54.61) (xy 254 54.61)
-		)
-		(stroke
-			(width 0)
-			(type default)
-		)
-	)
-	(wire
-		(pts
-			(xy 248.92 82.55) (xy 254 82.55)
-		)
-		(stroke
-			(width 0)
-			(type default)
-		)
-	)
-	(wire
-		(pts
-			(xy 248.92 97.79) (xy 254 97.79)
-		)
-		(stroke
-			(width 0)
-			(type default)
-		)
-	)
-	(wire
-		(pts
-			(xy 76.2 44.45) (xy 76.2 46.99)
-		)
-		(stroke
-			(width 0)
-			(type default)
-		)
-	)
-	(wire
-		(pts
-			(xy 127 101.6) (xy 137.16 101.6)
-		)
-		(stroke
-			(width 0)
-			(type default)
-		)
-	)
-	(wire
-		(pts
-			(xy 223.52 127) (xy 223.52 147.32)
-		)
-		(stroke
-			(width 0)
-			(type default)
-		)
-	)
-	(wire
-		(pts
-			(xy 24.13 135.89) (xy 34.29 135.89)
-		)
-		(stroke
-			(width 0)
-			(type default)
-		)
-	)
-	(wire
-		(pts
-			(xy 167.64 97.79) (xy 175.26 97.79)
-		)
-		(stroke
-			(width 0)
-			(type default)
-		)
-	)
-	(wire
-		(pts
-			(xy 184.15 53.34) (xy 184.15 55.88)
-		)
-		(stroke
-			(width 0)
-			(type default)
-		)
-	)
-	(wire
-		(pts
-			(xy 24.13 138.43) (xy 34.29 138.43)
-		)
-		(stroke
-			(width 0)
-			(type default)
-		)
-	)
-	(wire
-		(pts
-			(xy 69.85 46.99) (xy 76.2 46.99)
-		)
-		(stroke
-			(width 0)
-			(type default)
-		)
-	)
-	(wire
-		(pts
-			(xy 69.85 26.67) (xy 76.2 26.67)
 		)
 		(stroke
@@
 	)
 	(label "GPIO23"
-		(at 49.53 73.66 0)
+		(at 49.53 86.36 0)
 		(fields_autoplaced yes)
 		(effects
@@
 	)
 	(label "GPIO17"
-		(at 49.53 86.36 0)
-		(fields_autoplaced yes)
-		(effects
+		(at 49.53 73.66 0)
+		(fields_autoplaced yes)
+		(effects

Commit message: .
Connections:
- net GPIO19: now also J14.6; no longer J14.4
- net GPIO23: now also J14.5; no longer J14.6
- net GPIO5: now also J14.4; no longer J14.5
