File: ESP32-WROOM-Socket-v4-SMD/ESP32-WROOM-Socket-v4-SMD.kicad_sch (KiCad schematic)
At the start: 9 parts, among them SW1 PRG, U1 ESP32-WROOM-32D

Commit message: .
Parts:
- added R2: R, Alexander Footprints Library:R_2.5mm, symbol Device:R
Connections:
- net GND: now also R2.2
- net at D1.1 (K), R1.1: no longer D2.1 (K)
- new net: D2.1 (K), R2.1
Other:
- moved on the sheet: U1
Changed lines of the file:
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@@
 	(paper "A4")
 	(junction
-		(at 80.01 78.74)
+		(at 80.01 97.79)
 		(diameter 0)
 		(color 0 0 0 0)
@@
 	(wire
 		(pts
-			(xy 80.01 88.9) (xy 80.01 99.06)
+			(xy 67.31 88.9) (xy 67.31 97.79)
+		)
+		(stroke
+			(width 0)
+			(type default)
+		)
+	)
+	(wire
+		(pts
+			(xy 80.01 88.9) (xy 80.01 97.79)
 		)
 		(stroke
@@
 	(wire
 		(pts
-			(xy 134.62 133.35) (xy 134.62 137.16)
-		)
-		(stroke
-			(width 0)
-			(type default)
-		)
-	)
-	(wire
-		(pts
-			(xy 80.01 72.39) (xy 80.01 78.74)
+			(xy 67.31 97.79) (xy 80.01 97.79)
+		)
+		(stroke
+			(width 0)
+			(type default)
+		)
+	)
+	(wire
+		(pts
+			(xy 252.73 106.68) (xy 252.73 110.49)
 		)
 		(stroke
@@
 	(wire
 		(pts
-			(xy 80.01 78.74) (xy 80.01 81.28)
+			(xy 80.01 72.39) (xy 80.01 81.28)
 		)
 		(stroke
@@
 	(wire
 		(pts
-			(xy 67.31 72.39) (xy 67.31 78.74)
-		)
-		(stroke
-			(width 0)
-			(type default)
-		)
-	)
-	(wire
-		(pts
-			(xy 67.31 78.74) (xy 80.01 78.74)
-		)
-		(stroke
-			(width 0)
-			(type default)
-		)
-	)
-	(wire
-		(pts
-			(xy 134.62 57.15) (xy 134.62 62.23)
-		)
-		(stroke
-			(width 0)
-			(type default)
-		)
-	)
-	(wire
-		(pts
-			(xy 149.86 67.31) (xy 152.4 67.31)
+			(xy 80.01 97.79) (xy 80.01 99.06)
+		)
+		(stroke
+			(width 0)
+			(type default)
+		)
+	)
+	(wire
+		(pts
+			(xy 67.31 72.39) (xy 67.31 81.28)
+		)
+		(stroke
+			(width 0)
+			(type default)
+		)
+	)
+	(wire
+		(pts
+			(xy 252.73 30.48) (xy 252.73 35.56)
+		)
+		(stroke
+			(width 0)
+			(type default)
+		)
+	)
+	(wire
+		(pts
+			(xy 267.97 40.64) (xy 270.51 40.64)
 		)
 		(stroke
@@
 	)
 	(label "GND"
-		(at 134.62 137.16 90)
+		(at 252.73 110.49 90)
 		(fields_autoplaced yes)
 		(effects
@@
 	)
 	(label "3V3"
-		(at 134.62 57.15 270)
+		(at 252.73 30.48 270)
 		(fields_autoplaced yes)
 		(effects
@@
 	)
 	(label "PRG"
-		(at 152.4 67.31 0)
+		(at 270.51 40.64 0)
 		(fields_autoplaced yes)
 		(effects
@@
 	(symbol
 		(lib_id "RF_Module:ESP32-WROOM-32D")
-		(at 134.62 97.79 0)
+		(at 252.73 71.12 0)
 		(unit 1)
 		(exclude_from_sim no)
@@
 		(fields_autoplaced yes)
 		(property "Reference" "U1"
-			(at 136.8141 59.69 0)
+			(at 254.9241 33.02 0)
 			(effects
 				(font
@@
 		)
 		(property "Value" "ESP32-WROOM-32D"
-			(at 136.8141 62.23 0)
+			(at 254.9241 35.56 0)
 			(effects
 				(font
@@
 		)
 		(property "Footprint" "Alexander Footprints Library:ESP32-WROOM-Adapter-2"
-			(at 151.13 132.08 0)
+			(at 269.24 105.41 0)
 			(effects
 				(font
@@
 		)
 		(property "Datasheet" "https://www.espressif.com/sites/default/files/documentation/esp32-wroom-32d_esp32-wroom-32u_datasheet_en.pdf"
-			(at 127 96.52 0)
+			(at 245.11 69.85 0)
 			(effects
 				(font
@@
 		)
 		(property "Description" ""
-			(at 134.62 97.79 0)
+			(at 252.73 71.12 0)
 			(effects
 				(font
@@
 	)
 	(symbol
+		(lib_id "Device:R")
+		(at 67.31 85.09 0)
+		(unit 1)
+		(exclude_from_sim no)
+		(in_bom yes)
+		(on_board yes)
+		(dnp no)
+		(fields_autoplaced yes)
+		(property "Reference" "R2"
+			(at 69.85 83.82 0)
+			(effects
+				(font
+					(size 1.27 1.27)
+				)
+				(justify left)
+			)
+		)
+		(property "Value" "R"
+			(at 69.85 86.36 0)
+			(effects
+				(font
+					(size 1.27 1.27)
+				)
+				(justify left)
+			)
+		)
+		(property "Footprint" "Alexander Footprints Library:R_2.5mm"
+			(at 65.532 85.09 90)
+			(effects
+				(font
+					(size 1.27 1.27)
+				)
+				(hide yes)
+			)
+		)
+		(property "Datasheet" "~"
+			(at 67.31 85.09 0)
+			(effects
+				(font
+					(size 1.27 1.27)
+				)
+				(hide yes)
+			)
+		)
+		(property "Description" ""
+			(at 67.31 85.09 0)
+			(effects
+				(font
+					(size 1.27 1.27)
+				)
+				(hide yes)
+			)
+		)
+		(pin "1"
+		)
+		(pin "2"
+		)
+		(instances
+			(project "ESP32-WROOM-Socket-v4-SMD"
+				(path "/b6a3c81b-cf0c-432f-80e1-65c551ea51bb"
+					(reference "R2")
+					(unit 1)
+				)
+			)
+		)
+	)
+	(symbol
 		(lib_id "Device:LED")
 		(at 80.01 68.58 90)
@@
 		)
 		(instances
-			(project "esp32-wroom-socket-v2"
+			(project "ESP32-WROOM-Socket-v4-SMD"
 				(path "/b6a3c81b-cf0c-432f-80e1-65c551ea51bb"
 					(page "2")
