File: ESP32-C3-WROOM-Node-Temperature/ESP32-C3-WROOM-Node-Temperature/ESP32-C3-WROOM-Node-Temperature.kicad_pcb (KiCad board)
At the start: 2 copper layers, 65 x 40 mm, 22 parts, among them J1 PWR, K1 Relay_DPDT_HK19F_HUI, Q1 NPN, U2 AMS1117-3V3, U4 L7805

Commit message: .
Parts:
- R1, R3: footprint Resistor_SMD:R_2512_6332Metric_Pad1.40x3.35mm_HandSolder -> Resistor_SMD:R_1206_3216Metric_Pad1.30x1.75mm_HandSolder
- moved R1 2.07 mm to (150.0, 72.8), turned to -90 degrees
Changed lines of the file:
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@@
 		)
 	)
-	(footprint "Resistor_SMD:R_2512_6332Metric_Pad1.40x3.35mm_HandSolder"
+	(footprint "Resistor_SMD:R_1206_3216Metric_Pad1.30x1.75mm_HandSolder"
 		(layer "F.Cu")
-		(at 147.95 72.5)
-		(descr "Resistor SMD 2512 (6332 Metric), square (rectangular) end terminal, IPC_7351 nominal with elongated pad for handsoldering. (Body size source: IPC-SM-782 page 72, https://www.pcb-3d.com/wordpress/wp-content/uploads/ipc-sm-782a_amendment_1_and_2.pdf), generated with kicad-footprint-generator")
+		(at 150 72.75 -90)
+		(descr "Resistor SMD 1206 (3216 Metric), square (rectangular) end terminal, IPC_7351 nominal with elongated pad for handsoldering. (Body size source: IPC-SM-782 page 72, https://www.pcb-3d.com/wordpress/wp-content/uploads/ipc-sm-782a_amendment_1_and_2.pdf), generated with kicad-footprint-generator")
 		(tags "resistor handsolder")
 		(property "Reference" "R1"
-			(at 0 -2.62 0)
+			(at 0 -1.82 90)
 			(layer "F.SilkS")
 			(effects
@@
 		)
 		(property "Value" "10K"
-			(at 0 2.62 0)
+			(at 0 1.82 90)
 			(layer "F.Fab")
 			(effects
@@
 			)
 		)
-		(property "Footprint" "Resistor_SMD:R_2512_6332Metric_Pad1.40x3.35mm_HandSolder"
-			(at 0 0 0)
+		(property "Footprint" "Resistor_SMD:R_1206_3216Metric_Pad1.30x1.75mm_HandSolder"
+			(at 0 0 -90)
 			(unlocked yes)
 			(layer "F.Fab")
@@
 		)
 		(property "Datasheet" ""
-			(at 0 0 0)
+			(at 0 0 -90)
 			(unlocked yes)
 			(layer "F.Fab")
@@
 		)
 		(property "Description" "Resistor"
-			(at 0 0 0)
+			(at 0 0 -90)
 			(unlocked yes)
 			(layer "F.Fab")
@@
 		(attr smd)
 		(fp_line
-			(start -2.177064 -1.71)
-			(end 2.177064 -1.71)
+			(start -0.727064 0.91)
+			(end 0.727064 0.91)
 			(stroke
 				(width 0.12)
@@
 		)
 		(fp_line
-			(start -2.177064 1.71)
-			(end 2.177064 1.71)
+			(start -0.727064 -0.91)
+			(end 0.727064 -0.91)
 			(stroke
 				(width 0.12)
@@
 		)
 		(fp_line
-			(start -4 -1.92)
-			(end 4 -1.92)
+			(start -2.45 1.12)
+			(end -2.45 -1.12)
 			(stroke
 				(width 0.05)
@@
 		)
 		(fp_line
-			(start -4 1.92)
-			(end -4 -1.92)
+			(start 2.45 1.12)
+			(end -2.45 1.12)
 			(stroke
 				(width 0.05)
@@
 		)
 		(fp_line
-			(start 4 -1.92)
-			(end 4 1.92)
+			(start -2.45 -1.12)
+			(end 2.45 -1.12)
 			(stroke
 				(width 0.05)
@@
 		)
 		(fp_line
-			(start 4 1.92)
-			(end -4 1.92)
+			(start 2.45 -1.12)
+			(end 2.45 1.12)
 			(stroke
 				(width 0.05)
@@
 		)
 		(fp_line
-			(start -3.15 -1.6)
-			(end 3.15 -1.6)
+			(start -1.6 0.8)
+			(end -1.6 -0.8)
 			(stroke
 				(width 0.1)
@@
 		)
 		(fp_line
-			(start -3.15 1.6)
-			(end -3.15 -1.6)
+			(start 1.6 0.8)
+			(end -1.6 0.8)
 			(stroke
 				(width 0.1)
@@
 		)
 		(fp_line
-			(start 3.15 -1.6)
-			(end 3.15 1.6)
+			(start -1.6 -0.8)
+			(end 1.6 -0.8)
 			(stroke
 				(width 0.1)
@@
 		)
 		(fp_line
-			(start 3.15 1.6)
-			(end -3.15 1.6)
+			(start 1.6 -0.8)
+			(end 1.6 0.8)
 			(stroke
 				(width 0.1)
@@
 		)
 		(fp_text user "${REFERENCE}"
-			(at 0 0 0)
+			(at 0 0 90)
 			(layer "F.Fab")
 			(effects
 				(font
-					(size 1 1)
-					(thickness 0.15)
+					(size 0.8 0.8)
+					(thickness 0.12)
 				)
 			)
 		)
 		(pad "1" smd roundrect
-			(at -3.05 0)
-			(size 1.4 3.35)
+			(at -1.55 0 270)
+			(size 1.3 1.75)
 			(layers "F.Cu" "F.Paste" "F.Mask")
-			(roundrect_rratio 0.178571)
+			(roundrect_rratio 0.192308)
 			(net 1 "Net-(Q1-B)")
 			(pintype "passive")
 		)
 		(pad "2" smd roundrect
-			(at 3.05 0)
-			(size 1.4 3.35)
+			(at 1.55 0 270)
+			(size 1.3 1.75)
 			(layers "F.Cu" "F.Paste" "F.Mask")
-			(roundrect_rratio 0.178571)
+			(roundrect_rratio 0.192308)
 			(net 7 "/GPIO10")
 			(pintype "passive")
 		)
-		(model "${KICAD8_3DMODEL_DIR}/Resistor_SMD.3dshapes/R_2512_6332Metric.wrl"
+		(model "${KICAD8_3DMODEL_DIR}/Resistor_SMD.3dshapes/R_1206_3216Metric.wrl"
 			(offset
 				(xyz 0 0 0)
@@
 		)
 	)
-	(footprint "Resistor_SMD:R_2512_6332Metric_Pad1.40x3.35mm_HandSolder"
+	(footprint "Resistor_SMD:R_1206_3216Metric_Pad1.30x1.75mm_HandSolder"
 		(layer "F.Cu")
 		(at 96.01 71.12)
-		(descr "Resistor SMD 2512 (6332 Metric), square (rectangular) end terminal, IPC_7351 nominal with elongated pad for handsoldering. (Body size source: IPC-SM-782 page 72, https://www.pcb-3d.com/wordpress/wp-content/uploads/ipc-sm-782a_amendment_1_and_2.pdf), generated with kicad-footprint-generator")
+		(descr "Resistor SMD 1206 (3216 Metric), square (rectangular) end terminal, IPC_7351 nominal with elongated pad for handsoldering. (Body size source: IPC-SM-782 page 72, https://www.pcb-3d.com/wordpress/wp-content/uploads/ipc-sm-782a_amendment_1_and_2.pdf), generated with kicad-footprint-generator")
 		(tags "resistor handsolder")
 		(property "Reference" "R3"
-			(at 0 -2.62 0)
+			(at 0 -1.82 0)
 			(layer "F.SilkS")
 			(effects
@@
 		)
 		(property "Value" "R"
-			(at 0 2.62 0)
+			(at 0 1.82 0)
 			(layer "F.Fab")
 			(effects
@@
 			)
 		)
-		(property "Footprint" "Resistor_SMD:R_2512_6332Metric_Pad1.40x3.35mm_HandSolder"
+		(property "Footprint" "Resistor_SMD:R_1206_3216Metric_Pad1.30x1.75mm_HandSolder"
 			(at 0 0 0)
 			(unlocked yes)
@@
 		(attr smd)
 		(fp_line
-			(start -2.177064 -1.71)
-			(end 2.177064 -1.71)
+			(start -0.727064 -0.91)
+			(end 0.727064 -0.91)
 			(stroke
 				(width 0.12)
@@
 		)
 		(fp_line
-			(start -2.177064 1.71)
-			(end 2.177064 1.71)
+			(start -0.727064 0.91)
+			(end 0.727064 0.91)
 			(stroke
 				(width 0.12)
@@
 		)
 		(fp_line
-			(start -4 -1.92)
-			(end 4 -1.92)
+			(start -2.45 -1.12)
+			(end 2.45 -1.12)
 			(stroke
 				(width 0.05)
@@
 		)
 		(fp_line
-			(start -4 1.92)
-			(end -4 -1.92)
+			(start -2.45 1.12)
+			(end -2.45 -1.12)
 			(stroke
 				(width 0.05)
@@
 		)
 		(fp_line
-			(start 4 -1.92)
-			(end 4 1.92)
+			(start 2.45 -1.12)
+			(end 2.45 1.12)
 			(stroke
 				(width 0.05)
@@
 		)
 		(fp_line
-			(start 4 1.92)
-			(end -4 1.92)
+			(start 2.45 1.12)
+			(end -2.45 1.12)
 			(stroke
 				(width 0.05)
@@
 		)
 		(fp_line
-			(start -3.15 -1.6)
-			(end 3.15 -1.6)
+			(start -1.6 -0.8)
+			(end 1.6 -0.8)
 			(stroke
 				(width 0.1)
@@
 		)
 		(fp_line
-			(start -3.15 1.6)
-			(end -3.15 -1.6)
+			(start -1.6 0.8)
+			(end -1.6 -0.8)
 			(stroke
 				(width 0.1)
@@
 		)
 		(fp_line
-			(start 3.15 -1.6)
-			(end 3.15 1.6)
+			(start 1.6 -0.8)
+			(end 1.6 0.8)
 			(stroke
 				(width 0.1)
@@
 		)
 		(fp_line
-			(start 3.15 1.6)
-			(end -3.15 1.6)
+			(start 1.6 0.8)
+			(end -1.6 0.8)
 			(stroke
 				(width 0.1)
@@
 			(effects
 				(font
-					(size 1 1)
-					(thickness 0.15)
+					(size 0.8 0.8)
+					(thickness 0.12)
 				)
 			)
 		)
 		(pad "1" smd roundrect
-			(at -3.05 0)
-			(size 1.4 3.35)
+			(at -1.55 0)
+			(size 1.3 1.75)
 			(layers "F.Cu" "F.Paste" "F.Mask")
-			(roundrect_rratio 0.178571)
+			(roundrect_rratio 0.192308)
 			(net 29 "+3.3V")
 			(pintype "passive")
 		)
 		(pad "2" smd roundrect
-			(at 3.05 0)
-			(size 1.4 3.35)
+			(at 1.55 0)
+			(size 1.3 1.75)
 			(layers "F.Cu" "F.Paste" "F.Mask")
-			(roundrect_rratio 0.178571)
+			(roundrect_rratio 0.192308)
 			(net 9 "/ADC1")
 			(pintype "passive")
 		)
-		(model "${KICAD8_3DMODEL_DIR}/Resistor_SMD.3dshapes/R_2512_6332Metric.wrl"
+		(model "${KICAD8_3DMODEL_DIR}/Resistor_SMD.3dshapes/R_1206_3216Metric.wrl"
 			(offset
 				(xyz 0 0 0)

Commit message: .
Parts:
- moved C4 55.8 mm to (136.2, 73.0), turned to -90 degrees
- moved U2 54.8 mm to (133.7, 65.5)
- moved R3 52.7 mm to (142.2, 96.5)
- moved C5 51.3 mm to (130.8, 73.0), turned to -90 degrees
- moved D2 40.1 mm to (126.8, 64.2), turned to 90 degrees
- moved J1 38.1 mm to (121.9, 66.0), turned to 180 degrees
- moved U4 33.7 mm to (113.6, 68.2), turned to -90 degrees
- moved K1 10.5 mm to (142.0, 83.9)

Commit message: .
Parts:
- moved C3 50.7 mm to (118.2, 93.8)
- moved C2 46.5 mm to (113.8, 88.5)
- moved C1 45.9 mm to (113.8, 81.0)
- moved R1 23.8 mm to (172.7, 79.7)
- moved U1 23.4 mm to (167.6, 73.7), turned to 180 degrees
- moved R2 18.5 mm to (150.5, 66.8), turned to 90 degrees
- moved U3 15.4 mm to (168.9, 72.3), turned to 180 degrees
- moved D1 14.8 mm to (157.5, 53.3)
Changed lines of the file:
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@@
 	(footprint "Alexander Footprint Library:BME280_BMP280_I2C"
 		(layer "F.Cu")
-		(at 153.72 74.96 90)
+		(at 168.94 72.34 180)
 		(descr "Temperature, Humidity and Pressure sensor")
 		(tags "BME BMP 280 sensor")
 		(property "Reference" "U3"
-			(at 0 -0.6 90)
+			(at 0 -0.6 180)
 			(unlocked yes)
 			(layer "F.SilkS")
@@
 		)
 		(property "Value" "~"
-			(at 0 1 90)
+			(at 0 1 180)
 			(unlocked yes)
 			(layer "F.Fab")
@@
 		)
 		(property "Footprint" "Alexander Footprint Library:BME280_BMP280_I2C"
-			(at 0 0 90)
+			(at 0 0 180)
 			(unlocked yes)
 			(layer "F.Fab")
@@
 		)
 		(property "Datasheet" ""
-			(at 0 0 90)
+			(at 0 0 180)
 			(unlocked yes)
 			(layer "F.Fab")
@@
 		)
 		(property "Description" "BME(P)-280 I2C Environment Sensor"
-			(at 0 0 90)
+			(at 0 0 180)
 			(unlocked yes)
 			(layer "F.Fab")
@@
 		)
 		(fp_text user "BME(P) 280"
-			(at 6.8 5 180)
+			(at 6.8 5 -90)
 			(unlocked yes)
 			(layer "F.SilkS")
@@
 		)
 		(fp_text user "${REFERENCE}"
-			(at 0 2.5 90)
+			(at 0 2.5 180)
 			(unlocked yes)
 			(layer "F.Fab")
@@
 		)
 		(pad "1" thru_hole rect
-			(at 1.3 1.22 90)
+			(at 1.3 1.22 180)
 			(size 1.524 1.524)
 			(drill 0.762)
@@
 		)
 		(pad "2" thru_hole circle
-			(at 1.3 3.76 90)
+			(at 1.3 3.76 180)
 			(size 1.524 1.524)
 			(drill 0.762)
@@
 		)
 		(pad "3" thru_hole circle
-			(at 1.3 6.3 90)
+			(at 1.3 6.3 180)
 			(size 1.524 1.524)
 			(drill 0.762)
@@
 		)
 		(pad "4" thru_hole circle
-			(at 1.3 8.84 90)
+			(at 1.3 8.84 180)
 			(size 1.524 1.524)
 			(drill 0.762)
@@
 	(footprint "Resistor_SMD:R_1206_3216Metric_Pad1.30x1.75mm_HandSolder"
 		(layer "F.Cu")
-		(at 150 72.75 -90)
+		(at 172.72 79.73 -90)
 		(descr "Resistor SMD 1206 (3216 Metric), square (rectangular) end terminal, IPC_7351 nominal with elongated pad for handsoldering. (Body size source: IPC-SM-782 page 72, https://www.pcb-3d.com/wordpress/wp-content/uploads/ipc-sm-782a_amendment_1_and_2.pdf), generated with kicad-footprint-generator")
 		(tags "resistor handsolder")
@@
 	(footprint "LED_THT:LED_D5.0mm"
 		(layer "F.Cu")
-		(at 149.86 66.04 90)
+		(at 157.48 53.34 90)
 		(descr "LED, diameter 5.0mm, 2 pins, http://cdn-reichelt.de/documents/datenblatt/A500/LL-504BC2E-009.pdf")
 		(tags "LED diameter 5.0mm 2 pins")
@@
 	(footprint "Alexander Footprint Library:ESP32-C3_SuperMini"
 		(layer "F.Cu")
-		(at 144.78 78.74 -90)
+		(at 167.64 73.66 180)
 		(descr "ESP32 C3 Super Mini")
 		(tags "ESP32 C3")
 		(property "Reference" "U1"
-			(at 0 -0.5 -90)
+			(at 0 -0.5 180)
 			(unlocked yes)
 			(layer "F.SilkS")
@@
 		)
 		(property "Value" "~"
-			(at 0 1 -90)
+			(at 0 1 180)
 			(unlocked yes)
 			(layer "F.Fab")
@@
 		)
 		(property "Footprint" "Alexander Footprint Library:ESP32-C3_SuperMini"
-			(at 0 0 -90)
+			(at 0 0 180)
 			(unlocked yes)
 			(layer "F.Fab")
@@
 		)
 		(property "Datasheet" ""
-			(at 0 0 -90)
+			(at 0 0 180)
 			(unlocked yes)
 			(layer "F.Fab")
@@
 		)
 		(property "Description" ""
-			(at 0 0 -90)
+			(at 0 0 180)
 			(unlocked yes)
 			(layer "F.Fab")
@@
 		(attr through_hole)
 		(fp_text user "${REFERENCE}"
-			(at 0 2.5 -90)
+			(at 0 2.5 180)
 			(unlocked yes)
 			(layer "F.Fab")
@@
 		)
 		(pad "1" thru_hole roundrect
-			(at 0 -20.32 270)
+			(at 0 -20.32 180)
 			(size 1.7 1.7)
 			(drill 1)
@@
 		)
 		(pad "2" thru_hole oval
-			(at 0 -17.78 270)
+			(at 0 -17.78 180)
 			(size 1.7 1.7)
 			(drill 1)
@@
 		)
 		(pad "3" thru_hole oval
-			(at 0 -15.24 270)
+			(at 0 -15.24 180)
 			(size 1.7 1.7)
 			(drill 1)
@@
 		)
 		(pad "4" thru_hole oval
-			(at 0 -12.7 270)
+			(at 0 -12.7 180)
 			(size 1.7 1.7)
 			(drill 1)
@@
 		)
 		(pad "5" thru_hole oval
-			(at 0 -10.16 270)
+			(at 0 -10.16 180)
 			(size 1.7 1.7)
 			(drill 1)
@@
 		)
 		(pad "6" thru_hole oval
-			(at 0 -7.62 270)
+			(at 0 -7.62 180)
 			(size 1.7 1.7)
 			(drill 1)
@@
 		)
 		(pad "7" thru_hole oval
-			(at 0 -5.08 270)
+			(at 0 -5.08 180)
 			(size 1.7 1.7)
 			(drill 1)
@@
 		)
 		(pad "8" thru_hole oval
-			(at 0 -2.54 270)
+			(at 0 -2.54 180)
 			(size 1.7 1.7)
 			(drill 1)
@@
 		)
 		(pad "9" thru_hole oval
-			(at 15.24 -2.54 270)
+			(at 15.24 -2.54 180)
 			(size 1.7 1.7)
 			(drill 1)
@@
 		)
 		(pad "10" thru_hole oval
-			(at 15.24 -5.08 270)
+			(at 15.24 -5.08 180)
 			(size 1.7 1.7)
 			(drill 1)
@@
 		)
 		(pad "11" thru_hole oval
-			(at 15.24 -7.62 270)
+			(at 15.24 -7.62 180)
 			(size 1.7 1.7)
 			(drill 1)
@@
 		)
 		(pad "12" thru_hole oval
-			(at 15.24 -10.16 270)
+			(at 15.24 -10.16 180)
 			(size 1.7 1.7)
 			(drill 1)
@@
 		)
 		(pad "13" thru_hole oval
-			(at 15.24 -12.7 270)
+			(at 15.24 -12.7 180)
 			(size 1.7 1.7)
 			(drill 1)
@@
 		)
 		(pad "14" thru_hole oval
-			(at 15.24 -15.24 270)
+			(at 15.24 -15.24 180)
 			(size 1.7 1.7)
 			(drill 1)
@@
 		)
 		(pad "15" thru_hole rect
-			(at 15.24 -17.78 270)
+			(at 15.24 -17.78 180)
 			(size 1.7 1.7)
 			(drill 1)
@@
 		)
 		(pad "16" thru_hole oval
-			(at 15.24 -20.32 270)
+			(at 15.24 -20.32 180)
 			(size 1.7 1.7)
 			(drill 1)
@@
 	(footprint "Capacitor_THT:CP_Radial_D4.0mm_P2.00mm"
 		(layer "F.Cu")
-		(at 70.214801 77.66)
+		(at 118.25 93.75)
 		(descr "CP, Radial series, Radial, pin pitch=2.00mm, , diameter=4mm, Electrolytic Capacitor")
 		(tags "CP Radial series Radial pin pitch 2.00mm  diameter 4mm Electrolytic Capacitor")
@@
 	(footprint "Package_TO_SOT_THT:TO-46-2_Pin2Center"
 		(layer "F.Cu")
-		(at 168.91 68.58)
+		(at 150.5 66.77 90)
 		(descr "TO-46-2, Pin2 at center of package, Thorlabs photodiodes")
 		(tags "TO-46-2 Thorlabs")
 		(property "Reference" "R2"
-			(at 1.27 -4.02 0)
+			(at 1.27 -4.02 90)
 			(layer "F.SilkS")
 			(effects
@@
 		)
 		(property "Value" "R_Photo"
-			(at 1.27 4.02 0)
+			(at 1.27 4.02 90)
 			(layer "F.Fab")
 			(effects
@@
 		)
 		(property "Footprint" "Package_TO_SOT_THT:TO-46-2_Pin2Center"
-			(at 0 0 0)
+			(at 0 0 90)
 			(unlocked yes)
 			(layer "F.Fab")
@@
 		)
 		(property "Datasheet" ""
-			(at 0 0 0)
+			(at 0 0 90)
 			(unlocked yes)
 			(layer "F.Fab")
@@
 		)
 		(property "Description" "Photoresistor"
-			(at 0 0 0)
+			(at 0 0 90)
 			(unlocked yes)
 			(layer "F.Fab")
@@
 		(attr through_hole)
 		(fp_line
-			(start -2.58 -0.6)
-			(end -2.58 0.75)
+			(start -1.68 -0.6)
+			(end -2.58 -0.6)
 			(stroke
 				(width 0.12)
@@
 		)
 		(fp_line
-			(start -2.58 0.75)
-			(end -1.68 0.75)
+			(start -2.58 -0.6)
+			(end -2.58 0.75)
 			(stroke
 				(width 0.12)
@@
 		)
 		(fp_line
-			(start -1.68 -0.6)
-			(end -2.58 -0.6)
+			(start -2.58 0.75)
+			(end -1.68 0.75)
 			(stroke
 				(width 0.12)
@@
 		(fp_line
 			(start -2.73 -3.15)
-			(end -2.73 3.14)
+			(end 4.42 -3.15)
 			(stroke
 				(width 0.05)
@@
 		(fp_line
 			(start -2.73 -3.15)
-			(end 4.42 -3.15)
+			(end -2.73 3.14)
 			(stroke
 				(width 0.05)
@@
 		(fp_line
 			(start 4.42 3.14)
-			(end -2.73 3.14)
+			(end 4.42 -3.15)
 			(stroke
 				(width 0.05)
@@
 		(fp_line
 			(start 4.42 3.14)
-			(end 4.42 -3.15)
+			(end -2.73 3.14)
 			(stroke
 				(width 0.05)
@@
 		)
 		(fp_line
-			(start -2.48 -0.5)
-			(end -2.48 0.65)
+			(start -1.58 -0.5)
+			(end -2.48 -0.5)
 			(stroke
 				(width 0.1)
@@
 		)
 		(fp_line
-			(start -2.48 0.65)
-			(end -1.58 0.65)
+			(start -2.48 -0.5)
+			(end -2.48 0.65)
 			(stroke
 				(width 0.1)
@@
 		)
 		(fp_line
-			(start -1.58 -0.5)
-			(end -2.48 -0.5)
+			(start -2.48 0.65)
+			(end -1.58 0.65)
 			(stroke
 				(width 0.1)
@@
 		)
 		(fp_text user "${REFERENCE}"
-			(at 1.27 -4.02 0)
+			(at 1.27 -4.02 90)
 			(layer "F.Fab")
 			(effects
@@
 		)
 		(pad "1" thru_hole oval
-			(at 0 0 90)
+			(at 0 0 180)
 			(size 1.5 1)
 			(drill 0.7)
@@
 		)
 		(pad "2" thru_hole oval
-			(at 1.27 0)
+			(at 1.27 0 90)
 			(size 1 1)
 			(drill 0.6)
@@
 	(footprint "Capacitor_THT:CP_Radial_D4.0mm_P2.00mm"
 		(layer "F.Cu")
-		(at 70.214801 66.56)
+		(at 113.75 81)
 		(descr "CP, Radial series, Radial, pin pitch=2.00mm, , diameter=4mm, Electrolytic Capacitor")
 		(tags "CP Radial series Radial pin pitch 2.00mm  diameter 4mm Electrolytic Capacitor")
@@
 	(footprint "Capacitor_THT:CP_Radial_D4.0mm_P2.00mm"
 		(layer "F.Cu")
-		(at 70.214801 72.11)
+		(at 113.75 88.5)
 		(descr "CP, Radial series, Radial, pin pitch=2.00mm, , diameter=4mm, Electrolytic Capacitor")
 		(tags "CP Radial series Radial pin pitch 2.00mm  diameter 4mm Electrolytic Capacitor")

Commit message: .
Parts:
- moved Q1 0.23 mm to (142.2, 63.7)
Routing:
- added copper zone on F.Cu, net GND
Changed lines of the file:
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@@
 	(footprint "Package_TO_SOT_THT:TO-92"
 		(layer "F.Cu")
-		(at 142.24 63.5 -90)
+		(at 142.24 63.73 -90)
 		(descr "TO-92 leads molded, narrow, drill 0.75mm (see NXP sot054_po.pdf)")
 		(tags "to-92 sc-43 sc-43a sot54 PA33 transistor")
@@
 			)
 		)
+	)
+	(zone
+		(net 3)
+		(net_name "GND")
+		(layer "F.Cu")
+		(hatch edge 0.5)
+		(priority 1)
+		(connect_pads
+			(clearance 0.5)
+		)
+		(min_thickness 0.25)
+		(filled_areas_thickness no)
+		(fill yes
+			(thermal_gap 0.5)
+			(thermal_bridge_width 0.5)
+		)
+		(polygon
+			(pts
+				(xy 110.5 59.25) (xy 175.75 59.25) (xy 175.75 99.25) (xy 110.5 99.25)
+			)
+		)

Commit message: .
Parts:
- moved Q1 36.5 mm to (171.8, 85.2)
- moved U1 3.59 mm to (165.1, 76.2)
Changed lines of the file:
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@@
 	(footprint "Package_TO_SOT_THT:TO-92"
 		(layer "F.Cu")
-		(at 142.24 63.73 -90)
+		(at 171.75 85.21 -90)
 		(descr "TO-92 leads molded, narrow, drill 0.75mm (see NXP sot054_po.pdf)")
 		(tags "to-92 sc-43 sc-43a sot54 PA33 transistor")
@@
 	(footprint "Alexander Footprint Library:ESP32-C3_SuperMini"
 		(layer "F.Cu")
-		(at 167.64 73.66 180)
+		(at 165.1 76.2 180)
 		(descr "ESP32 C3 Super Mini")
 		(tags "ESP32 C3")

Commit message: .
Parts:
- moved R3 31.4 mm to (145.2, 65.2), turned to -90 degrees
Connections:
- D1 pad 2: /3V3 -> +3V3
- Q1 pad 1: /3V3 -> +3V3
- R3 pad 1: +3.3V -> +3V3
- U1 pad 14: /3V3 -> +3V3
- U1 pad 15: unconnected-(U1-5V-Pad15) -> +5V
