File: ESP32-C3-WROOM-Node-Temperature/ESP32-C3-WROOM-Node-Temperature/ESP32-C3-WROOM-Node-Temperature.kicad_pcb (KiCad board)
At the start: 2 copper layers, 65 x 40 mm, 22 parts, among them J1 PWR, K1 Relay_DPDT_HK19F_HUI, Q1 NPN, U2 AMS1117-3V3, U4 L7805

Commit message: .
Parts:
- moved C4 13.3 mm to (123.2, 70.2)
- moved J1 4.42 mm to (119.3, 62.5), turned to 0 degrees
- moved U2 4.35 mm to (138.0, 65.5)
- moved C5 3.13 mm to (129.2, 70.2)
- moved D2 2.02 mm to (128.8, 64.0), turned to -90 degrees
Changed lines of the file:
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@@
 	(footprint "Connector_PinSocket_2.54mm:PinSocket_1x02_P2.54mm_Vertical"
 		(layer "F.Cu")
-		(at 121.92 66.04 180)
+		(at 119.275 62.5)
 		(descr "Through hole straight socket strip, 1x02, 2.54mm pitch, single row (from Kicad 4.0.7), script generated")
 		(tags "Through hole socket strip THT 1x02 2.54mm single row")
@@
 		)
 		(property "Footprint" "Connector_PinSocket_2.54mm:PinSocket_1x02_P2.54mm_Vertical"
-			(at 0 0 180)
+			(at 0 0 0)
 			(unlocked yes)
 			(layer "F.Fab")
@@
 		)
 		(property "Datasheet" ""
-			(at 0 0 180)
+			(at 0 0 0)
 			(unlocked yes)
 			(layer "F.Fab")
@@
 		)
 		(property "Description" ""
-			(at 0 0 180)
+			(at 0 0 0)
 			(unlocked yes)
 			(layer "F.Fab")
@@
 		(attr through_hole)
 		(fp_line
-			(start 1.33 1.27)
-			(end 1.33 3.87)
+			(start -1.33 1.27)
+			(end -1.33 3.87)
 			(stroke
 				(width 0.12)
@@
 		)
 		(fp_line
-			(start 1.33 -1.33)
-			(end 1.33 0)
+			(start -1.33 1.27)
+			(end 1.33 1.27)
 			(stroke
 				(width 0.12)
@@
 		)
 		(fp_line
-			(start 0 -1.33)
-			(end 1.33 -1.33)
+			(start -1.33 3.87)
+			(end 1.33 3.87)
 			(stroke
 				(width 0.12)
@@
 		)
 		(fp_line
-			(start -1.33 3.87)
-			(end 1.33 3.87)
+			(start 0 -1.33)
+			(end 1.33 -1.33)
 			(stroke
 				(width 0.12)
@@
 		)
 		(fp_line
-			(start -1.33 1.27)
-			(end 1.33 1.27)
+			(start 1.33 -1.33)
+			(end 1.33 0)
 			(stroke
 				(width 0.12)
@@
 		)
 		(fp_line
-			(start -1.33 1.27)
-			(end -1.33 3.87)
+			(start 1.33 1.27)
+			(end 1.33 3.87)
 			(stroke
 				(width 0.12)
@@
 		)
 		(fp_line
-			(start 1.75 4.3)
-			(end -1.8 4.3)
+			(start -1.8 -1.8)
+			(end 1.75 -1.8)
 			(stroke
 				(width 0.05)
@@
 		)
 		(fp_line
-			(start 1.75 -1.8)
-			(end 1.75 4.3)
+			(start -1.8 4.3)
+			(end -1.8 -1.8)
 			(stroke
 				(width 0.05)
@@
 		)
 		(fp_line
-			(start -1.8 4.3)
-			(end -1.8 -1.8)
+			(start 1.75 -1.8)
+			(end 1.75 4.3)
 			(stroke
 				(width 0.05)
@@
 		)
 		(fp_line
-			(start -1.8 -1.8)
-			(end 1.75 -1.8)
+			(start 1.75 4.3)
+			(end -1.8 4.3)
 			(stroke
 				(width 0.05)
@@
 		)
 		(fp_line
-			(start 1.27 3.81)
-			(end -1.27 3.81)
+			(start -1.27 -1.27)
+			(end 0.635 -1.27)
 			(stroke
 				(width 0.1)
@@
 		)
 		(fp_line
-			(start 1.27 -0.635)
-			(end 1.27 3.81)
+			(start -1.27 3.81)
+			(end -1.27 -1.27)
 			(stroke
 				(width 0.1)
@@
 		)
 		(fp_line
-			(start -1.27 3.81)
-			(end -1.27 -1.27)
+			(start 1.27 -0.635)
+			(end 1.27 3.81)
 			(stroke
 				(width 0.1)
@@
 		)
 		(fp_line
-			(start -1.27 -1.27)
-			(end 0.635 -1.27)
+			(start 1.27 3.81)
+			(end -1.27 3.81)
 			(stroke
 				(width 0.1)
@@
 		)
 		(pad "1" thru_hole rect
-			(at 0 0 180)
+			(at 0 0)
 			(size 1.7 1.7)
 			(drill 1)
@@
 		)
 		(pad "2" thru_hole oval
-			(at 0 2.54 180)
+			(at 0 2.54)
 			(size 1.7 1.7)
 			(drill 1)
@@
 	(footprint "Package_TO_SOT_SMD:SOT-223-3_TabPin2"
 		(layer "F.Cu")
-		(at 133.65 65.55)
+		(at 138 65.5)
 		(descr "module CMS SOT223 4 pins")
 		(tags "CMS SOT")
@@
 	(footprint "Diode_SMD:D_1210_3225Metric"
 		(layer "F.Cu")
-		(at 126.75 64.25 90)
+		(at 128.75 64 -90)
 		(descr "Diode SMD 1210 (3225 Metric), square (rectangular) end terminal, IPC_7351 nominal, (Body size source: http://www.tortai-tech.com/upload/download/2011102023233369053.pdf), generated with kicad-footprint-generator")
 		(tags "diode")
@@
 		)
 		(property "Footprint" "Diode_SMD:D_1210_3225Metric"
-			(at 0 0 90)
+			(at 0 0 -90)
 			(unlocked yes)
 			(layer "F.Fab")
@@
 		)
 		(property "Datasheet" ""
-			(at 0 0 90)
+			(at 0 0 -90)
 			(unlocked yes)
 			(layer "F.Fab")
@@
 		)
 		(property "Description" "Diode"
-			(at 0 0 90)
+			(at 0 0 -90)
 			(unlocked yes)
 			(layer "F.Fab")
@@
 		)
 		(property "Sim.Device" "D"
-			(at 0 0 90)
+			(at 0 0 -90)
 			(unlocked yes)
 			(layer "F.Fab")
@@
 		)
 		(property "Sim.Pins" "1=K 2=A"
-			(at 0 0 90)
+			(at 0 0 -90)
 			(unlocked yes)
 			(layer "F.Fab")
@@
 		(attr smd)
 		(fp_line
-			(start 1.6 -1.585)
-			(end -2.285 -1.585)
+			(start -2.285 1.585)
+			(end 1.6 1.585)
 			(stroke
 				(width 0.12)
@@
 		)
 		(fp_line
-			(start -2.285 1.585)
-			(end 1.6 1.585)
+			(start 1.6 -1.585)
+			(end -2.285 -1.585)
 			(stroke
 				(width 0.12)
@@
 		)
 		(fp_line
-			(start 2.28 -1.58)
-			(end 2.28 1.58)
+			(start -2.28 1.58)
+			(end -2.28 -1.58)
 			(stroke
 				(width 0.05)
@@
 		)
 		(fp_line
-			(start -2.28 -1.58)
-			(end 2.28 -1.58)
+			(start 2.28 1.58)
+			(end -2.28 1.58)
 			(stroke
 				(width 0.05)
@@
 		)
 		(fp_line
-			(start 2.28 1.58)
-			(end -2.28 1.58)
+			(start -2.28 -1.58)
+			(end 2.28 -1.58)
 			(stroke
 				(width 0.05)
@@
 		)
 		(fp_line
-			(start -2.28 1.58)
-			(end -2.28 -1.58)
+			(start 2.28 -1.58)
+			(end 2.28 1.58)
 			(stroke
 				(width 0.05)
@@
 		)
 		(fp_line
-			(start 1.6 -1.25)
-			(end -0.975 -1.25)
+			(start -1.6 1.25)
+			(end 1.6 1.25)
 			(stroke
 				(width 0.1)
@@
 		)
 		(fp_line
-			(start -0.975 -1.25)
-			(end -1.6 -0.625)
+			(start 1.6 1.25)
+			(end 1.6 -1.25)
 			(stroke
 				(width 0.1)
@@
 		)
 		(fp_line
-			(start 1.6 1.25)
-			(end 1.6 -1.25)
+			(start -0.975 -1.25)
+			(end -1.6 -0.625)
 			(stroke
 				(width 0.1)
@@
 		)
 		(fp_line
-			(start -1.6 1.25)
-			(end 1.6 1.25)
+			(start 1.6 -1.25)
+			(end -0.975 -1.25)
 			(stroke
 				(width 0.1)
@@
 		)
 		(pad "1" smd roundrect
-			(at -1.4 0 90)
+			(at -1.4 0 270)
 			(size 1.25 2.65)
 			(layers "F.Cu" "F.Paste" "F.Mask")
@@
 		)
 		(pad "2" smd roundrect
-			(at 1.4 0 90)
+			(at 1.4 0 270)
 			(size 1.25 2.65)
 			(layers "F.Cu" "F.Paste" "F.Mask")
@@
 	(footprint "Capacitor_SMD:CP_Elec_3x5.3"
 		(layer "F.Cu")
-		(at 136.25 73 -90)
+		(at 123.25 70.25 -90)
 		(descr "SMT capacitor, aluminium electrolytic, 3x5.3, Cornell Dubilier Electronics ")
 		(tags "Capacitor Electrolytic")
@@
 	(footprint "Capacitor_SMD:CP_Elec_3x5.3"
 		(layer "F.Cu")
-		(at 130.75 73 -90)
+		(at 129.25 70.25 -90)
 		(descr "SMT capacitor, aluminium electrolytic, 3x5.3, Cornell Dubilier Electronics ")
 		(tags "Capacitor Electrolytic")

Commit message: .
Parts:
- moved TP3 52.5 mm to (127.0, 69.8)
- moved TP1 41.7 mm to (116.8, 66.2)
- moved TP4 38.6 mm to (114.2, 81.5)
- moved C2 20.3 mm to (127.5, 73.5), turned to -90 degrees
- moved C3 17.0 mm to (121.3, 77.0)
- moved C4 15.8 mm to (138.5, 74.5)
- moved C1 12.9 mm to (121.2, 70.5)
- moved C5 6.02 mm to (133.2, 74.8)
- moved U2 4.50 mm to (133.5, 65.5), turned to 90 degrees
- moved U4 3.00 mm to (114.3, 71.1)
- moved J1 2.72 mm to (120.2, 65.0), turned to 180 degrees
- moved D2 2.26 mm to (126.5, 63.8), turned to 90 degrees
- moved K1 1.38 mm to (142.1, 85.2)
