File: Production/prod_esp32-wroom-table-lights/esp32-wroom-table-lights.kicad_sch (KiCad schematic)
At the start: 13 parts, among them J2 I2C, J4 I2C, J5 USB-C, U1 ESP32-C3 SuperMini, U4 ESP32-C3 SuperMini

Commit message: .
Other:
- company: (none) -> Alexander Bobkov
- title: (none) -> Smart Work Desk Lights
Changed lines of the file:
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@@
 	(generator "eeschema")
 	(generator_version "8.0")
-	(paper "A4")
+	(paper "USLetter")
+	(title_block
+		(title "Smart Work Desk Lights")
+		(date "2024-07-24")
+		(rev "Final")
+		(company "Alexander Bobkov")
+		(comment 1 "Specialized Accounting Offices")
+		(comment 2 "ESP32-C3 SuperMini")
+	)
 	(junction
 		(at 203.2 132.08)

Commit message: .
Parts:
- removed BRD1: ~, Alexander Footprint Library:Circle-44R, symbol Alexander_Library_Symbols:CircleBoard
- removed D2: 5050, LED_SMD:LED_1210_3225Metric_Pad1.42x2.65mm_HandSolder, symbol Device:LED
- removed H1: MountingHole_M3, MountingHole:MountingHole_3.2mm_M3, symbol PCM_SL_Mechanical:MountingHole_M3
- removed J4: I2C, Alexander Footprint Library:Conn_I2C, symbol Alexander Symbol Library:Conn_I2C
- removed J5: USB-C, Alexander Footprint Library:USB-C MOLEX 2171750001, symbol Alexander_Library_Symbols:USB-C RCP USB2.0 6POS
- removed R4: 10R, Resistor_SMD:R_1206_3216Metric_Pad1.30x1.75mm_HandSolder, symbol Device:R
- removed U1: ESP32-C3 SuperMini, Alexander Footprint Library:ESP32-C3_SuperMini, symbol Alexander Symbol Library:ESP32-C3-SuperMini
Other:
- added sheet Interfaces (interfaces.kicad_sch)
- moved on the sheet: D6, R5, U4

Commit message: .
Parts:
- removed J2: I2C, Alexander Footprint Library:Conn_I2C, symbol Alexander Symbol Library:Conn_I2C
Changed lines of the file:
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@@
 	(wire
 		(pts
-			(xy 72.39 60.96) (xy 77.47 60.96)
+			(xy 129.54 30.48) (xy 133.35 30.48)
 		)
 		(stroke
@@
 	(wire
 		(pts
-			(xy 129.54 30.48) (xy 133.35 30.48)
+			(xy 119.38 68.58) (xy 119.38 74.93)
 		)
 		(stroke
@@
 	(wire
 		(pts
-			(xy 72.39 58.42) (xy 77.47 58.42)
+			(xy 97.79 45.72) (xy 104.14 45.72)
 		)
 		(stroke
@@
 	(wire
 		(pts
-			(xy 72.39 66.04) (xy 77.47 66.04)
+			(xy 97.79 48.26) (xy 104.14 48.26)
 		)
 		(stroke
@@
 	(wire
 		(pts
-			(xy 119.38 68.58) (xy 119.38 74.93)
+			(xy 134.62 50.8) (xy 138.43 50.8)
 		)
 		(stroke
@@
 	(wire
 		(pts
-			(xy 97.79 45.72) (xy 104.14 45.72)
+			(xy 134.62 58.42) (xy 138.43 58.42)
 		)
 		(stroke
@@
 	(wire
 		(pts
-			(xy 97.79 48.26) (xy 104.14 48.26)
+			(xy 120.65 34.29) (xy 120.65 30.48)
 		)
 		(stroke
@@
 		)
 	)
-	(wire
-		(pts
-			(xy 134.62 50.8) (xy 138.43 50.8)
-		)
-		(stroke
-			(width 0)
-			(type default)
-		)
-	)
-	(wire
-		(pts
-			(xy 134.62 58.42) (xy 138.43 58.42)
-		)
-		(stroke
-			(width 0)
-			(type default)
-		)
-	)
-	(wire
-		(pts
-			(xy 72.39 63.5) (xy 77.47 63.5)
-		)
-		(stroke
-			(width 0)
-			(type default)
-		)
-	)
-	(wire
-		(pts
-			(xy 120.65 34.29) (xy 120.65 30.48)
-		)
-		(stroke
-			(width 0)
-			(type default)
-		)
-	)
-	(label "GND"
-		(at 77.47 58.42 180)
+	(label "SCK"
+		(at 97.79 48.26 0)
 		(fields_autoplaced yes)
 		(effects
@@
 				(size 1.27 1.27)
 			)
-			(justify right bottom)
-		)
-	)
-	(label "SCK"
-		(at 97.79 48.26 0)
-		(fields_autoplaced yes)
-		(effects
-			(font
-				(size 1.27 1.27)
-			)
 			(justify left bottom)
-		)
-	)
-	(label "SDA"
-		(at 77.47 63.5 180)
-		(fields_autoplaced yes)
-		(effects
-			(font
-				(size 1.27 1.27)
-			)
-			(justify right bottom)
-		)
-	)
-	(label "SCK"
-		(at 77.47 66.04 180)
-		(fields_autoplaced yes)
-		(effects
-			(font
-				(size 1.27 1.27)
-			)
-			(justify right bottom)
 		)
 	)
@@
 	)
 	(symbol
-		(lib_id "Alexander Symbol Library:Conn_I2C")
-		(at 67.31 60.96 0)
-		(unit 1)
-		(exclude_from_sim no)
-		(in_bom yes)
-		(on_board yes)
-		(dnp no)
-		(fields_autoplaced yes)
-		(property "Reference" "J2"
-			(at 67.945 53.34 0)
-			(effects
-				(font
-					(size 1.27 1.27)
-				)
-			)
-		)
-		(property "Value" "I2C"
-			(at 67.945 55.88 0)
-			(effects
-				(font
-					(size 1.27 1.27)
-				)
-			)
-		)
-		(property "Footprint" "Alexander Footprint Library:Conn_I2C"
-			(at 67.31 60.96 0)
-			(effects
-				(font
-					(size 1.27 1.27)
-				)
-				(hide yes)
-			)
-		)
-		(property "Datasheet" "~"
-			(at 67.31 60.96 0)
-			(effects
-				(font
-					(size 1.27 1.27)
-				)
-				(hide yes)
-			)
-		)
-		(property "Description" "I2C connector, single row, 01x04"
-			(at 67.31 60.96 0)
-			(effects
-				(font
-					(size 1.27 1.27)
-				)
-				(hide yes)
-			)
-		)
-		(pin "GND"
-		)
-		(pin "Vcc"
-		)
-		(pin "SDA"
-		)
-		(pin "SCL"
-		)
-		(instances
-			(project "esp32-wroom-table-lights"
-				(path "/d3041bbb-21f1-431e-bbf9-53a09e8890bd"
-					(reference "J2")
-					(unit 1)
-				)
-			)
-		)
-	)
-	(symbol
 		(lib_id "power:GND")
 		(at 144.78 30.48 90)
@@
 					(unit 1)
 				)
-			)
-		)
-	)
-	(symbol
-		(lib_id "power:+3V3")
-		(at 77.47 60.96 270)
-		(unit 1)
-		(exclude_from_sim no)
-		(in_bom yes)
-		(on_board yes)
-		(dnp no)
-		(property "Reference" "#PWR01"
-			(at 73.66 60.96 0)
-			(effects
-				(font
-					(size 1.27 1.27)
-				)
-				(hide yes)
-			)
-		)
-		(property "Value" "+3V3"
-			(at 83.82 60.96 90)
-			(effects
-				(font
-					(size 1.27 1.27)
-				)
-			)
-		)
-		(property "Footprint" ""
-			(at 77.47 60.96 0)
-			(effects
-				(font
-					(size 1.27 1.27)
-				)
-				(hide yes)
-			)
-		)
-		(property "Datasheet" ""
-			(at 77.47 60.96 0)
-			(effects
-				(font
-					(size 1.27 1.27)
-				)
-				(hide yes)
-			)
-		)
-		(property "Description" ""
-			(at 77.47 60.96 0)
-			(effects
-				(font
-					(size 1.27 1.27)
-				)
-				(hide yes)
-			)
-		)
-		(pin "1"
-		)
-		(instances
-			(project "esp32-wroom-table-lights"
-				(path "/d3041bbb-21f1-431e-bbf9-53a09e8890bd"
-					(reference "#PWR01")
-					(unit 1)
-				)

Commit message: .
Parts:
- added J1: I2C, Alexander Footprint Library:Conn_I2C, symbol Alexander Symbol Library:Conn_I2C
Connections:
- net GND: now also J1.GND
- net SCK: now also J1.SCL
- net SDA: now also J1.SDA
- new net +3V3: J1.Vcc (VCC)
Changed lines of the file:
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@@
+	(wire
+		(pts
+			(xy 77.47 76.2) (xy 82.55 76.2)
+		)
+		(stroke
+			(width 0)
+			(type default)
+		)
+	)
 	(wire
 		(pts
@@
 	(wire
 		(pts
+			(xy 77.47 68.58) (xy 82.55 68.58)
+		)
+		(stroke
+			(width 0)
+			(type default)
+		)
+	)
+	(wire
+		(pts
 			(xy 96.52 40.64) (xy 104.14 40.64)
 		)
@@
 	(wire
 		(pts
+			(xy 77.47 73.66) (xy 82.55 73.66)
+		)
+		(stroke
+			(width 0)
+			(type default)
+		)
+	)
+	(wire
+		(pts
 			(xy 96.52 50.8) (xy 104.14 50.8)
 		)
@@
 		(pts
 			(xy 119.38 68.58) (xy 119.38 74.93)
+		)
+		(stroke
+			(width 0)
+			(type default)
+		)
+	)
+	(wire
+		(pts
+			(xy 77.47 71.12) (xy 82.55 71.12)
 		)
 		(stroke
@@
 			)
 			(justify left bottom)
+		)
+	)
+	(label "GND"
+		(at 82.55 68.58 180)
+		(fields_autoplaced yes)
+		(effects
+			(font
+				(size 1.27 1.27)
+			)
+			(justify right bottom)
+		)
+	)
+	(label "SDA"
+		(at 82.55 73.66 180)
+		(fields_autoplaced yes)
+		(effects
+			(font
+				(size 1.27 1.27)
+			)
+			(justify right bottom)
+		)
+	)
+	(label "SCK"
+		(at 82.55 76.2 180)
+		(fields_autoplaced yes)
+		(effects
+			(font
+				(size 1.27 1.27)
+			)
+			(justify right bottom)
 		)
 	)
@@
 	)
 	(symbol
+		(lib_id "power:+3V3")
+		(at 82.55 71.12 270)
+		(unit 1)
+		(exclude_from_sim no)
+		(in_bom yes)
+		(on_board yes)
+		(dnp no)
+		(property "Reference" "#PWR01"
+			(at 78.74 71.12 0)
+			(effects
+				(font
+					(size 1.27 1.27)
+				)
+				(hide yes)
+			)
+		)
+		(property "Value" "+3V3"
+			(at 88.9 71.12 90)
+			(effects
+				(font
+					(size 1.27 1.27)
+				)
+			)
+		)
+		(property "Footprint" ""
+			(at 82.55 71.12 0)
+			(effects
+				(font
+					(size 1.27 1.27)
+				)
+				(hide yes)
+			)
+		)
+		(property "Datasheet" ""
+			(at 82.55 71.12 0)
+			(effects
+				(font
+					(size 1.27 1.27)
+				)
+				(hide yes)
+			)
+		)
+		(property "Description" ""
+			(at 82.55 71.12 0)
+			(effects
+				(font
+					(size 1.27 1.27)
+				)
+				(hide yes)
+			)
+		)
+		(pin "1"
+		)
+		(instances
+			(project "esp32-wroom-table-lights"
+				(path "/d3041bbb-21f1-431e-bbf9-53a09e8890bd"
+					(reference "#PWR01")
+					(unit 1)
+				)
+			)
+		)
+	)
+	(symbol
 		(lib_id "Alexander Symbol Library:ESP32-C3-SuperMini")
 		(at 106.68 34.29 0)
@@
 					(unit 1)
 				)
+			)
+		)
+	)
+	(symbol
+		(lib_id "Alexander Symbol Library:Conn_I2C")
+		(at 72.39 71.12 0)
+		(unit 1)
+		(exclude_from_sim no)
+		(in_bom yes)
+		(on_board yes)
+		(dnp no)
+		(fields_autoplaced yes)
+		(property "Reference" "J1"
+			(at 73.025 63.5 0)
+			(effects
+				(font
+					(size 1.27 1.27)
+				)
+			)
+		)
+		(property "Value" "I2C"
+			(at 73.025 66.04 0)
+			(effects
+				(font
+					(size 1.27 1.27)
+				)
+			)
+		)
+		(property "Footprint" "Alexander Footprint Library:Conn_I2C"
+			(at 72.39 71.12 0)
+			(effects
+				(font
+					(size 1.27 1.27)
+				)
+				(hide yes)
+			)
+		)
+		(property "Datasheet" "~"
+			(at 72.39 71.12 0)
+			(effects
+				(font
+					(size 1.27 1.27)
+				)
+				(hide yes)
+			)
+		)
+		(property "Description" "I2C connector, single row, 01x04"
+			(at 72.39 71.12 0)
+			(effects
+				(font
+					(size 1.27 1.27)
+				)
+				(hide yes)
+			)
+		)
+		(pin "GND"
+		)
+		(pin "Vcc"
+		)
+		(pin "SDA"
+		)
+		(pin "SCL"
+		)
+		(instances
+			(project "esp32-wroom-table-lights"
+				(path "/d3041bbb-21f1-431e-bbf9-53a09e8890bd"
+					(reference "J1")
+					(unit 1)
+				)

Commit message: .
Other:
- note added: "Hardware"
- note added: "Round PCB board with 3 mounting holes."
- note added: "Terminals"
- moved on the sheet: BRD2, D6, H2, J1, R5, U4

Commit message: .
Other:
- removed sheet Interfaces
Changed lines of the file:
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@@
-	)
-	(sheet
-		(at 25.4 139.7)
-		(size 63.5 12.7)
-		(fields_autoplaced yes)
-		(stroke
-			(width 0.1524)
-			(type solid)
-		)
-		(fill
-			(color 0 0 0 0.0000)
-		)
-		(property "Sheetname" "Interfaces"
-			(at 25.4 138.9884 0)
-			(effects
-				(font
-					(size 1.27 1.27)
-				)
-				(justify left bottom)
-			)
-		)
-		(property "Sheetfile" "interfaces.kicad_sch"
-			(at 25.4 152.9846 0)
-			(effects
-				(font
-					(size 1.27 1.27)
-				)
-				(justify left top)
-			)
-		)
-		(instances
-			(project "esp32-wroom-table-lights"
-				(path "/d3041bbb-21f1-431e-bbf9-53a09e8890bd"
-					(page "4")
-				)
-			)
-		)
 	)
 	(sheet
