File: Production/prod_esp32-wroom-table-lights/esp32-wroom-table-lights.kicad_pcb (KiCad board)
At the start: 2 copper layers, 88 x 88 mm, 135 parts, among them J1 PWR, J2 I2C, J3 PWR, J4 I2C, Q1 NPN, U1 ESP32-C3 SuperMini, U2 AMS1117-3V3, U3 AMS1117-5V, U4 ESP32-C3 SuperMini, U5 AMS1117-3V3, U6 AMS1117-5V

Commit message: .
Parts:
- removed BRD1: ~, Alexander Footprint Library:Circle-44R
- removed C1, C2, C3: 1uF, Capacitor_SMD:CP_Elec_3x5.3
- removed C4, C6: 10uF, Capacitor_SMD:CP_Elec_3x5.3
- removed C5, C7: 0.1uF, Capacitor_SMD:CP_Elec_3x5.3
- removed D1: D, Diode_SMD:D_1206_3216Metric_Pad1.42x1.75mm_HandSolder
- removed D2: 5050, LED_SMD:LED_1210_3225Metric_Pad1.42x2.65mm_HandSolder
- removed D3 (x20): LED-5050, Alexander Footprint Library:LED_5050-6
- removed D4: LED-5050, Alexander Footprint Library:PinSocket_1x02_P2.54
- removed H1 (x5): MountingHole_M3, MountingHole:MountingHole_3.2mm_M3
- removed J1: PWR, Connector_PinSocket_2.54mm:PinSocket_1x02_P2.54mm_Vertical
- removed J2: I2C, Alexander Footprint Library:Conn_I2C
- removed R1 (x20), R2, R4: 10R, Resistor_SMD:R_1206_3216Metric_Pad1.30x1.75mm_HandSolder
- removed TP1: VIN, TestPoint:TestPoint_Pad_D1.5mm
- removed TP2: GND, TestPoint:TestPoint_Pad_D1.5mm
- removed TP3: 3V3, TestPoint:TestPoint_Pad_D1.5mm
- removed TP4: 5V, TestPoint:TestPoint_Pad_D1.5mm
- removed U1: ESP32-C3 SuperMini, Alexander Footprint Library:ESP32-C3_SuperMini
- removed U2: AMS1117-3V3, Alexander Footprint Library:AMS1117 SOT-223
- removed U3: AMS1117-5V, Alexander Footprint Library:AMS1117 SOT-223
- moved BRD2 0.10 mm to (200.1, 99.6)
Routing:
- net GPIO3: track 560.5 -> 68.9 mm
- net Net-(D3-AB): track 163.4 -> 0.00 mm
- net /Power Supply/VIN: track 104.1 -> 37.1 mm
- net +3V3: track 134.6 -> 68.7 mm, vias 1 -> 0
- net +5V: track 82.9 -> 34.2 mm
- net /SCK: track 55.0 -> 17.5 mm
- net /SDA: track 57.4 -> 23.5 mm
- net GPIO2: track 19.1 -> 0.00 mm
- net Net-(D4-AB): track 16.4 -> 0.00 mm, vias 1 -> 0
- net /Power Supply/VDC: track 20.0 -> 11.3 mm

Commit message: .
Parts:
- removed J4: I2C, Alexander Footprint Library:Conn_I2C
- added J1: I2C, Alexander Footprint Library:Conn_I2C, F.Cu at (212.2, 102.9)
Changed lines of the file:
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@@
 		(pad_to_mask_clearance 0)
 		(allow_soldermask_bridges_in_footprints no)
-		(grid_origin 100.1 99.7)
+		(grid_origin 200.1 99.7)
 		(pcbplotparams
 			(layerselection 0x00010fc_ffffffff)
@@
 		)
 	)
+	(footprint "Alexander Footprint Library:Conn_I2C"
+		(layer "F.Cu")
+		(at 212.225 102.86)
+		(property "Reference" "J1"
+			(at 0 -0.5 0)
+			(unlocked yes)
+			(layer "F.SilkS")
+			(effects
+				(font
+					(size 1 1)
+					(thickness 0.1)
+				)
+			)
+		)
+		(property "Value" "I2C"
+			(at 0 1 0)
+			(unlocked yes)
+			(layer "F.Fab")
+			(effects
+				(font
+					(size 1 1)
+					(thickness 0.15)
+				)
+			)
+		)
+		(property "Footprint" "Alexander Footprint Library:Conn_I2C"
+			(at 0 0 0)
+			(unlocked yes)
+			(layer "F.Fab")
+			(hide yes)
+			(effects
+				(font
+					(size 1.27 1.27)
+					(thickness 0.15)
+				)
+			)
+		)
+		(property "Datasheet" ""
+			(at 0 0 0)
+			(unlocked yes)
+			(layer "F.Fab")
+			(hide yes)
+			(effects
+				(font
+					(size 1.27 1.27)
+					(thickness 0.15)
+				)
+			)
+		)
+		(property "Description" "I2C connector, single row, 01x04"
+			(at 0 0 0)
+			(unlocked yes)
+			(layer "F.Fab")
+			(hide yes)
+			(effects
+				(font
+					(size 1.27 1.27)
+					(thickness 0.15)
+				)
+			)
+		)
+		(property ki_fp_filters "Connector*:*_1x??_*")
+		(sheetname "Root")
+		(sheetfile "esp32-wroom-table-lights.kicad_sch")
+		(attr through_hole)
+		(fp_text user "I2C"
+			(at 0 17.78 0)
+			(unlocked yes)
+			(layer "F.SilkS" knockout)
+			(effects
+				(font
+					(size 1 1)
+					(thickness 0.2)
+					(bold yes)
+				)
+				(justify bottom)
+			)
+		)
+		(fp_text user "Vcc"
+			(at 2.54 10.16 0)
+			(unlocked yes)
+			(layer "F.SilkS")
+			(effects
+				(font
+					(size 0.8 1)
+					(thickness 0.1)
+				)
+			)
+		)
+		(fp_text user "SDA"
+			(at 2.54 12.7 0)
+			(unlocked yes)
+			(layer "F.SilkS")
+			(effects
+				(font
+					(size 0.8 1)
+					(thickness 0.1)
+				)
+			)
+		)
+		(fp_text user "GND"
+			(at 2.54 7.62 0)
+			(unlocked yes)
+			(layer "F.SilkS")
+			(effects
+				(font
+					(size 0.8 1)
+					(thickness 0.1)
+				)
+			)
+		)
+		(fp_text user "SCL"
+			(at 2.54 15.24 0)
+			(unlocked yes)
+			(layer "F.SilkS")
+			(effects
+				(font
+					(size 0.8 1)
+					(thickness 0.1)
+				)
+			)
+		)
+		(fp_text user "${REFERENCE}"
+			(at 0 2.5 0)
+			(unlocked yes)
+			(layer "F.Fab")
+			(effects
+				(font
+					(size 1 1)
+					(thickness 0.15)
+				)
+			)
+		)
+		(pad "GND" thru_hole rect
+			(at 0 7.62)
+			(size 1.524 1.524)
+			(drill 0.762)
+			(layers "*.Cu" "*.Mask")
+			(remove_unused_layers no)
+			(net 2 "GND")
+			(pinfunction "GND")
+			(pintype "power_out")
+		)
+		(pad "SCL" thru_hole circle
+			(at 0 15.24)
+			(size 1.524 1.524)
+			(drill 0.762)
+			(layers "*.Cu" "*.Mask")
+			(remove_unused_layers no)
+			(net 8 "/SCK")
+			(pinfunction "SCL")
+			(pintype "bidirectional")
+		)
+		(pad "SDA" thru_hole circle
+			(at 0 12.7)
+			(size 1.524 1.524)
+			(drill 0.762)
+			(layers "*.Cu" "*.Mask")
+			(remove_unused_layers no)
+			(net 1 "/SDA")
+			(pinfunction "SDA")
+			(pintype "bidirectional")
+		)
+		(pad "Vcc" thru_hole circle
+			(at 0 10.16)
+			(size 1.524 1.524)
+			(drill 0.762)
+			(layers "*.Cu" "*.Mask")
+			(remove_unused_layers no)
+			(net 4 "+3V3")
+			(pinfunction "VCC")
+			(pintype "power_in")
+		)
+	)
 	(footprint "TestPoint:TestPoint_Pad_D1.5mm"
 		(layer "F.Cu")
@@
 		)
 	)
-	(footprint "Alexander Footprint Library:Conn_I2C"
-		(layer "F.Cu")
-		(at 212.2 102.86)
-		(property "Reference" "J4"
-			(at 0 -0.5 0)
-			(unlocked yes)
-			(layer "F.SilkS")
-			(effects
-				(font
-					(size 1 1)
-					(thickness 0.1)
-				)
-			)
-		)
-		(property "Value" "I2C"
-			(at 0 1 0)
-			(unlocked yes)
-			(layer "F.Fab")
-			(effects
-				(font
-					(size 1 1)
-					(thickness 0.15)
-				)
-			)
-		)
-		(property "Footprint" "Alexander Footprint Library:Conn_I2C"
-			(at 0 0 0)
-			(unlocked yes)
-			(layer "F.Fab")
-			(hide yes)
-			(effects
-				(font
-					(size 1.27 1.27)
-					(thickness 0.15)
-				)
-			)
-		)
-		(property "Datasheet" ""
-			(at 0 0 0)
-			(unlocked yes)
-			(layer "F.Fab")
-			(hide yes)
-			(effects
-				(font
-					(size 1.27 1.27)
-					(thickness 0.15)
-				)
-			)
-		)
-		(property "Description" "I2C connector, single row, 01x04"
-			(at 0 0 0)
-			(unlocked yes)
-			(layer "F.Fab")
-			(hide yes)
-			(effects
-				(font
-					(size 1.27 1.27)
-					(thickness 0.15)
-				)
-			)
-		)
-		(property ki_fp_filters "Connector*:*_1x??_*")
-		(sheetname "Root")
-		(sheetfile "esp32-wroom-table-lights.kicad_sch")
-		(attr through_hole)
-		(fp_text user "I2C"
-			(at -0.05 18.19 0)
-			(unlocked yes)
-			(layer "F.SilkS" knockout)
-			(effects
-				(font
-					(size 1 1)
-					(thickness 0.2)
-					(bold yes)
-				)
-				(justify bottom)
-			)
-		)
-		(fp_text user "GND"
-			(at -3.275 7.71 0)
-			(unlocked yes)
-			(layer "F.SilkS")
-			(effects
-				(font
-					(size 0.8 1)
-					(thickness 0.1)
-				)
-			)
-		)
-		(fp_text user "SDA"
-			(at -3.275 12.79 0)
-			(unlocked yes)
-			(layer "F.SilkS")
-			(effects
-				(font
-					(size 0.8 1)
-					(thickness 0.1)
-				)
-			)
-		)
-		(fp_text user "SCL"
-			(at -3.275 15.33 0)
-			(unlocked yes)
-			(layer "F.SilkS")
-			(effects
-				(font
-					(size 0.8 1)
-					(thickness 0.1)
-				)
-			)
-		)
-		(fp_text user "Vcc"
-			(at -3.275 10.25 0)
-			(unlocked yes)
-			(layer "F.SilkS")
-			(effects
-				(font
-					(size 0.8 1)
-					(thickness 0.1)
-				)
-			)
-		)
-		(fp_text user "${REFERENCE}"
-			(at 0 2.5 0)
-			(unlocked yes)
-			(layer "F.Fab")
-			(effects
-				(font
-					(size 1 1)
-					(thickness 0.15)
-				)
-			)
-		)
-		(pad "GND" thru_hole rect
-			(at 0 7.62)
-			(size 1.524 1.524)
-			(drill 0.762)
-			(layers "*.Cu" "*.Mask")
-			(remove_unused_layers no)
-			(net 2 "GND")
-			(pinfunction "GND")
-			(pintype "power_out")
-		)
-		(pad "SCL" thru_hole circle
-			(at 0 15.24)
-			(size 1.524 1.524)
-			(drill 0.762)
-			(layers "*.Cu" "*.Mask")
-			(remove_unused_layers no)
-			(net 8 "/SCK")
-			(pinfunction "SCL")
-			(pintype "bidirectional")
-		)
-		(pad "SDA" thru_hole circle
-			(at 0 12.7)
-			(size 1.524 1.524)
-			(drill 0.762)
-			(layers "*.Cu" "*.Mask")
-			(remove_unused_layers no)
-			(net 1 "/SDA")
-			(pinfunction "SDA")
-			(pintype "bidirectional")
-		)
-		(pad "Vcc" thru_hole circle
-			(at 0 10.16)
-			(size 1.524 1.524)
-			(drill 0.762)
-			(layers "*.Cu" "*.Mask")
-			(remove_unused_layers no)
-			(net 4 "+3V3")
-			(pinfunction "VCC")
-			(pintype "power_in")
-		)
-	)

Commit message: .
Routing:
- net GPIO3: track 68.9 -> 16.0 mm
Changed lines of the file:
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@@
-	)
-	(segment
-		(start 173.61091 136.423712)
-		(end 174.598036 136.423712)
-		(width 0.25)
-		(layer "F.Cu")
-		(net 7)
-	)
-	(segment
-		(start 155.472509 118.285311)
-		(end 173.61091 136.423712)
-		(width 0.25)
-		(layer "F.Cu")
-		(net 7)
-	)
-	(segment
-		(start 155.472509 92.059707)
-		(end 155.472509 118.285311)
-		(width 0.25)
-		(layer "F.Cu")
-		(net 7)
 	)
 	(segment
