File: Production/prod_esp32-wroom-table-lights/led-lights-array.kicad_sch (KiCad schematic)
At the start: 7 parts, among them Q1 NPN

Commit message: .
Parts:
- R3: value 10R -> 470
- R6: value R -> 1k
- R8: value R -> 1M
Changed lines of the file:
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@@
 			)
 		)
-		(property "Value" "10R"
+		(property "Value" "470"
 			(at 44.45 34.29 90)
 			(effects
@@
 			)
 		)
-		(property "Value" "R"
+		(property "Value" "1M"
 			(at 36.83 96.5199 0)
 			(effects
@@
 			)
 		)
-		(property "Value" "R"
+		(property "Value" "1k"
 			(at 57.15 67.3099 0)
 			(effects

Commit message: .
Parts:
- removed R3: 470, Resistor_SMD:R_1206_3216Metric_Pad1.30x1.75mm_HandSolder, symbol Device:R
- added R1: 470, Resistor_SMD:R_1206_3216Metric_Pad1.30x1.75mm_HandSolder, symbol Device:R
Connections:
- net LED_RING: now also D5.1 (AB), D5.2 (KB), D5.3 (AR), R1.1; no longer Q1.3 (E)
- new net: Q1.3 (E), R1.2
Changed lines of the file:
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@@
-	(wire
-		(pts
-			(xy 48.26 38.1) (xy 50.8 38.1)
-		)
-		(stroke
-			(width 0)
-			(type default)
-		)
-	)
 	(wire
 		(pts
@@
 	(wire
 		(pts
-			(xy 38.1 38.1) (xy 40.64 38.1)
-		)
-		(stroke
-			(width 0)
-			(type default)
-		)
-	)
-	(wire
-		(pts
-			(xy 59.69 53.34) (xy 66.04 53.34)
+			(xy 38.1 38.1) (xy 50.8 38.1)
 		)
 		(stroke
@@
 		(pts
 			(xy 34.29 88.9) (xy 34.29 91.44)
+		)
+		(stroke
+			(width 0)
+			(type default)
+		)
+	)
+	(wire
+		(pts
+			(xy 59.69 53.34) (xy 64.77 53.34)
+		)
+		(stroke
+			(width 0)
+			(type default)
+		)
+	)
+	(wire
+		(pts
+			(xy 72.39 53.34) (xy 77.47 53.34)
 		)
 		(stroke
@@
 	(global_label "LED_RING"
 		(shape output)
-		(at 66.04 53.34 0)
+		(at 77.47 53.34 0)
 		(fields_autoplaced yes)
 		(effects
@@
 		)
 		(property "Intersheetrefs" "${INTERSHEET_REFS}"
-			(at 77.9152 53.34 0)
+			(at 89.3452 53.34 0)
 			(effects
 				(font
@@
 	(symbol
 		(lib_id "Device:R")
-		(at 44.45 38.1 270)
+		(at 68.58 53.34 270)
 		(unit 1)
 		(exclude_from_sim no)
@@
 		(on_board yes)
 		(dnp no)
-		(property "Reference" "R3"
-			(at 44.45 31.75 90)
+		(property "Reference" "R1"
+			(at 68.58 46.99 90)
 			(effects
 				(font
@@
 		)
 		(property "Value" "470"
-			(at 44.45 34.29 90)
+			(at 68.58 49.53 90)
 			(effects
 				(font
@@
 		)
 		(property "Footprint" "Resistor_SMD:R_1206_3216Metric_Pad1.30x1.75mm_HandSolder"
-			(at 44.45 36.322 90)
+			(at 68.58 51.562 90)
 			(effects
 				(font
@@
 		)
 		(property "Datasheet" "~"
-			(at 44.45 38.1 0)
+			(at 68.58 53.34 0)
 			(effects
 				(font
@@
 		)
 		(property "Description" "Resistor"
-			(at 44.45 38.1 0)
+			(at 68.58 53.34 0)
 			(effects
 				(font
@@
 			(project "esp32-wroom-table-lights"
 				(path "/d3041bbb-21f1-431e-bbf9-53a09e8890bd/d5fc8cf4-d8a2-46b6-9b2c-3f15f2406209"
-					(reference "R3")
+					(reference "R1")
 					(unit 1)
 				)
