File: esp32-mqtt-bot/esp32-mqtt-bot/esp32-mqtt-bot.kicad_sch (KiCad schematic)
At the start: 1 part, among them U1 ESP32-WROOM-32

Commit message: .
Connections:
- net GND: now reaches U1.1 (GND), U1.15 (GND), U1.38 (GND), U1.39 (GND)
Changed lines of the file:
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@@
 	(generator_version "8.0")
 	(paper "A4")
+	(wire
+		(pts
+			(xy 119.38 134.62) (xy 119.38 137.16)
+		)
+		(stroke
+			(width 0)
+			(type default)
+		)
+	)
+	(symbol
+		(lib_id "power:GND")
+		(at 119.38 137.16 0)
+		(unit 1)
+		(exclude_from_sim no)
+		(in_bom yes)
+		(on_board yes)
+		(dnp no)
+		(fields_autoplaced yes)
+		(property "Reference" "#PWR01"
+			(at 119.38 143.51 0)
+			(effects
+				(font
+					(size 1.27 1.27)
+				)
+				(hide yes)
+			)
+		)
+		(property "Value" "GND"
+			(at 119.38 142.24 0)
+			(effects
+				(font
+					(size 1.27 1.27)
+				)
+			)
+		)
+		(property "Footprint" ""
+			(at 119.38 137.16 0)
+			(effects
+				(font
+					(size 1.27 1.27)
+				)
+				(hide yes)
+			)
+		)
+		(property "Datasheet" ""
+			(at 119.38 137.16 0)
+			(effects
+				(font
+					(size 1.27 1.27)
+				)
+				(hide yes)
+			)
+		)
+		(property "Description" "Power symbol creates a global label with name \"GND\" , ground"
+			(at 119.38 137.16 0)
+			(effects
+				(font
+					(size 1.27 1.27)
+				)
+				(hide yes)
+			)
+		)
+		(pin "1"
+		)
+		(instances
+			(project ""
+				(path "/0b74e088-c891-4ff7-bf69-53ac2ddf47f3"
+					(reference "#PWR01")
+					(unit 1)
+				)
+			)
+		)
+	)
 	(symbol
 		(lib_id "Alexander Symbol Library:ESP32-WROOM-32")

Commit message: .
Parts:
- added D1: LED_SMD_5050, Alexander Footprint Library:LED_5050-6, symbol Alexander Symbol Library:LED_SMD_5050
- added R1: A1050, OptoDevice:R_LDR_D6.4mm_P3.4mm_Vertical, symbol Sensor_Optical:A1050
Connections:
- net GND: now also D1.4 (KR), D1.5 (AG), D1.6 (KR)
- net GPIO23: now reaches U1.37 (IO23)
- net GPIO23: now also R1.2
- new net +3V3: D1.1 (AB), D1.2 (KB), D1.3 (AR), R1.1

Commit message: .
Parts:
- added D2, D3: LED_SMD_5050, Alexander Footprint Library:LED_5050-6, symbol Alexander Symbol Library:LED_SMD_5050
Connections:
- net +3V3: now also D2.1 (AB), D2.2 (KB), D2.3 (AR), D3.1 (AB), D3.2 (KB), D3.3 (AR)
- net GND: now also D2.4 (KR), D2.5 (AG), D2.6 (KR), D3.4 (KR), D3.5 (AG), D3.6 (KR)
Other:
- moved on the sheet: R1
