File: esp32-c3-wroom-socket/esp32-c3-wroom-socket/esp32-c3-wroom-socket.kicad_pcb (KiCad board)
At the start: 2 copper layers, 30.5 x 25.4 mm, 7 parts, among them J1 USB-C_Receptacle_Data_16P_GCT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, U1 ESP32-C3-WROOM-02-N4

Commit message: .
Parts:
- moved R3 1.81 mm to (149.0, 76.6)
- moved R2 1.74 mm to (165.1, 76.6)
- moved J1 1.73 mm to (154.2, 75.2)
Routing:
- net Net-(J1-VBUS-PadA4): track 9.30 -> 0.00 mm
- net Net-(J1-CC1): track 8.58 -> 9.80 mm
- net USB_D+: track 25.5 -> 26.3 mm
- net USB_D-: track 24.0 -> 24.6 mm
Changed lines of the file:
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@@
 	(footprint "Alexander Footprint Library:USB-C GCT CONN16_USB4085-GF-A"
 		(layer "F.Cu")
-		(at 154.124444 76.932435)
+		(at 154.15 75.2)
 		(tags "USB4085-GF-A ")
 		(property "Reference" "J1"
@@
 	(footprint "Resistor_SMD:R_1206_3216Metric_Pad1.30x1.75mm_HandSolder"
 		(layer "B.Cu")
-		(at 164.75 78.3 -90)
+		(at 165.1 76.6 -90)
 		(descr "Resistor SMD 1206 (3216 Metric), square (rectangular) end terminal, IPC_7351 nominal with elongated pad for handsoldering. (Body size source: IPC-SM-782 page 72, https://www.pcb-3d.com/wordpress/wp-content/uploads/ipc-sm-782a_amendment_1_and_2.pdf), generated with kicad-footprint-generator")
 		(tags "resistor handsolder")
@@
 	(footprint "Resistor_SMD:R_1206_3216Metric_Pad1.30x1.75mm_HandSolder"
 		(layer "B.Cu")
-		(at 149.75 78.25 90)
+		(at 149 76.6 90)
 		(descr "Resistor SMD 1206 (3216 Metric), square (rectangular) end terminal, IPC_7351 nominal with elongated pad for handsoldering. (Body size source: IPC-SM-782 page 72, https://www.pcb-3d.com/wordpress/wp-content/uploads/ipc-sm-782a_amendment_1_and_2.pdf), generated with kicad-footprint-generator")
 		(tags "resistor handsolder")
@@
 	)
 	(segment
-		(start 160.074445 76.932435)
-		(end 160.074445 78.282435)
+		(start 154.15 75.2)
+		(end 154.15 76.55)
 		(width 0.5)
-		(layer "F.Cu")
+		(layer "B.Cu")
 		(net 2)
 	)
 	(segment
-		(start 154.124444 76.932435)
-		(end 154.124444 78.282435)
+		(start 160.100001 75.2)
+		(end 160.100001 76.55)
 		(width 0.5)
-		(layer "F.Cu")
+		(layer "B.Cu")
 		(net 2)
 	)
@@
 	)
 	(segment
-		(start 155.5 79.75)
-		(end 158.75 79.75)
-		(width 0.2)
-		(layer "F.Cu")
-		(net 7)
-	)
-	(segment
-		(start 158.75 79.75)
-		(end 159.224444 79.275556)
-		(width 0.2)
-		(layer "F.Cu")
-		(net 7)
-	)
-	(segment
-		(start 154.974445 79.224445)
-		(end 155.5 79.75)
-		(width 0.2)
-		(layer "F.Cu")
-		(net 7)
-	)
-	(segment
-		(start 154.974445 78.282435)
-		(end 154.974445 79.224445)
-		(width 0.2)
-		(layer "F.Cu")
-		(net 7)
-	)
-	(segment
-		(start 159.224444 79.275556)
-		(end 159.224444 78.282435)
-		(width 0.2)
-		(layer "F.Cu")
-		(net 7)
-	)
-	(segment
-		(start 159.224444 76.932435)
-		(end 159.224444 78.282435)
-		(width 0.2)
-		(layer "B.Cu")
-		(net 7)
-	)
-	(segment
-		(start 154.974445 76.932435)
-		(end 154.974445 78.282435)
-		(width 0.2)
-		(layer "B.Cu")
-		(net 7)
-	)
-	(segment
-		(start 158.374446 78.282435)
-		(end 158.374446 79.374446)
+		(start 158.400002 77.800002)
+		(end 158.75 78.15)
 		(width 0.2)
 		(layer "B.Cu")
@@
 	)
 	(segment
-		(start 158.374446 79.374446)
-		(end 158.85 79.85)
+		(start 158.75 78.15)
+		(end 165.1 78.15)
 		(width 0.2)
 		(layer "B.Cu")
@@
 	)
 	(segment
-		(start 158.85 79.85)
-		(end 164.75 79.85)
+		(start 158.400002 76.55)
+		(end 158.400002 77.800002)
 		(width 0.2)
 		(layer "B.Cu")
@@
 	)
 	(segment
-		(start 149.75 76.7)
-		(end 149.75 75.75)
+		(start 155.849999 73.849999)
+		(end 155.849999 75.2)
 		(width 0.2)
 		(layer "B.Cu")
@@
 	)
 	(segment
-		(start 155.25 75.25)
-		(end 155.824443 75.824443)
+		(start 149 75.05)
+		(end 149 73.8)
 		(width 0.2)
 		(layer "B.Cu")
@@
 	)
 	(segment
-		(start 149.75 75.75)
-		(end 150.25 75.25)
+		(start 149 73.8)
+		(end 149.4 73.4)
 		(width 0.2)
 		(layer "B.Cu")
@@
 	)
 	(segment
-		(start 150.25 75.25)
-		(end 155.25 75.25)
+		(start 155.4 73.4)
+		(end 155.849999 73.849999)
 		(width 0.2)
 		(layer "B.Cu")
@@
 	)
 	(segment
-		(start 155.824443 75.824443)
-		(end 155.824443 76.932435)
+		(start 149.4 73.4)
+		(end 155.4 73.4)
 		(width 0.2)
 		(layer "B.Cu")
@@
 	)
 	(segment
-		(start 156.674444 76.932435)
-		(end 156.674444 77.174444)
+		(start 157.62 71.78)
+		(end 165.72 71.78)
 		(width 0.2)
 		(layer "B.Cu")
@@
 	)
 	(segment
+		(start 157.550001 76.083027)
+		(end 157.266974 75.8)
+		(width 0.2)
+		(layer "B.Cu")
+		(net 13)
+	)
+	(segment
+		(start 157.550001 76.55)
+		(end 157.550001 76.083027)
+		(width 0.2)
+		(layer "B.Cu")
+		(net 13)
+	)
+	(segment
+		(start 156.7 75.7)
+		(end 156.7 75.2)
+		(width 0.2)
+		(layer "B.Cu")
+		(net 13)
+	)
+	(segment
+		(start 157.266974 75.8)
+		(end 156.8 75.8)
+		(width 0.2)
+		(layer "B.Cu")
+		(net 13)
+	)
+	(segment
+		(start 156.7 75.2)
+		(end 156.7 72.7)
+		(width 0.2)
+		(layer "B.Cu")
+		(net 13)
+	)
+	(segment
+		(start 165.72 71.78)
+		(end 167.86 69.64)
+		(width 0.2)
+		(layer "B.Cu")
+		(net 13)
+	)
+	(segment
+		(start 156.8 75.8)
+		(end 156.7 75.7)
+		(width 0.2)
+		(layer "B.Cu")
+		(net 13)
+	)
+	(segment
 		(start 167.86 69.64)
-		(end 165.72 71.78)
+		(end 169.41 69.64)
 		(width 0.2)
 		(layer "B.Cu")
@@
 	)
 	(segment
-		(start 169.41 69.64)
-		(end 167.86 69.64)
-		(width 0.2)
-		(layer "B.Cu")
-		(net 13)
-	)
-	(segment
-		(start 156.674444 77.174444)
-		(end 157.524445 78.024445)
-		(width 0.2)
-		(layer "B.Cu")
-		(net 13)
-	)
-	(segment
-		(start 157.524445 78.024445)
-		(end 157.524445 78.282435)
-		(width 0.2)
-		(layer "B.Cu")
-		(net 13)
-	)
-	(segment
-		(start 156.674444 76.465462)
-		(end 156.674444 76.932435)
-		(width 0.2)
-		(layer "B.Cu")
-		(net 13)
-	)
-	(segment
-		(start 161.359906 71.78)
-		(end 156.674444 76.465462)
-		(width 0.2)
-		(layer "B.Cu")
-		(net 13)
-	)
-	(segment
-		(start 165.72 71.78)
-		(end 161.359906 71.78)
+		(start 156.7 72.7)
+		(end 157.62 71.78)
 		(width 0.2)
 		(layer "B.Cu")
@@
 	)
 	(segment
+		(start 157.550001 75.649999)
+		(end 157.550001 75.2)
+		(width 0.2)
+		(layer "F.Cu")
+		(net 15)
+	)
+	(segment
+		(start 156.7 76.55)
+		(end 156.7 76.091238)
+		(width 0.2)
+		(layer "F.Cu")
+		(net 15)
+	)
+	(segment
 		(start 167.8 68.595686)
 		(end 167.8 70.57)
@@
 	)
 	(segment
-		(start 156.674444 78.241198)
-		(end 157.524445 77.391197)
+		(start 156.991238 75.8)
+		(end 157.4 75.8)
 		(width 0.2)
 		(layer "F.Cu")
@@
 	)
 	(segment
-		(start 157.524445 77.391197)
-		(end 157.524445 76.932435)
+		(start 157.4 75.8)
+		(end 157.550001 75.649999)
 		(width 0.2)
 		(layer "F.Cu")
@@
 	)
 	(segment
-		(start 156.674444 78.282435)
-		(end 156.674444 78.241198)
+		(start 156.7 76.091238)
+		(end 156.991238 75.8)
 		(width 0.2)
 		(layer "F.Cu")
@@
 	)
 	(segment
-		(start 161.809907 72.18)
-		(end 157.524445 76.465462)
+		(start 158.2 72.18)
+		(end 169.41 72.18)
 		(width 0.2)
 		(layer "B.Cu")
@@
 	)
 	(segment
-		(start 157.524445 76.465462)
-		(end 157.524445 76.932435)
+		(start 157.550001 75.2)
+		(end 157.550001 72.829999)
 		(width 0.2)
 		(layer "B.Cu")
@@
 	)
 	(segment
-		(start 169.41 72.18)
-		(end 161.809907 72.18)
-		(width 0.2)
-		(layer "B.Cu")
+		(start 157.550001 72.829999)
+		(end 158.2 72.18)
+		(width 0.2)
+		(layer "B.Cu")

Commit message: .
Parts:
- removed C1: 1uF, Resistor_SMD:R_0612_1632Metric_Pad1.18x3.40mm_HandSolder
- added U2: AMS1117-3V3, Package_TO_SOT_SMD:SOT-223-3_TabPin2, B.Cu at (151.6, 67.6)
- moved R3 14.1 mm to (161.2, 69.5), turned to 180 degrees
- moved R1 3.40 mm to (148.4, 60.7)
- moved R2 0.14 mm to (165.0, 76.5)
Connections:
- net Net-(J1-VBUS-PadA4) renamed VBUS
Routing:
- net VBUS: track 0.00 -> 21.8 mm
- net EN: track 13.6 -> 10.2 mm
- net 3V3: track 12.7 -> 9.27 mm
- net Net-(J1-CC1): track 9.80 -> 8.24 mm

Commit message: .
Parts:
- moved R1 2.05 mm to (149.9, 62.1), turned to 180 degrees
- moved U2 1.20 mm to (151.7, 68.8)
Routing:
- net 3V3: track 9.27 -> 21.3 mm
- net VBUS: track 21.8 -> 20.0 mm
Changed lines of the file:
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@@
 	(footprint "Package_TO_SOT_SMD:SOT-223-3_TabPin2"
 		(layer "B.Cu")
-		(at 151.6 67.6)
+		(at 151.7 68.8)
 		(descr "module CMS SOT223 4 pins")
 		(tags "CMS SOT")
@@
 	(footprint "Resistor_SMD:R_1206_3216Metric_Pad1.30x1.75mm_HandSolder"
 		(layer "B.Cu")
-		(at 148.4 60.7 -90)
+		(at 149.9 62.1 180)
 		(descr "Resistor SMD 1206 (3216 Metric), square (rectangular) end terminal, IPC_7351 nominal with elongated pad for handsoldering. (Body size source: IPC-SM-782 page 72, https://www.pcb-3d.com/wordpress/wp-content/uploads/ipc-sm-782a_amendment_1_and_2.pdf), generated with kicad-footprint-generator")
 		(tags "resistor handsolder")
 		(property "Reference" "R1"
-			(at 0 1.82 90)
+			(at 0 1.82 0)
 			(layer "B.SilkS")
 			(effects
@@
 		)
 		(property "Value" "10k"
-			(at 0 -1.82 90)
+			(at 0 -1.82 0)
 			(layer "B.Fab")
 			(effects
@@
 		)
 		(property "Footprint" "Resistor_SMD:R_1206_3216Metric_Pad1.30x1.75mm_HandSolder"
-			(at 0 0 90)
+			(at 0 0 0)
 			(unlocked yes)
 			(layer "B.Fab")
@@
 		)
 		(property "Datasheet" ""
-			(at 0 0 90)
+			(at 0 0 0)
 			(unlocked yes)
 			(layer "B.Fab")
@@
 		)
 		(property "Description" "Resistor"
-			(at 0 0 90)
+			(at 0 0 0)
 			(unlocked yes)
 			(layer "B.Fab")
@@
 		)
 		(fp_line
+			(start 2.45 1.12)
+			(end -2.45 1.12)
+			(stroke
+				(width 0.05)
+				(type solid)
+			)
+			(layer "B.CrtYd")
+		)
+		(fp_line
+			(start 2.45 -1.12)
+			(end 2.45 1.12)
+			(stroke
+				(width 0.05)
+				(type solid)
+			)
+			(layer "B.CrtYd")
+		)
+		(fp_line
 			(start -2.45 1.12)
 			(end -2.45 -1.12)
@@
 		)
 		(fp_line
-			(start 2.45 1.12)
-			(end -2.45 1.12)
-			(stroke
-				(width 0.05)
-				(type solid)
-			)
-			(layer "B.CrtYd")
-		)
-		(fp_line
 			(start -2.45 -1.12)
 			(end 2.45 -1.12)
@@
 		)
 		(fp_line
-			(start 2.45 -1.12)
-			(end 2.45 1.12)
-			(stroke
-				(width 0.05)
-				(type solid)
-			)
-			(layer "B.CrtYd")
+			(start 1.6 0.8)
+			(end -1.6 0.8)
+			(stroke
+				(width 0.1)
+				(type solid)
+			)
+			(layer "B.Fab")
+		)
+		(fp_line
+			(start 1.6 -0.8)
+			(end 1.6 0.8)
+			(stroke
+				(width 0.1)
+				(type solid)
+			)
+			(layer "B.Fab")
 		)
 		(fp_line
@@
 		)
 		(fp_line
-			(start 1.6 0.8)
-			(end -1.6 0.8)
-			(stroke
-				(width 0.1)
-				(type solid)
-			)
-			(layer "B.Fab")
-		)
-		(fp_line
 			(start -1.6 -0.8)
 			(end 1.6 -0.8)
@@
 			(layer "B.Fab")
 		)
-		(fp_line
-			(start 1.6 -0.8)
-			(end 1.6 0.8)
-			(stroke
-				(width 0.1)
-				(type solid)
-			)
-			(layer "B.Fab")
-		)
 		(fp_text user "${REFERENCE}"
-			(at 0 0 90)
+			(at 0 0 0)
 			(layer "B.Fab")
 			(effects
@@
 		)
 		(pad "1" smd roundrect
-			(at -1.55 0 270)
+			(at -1.55 0 180)
 			(size 1.3 1.75)
 			(layers "B.Cu" "B.Paste" "B.Mask")
@@
 		)
 		(pad "2" smd roundrect
-			(at 1.55 0 270)
+			(at 1.55 0 180)
 			(size 1.3 1.75)
 			(layers "B.Cu" "B.Paste" "B.Mask")
@@
 	)
 	(segment
-		(start 154.4 71.8)
-		(end 148.8 71.8)
+		(start 155.000001 73.900001)
+		(end 154.1 73)
 		(width 0.5)
 		(layer "B.Cu")
@@
 	)
 	(segment
+		(start 148.55 71.1)
+		(end 148.55 72.15)
+		(width 0.5)
+		(layer "B.Cu")
+		(net 7)
+	)
+	(segment
+		(start 149.4 73)
+		(end 154.1 73)
+		(width 0.5)
+		(layer "B.Cu")
+		(net 7)
+	)
+	(segment
 		(start 155.000001 75.2)
-		(end 155.000001 72.400001)
+		(end 155.000001 73.900001)
 		(width 0.5)
 		(layer "B.Cu")
@@
 	)
 	(segment
-		(start 148.8 71.8)
-		(end 148.45 71.45)
-		(width 0.5)
-		(layer "B.Cu")
-		(net 7)
-	)
-	(segment
-		(start 148.45 71.45)
-		(end 148.45 69.9)
-		(width 0.5)
-		(layer "B.Cu")
-		(net 7)
-	)
-	(segment
-		(start 155.000001 72.400001)
-		(end 154.4 71.8)
+		(start 148.55 72.15)
+		(end 149.4 73)
 		(width 0.5)
 		(layer "B.Cu")
@@
 	)
 	(segment
-		(start 148.4 62.25)
-		(end 146.3 62.25)
+		(start 144.01 62.02)
+		(end 145.9 62.02)
 		(width 0.2)
 		(layer "B.Cu")
@@
 	)
 	(segment
-		(start 146.07 62.02)
-		(end 146.3 62.25)
+		(start 145.98 62.1)
+		(end 145.9 62.02)
 		(width 0.2)
 		(layer "B.Cu")
@@
 	)
 	(segment
-		(start 144.01 62.02)
+		(start 148.35 62.1)
+		(end 145.98 62.1)
+		(width 0.2)
+		(layer "B.Cu")
+		(net 20)
+	)
+	(segment
+		(start 145.9 62.02)
 		(end 146.07 62.02)
 		(width 0.2)
@@
 	)
 	(segment
-		(start 145.92 59.48)
-		(end 144.01 59.48)
+		(start 150.68 59.48)
+		(end 151.45 60.25)
+		(width 0.5)
+		(layer "B.Cu")
+		(net 22)
+	)
+	(segment
+		(start 148.55 66.5)
+		(end 150.8 66.5)
 		(width 0.5)
 		(layer "B.Cu")
@@
 	)
 	(segment
-		(start 146.25 59.15)
-		(end 145.92 59.48)
+		(start 151.45 65.85)
+		(end 151.45 62.1)
 		(width 0.5)
 		(layer "B.Cu")
@@
 	)
 	(segment
-		(start 148.4 59.15)
-		(end 146.25 59.15)
-		(width 0.5)
-		(layer "B.Cu")
+		(start 144.01 59.48)
+		(end 150.68 59.48)
+		(width 0.5)
+		(layer "B.Cu")
+		(net 22)
+	)
+	(segment
+		(start 150.8 66.5)
+		(end 151.45 65.85)
+		(width 0.5)
+		(layer "B.Cu")
+		(net 22)
+	)
+	(segment
+		(start 151.45 60.25)
+		(end 151.45 62.1)
+		(width 0.5)
+		(layer "B.Cu")

Commit message: .
Parts:
- added EN: SW_Push, Alexander Footprint Library:SW_SPST_6x3, B.Cu at (160.3, 59.6)
Routing:
- net EN: track 10.2 -> 17.8 mm, vias 0 -> 1

Commit message: .
Parts:
- removed EN: SW_Push, Alexander Footprint Library:SW_SPST_6x3
- added C1: 1uF, Resistor_SMD:R_0612_1632Metric_Pad1.18x3.40mm_HandSolder, F.Cu at (136.3, 55.9)
- added LED1: LED-RED-GREEN-B1552USUG20D, Alexander Footprint Library:B1552_HVK-M, F.Cu at (149.0, 78.2)
- added SW1: SW_Push, Alexander Footprint Library:SW_SPST_6x3, F.Cu at (160.2, 59.5)
Routing:
- net 3V3: track 21.3 -> 41.5 mm, vias 0 -> 1

Commit message: .
Parts:
- SW1: moved to B.Cu

Commit message: .
Routing:
- net 3V3: track 41.5 -> 33.8 mm
Changed lines of the file:
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@@
+	)
+	(segment
+		(start 148.249999 74.849999)
+		(end 148.2 74.8)
+		(width 0.5)
+		(layer "F.Cu")
+		(net 22)
 	)
 	(segment
@@
 		(end 145.62 59.48)
 		(width 0.2)
-		(layer "F.Cu")
-		(net 22)
-	)
-	(segment
-		(start 153.4 72.1)
-		(end 152.6 72.9)
-		(width 0.25)
 		(layer "F.Cu")
 		(net 22)
@@
 	)
 	(segment
-		(start 153.4 62.7)
-		(end 153.4 72.1)
-		(width 0.25)
-		(layer "F.Cu")
-		(net 22)
-	)
-	(segment
-		(start 148.249999 73.750001)
-		(end 148.249999 76.5998)
-		(width 0.25)
-		(layer "F.Cu")
-		(net 22)
-	)
-	(segment
-		(start 149.1 72.9)
-		(end 148.249999 73.750001)
+		(start 148.249999 76.5998)
+		(end 148.249999 74.849999)
 		(width 0.25)
 		(layer "F.Cu")
@@
 		(net 22)
 	)
-	(segment
-		(start 152.6 72.9)
-		(end 149.1 72.9)
-		(width 0.25)
-		(layer "F.Cu")
-		(net 22)
-	)
 	(via
-		(at 153.4 62.7)
+		(at 148.2 74.8)
 		(size 0.6)
 		(drill 0.3)
@@
 	)
 	(segment
+		(start 148.2 74.8)
+		(end 146.4 73)
+		(width 0.25)
+		(layer "B.Cu")
+		(net 22)
+	)
+	(segment
 		(start 150.68 59.48)
 		(end 151.45 60.25)
 		(width 0.5)
+		(layer "B.Cu")
+		(net 22)
+	)
+	(segment
+		(start 147.2 66.5)
+		(end 148.55 66.5)
+		(width 0.25)
 		(layer "B.Cu")
 		(net 22)
@@
 	)
 	(segment
-		(start 153.4 62.7)
-		(end 152.8 62.1)
+		(start 146.4 73)
+		(end 146.4 67.3)
 		(width 0.25)
 		(layer "B.Cu")
@@
 	)
 	(segment
-		(start 152.8 62.1)
-		(end 151.45 62.1)
+		(start 146.4 67.3)
+		(end 147.2 66.5)
 		(width 0.25)
 		(layer "B.Cu")

Commit message: .
Connections:
- LED1 pad 2: 3V3 -> EN
- LED1 pad 3: 3V3 -> unconnected-(LED1-GRN-Pad3)
Routing:
- net EN: track 17.8 -> 33.0 mm, vias 1 -> 2
- net 3V3: track 33.8 -> 21.3 mm, vias 1 -> 0
Changed lines of the file:
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@@
 	(net 22 "3V3")
 	(net 23 "GPIO6")
+	(net 24 "unconnected-(LED1-GRN-Pad3)")
 	(footprint "Alexander Footprint Library:ESP32-C3-WROOM-02-H4"
 		(layer "F.Cu")
@@
 			(size 1.1176 1.0414)
 			(layers "F.Cu" "F.Paste" "F.Mask")
-			(net 22 "3V3")
+			(net 20 "EN")
 			(pinfunction "RED")
 			(pintype "power_out")
@@
 			(size 1.1176 1.0414)
 			(layers "F.Cu" "F.Paste" "F.Mask")
-			(net 22 "3V3")
+			(net 24 "unconnected-(LED1-GRN-Pad3)")
 			(pinfunction "GRN")
 			(pintype "power_in")
@@
 	)
 	(segment
+		(start 148.249999 74.849999)
+		(end 148.2 74.8)
+		(width 0.5)
+		(layer "F.Cu")
+		(net 20)
+	)
+	(segment
 		(start 146.8 59.7)
 		(end 146.1 60.4)
@@
 	)
 	(segment
+		(start 148.249999 76.5998)
+		(end 148.249999 74.849999)
+		(width 0.25)
+		(layer "F.Cu")
+		(net 20)
+	)
+	(segment
 		(start 148.19 59.7)
 		(end 153.3 59.7)
@@
 		(net 20)
 	)
+	(via
+		(at 148.2 74.8)
+		(size 0.6)
+		(drill 0.3)
+		(layers "F.Cu" "B.Cu")
+		(net 20)
+	)
 	(segment
 		(start 144.01 62.02)
 		(end 145.9 62.02)
-		(width 0.2)
+		(width 0.25)
 		(layer "B.Cu")
 		(net 20)
 	)
 	(segment
-		(start 145.98 62.1)
-		(end 145.9 62.02)
-		(width 0.2)
+		(start 146.4 62.52)
+		(end 146.4 73)
+		(width 0.25)
+		(layer "B.Cu")
+		(net 20)
+	)
+	(segment
+		(start 145.9 62.02)
+		(end 146.4 62.52)
+		(width 0.25)
 		(layer "B.Cu")
 		(net 20)
@@
 		(start 148.35 62.1)
 		(end 145.98 62.1)
-		(width 0.2)
+		(width 0.25)
 		(layer "B.Cu")
 		(net 20)
 	)
 	(segment
-		(start 145.9 62.02)
-		(end 146.07 62.02)
-		(width 0.2)
+		(start 146.4 73)
+		(end 148.2 74.8)
+		(width 0.25)
 		(layer "B.Cu")
 		(net 20)
@@
 	)
 	(segment
-		(start 148.249999 74.849999)
-		(end 148.2 74.8)
-		(width 0.5)
-		(layer "F.Cu")
-		(net 22)
-	)
-	(segment
 		(start 146.9 58.2)
 		(end 145.62 59.48)
@@
 	)
 	(segment
-		(start 148.249999 76.5998)
-		(end 148.249999 74.849999)
-		(width 0.25)
-		(layer "F.Cu")
-		(net 22)
-	)
-	(segment
 		(start 148.19 58.2)
 		(end 146.9 58.2)
@@
 		(net 22)
 	)
-	(via
-		(at 148.2 74.8)
-		(size 0.6)
-		(drill 0.3)
-		(layers "F.Cu" "B.Cu")
-		(net 22)
-	)
-	(segment
-		(start 148.2 74.8)
-		(end 146.4 73)
-		(width 0.25)
-		(layer "B.Cu")
-		(net 22)
-	)
 	(segment
 		(start 150.68 59.48)
@@
 	)
 	(segment
-		(start 147.2 66.5)
-		(end 148.55 66.5)
-		(width 0.25)
-		(layer "B.Cu")
-		(net 22)
-	)
-	(segment
 		(start 148.55 66.5)
 		(end 150.8 66.5)
@@
 	)
 	(segment
-		(start 146.4 73)
-		(end 146.4 67.3)
-		(width 0.25)
-		(layer "B.Cu")
-		(net 22)
-	)
-	(segment
 		(start 150.8 66.5)
 		(end 151.45 65.85)
@@
 		(layer "B.Cu")
 		(net 22)
-	)
-	(segment
-		(start 146.4 67.3)
-		(end 147.2 66.5)
-		(width 0.25)
-		(layer "B.Cu")
-		(net 22)
