File: ESP32-C3-WROOM-Node-Temperature_USB-C/ESP32-C3-WROOM-Node-Temperature/ESP32-C3-WROOM-Node-Temperature.kicad_pcb (KiCad board)
At the start: 2 copper layers, 65 x 40 mm, 30 parts, among them J1 PWR, J2 Conn_01x02_Socket, J3 Conn_01x02_Socket, J4 I2C, J5 USB-C_Receptacle_PowerOnly_6P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, K1 Relay_DPDT_HK19F_HUI, Q1 NPN, SW1 SW_SPDT, U2 AMS1117-3V3, U4 L7805

Commit message: .
Parts:
- moved R5 29.8 mm to (149.1, 71.4), turned to 90 degrees
- moved R6 23.3 mm to (144.9, 71.3), turned to 90 degrees
- moved GND 11.1 mm to (159.8, 55.0)
- moved J5 2.01 mm to (145.6, 58.9)
- moved C3 2.00 mm to (134.0, 71.3)
- moved C6 2.00 mm to (139.8, 71.3)
- moved U2 1.10 mm to (129.0, 66.2)
Connections:
- J1 pad 2: Net-(J1-Pin_2) -> /Power Supply/PWR
- J5 pad A9: unconnected-(J5-VBUS-PadA9) -> /Power Supply/PWR
- J5 pad B9: unconnected-(J5-VBUS-PadB9) -> /Power Supply/PWR
- SW1 pad 3: Net-(J1-Pin_2) -> /Power Supply/PWR
Routing:
- net /Power Supply/PWR: track 0.00 -> 66.8 mm, vias 0 -> 1
- net Net-(J5-CC1): track 0.00 -> 6.98 mm
- net Net-(J1-Pin_2): track 5.92 -> 0.00 mm
- net Net-(J5-CC2): track 0.00 -> 4.43 mm
- net +3V3: track 167.1 -> 169.5 mm
- net +5V: track 71.6 -> 72.9 mm

Commit message: .
Parts:
- moved GND 10.5 mm to (153.5, 63.4)
- moved 5V 1.90 mm to (156.9, 62.3)
- moved 3V3 1.61 mm to (160.1, 62.2)
Routing:
- net +3V3: track 169.5 -> 170.4 mm
Changed lines of the file:
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@@
 	(footprint "TestPoint:TestPoint_Pad_D1.5mm"
 		(layer "F.Cu")
-		(at 158.5 62.4)
+		(at 160.1 62.2)
 		(descr "SMD pad as test Point, diameter 1.5mm")
 		(tags "test point SMD pad")
@@
 	(footprint "TestPoint:TestPoint_Pad_D1.5mm"
 		(layer "F.Cu")
-		(at 155 62.4)
+		(at 156.9 62.3)
 		(descr "SMD pad as test Point, diameter 1.5mm")
 		(tags "test point SMD pad")
@@
 	(footprint "TestPoint:TestPoint_Pad_D1.5mm"
 		(layer "F.Cu")
-		(at 159.8 55)
+		(at 153.5 63.4)
 		(descr "SMD pad as test Point, diameter 1.5mm")
 		(tags "test point SMD pad")
@@
 	)
 	(segment
-		(start 145.86 76.8)
-		(end 145.83 76.83)
-		(width 0.2)
+		(start 157.92 66.68)
+		(end 160.1 64.5)
+		(width 0.25)
 		(layer "F.Cu")
 		(net 16)
 	)
 	(segment
-		(start 157.92 66.68)
-		(end 158.5 66.1)
-		(width 0.25)
+		(start 145.86 76.8)
+		(end 145.83 76.83)
+		(width 0.2)
 		(layer "F.Cu")
 		(net 16)
@@
 	)
 	(segment
-		(start 158.5 66.1)
-		(end 158.5 62.4)
+		(start 160.1 64.5)
+		(end 160.1 62.2)
 		(width 0.25)
 		(layer "F.Cu")
@@
 	(segment
 		(start 155.38 66.78)
-		(end 155 66.4)
-		(width 0.25)
-		(layer "F.Cu")
-		(net 18)
-	)
-	(segment
-		(start 155 66.4)
-		(end 155 62.4)
-		(width 0.25)
-		(layer "F.Cu")
-		(net 18)
-	)
-	(segment
-		(start 155.38 69.68)
-		(end 155.38 66.78)
+		(end 156.9 65.26)
 		(width 0.25)
 		(layer "F.Cu")
@@
 	(segment
 		(start 155.38 69.68)
-		(end 155.4 69.7)
-		(width 0.5)
-		(layer "B.Cu")
+		(end 155.38 66.78)
+		(width 0.25)
+		(layer "F.Cu")
 		(net 18)
 	)
 	(segment
-		(start 154 73.2)
-		(end 130 73.2)
-		(width 0.5)
-		(layer "B.Cu")
+		(start 156.9 65.26)
+		(end 156.9 62.3)
+		(width 0.25)
+		(layer "F.Cu")
 		(net 18)
 	)
@@
 	)
 	(segment
-		(start 155.4 71.8)
-		(end 154 73.2)
+		(start 155.38 69.68)
+		(end 155.4 69.7)
 		(width 0.5)
 		(layer "B.Cu")
@@
 	)
 	(segment
-		(start 129.445 72.645)
-		(end 126.14 72.645)
+		(start 155.4 71.8)
+		(end 154.555 72.645)
 		(width 0.5)
 		(layer "B.Cu")
@@
 	)
 	(segment
-		(start 130 73.2)
-		(end 129.445 72.645)
+		(start 154.555 72.645)
+		(end 126.14 72.645)
 		(width 0.5)
 		(layer "B.Cu")
@@
 		(end 113.8 76.22)
 		(width 0.5)
-		(layer "B.Cu")
+		(layer "F.Cu")
 		(net 19)
 	)
 	(segment
-		(start 120.52 79.3)
-		(end 120.52 86.8)
-		(width 1)
-		(layer "B.Cu")
-		(net 20)
-	)
-	(segment
 		(start 120.52 89.52)
 		(end 121.1 90.1)
 		(width 1)
-		(layer "B.Cu")
+		(layer "F.Cu")
 		(net 20)
 	)
@@
 		(end 120.52 89.52)
 		(width 1)
-		(layer "B.Cu")
+		(layer "F.Cu")
 		(net 20)
 	)
@@
 		(end 121.1 95.2)
 		(width 1)
-		(layer "B.Cu")
+		(layer "F.Cu")
 		(net 20)
 	)
 	(segment
-		(start 125.6 86.8)
-		(end 125.6 79.3)
+		(start 120.52 86.8)
+		(end 120.52 79.3)
 		(width 1)
 		(layer "B.Cu")
+		(net 20)
+	)
+	(segment
+		(start 126.18 90.28)
+		(end 126.18 95.2)
+		(width 1)
+		(layer "F.Cu")
 		(net 21)
 	)
 	(segment
-		(start 126.18 95.2)
-		(end 131.7 95.2)
+		(start 125.6 89.7)
+		(end 126.18 90.28)
 		(width 1)
-		(layer "B.Cu")
+		(layer "F.Cu")
 		(net 21)
 	)
 	(segment
-		(start 126.18 89.88)
-		(end 126.18 95.2)
+		(start 126.18 95.2)
+		(end 131.7 95.2)
 		(width 1)
-		(layer "B.Cu")
+		(layer "F.Cu")
 		(net 21)
 	)
 	(segment
 		(start 125.6 86.8)
-		(end 125.6 89.3)
+		(end 125.6 89.7)
 		(width 1)
-		(layer "B.Cu")
+		(layer "F.Cu")
 		(net 21)
 	)
 	(segment
-		(start 125.6 89.3)
-		(end 126.18 89.88)
+		(start 125.6 86.8)
+		(end 125.6 79.3)
 		(width 1)
 		(layer "B.Cu")
@@
 	)
 	(segment
-		(start 130.68 86.8)
-		(end 130.68 79.3)
+		(start 136.78 92.48)
+		(end 136.78 95.2)
 		(width 1)
-		(layer "B.Cu")
+		(layer "F.Cu")
 		(net 22)
 	)
 	(segment
-		(start 130.68 89.38)
-		(end 132 90.7)
+		(start 134.9 90.6)
+		(end 136.78 92.48)
 		(width 1)
-		(layer "B.Cu")
+		(layer "F.Cu")
 		(net 22)
 	)
 	(segment
-		(start 132 90.7)
-		(end 135.6 90.7)
+		(start 132 90.6)
+		(end 134.9 90.6)
 		(width 1)
-		(layer "B.Cu")
+		(layer "F.Cu")
 		(net 22)
 	)
 	(segment
-		(start 130.68 86.8)
-		(end 130.68 89.38)
+		(start 130.68 89.28)
+		(end 132 90.6)
 		(width 1)
-		(layer "B.Cu")
+		(layer "F.Cu")
 		(net 22)
 	)
 	(segment
-		(start 135.6 90.7)
-		(end 136.78 91.88)
+		(start 130.68 86.8)
+		(end 130.68 89.28)
 		(width 1)
-		(layer "B.Cu")
+		(layer "F.Cu")
 		(net 22)
 	)
 	(segment
-		(start 136.78 91.88)
-		(end 136.78 95.2)
+		(start 130.68 86.8)
+		(end 130.68 79.3)
 		(width 1)
 		(layer "B.Cu")
@@
 	)
 	(segment
-		(start 138.4 63.5)
-		(end 145.1 63.5)
-		(width 0.5)
-		(layer "F.Cu")
-		(net 27)
-	)
-	(segment
 		(start 113.775 81.325)
 		(end 113.8 81.3)
@@
 	)
 	(segment
+		(start 143.2 63.5)
+		(end 145.1 63.5)
+		(width 0.5)
+		(layer "F.Cu")
+		(net 27)
+	)
+	(segment
 		(start 147.12 64.12)
 		(end 146.5 63.5)
@@
 		(net 27)
 	)
-	(segment
-		(start 138.1 63.2)
-		(end 138.4 63.5)
-		(width 0.5)
-		(layer "F.Cu")
-		(net 27)
-	)
 	(via
-		(at 138.1 63.2)
+		(at 143.2 63.5)
 		(size 0.6)
 		(drill 0.3)
@@
 	)
 	(segment
-		(start 115.9 81.3)
-		(end 116.8 80.4)
+		(start 120.9 61.5)
+		(end 119.2 63.2)
 		(width 0.5)
 		(layer "B.Cu")
@@
 	)
 	(segment
-		(start 119.2 68.4)
-		(end 119.2 63.2)
+		(start 138.4 63.5)
+		(end 136.4 61.5)
 		(width 0.5)
 		(layer "B.Cu")
@@
 	)
 	(segment
-		(start 113.8 81.3)
+		(start 116.8 80.4)
 		(end 115.9 81.3)
 		(width 0.5)
@@
 	)
 	(segment
-		(start 136.4 61.5)
-		(end 138.1 63.2)
+		(start 116.8 70.8)
+		(end 116.8 80.4)
 		(width 0.5)
 		(layer "B.Cu")
@@
 	)
 	(segment
-		(start 113.775 87.21)
-		(end 113.775 81.325)
+		(start 119.2 63.2)
+		(end 119.2 68.4)
 		(width 0.5)
 		(layer "B.Cu")
@@
 	)
 	(segment
-		(start 116.8 80.4)
-		(end 116.8 70.8)
+		(start 136.4 61.5)
+		(end 120.9 61.5)
 		(width 0.5)
 		(layer "B.Cu")
@@
 	)
 	(segment
-		(start 116.8 70.8)
-		(end 119.2 68.4)
+		(start 113.775 87.21)
+		(end 113.775 81.325)
 		(width 0.5)
 		(layer "B.Cu")
@@
 	)
 	(segment
-		(start 119.2 63.2)
-		(end 120.9 61.5)
+		(start 115.9 81.3)
+		(end 113.8 81.3)
 		(width 0.5)
 		(layer "B.Cu")
@@
 	)
 	(segment
-		(start 120.9 61.5)
-		(end 136.4 61.5)
+		(start 119.2 68.4)
+		(end 116.8 70.8)
+		(width 0.5)
+		(layer "B.Cu")
+		(net 27)
+	)
+	(segment
+		(start 143.2 63.5)
+		(end 138.4 63.5)
 		(width 0.5)
 		(layer "B.Cu")
