File: esp32-c3-wroom-socket-USB-C_4layers/esp32-c3-wroom-socket/esp32-c3-wroom-socket.kicad_pcb (KiCad board)
At the start: 2 copper layers, 30.5 x 25.4 mm, 10 parts, among them J3 USB-C_KUSBX-SL-CS1N14-B, SW1 SW_Push, U1 ESP32-C3-WROOM-02-N4, U2 AMS1117-3V3

Commit message: .
Parts:
- moved R4 1.61 mm to (165.6, 74.8), turned to 90 degrees
- moved LED1 0.68 mm to (157.4, 74.8), turned to -90 degrees
Routing:
- net Net-(LED1-GND-Pad1): track 6.87 -> 0.00 mm
- net GND: track 7.28 -> 12.2 mm, vias 17 -> 14
- net 3V3: track 41.4 -> 39.7 mm
- added copper zone on In2.Cu, net 3V3
- added copper zone on In1.Cu, net GND
- removed copper zone on B.Cu, net GND
- removed copper zone on F.Cu, net GND
Other:
- copper layers 2 -> 4

Commit message: .
Routing:
- net GND: vias 14 -> 0
Changed lines of the file:
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@@
 	(layers
 		(0 "F.Cu" signal)
-		(1 "In1.Cu" signal)
-		(2 "In2.Cu" signal)
+		(1 "In1.Cu" signal "Layer 3")
+		(2 "In2.Cu" mixed "Layer 4")
 		(31 "B.Cu" signal)
 		(32 "B.Adhes" user "B.Adhesive")
@@
 		(net 2)
 	)
-	(via
-		(at 151.2 68.2)
-		(size 0.6)
-		(drill 0.3)
-		(layers "F.Cu" "B.Cu")
-		(free yes)
-		(net 2)
-	)
-	(via
-		(at 153.4 58)
-		(size 0.6)
-		(drill 0.3)
-		(layers "F.Cu" "B.Cu")
-		(free yes)
-		(net 2)
-	)
-	(via
-		(at 156.2 71.2)
-		(size 0.6)
-		(drill 0.3)
-		(layers "F.Cu" "B.Cu")
-		(free yes)
-		(net 2)
-	)
-	(via
-		(at 152 68.2)
-		(size 0.6)
-		(drill 0.3)
-		(layers "F.Cu" "B.Cu")
-		(free yes)
-		(net 2)
-	)
-	(via
-		(at 156.2 69.6)
-		(size 0.6)
-		(drill 0.3)
-		(layers "F.Cu" "B.Cu")
-		(free yes)
-		(net 2)
-	)
-	(via
-		(at 154.2 58)
-		(size 0.6)
-		(drill 0.3)
-		(layers "F.Cu" "B.Cu")
-		(free yes)
-		(net 2)
-	)
-	(via
-		(at 154 81.2)
-		(size 0.6)
-		(drill 0.3)
-		(layers "F.Cu" "B.Cu")
-		(free yes)
-		(net 2)
-	)
-	(via
-		(at 152.6 58)
-		(size 0.6)
-		(drill 0.3)
-		(layers "F.Cu" "B.Cu")
-		(free yes)
-		(net 2)
-	)
-	(via
-		(at 154 80)
-		(size 0.6)
-		(drill 0.3)
-		(layers "F.Cu" "B.Cu")
-		(free yes)
-		(net 2)
-	)
-	(via
-		(at 156.2 70.4)
-		(size 0.6)
-		(drill 0.3)
-		(layers "F.Cu" "B.Cu")
-		(free yes)
-		(net 2)
-	)
-	(via
-		(at 156.2 68.8)
-		(size 0.6)
-		(drill 0.3)
-		(layers "F.Cu" "B.Cu")
-		(free yes)
-		(net 2)
-	)
-	(via
-		(at 152.8 68.2)
-		(size 0.6)
-		(drill 0.3)
-		(layers "F.Cu" "B.Cu")
-		(free yes)
-		(net 2)
-	)
-	(via
-		(at 155 58)
-		(size 0.6)
-		(drill 0.3)
-		(layers "F.Cu" "B.Cu")
-		(free yes)
-		(net 2)
-	)
-	(via
-		(at 150.4 68.2)
-		(size 0.6)
-		(drill 0.3)
-		(layers "F.Cu" "B.Cu")
-		(free yes)
-		(net 2)
-	)

Commit message: .
Routing:
- net 3V3: track 39.7 -> 14.0 mm
- net Net-(LED1-GND-Pad1): track 0.00 -> 10.6 mm
- net GND: track 12.2 -> 18.0 mm, vias 0 -> 2
- added copper zone on F.Cu, net 3V3
- added copper zone on B.Cu, net GND
Changed lines of the file:
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@@
+	)
+	(segment
+		(start 165.79 79.6)
+		(end 165.79 76.54)
+		(width 0.25)
+		(layer "F.Cu")
+		(net 2)
 	)
 	(segment
@@
 	)
 	(segment
+		(start 165.79 76.54)
+		(end 165.6 76.35)
+		(width 0.25)
+		(layer "F.Cu")
+		(net 2)
+	)
+	(segment
 		(start 147.8 70.2)
 		(end 147.025 70.975)
@@
 	)
 	(segment
+		(start 164.35 76.35)
+		(end 163.6 75.6)
+		(width 0.25)
+		(layer "F.Cu")
+		(net 2)
+	)
+	(segment
+		(start 165.6 76.35)
+		(end 164.35 76.35)
+		(width 0.25)
+		(layer "F.Cu")
+		(net 2)
+	)
+	(segment
 		(start 146.225 73.671726)
 		(end 146.225 77.585)
 		(width 0.25)
 		(layer "F.Cu")
+		(net 2)
+	)
+	(via
+		(at 163.6 75.6)
+		(size 0.6)
+		(drill 0.3)
+		(layers "F.Cu" "B.Cu")
+		(net 2)
+	)
+	(via
+		(at 151.8 64.2)
+		(size 0.6)
+		(drill 0.3)
+		(layers "F.Cu" "B.Cu")
+		(net 2)
+	)
+	(segment
+		(start 151.7 64.2)
+		(end 151.8 64.2)
+		(width 0.5)
+		(layer "B.Cu")
 		(net 2)
 	)
@@
 	)
 	(segment
-		(start 150.8 58.2)
-		(end 154.8 62.2)
-		(width 0.25)
-		(layer "F.Cu")
-		(net 18)
-	)
-	(segment
-		(start 146.9 58.2)
-		(end 145.62 59.48)
-		(width 0.5)
-		(layer "F.Cu")
-		(net 18)
-	)
-	(segment
-		(start 154.8 72.8)
-		(end 155.2 73.2)
-		(width 0.25)
-		(layer "F.Cu")
-		(net 18)
-	)
-	(segment
-		(start 154.8 62.2)
-		(end 154.8 72.8)
-		(width 0.25)
-		(layer "F.Cu")
-		(net 18)
-	)
-	(segment
-		(start 145.62 59.48)
-		(end 144.01 59.48)
-		(width 0.5)
-		(layer "F.Cu")
-		(net 18)
-	)
-	(segment
-		(start 148.19 58.2)
-		(end 146.9 58.2)
-		(width 0.5)
-		(layer "F.Cu")
-		(net 18)
-	)
-	(segment
-		(start 155.2 73.2)
-		(end 156.699998 73.2)
-		(width 0.25)
-		(layer "F.Cu")
-		(net 18)
-	)
-	(segment
-		(start 148.19 58.2)
-		(end 150.8 58.2)
-		(width 0.25)
-		(layer "F.Cu")
-		(net 18)
-	)
-	(segment
 		(start 154 61.8)
 		(end 154 64.2)
@@
 	)
 	(segment
+		(start 165.55 73.2)
+		(end 165.6 73.25)
+		(width 0.25)
+		(layer "F.Cu")
+		(net 21)
+	)
+	(segment
+		(start 158.2 76.4004)
+		(end 158.2 73.2)
+		(width 0.25)
+		(layer "F.Cu")
+		(net 21)
+	)
+	(segment
+		(start 158.2 73.2)
+		(end 165.55 73.2)
+		(width 0.25)
+		(layer "F.Cu")
+		(net 21)
+	)
+	(segment
 		(start 153.35 76.95)
 		(end 155.2 76.95)
@@
 		(layer "B.Cu")
 		(net 23)
+	)
+	(zone
+		(net 18)
+		(net_name "3V3")
+		(layer "F.Cu")
+		(hatch edge 0.5)
+		(priority 2)
+		(connect_pads
+			(clearance 0.5)
+		)
+		(min_thickness 0.25)
+		(filled_areas_thickness no)
+		(fill yes
+			(thermal_gap 0.5)
+			(thermal_bridge_width 0.5)
+		)
+		(polygon
+			(pts
+				(xy 141 56.6) (xy 172.6 56.6) (xy 172.6 83) (xy 141 83)
+			)
+		)
 	)
 	(zone
@@
 			)
 		)
+	)
+	(zone
+		(net 2)
+		(net_name "GND")
+		(layer "B.Cu")
+		(hatch edge 0.5)
+		(priority 3)
+		(connect_pads
+			(clearance 0.5)
+		)
+		(min_thickness 0.25)
+		(filled_areas_thickness no)
+		(fill yes
+			(thermal_gap 0.5)
+			(thermal_bridge_width 0.5)
+		)
+		(polygon
+			(pts
+				(xy 140.8 56.4) (xy 172.8 56.4) (xy 172.8 83.2) (xy 140.8 83.2)
+			)
+		)
