File: Production/prod_esp32-c3-wroom-socket/esp32-c3-wroom-socket.kicad_pcb (KiCad board)
At the start: 2 copper layers, 30.5 x 25.4 mm, 10 parts, among them J3 USB-C_KUSBX-SL-CS1N14-B, SW1 SW_Push, U1 ESP32-C3-WROOM-02-N4, U2 AMS1117-3V3

Commit message: .
Parts:
- removed SW1: SW_Push, Alexander Footprint Library:SW_SPST_6x3
- added SW2: SW_Push_SMD_6x3.5, Alexander Footprint Library:SW_PUSH_6x3.5mm, F.Cu at (165.7, 79.4)
Routing:
- net EN: track 35.6 -> 38.0 mm

Commit message: .
Parts:
- added R7: 10k, Resistor_SMD:R_1206_3216Metric_Pad1.30x1.75mm_HandSolder, F.Cu at (155.8, 75.6)
- added SW1: SW_Push_SMD_6x3.5, Alexander Footprint Library:SW_PUSH_6x3.5mm, F.Cu at (165.4, 79.4)
- moved LED1 24.6 mm to (180.8, 65.2)
- moved R4 20.1 mm to (183.6, 70.4)
- moved SW2 4.80 mm to (165.4, 74.6)
Routing:
- net EN: track 38.0 -> 17.7 mm
- net GPIO9: track 10.9 -> 29.8 mm
- net GPIO8: track 10.0 -> 27.0 mm
- net 3V3: track 41.4 -> 30.0 mm, vias 0 -> 1
- net Net-(LED1-GND-Pad1): track 6.87 -> 0.00 mm

Commit message: .
Parts:
- LED1, R4: moved to B.Cu
- moved LED1 24.8 mm to (156.7, 59.2)
- moved R4 22.9 mm to (161.8, 63.5), turned to 90 degrees
Routing:
- net EN: track 17.7 -> 33.3 mm

Commit message: .
Parts:
- moved R4 0.21 mm to (161.6, 63.6)
- moved LED1 0.15 mm to (156.7, 59.4)
Routing:
- net Net-(LED1-GND-Pad1): track 0.00 -> 8.03 mm
- net GND: vias 17 -> 13
Changed lines of the file:
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@@
 	(footprint "Alexander Footprint Library:B1552_HVK-M"
 		(layer "B.Cu")
-		(at 156.71 59.2)
+		(at 156.71 59.350001)
 		(tags "B1552USUG20D000113U1930 ")
 		(property "Reference" "LED1"
@@
 	(footprint "Resistor_SMD:R_1206_3216Metric_Pad1.30x1.75mm_HandSolder"
 		(layer "B.Cu")
-		(at 161.8 63.55 90)
+		(at 161.6 63.6 90)
 		(descr "Resistor SMD 1206 (3216 Metric), square (rectangular) end terminal, IPC_7351 nominal with elongated pad for handsoldering. (Body size source: IPC-SM-782 page 72, https://www.pcb-3d.com/wordpress/wp-content/uploads/ipc-sm-782a_amendment_1_and_2.pdf), generated with kicad-footprint-generator")
 		(tags "resistor handsolder")
@@
 	)
 	(via
-		(at 151.4 58)
-		(size 0.6)
-		(drill 0.3)
-		(layers "F.Cu" "B.Cu")
-		(free yes)
-		(net 2)
-	)
-	(via
 		(at 156.2 71.2)
 		(size 0.6)
@@
 	)
 	(via
-		(at 152.2 58)
-		(size 0.6)
-		(drill 0.3)
-		(layers "F.Cu" "B.Cu")
-		(free yes)
-		(net 2)
-	)
-	(via
 		(at 154 81.2)
 		(size 0.6)
@@
 	)
 	(via
-		(at 150.6 58)
-		(size 0.6)
-		(drill 0.3)
-		(layers "F.Cu" "B.Cu")
-		(free yes)
-		(net 2)
-	)
-	(via
-		(at 154 80)
+		(at 155.2 81.2)
 		(size 0.6)
 		(drill 0.3)
@@
 	)
 	(via
-		(at 153 58)
-		(size 0.6)
-		(drill 0.3)
-		(layers "F.Cu" "B.Cu")
-		(free yes)
-		(net 2)
-	)
-	(via
 		(at 150.4 68.2)
 		(size 0.6)
@@
 	)
 	(segment
+		(start 152.4 61.4)
+		(end 154 63)
+		(width 0.5)
+		(layer "B.Cu")
+		(net 18)
+	)
+	(segment
+		(start 154 63)
+		(end 154 64.2)
+		(width 0.5)
+		(layer "B.Cu")
+		(net 18)
+	)
+	(segment
 		(start 144.03 59.5)
 		(end 144.01 59.48)
@@
 	(segment
 		(start 151.45 61.4)
-		(end 152.8 61.4)
-		(width 0.5)
-		(layer "B.Cu")
-		(net 18)
-	)
-	(segment
-		(start 152.8 61.4)
-		(end 154 62.6)
-		(width 0.5)
-		(layer "B.Cu")
-		(net 18)
-	)
-	(segment
-		(start 154 62.6)
-		(end 154 64.2)
+		(end 152.4 61.4)
 		(width 0.5)
 		(layer "B.Cu")
@@
 	)
 	(segment
+		(start 155.1098 60.100002)
+		(end 158.3102 60.100002)
+		(width 0.2)
+		(layer "B.Cu")
+		(net 21)
+	)
+	(segment
+		(start 161.6 62.05)
+		(end 161.6 60.8)
+		(width 0.2)
+		(layer "B.Cu")
+		(net 21)
+	)
+	(segment
+		(start 158.3102 60.100002)
+		(end 160.900002 60.100002)
+		(width 0.2)
+		(layer "B.Cu")
+		(net 21)
+	)
+	(segment
+		(start 160.900002 60.100002)
+		(end 161.6 60.8)
+		(width 0.2)
+		(layer "B.Cu")
+		(net 21)
+	)
+	(segment

Commit message: .
Parts:
- moved R4 1.85 mm to (161.6, 61.8)
Routing:
- net Net-(LED1-GND-Pad1): track 8.03 -> 6.53 mm
- net VBUS: track 32.3 -> 31.4 mm
- net USB_D-: track 62.0 -> 61.5 mm

Commit message: .
Parts:
- turned LED1 to 180 degrees
Routing:
- net Net-(LED1-GND-Pad1): track 6.53 -> 0.14 mm
- net GND: track 7.28 -> 9.54 mm, vias 13 -> 10

Commit message: .
Parts:
- moved R4 3.24 mm to (163.6, 59.2), turned to 180 degrees
- turned LED1 to 0 degrees
Connections:
- LED1 pad 2: 3V3 -> unconnected-(LED1-RED-Pad2)
- LED1 pad 3: unconnected-(LED1-GRN-Pad3) -> 3V3
Routing:
- net 3V3: track 29.3 -> 34.5 mm, vias 1 -> 2
- net Net-(LED1-GND-Pad1): track 0.14 -> 1.65 mm

Commit message: .
Parts:
- moved R4 3.61 mm to (163.4, 62.8), turned to 90 degrees
Connections:
- LED1 pad 2: unconnected-(LED1-RED-Pad2) -> 3V3
- LED1 pad 3: 3V3 -> unconnected-(LED1-GRN-Pad3)
Routing:
- net 3V3: track 34.5 -> 36.6 mm
- net Net-(LED1-GND-Pad1): track 1.65 -> 3.20 mm
Changed lines of the file:
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@@
 	(net 18 "3V3")
 	(net 19 "GPIO6")
-	(net 20 "unconnected-(LED1-RED-Pad2)")
-	(net 21 "Net-(LED1-GND-Pad1)")
-	(net 22 "Net-(J3-CC2)")
-	(net 23 "Net-(J3-CC1)")
+	(net 20 "Net-(LED1-GND-Pad1)")
+	(net 21 "Net-(J3-CC2)")
+	(net 22 "Net-(J3-CC1)")
+	(net 23 "unconnected-(LED1-GRN-Pad3)")
 	(footprint "Alexander Footprint Library:ESP32-C3-WROOM-02-H4"
 		(layer "F.Cu")
@@
 			(layers "*.Cu" "*.Mask")
 			(remove_unused_layers no)
-			(net 23 "Net-(J3-CC1)")
+			(net 22 "Net-(J3-CC1)")
 			(pinfunction "CC1")
 			(pintype "bidirectional")
@@
 			(layers "*.Cu" "*.Mask")
 			(remove_unused_layers no)
-			(net 22 "Net-(J3-CC2)")
+			(net 21 "Net-(J3-CC2)")
 			(pinfunction "CC2")
 			(pintype "bidirectional")
@@
 			(size 1.1176 1.0414)
 			(layers "B.Cu" "B.Paste" "B.Mask")
-			(net 21 "Net-(LED1-GND-Pad1)")
+			(net 20 "Net-(LED1-GND-Pad1)")
 			(pinfunction "GND")
 			(pintype "power_in")
@@
 			(size 1.1176 1.0414)
 			(layers "B.Cu" "B.Paste" "B.Mask")
-			(net 20 "unconnected-(LED1-RED-Pad2)")
+			(net 18 "3V3")
 			(pinfunction "RED")
 			(pintype "power_out")
@@
 			(size 1.1176 1.0414)
 			(layers "B.Cu" "B.Paste" "B.Mask")
-			(net 18 "3V3")
+			(net 23 "unconnected-(LED1-GRN-Pad3)")
 			(pinfunction "GRN")
 			(pintype "power_in")
@@
 			(size 1.1176 1.0414)
 			(layers "B.Cu" "B.Paste" "B.Mask")
-			(net 21 "Net-(LED1-GND-Pad1)")
+			(net 20 "Net-(LED1-GND-Pad1)")
 			(pinfunction "GND")
 			(pintype "power_out")
@@
 			(layers "B.Cu" "B.Paste" "B.Mask")
 			(roundrect_rratio 0.192308)
-			(net 23 "Net-(J3-CC1)")
+			(net 22 "Net-(J3-CC1)")
 			(pintype "passive")
 		)
@@
 	(footprint "Resistor_SMD:R_1206_3216Metric_Pad1.30x1.75mm_HandSolder"
 		(layer "B.Cu")
-		(at 163.6 59.2 180)
+		(at 163.4 62.8 90)
 		(descr "Resistor SMD 1206 (3216 Metric), square (rectangular) end terminal, IPC_7351 nominal with elongated pad for handsoldering. (Body size source: IPC-SM-782 page 72, https://www.pcb-3d.com/wordpress/wp-content/uploads/ipc-sm-782a_amendment_1_and_2.pdf), generated with kicad-footprint-generator")
 		(tags "resistor handsolder")
 		(property "Reference" "R4"
-			(at 0 1.82 360)
+			(at 0 1.82 90)
 			(layer "B.SilkS")
 			(effects
@@
 		)
 		(property "Value" "5k1"
-			(at 0 -1.82 360)
+			(at 0 -1.82 90)
 			(layer "B.Fab")
 			(effects
@@
 		)
 		(property "Footprint" "Resistor_SMD:R_1206_3216Metric_Pad1.30x1.75mm_HandSolder"
-			(at 0 0 0)
+			(at 0 0 -90)
 			(unlocked yes)
 			(layer "B.Fab")
@@
 		)
 		(property "Datasheet" ""
-			(at 0 0 0)
+			(at 0 0 -90)
 			(unlocked yes)
 			(layer "B.Fab")
@@
 		)
 		(property "Description" "Resistor"
-			(at 0 0 0)
+			(at 0 0 -90)
 			(unlocked yes)
 			(layer "B.Fab")
@@
 		(attr smd)
 		(fp_line
-			(start 0.727064 0.91)
-			(end -0.727064 0.91)
+			(start 0.727064 -0.91)
+			(end -0.727064 -0.91)
 			(stroke
 				(width 0.12)
@@
 		)
 		(fp_line
-			(start 0.727064 -0.91)
-			(end -0.727064 -0.91)
+			(start 0.727064 0.91)
+			(end -0.727064 0.91)
 			(stroke
 				(width 0.12)
@@
 		)
 		(fp_line
-			(start 2.45 1.12)
-			(end -2.45 1.12)
+			(start 2.45 -1.12)
+			(end 2.45 1.12)
 			(stroke
 				(width 0.05)
@@
 		)
 		(fp_line
-			(start 2.45 -1.12)
-			(end 2.45 1.12)
+			(start -2.45 -1.12)
+			(end 2.45 -1.12)
 			(stroke
 				(width 0.05)
@@
 		)
 		(fp_line
-			(start -2.45 1.12)
-			(end -2.45 -1.12)
+			(start 2.45 1.12)
+			(end -2.45 1.12)
 			(stroke
 				(width 0.05)
@@
 		)
 		(fp_line
-			(start -2.45 -1.12)
-			(end 2.45 -1.12)
+			(start -2.45 1.12)
+			(end -2.45 -1.12)
 			(stroke
 				(width 0.05)
@@
 		)
 		(fp_line
-			(start 1.6 0.8)
-			(end -1.6 0.8)
+			(start 1.6 -0.8)
+			(end 1.6 0.8)
 			(stroke
 				(width 0.1)
@@
 		)
 		(fp_line
-			(start 1.6 -0.8)
-			(end 1.6 0.8)
+			(start -1.6 -0.8)
+			(end 1.6 -0.8)
 			(stroke
 				(width 0.1)
@@
 		)
 		(fp_line
-			(start -1.6 0.8)
-			(end -1.6 -0.8)
+			(start 1.6 0.8)
+			(end -1.6 0.8)
 			(stroke
 				(width 0.1)
@@
 		)
 		(fp_line
-			(start -1.6 -0.8)
-			(end 1.6 -0.8)
+			(start -1.6 0.8)
+			(end -1.6 -0.8)
 			(stroke
 				(width 0.1)
@@
 		)
 		(fp_text user "${REFERENCE}"
-			(at 0 0 360)
+			(at 0 0 90)
 			(layer "B.Fab")
 			(effects
@@
 		)
 		(pad "1" smd roundrect
-			(at -1.55 0 180)
+			(at -1.55 0 90)
 			(size 1.3 1.75)
 			(layers "B.Cu" "B.Paste" "B.Mask")
@@
 		)
 		(pad "2" smd roundrect
-			(at 1.55 0 180)
+			(at 1.55 0 90)
 			(size 1.3 1.75)
 			(layers "B.Cu" "B.Paste" "B.Mask")
 			(roundrect_rratio 0.192308)
-			(net 21 "Net-(LED1-GND-Pad1)")
+			(net 20 "Net-(LED1-GND-Pad1)")
 			(pintype "passive")
 		)
@@
 			(layers "B.Cu" "B.Paste" "B.Mask")
 			(roundrect_rratio 0.192308)
-			(net 22 "Net-(J3-CC2)")
+			(net 21 "Net-(J3-CC2)")
 			(pintype "passive")
 		)
@@
 	)
 	(segment
-		(start 153 59.2)
-		(end 152 58.2)
+		(start 153.2 58)
+		(end 149.8 58)
+		(width 0.2)
+		(layer "F.Cu")
+		(net 18)
+	)
+	(segment
+		(start 149.6 58.2)
+		(end 148.19 58.2)
+		(width 0.2)
+		(layer "F.Cu")
+		(net 18)
+	)
+	(segment
+		(start 149.8 58)
+		(end 149.6 58.2)
 		(width 0.2)
 		(layer "F.Cu")
@@
 	)
 	(segment
-		(start 152 58.2)
-		(end 148.19 58.2)
-		(width 0.2)
-		(layer "F.Cu")
-		(net 18)
-	)
-	(segment
 		(start 148.19 58.2)
 		(end 146.9 58.2)
@@
 	)
 	(via
-		(at 153 59.2)
+		(at 153.2 58)
 		(size 0.6)
 		(drill 0.3)
@@
 	)
 	(segment
+		(start 153.2 58)
+		(end 153.8 58.6)
+		(width 0.2)
+		(layer "B.Cu")
+		(net 18)
+	)
+	(segment
+		(start 153.8 58.6)
+		(end 155.1098 58.6)
+		(width 0.2)
+		(layer "B.Cu")
+		(net 18)
+	)
+	(segment
 		(start 146.2 64.8)
 		(end 146.2 65.95)
@@
 	)
 	(segment
-		(start 160.4 59.2)
-		(end 162.05 59.2)
+		(start 155.1098 60.100002)
+		(end 158.3102 60.100002)
 		(width 0.2)
 		(layer "B.Cu")
-		(net 21)
+		(net 20)
 	)
 	(segment
@@
 		(width 0.2)
 		(layer "B.Cu")
-		(net 22)
+		(net 21)
 	)
 	(segment
@@
 		(width 0.2)
 		(layer "B.Cu")
-		(net 22)
+		(net 21)
 	)
 	(segment
@@
 		(width 0.2)
 		(layer "B.Cu")
-		(net 22)
+		(net 21)
 	)
 	(segment
@@
 		(width 0.2)
 		(layer "B.Cu")
-		(net 23)
+		(net 22)
 	)
 	(segment
@@
 		(width 0.2)
 		(layer "B.Cu")
-		(net 23)
+		(net 22)
 	)
 	(segment
@@
 		(width 0.2)
 		(layer "B.Cu")
-		(net 23)
+		(net 22)
 	)
 	(zone
