File: Production/prod_esp32-c3-wroom-socket/esp32-c3-wroom-socket.kicad_sch (KiCad schematic)
At the start: 15 parts, among them J1 USB-C_Receptacle_Data_16P_GCT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, J3 USB-C_KUSBX-SL-CS1N14-B, SW1 SW_Push, U1 ESP32-C3-WROOM-02-N4, U2 AMS1117-3V3

Commit message: .
Parts:
- removed SW1: SW_Push, Alexander Footprint Library:SW_SPST_6x3, symbol Switch:SW_Push
- added SW2: SW_Push_SMD_6x3.5, Alexander Footprint Library:SW_PUSH_6x3.5mm, symbol Alexander_Library_Symbols:SW_Push_SMD_6x3.5
Connections:
- net EN: now also SW2.2
- net GND: now also SW2.1
Changed lines of the file:
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@@
+	)
+	(symbol
+		(lib_id "Alexander_Library_Symbols:SW_Push_SMD_6x3.5")
+		(at 29.21 72.39 90)
+		(unit 1)
+		(exclude_from_sim no)
+		(in_bom yes)
+		(on_board yes)
+		(dnp no)
+		(property "Reference" "SW2"
+			(at 24.892 70.612 0)
+			(effects
+				(font
+					(size 1.27 1.27)
+				)
+				(justify right)
+			)
+		)
+		(property "Value" "SW_Push_SMD_6x3.5"
+			(at 32.004 62.484 0)
+			(effects
+				(font
+					(size 1.27 1.27)
+				)
+				(justify right)
+			)
+		)
+		(property "Footprint" "Alexander Footprint Library:SW_PUSH_6x3.5mm"
+			(at 24.13 72.39 0)
+			(effects
+				(font
+					(size 1.27 1.27)
+				)
+				(hide yes)
+			)
+		)
+		(property "Datasheet" "~"
+			(at 24.13 72.39 0)
+			(effects
+				(font
+					(size 1.27 1.27)
+				)
+				(hide yes)
+			)
+		)
+		(property "Description" ""
+			(at 29.21 72.39 0)
+			(effects
+				(font
+					(size 1.27 1.27)
+				)
+				(hide yes)
+			)
+		)
+		(pin "2"
+		)
+		(pin "1"
+		)
+		(instances
+			(project ""
+				(path "/1aed2ed1-0515-43a4-a546-c7b070175ea1"
+					(reference "SW2")
+					(unit 1)
+				)
+			)
+		)
 	)
 	(symbol
@@
 					(unit 1)
 				)
-			)
-		)
-	)
-	(symbol
-		(lib_id "Switch:SW_Push")
-		(at 29.21 72.39 90)
-		(unit 1)
-		(exclude_from_sim no)
-		(in_bom yes)
-		(on_board yes)
-		(dnp no)
-		(fields_autoplaced yes)
-		(property "Reference" "SW1"
-			(at 30.48 71.1199 90)
-			(effects
-				(font
-					(size 1.27 1.27)
-				)
-				(justify right)
-			)
-		)
-		(property "Value" "SW_Push"
-			(at 30.48 73.6599 90)
-			(effects
-				(font
-					(size 1.27 1.27)
-				)
-				(justify right)
-			)
-		)
-		(property "Footprint" "Alexander Footprint Library:SW_SPST_6x3"
-			(at 24.13 72.39 0)
-			(effects
-				(font
-					(size 1.27 1.27)
-				)
-				(hide yes)
-			)
-		)
-		(property "Datasheet" "~"
-			(at 24.13 72.39 0)
-			(effects
-				(font
-					(size 1.27 1.27)
-				)
-				(hide yes)
-			)
-		)
-		(property "Description" "Push button switch, generic, two pins"
-			(at 29.21 72.39 0)
-			(effects
-				(font
-					(size 1.27 1.27)
-				)
-				(hide yes)
-			)
-		)
-		(pin "2"
-		)
-		(pin "1"
-		)
-		(instances
-			(project ""
-				(path "/1aed2ed1-0515-43a4-a546-c7b070175ea1"
-					(reference "SW1")
-					(unit 1)
-				)

Commit message: .
Parts:
- added C2: 1uF, Resistor_SMD:R_0612_1632Metric_Pad1.18x3.40mm_HandSolder, symbol Device:C
- added R7: 10k, Resistor_SMD:R_1206_3216Metric_Pad1.30x1.75mm_HandSolder, symbol Device:R
- added SW1: SW_Push_SMD_6x3.5, Alexander Footprint Library:SW_PUSH_6x3.5mm, symbol Alexander_Library_Symbols:SW_Push_SMD_6x3.5
Connections:
- net 3V3: now also R7.1
- net GND: now also C2.2, SW1.1
- net GPIO8: now also R7.2
- net GPIO9: now also C2.1, SW1.2
Other:
- note added: "Strapping Pins"
- moved on the sheet: C1, J2, LED1, R1, R4, SW2, U1, U2

Commit message: .
Connections:
- net 3V3: now also LED1.3 (GRN); no longer LED1.2 (RED)
Changed lines of the file:
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@@
+	(wire
+		(pts
+			(xy 25.4 88.9) (xy 31.75 88.9)
+		)
+		(stroke
+			(width 0)
+			(type default)
+		)
+	)
 	(wire
 		(pts
@@
 		(pts
 			(xy 90.17 60.96) (xy 93.98 60.96)
-		)
-		(stroke
-			(width 0)
-			(type default)
-		)
-	)
-	(wire
-		(pts
-			(xy 25.4 81.28) (xy 31.75 81.28)
 		)
 		(stroke
@@
 	)
 	(label "3V3"
-		(at 25.4 81.28 0)
+		(at 25.4 88.9 0)
 		(fields_autoplaced yes)
 		(effects

Commit message: .
Connections:
- net 3V3: now also LED1.2 (RED); no longer LED1.3 (GRN)
Changed lines of the file:
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@@
-	(wire
-		(pts
-			(xy 25.4 88.9) (xy 31.75 88.9)
-		)
-		(stroke
-			(width 0)
-			(type default)
-		)
-	)
 	(wire
 		(pts
@@
 		(pts
 			(xy 129.54 48.26) (xy 133.35 48.26)
+		)
+		(stroke
+			(width 0)
+			(type default)
+		)
+	)
+	(wire
+		(pts
+			(xy 25.4 81.28) (xy 31.75 81.28)
 		)
 		(stroke
@@
 	)
 	(label "3V3"
-		(at 25.4 88.9 0)
+		(at 25.4 81.28 0)
 		(fields_autoplaced yes)
 		(effects

Commit message: .
Parts:
- added R8: 2K2, Resistor_SMD:R_1206_3216Metric_Pad1.30x1.75mm_HandSolder, symbol Device:R
- C1, C2: value 1uF -> 0.1uF
- R7: value 10k -> 2K2
Connections:
- net 3V3: now also R8.1
- net GPIO10: now also LED1.3 (GRN)
- net GPIO9: now also R8.2
Changed lines of the file:
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@@
 	(wire
 		(pts
+			(xy 76.2 137.16) (xy 76.2 140.97)
+		)
+		(stroke
+			(width 0)
+			(type default)
+		)
+	)
+	(wire
+		(pts
 			(xy 62.23 165.1) (xy 62.23 168.91)
 		)
@@
 	(wire
 		(pts
+			(xy 76.2 148.59) (xy 76.2 152.4)
+		)
+		(stroke
+			(width 0)
+			(type default)
+		)
+	)
+	(wire
+		(pts
 			(xy 101.6 134.62) (xy 101.6 138.43)
 		)
@@
 	(wire
 		(pts
+			(xy 24.13 88.9) (xy 31.75 88.9)
+		)
+		(stroke
+			(width 0)
+			(type default)
+		)
+	)
+	(wire
+		(pts
 			(xy 39.37 135.89) (xy 39.37 140.97)
 		)
@@
 	(wire
 		(pts
-			(xy 25.4 81.28) (xy 31.75 81.28)
+			(xy 24.13 81.28) (xy 31.75 81.28)
 		)
 		(stroke
@@
 	)
 	(label "3V3"
-		(at 25.4 81.28 0)
+		(at 24.13 81.28 0)
+		(fields_autoplaced yes)
+		(effects
+			(font
+				(size 1.27 1.27)
+			)
+			(justify left bottom)
+		)
+	)
+	(label "GPIO10"
+		(at 24.13 88.9 0)
+		(fields_autoplaced yes)
+		(effects
+			(font
+				(size 1.27 1.27)
+			)
+			(justify left bottom)
+		)
+	)
+	(label "3V3"
+		(at 76.2 137.16 0)
 		(fields_autoplaced yes)
 		(effects
@@
 			)
 		)
-		(property "Value" "1uF"
+		(property "Value" "0.1uF"
 			(at 80.01 161.2899 0)
 			(effects
@@
 	)
 	(symbol
+		(lib_id "Device:R")
+		(at 76.2 144.78 0)
+		(unit 1)
+		(exclude_from_sim no)
+		(in_bom yes)
+		(on_board yes)
+		(dnp no)
+		(fields_autoplaced yes)
+		(property "Reference" "R8"
+			(at 78.74 143.5099 0)
+			(effects
+				(font
+					(size 1.27 1.27)
+				)
+				(justify left)
+			)
+		)
+		(property "Value" "2K2"
+			(at 78.74 146.0499 0)
+			(effects
+				(font
+					(size 1.27 1.27)
+				)
+				(justify left)
+			)
+		)
+		(property "Footprint" "Resistor_SMD:R_1206_3216Metric_Pad1.30x1.75mm_HandSolder"
+			(at 74.422 144.78 90)
+			(effects
+				(font
+					(size 1.27 1.27)
+				)
+				(hide yes)
+			)
+		)
+		(property "Datasheet" "~"
+			(at 76.2 144.78 0)
+			(effects
+				(font
+					(size 1.27 1.27)
+				)
+				(hide yes)
+			)
+		)
+		(property "Description" "Resistor"
+			(at 76.2 144.78 0)
+			(effects
+				(font
+					(size 1.27 1.27)
+				)
+				(hide yes)
+			)
+		)
+		(pin "1"
+		)
+		(pin "2"
+		)
+		(instances
+			(project "esp32-c3-wroom-socket"
+				(path "/1aed2ed1-0515-43a4-a546-c7b070175ea1"
+					(reference "R8")
+					(unit 1)
+				)
+			)
+		)
+	)
+	(symbol
 		(lib_id "power:GND")
 		(at 19.05 54.61 0)
@@
 			)
 		)
-		(property "Value" "10k"
+		(property "Value" "2K2"
 			(at 104.14 143.5099 0)
 			(effects
@@
 			)
 		)
-		(property "Value" "1uF"
+		(property "Value" "0.1uF"
 			(at 43.18 161.2899 0)
 			(effects
