File: ESP32-C3-WROOM-Socket-Legacy-v2/ESP32-C3-WROOM-Socket-Legacy-v2.kicad_pcb (KiCad board)
At the start: 2 copper layers, 35.6 x 35.6 mm, 5 parts, among them SW1 SW_Push, U1 ESP32-WROOM-32D

Commit message: .
Parts:
- added U2: ESP32-C3-WROOM-02-N4, Alexander Footprint Library:ESP32-C3-WROOM-02-H4, F.Cu at (205.2, 91.5)

Commit message: .
Parts:
- U2: footprint Alexander Footprint Library:ESP32-C3-WROOM-02-H4 -> Alexander Footprint Library:ESP32-C3-WROOM-Adapter-Legacy-v3
- moved U2 4.28 mm to (207.3, 87.8)
Connections:
- U2 pad 1: unconnected-(U2-3V3-Pad1) -> +3V3
- U2 pad 19: GND__1 -> GND
- U2 pad 20: GND__1 -> GND
- U2 pad 21: GND__1 -> GND
- U2 pad 22: GND__1 -> GND
- U2 pad 23: GND__1 -> GND
- U2 pad 24: GND__1 -> GND
- U2 pad 25: GND__1 -> GND
- U2 pad 26: GND__1 -> GND
- U2 pad 27: GND__1 -> GND
- U2 pad 28: GND__1 -> GND
- U2 pad 29: GND__1 -> GND
- U2 pad 30: GND__1 -> GND
- U2 pad 31: GND__1 -> GND
- U2 pad 32: GND__1 -> GND
- U2 pad 33: GND__1 -> GND
- U2 pad 34: GND__1 -> GND
- U2 pad 35: GND__17 -> GND
- U2 pad 36: GND__17 -> GND
- U2 pad 37: GND__17 -> GND
- U2 pad 38: GND__17 -> GND
- U2 pad 39: GND__17 -> GND
- U2 pad 9: GND__1 -> GND

Commit message: .
Parts:
- added U3: ~, Alexander Footprint Library:Conn_ESP32-C3_WROOM-Socket-20P-v3, F.Cu at (207.9, 88.9)
- U2: footprint Alexander Footprint Library:ESP32-C3-WROOM-Adapter-Legacy-v3 -> Alexander Footprint Library:ESP32-C3-WROOM-02-H4
- moved U2 1.45 mm to (208.1, 86.5)
Connections:
- U2 pad 13: unconnected-(U2-IO18-Pad13) -> /USB_D-
- U2 pad 14: unconnected-(U2-IO19-Pad14) -> /USB_D+

Commit message: .
Parts:
- removed U1: ESP32-WROOM-32D, Alexander Footprint Library:ESP32-WROOM-Adapter-Legacy-v3
- R1, R2: moved to F.Cu
- U3: footprint Alexander Footprint Library:Conn_ESP32-C3_WROOM-Socket-20P-v3 -> Alexander Footprint Library:CONN-ESP32-WROOM-Adapter-Legacy-v3
- moved SW1 27.3 mm to (168.7, 79.6), turned to 0 degrees
- moved D1 25.7 mm to (166.4, 85.4)
- moved R2 20.0 mm to (173.6, 87.1), turned to 0 degrees
- moved R1 18.9 mm to (173.6, 83.8), turned to 0 degrees
Connections:
- R2 pad 2: Net-(U1-EN) -> unconnected-(R2-Pad2)
- U2 pad 11: unconnected-(U2-RXD-Pad11) -> /UART_RX
- U2 pad 12: unconnected-(U2-TXD-Pad12) -> /UART_TX
- U2 pad 17: unconnected-(U2-IO1-Pad17) -> /GPIO1
- U2 pad 18: unconnected-(U2-IO0-Pad18) -> /GPIO0
- U2 pad 2: unconnected-(U2-EN-Pad2) -> /EN
Routing:
- net Net-(D1-AB): track 28.5 -> 0.00 mm, vias 1 -> 0
- net +3V3: track 25.9 -> 5.06 mm
- net /GPIO0: track 20.2 -> 0.00 mm
- net Net-(U1-EN): track 18.5 -> 0.00 mm
- net /UART_TX: track 0.00 -> 17.0 mm
- net /UART_RX: track 0.00 -> 14.3 mm, vias 0 -> 1
- net unconnected-(U1-IO2-Pad24): track 8.30 -> 0.00 mm
- net unconnected-(U1-IO15-Pad23): track 7.62 -> 0.00 mm
- net unconnected-(U1-IO26-Pad11): track 7.28 -> 0.00 mm
- net unconnected-(U1-IO14-Pad13): track 7.28 -> 0.00 mm
- net unconnected-(U1-IO33-Pad9): track 7.28 -> 0.00 mm
- net unconnected-(U1-TXD0/IO1-Pad35): track 7.28 -> 0.00 mm
- net unconnected-(U1-IO5-Pad29): track 7.28 -> 0.00 mm
- net unconnected-(U1-IO23-Pad37): track 7.28 -> 0.00 mm
- net unconnected-(U1-IO21-Pad33): track 7.28 -> 0.00 mm
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Other:
- board text removed: "PROG"

Commit message: .
Parts:
- moved SW1 56.6 mm to (218.7, 106.2), turned to 180 degrees
- moved D1 37.8 mm to (197.6, 106.8)
- moved R2 13.4 mm to (177.8, 99.8)
- moved R1 8.17 mm to (180.3, 88.4)
Connections:
- U3 pad 19: unconnected-(U3-GPIO1-Pad19) -> /GPIO1
- U3 pad 25: unconnected-(U3-GPIO0-Pad25) -> /GPIO0
- U3 pad 3: unconnected-(U3-EN-Pad3) -> /EN
Routing:
- net /GPIO1: track 0.00 -> 24.2 mm
- net /GPIO0: track 0.00 -> 20.3 mm, vias 0 -> 1
- net /EN: track 0.00 -> 7.17 mm

Commit message: .
Parts:
- R1, R2: moved to B.Cu
- moved R2 25.1 mm to (200.4, 88.9), turned to 45 degrees
- moved R1 21.5 mm to (200.4, 96.0), turned to -135 degrees
Connections:
- R2 pad 1: +3V3 -> /EN
- R2 pad 2: unconnected-(R2-Pad2) -> +3V3
Routing:
- net +3V3: track 5.06 -> 22.3 mm
- net Net-(D1-AB): track 0.00 -> 13.7 mm, vias 0 -> 1
- net /EN: track 7.17 -> 18.0 mm

Commit message: .
Parts:
- moved R2 4.36 mm to (202.7, 85.2), turned to 135 degrees
Connections:
- U2 pad 15: unconnected-(U2-IO3-Pad15) -> /GPIO3
- U2 pad 16: unconnected-(U2-IO2-Pad16) -> /GPIO2
- U2 pad 3: unconnected-(U2-IO4-Pad3) -> /GPIO4
- U2 pad 4: unconnected-(U2-IO5-Pad4) -> /GPIO5
- U2 pad 5: unconnected-(U2-IO6-Pad5) -> /GPIO6
- U3 pad 20: unconnected-(U3-GPIO6-Pad20) -> /GPIO6
- U3 pad 24: unconnected-(U3-GPIO2-Pad24) -> /GPIO2
- U3 pad 26: unconnected-(U3-GPIO5-Pad26) -> /GPIO5
- U3 pad 32: unconnected-(U3-GPIO4-Pad32) -> /GPIO4
- U3 pad 5: unconnected-(U3-GPIO3-Pad5) -> /GPIO3
Routing:
- net /GPIO4: track 0.00 -> 29.3 mm, vias 0 -> 1
- net /GPIO3: track 0.00 -> 24.9 mm, vias 0 -> 1
- net /GPIO5: track 0.00 -> 24.8 mm, vias 0 -> 1
- net /GPIO2: track 0.00 -> 24.0 mm
- net /GPIO6: track 0.00 -> 18.4 mm, vias 0 -> 1
- net +3V3: track 22.3 -> 12.6 mm
- net /GPIO0: track 20.3 -> 28.6 mm
- net /EN: track 18.0 -> 19.6 mm

Commit message: .
Parts:
- removed SW1: SW_Push, Alexander Footprint Library:SW_SPST_6x3
- added SW2: SW_Push_SMD_6x3.5, Alexander Footprint Library:SW_PUSH_6x3.5mm, F.Cu at (220.7, 106.2)
Routing:
- net /GPIO0: track 28.6 -> 30.9 mm
Changed lines of the file:
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@@
 		)
 	)
-	(footprint "Alexander Footprint Library:SW_SPST_6x3"
-		(layer "F.Cu")
-		(at 218.71 106.2 180)
-		(tags "SPST button tactile switch")
-		(property "Reference" "SW1"
-			(at 0 -4 0)
+	(footprint "Alexander Footprint Library:SW_PUSH_6x3.5mm"
+		(layer "F.Cu")
+		(at 220.65 106.2 180)
+		(descr "tactile push button, 6x3.5mm, https://www.apem.com/idec-apem/en_US/PCB-switches/Tactile-Switches/MJTP-6mm-through-hole/c/MJTP_6mm_through%20hole?page=1")
+		(tags "PHAP3362 6mm tact sw THT")
+		(property "Reference" "SW2"
+			(at 3.42 -2.7 0)
 			(layer "F.SilkS")
 			(effects
@@
 			)
 		)
-		(property "Value" "SW_Push"
-			(at 0 3 0)
+		(property "Value" "SW_Push_SMD_6x3.5"
+			(at 4.4 3.7 0)
 			(layer "F.Fab")
 			(effects
@@
 			)
 		)
-		(property "Footprint" "Alexander Footprint Library:SW_SPST_6x3"
+		(property "Footprint" "Alexander Footprint Library:SW_PUSH_6x3.5mm"
 			(at 0 0 180)
 			(unlocked yes)
@@
 			)
 		)
-		(property "Description" "Push button switch, generic, two pins"
+		(property "Description" ""
 			(at 0 0 180)
 			(unlocked yes)
@@
 		(sheetname "Root")
 		(sheetfile "ESP32-C3-WROOM-Socket-Legacy-v2.kicad_sch")
-		(attr smd)
-		(fp_line
-			(start 3.06 1.81)
-			(end -3.06 1.81)
+		(attr through_hole)
+		(fp_line
+			(start 6.35 1.39)
+			(end 6.35 1.85)
 			(stroke
 				(width 0.12)
@@
 		)
 		(fp_line
-			(start 3.06 -1.81)
-			(end 3.06 1.81)
+			(start 6.35 -1.85)
+			(end 6.35 -1.39)
 			(stroke
 				(width 0.12)
@@
 		)
 		(fp_line
-			(start -3.06 1.81)
-			(end -3.06 -1.81)
+			(start 6.35 -1.85)
+			(end 0.15 -1.85)
 			(stroke
 				(width 0.12)
@@
 		)
 		(fp_line
-			(start -3.06 -1.81)
-			(end 3.06 -1.81)
+			(start 0.15 1.85)
+			(end 6.35 1.85)
 			(stroke
 				(width 0.12)
@@
 		)
 		(fp_line
-			(start 5.95 -2)
-			(end 5.95 2)
-			(stroke
-				(width 0.05)
-				(type solid)
-			)
-			(layer "F.CrtYd")
-		)
-		(fp_line
-			(start -5.95 2)
-			(end 5.95 2)
-			(stroke
-				(width 0.05)
-				(type solid)
-			)
-			(layer "F.CrtYd")
-		)
-		(fp_line
-			(start -5.95 -2)
-			(end 5.95 -2)
-			(stroke
-				(width 0.05)
-				(type solid)
-			)
-			(layer "F.CrtYd")
-		)
-		(fp_line
-			(start -5.95 -2)
-			(end -5.95 2)
-			(stroke
-				(width 0.05)
-				(type solid)
-			)
-			(layer "F.CrtYd")
-		)
-		(fp_line
-			(start 3 -1.75)
-			(end 3 1.75)
-			(stroke
-				(width 0.1)
-				(type solid)
-			)
-			(layer "F.Fab")
-		)
-		(fp_line
-			(start 1.75 1)
-			(end -1.75 1)
-			(stroke
-				(width 0.1)
-				(type solid)
-			)
-			(layer "F.Fab")
-		)
-		(fp_line
-			(start 1.75 -1)
-			(end 1.75 1)
-			(stroke
-				(width 0.1)
-				(type solid)
-			)
-			(layer "F.Fab")
-		)
-		(fp_line
-			(start 1.5 -0.8)
-			(end 1.5 0.8)
-			(stroke
-				(width 0.1)
-				(type solid)
-			)
-			(layer "F.Fab")
-		)
-		(fp_line
-			(start -1.5 0.8)
-			(end 1.5 0.8)
-			(stroke
-				(width 0.1)
-				(type solid)
-			)
-			(layer "F.Fab")
-		)
-		(fp_line
-			(start -1.5 -0.8)
-			(end 1.5 -0.8)
-			(stroke
-				(width 0.1)
-				(type solid)
-			)
-			(layer "F.Fab")
-		)
-		(fp_line
-			(start -1.5 -0.8)
-			(end -1.5 0.8)
-			(stroke
-				(width 0.1)
-				(type solid)
-			)
-			(layer "F.Fab")
-		)
-		(fp_line
-			(start -1.75 1)
-			(end -1.75 -1)
-			(stroke
-				(width 0.1)
-				(type solid)
-			)
-			(layer "F.Fab")
-		)
-		(fp_line
-			(start -1.75 -1)
-			(end 1.75 -1)
-			(stroke
-				(width 0.1)
-				(type solid)
-			)
-			(layer "F.Fab")
-		)
-		(fp_line
-			(start -3 1.75)
-			(end 3 1.75)
-			(stroke
-				(width 0.1)
-				(type solid)
-			)
-			(layer "F.Fab")
-		)
-		(fp_line
-			(start -3 -1.75)
-			(end 3 -1.75)
-			(stroke
-				(width 0.1)
-				(type solid)
-			)
-			(layer "F.Fab")
-		)
-		(fp_line
-			(start -3 -1.75)
-			(end -3 1.75)
+			(start 0.15 1.39)
+			(end 0.15 1.85)
+			(stroke
+				(width 0.12)
+				(type solid)
+			)
+			(layer "F.SilkS")
+		)
+		(fp_line
+			(start 0.15 -1.39)
+			(end -0.85 -1.39)
+			(stroke
+				(width 0.12)
+				(type default)
+			)
+			(layer "F.SilkS")
+		)
+		(fp_line
+			(start 0.15 -1.85)
+			(end 0.15 -1.39)
+			(stroke
+				(width 0.12)
+				(type default)
+			)
+			(layer "F.SilkS")
+		)
+		(fp_rect
+			(start 1.75 -0.55)
+			(end 4.6 0.5)
+			(stroke
+				(width 0.12)
+				(type default)
+			)
+			(fill none)
+			(layer "F.SilkS")
+		)
+		(fp_line
+			(start 6.5 2)
+			(end 0 2)
+			(stroke
+				(width 0.05)
+				(type solid)
+			)
+			(layer "F.CrtYd")
+		)
+		(fp_line
+			(start 6.5 1.38)
+			(end 6.5 2)
+			(stroke
+				(width 0.05)
+				(type default)
+			)
+			(layer "F.CrtYd")
+		)
+		(fp_line
+			(start 6.5 -2)
+			(end 6.5 -1.38)
+			(stroke
+				(width 0.05)
+				(type default)
+			)
+			(layer "F.CrtYd")
+		)
+		(fp_line
+			(start 0 1.38)
+			(end 0 2)
+			(stroke
+				(width 0.05)
+				(type default)
+			)
+			(layer "F.CrtYd")
+		)
+		(fp_line
+			(start 0 -2)
+			(end 6.5 -2)
+			(stroke
+				(width 0.05)
+				(type solid)
+			)
+			(layer "F.CrtYd")
+		)
+		(fp_line
+			(start 0 -2)
+			(end 0 -1.38)
+			(stroke
+				(width 0.05)
+				(type default)
+			)
+			(layer "F.CrtYd")
+		)
+		(fp_line
+			(start -1.38 1.38)
+			(end 0 1.38)
+			(stroke
+				(width 0.05)
+				(type default)
+			)
+			(layer "F.CrtYd")
+		)
+		(fp_line
+			(start -1.38 1.38)
+			(end -1.38 -1.38)
+			(stroke
+				(width 0.05)
+				(type solid)
+			)
+			(layer "F.CrtYd")
+		)
+		(fp_line
+			(start -1.38 -1.38)
+			(end 0 -1.38)
+			(stroke
+				(width 0.05)
+				(type default)
+			)
+			(layer "F.CrtYd")
+		)
+		(fp_arc
+			(start 6.5 -1.38)
+			(mid 7.88 0)
+			(end 6.5 1.38)
+			(stroke
+				(width 0.05)
+				(type default)
+			)
+			(layer "F.CrtYd")
+		)
+		(fp_line
+			(start 6.25 1.75)
+			(end 0.25 1.75)
+			(stroke
+				(width 0.1)
+				(type solid)
+			)
+			(layer "F.Fab")
+		)
+		(fp_line
+			(start 6.25 -1.75)
+			(end 6.25 1.75)
+			(stroke
+				(width 0.1)
+				(type solid)
+			)
+			(layer "F.Fab")
+		)
+		(fp_line
+			(start 0.65 -1.75)
+			(end 6.25 -1.75)
+			(stroke
+				(width 0.1)
+				(type solid)
+			)
+			(layer "F.Fab")
+		)
+		(fp_line
+			(start 0.65 -1.75)
+			(end 0.25 -1.35)
+			(stroke
+				(width 0.1)
+				(type default)
+			)
+			(layer "F.Fab")
+		)
+		(fp_line
+			(start 0.25 1.75)
+			(end 0.25 -1.35)
 			(stroke
 				(width 0.1)
@@
 		)
 		(fp_text user "${REFERENCE}"
-			(at 0 -2.6 0)
+			(at 3 0 0)
 			(layer "F.Fab")
 			(effects
@@
 		)
 		(pad "1" smd rect
-			(at -4.59 0 180)
-			(size 2.18 1.6)
+			(at 0 0 270)
+			(size 2.25 2.25)
 			(layers "F.Cu" "F.Paste" "F.Mask")
 			(net 4 "/GPIO0")
@@
 			(pintype "passive")
 		)
-		(pad "2" smd rect
-			(at 4.59 0 180)
-			(size 2.18 1.6)
+		(pad "2" smd oval
+			(at 6.5 0 270)
+			(size 2.25 2.25)
 			(layers "F.Cu" "F.Paste" "F.Mask")
 			(net 1 "GND")
@@
 			(pintype "passive")
 		)
-		(model "${KICAD8_3DMODEL_DIR}/Button_Switch_SMD.3dshapes/SW_SPST_FSMSM.wrl"
+		(model "${KICAD8_3DMODEL_DIR}/Button_Switch_THT.3dshapes/SW_PUSH_1P1T_6x3.5mm_H4.3_APEM_MJTP1243.wrl"
 			(offset
 				(xyz 0 0 0)
@@
 	(segment
 		(start 223.3 101.76)
-		(end 220.61 99.07)
+		(end 223.3 105.7)
+		(width 0.25)
+		(layer "F.Cu")
+		(net 4)
+	)
+	(segment
+		(start 223.3 105.7)
+		(end 222.8 106.2)
+		(width 0.25)
+		(layer "F.Cu")
+		(net 4)
+	)
+	(segment
+		(start 222.8 106.2)
+		(end 220.65 106.2)
 		(width 0.25)
 		(layer "F.Cu")
@@
 	)
 	(segment
+		(start 220.61 99.07)
+		(end 223.3 101.76)
+		(width 0.25)
+		(layer "F.Cu")
+		(net 4)
+	)
+	(segment
 		(start 217.6 83.6)
 		(end 216.8125 83.6)
 		(width 0.25)
 		(layer "F.Cu")
-		(net 4)
-	)
-	(segment
-		(start 223.3 106.2)
-		(end 223.3 101.76)
-		(width 0.25)
-		(layer "F.Cu")
