File: Production/prod_esp32-c3-wroom-socket-minimal-USB-plug/esp32-c3-wroom-socket/esp32-c3-wroom-socket.kicad_sch (KiCad schematic)
At the start: 9 parts, among them J1 USB-C_Receptacle_Data_16P_GCT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, U1 ESP32-C3-WROOM-02-N4, U2 AMS1117-3V3

Commit message: .
Parts:
- added J3: USB-C_Plug_CX60-24S-UNIT, Alexander Footprint Library:USB-C_Plug_HIROSE_CX60-24S-UNIT, symbol Alexander_Library_Symbols:USB-C_Plug_CX60-24S-UNIT
Changed lines of the file:
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@@
+	)
+	(symbol
+		(lib_id "Alexander_Library_Symbols:USB-C_Plug_CX60-24S-UNIT")
+		(at 252.73 86.36 0)
+		(unit 1)
+		(exclude_from_sim no)
+		(in_bom yes)
+		(on_board yes)
+		(dnp no)
+		(fields_autoplaced yes)
+		(property "Reference" "J3"
+			(at 252.73 66.04 0)
+			(effects
+				(font
+					(size 1.27 1.27)
+				)
+			)
+		)
+		(property "Value" "USB-C_Plug_CX60-24S-UNIT"
+			(at 252.73 68.58 0)
+			(effects
+				(font
+					(size 1.27 1.27)
+				)
+			)
+		)
+		(property "Footprint" "Alexander Footprint Library:USB-C_Plug_HIROSE_CX60-24S-UNIT"
+			(at 252.73 86.36 0)
+			(effects
+				(font
+					(size 1.27 1.27)
+				)
+				(justify bottom)
+				(hide yes)
+			)
+		)
+		(property "Datasheet" ""
+			(at 252.73 86.36 0)
+			(effects
+				(font
+					(size 1.27 1.27)
+				)
+				(hide yes)
+			)
+		)
+		(property "Description" ""
+			(at 252.73 86.36 0)
+			(effects
+				(font
+					(size 1.27 1.27)
+				)
+				(hide yes)
+			)
+		)
+		(property "PARTREV" "5"
+			(at 252.73 86.36 0)
+			(effects
+				(font
+					(size 1.27 1.27)
+				)
+				(justify bottom)
+				(hide yes)
+			)
+		)
+		(property "STANDARD" "Manufacturer Recommendations"
+			(at 252.73 86.36 0)
+			(effects
+				(font
+					(size 1.27 1.27)
+				)
+				(justify bottom)
+				(hide yes)
+			)
+		)
+		(property "MAXIMUM_PACKAGE_HEIGHT" "2.6 mm"
+			(at 252.73 86.36 0)
+			(effects
+				(font
+					(size 1.27 1.27)
+				)
+				(justify bottom)
+				(hide yes)
+			)
+		)
+		(property "MANUFACTURER" "Hirose"
+			(at 252.73 86.36 0)
+			(effects
+				(font
+					(size 1.27 1.27)
+				)
+				(justify bottom)
+				(hide yes)
+			)
+		)
+		(pin "B12"
+		)
+		(pin "B2"
+		)
+		(pin "A3"
+		)
+		(pin "S2"
+		)
+		(pin "A9"
+		)
+		(pin "B10"
+		)
+		(pin "A10"
+		)
+		(pin "B5"
+		)
+		(pin "B9"
+		)
+		(pin "S3"
+		)
+		(pin "A2"
+		)
+		(pin "B3"
+		)
+		(pin "B4"
+		)
+		(pin "B8"
+		)
+		(pin "S4"
+		)
+		(pin "B1"
+		)
+		(pin "A11"
+		)
+		(pin "A6"
+		)
+		(pin "A1"
+		)
+		(pin "S1"
+		)
+		(pin "A5"
+		)
+		(pin "A7"
+		)
+		(pin "A12"
+		)
+		(pin "A4"
+		)
+		(pin "A8"
+		)
+		(pin "B11"
+		)
+		(instances
+			(project ""
+				(path "/1aed2ed1-0515-43a4-a546-c7b070175ea1"
+					(reference "J3")
+					(unit 1)
+				)
+			)
+		)
 	)
 	(symbol
