File: 555_toggle-switch_v2.0/555_toggle-switch_v2.kicad_pcb (KiCad board)
At the start: 2 copper layers, 29.8 x 39.8 mm, 17 parts, among them J1 3V3, J3 OUT, J4 USB-C_Receptacle_PowerOnly_6P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, SW1 SW_Push, SW2 SW_SPDT, SW3 SW_Reed, U1 NE555D, U2 AMS1117-3V3

Commit message: .
Parts:
- U2: moved to F.Cu
- moved J3 1.86 mm to (124.4, 89.7)
- turned U2 to 180 degrees
Routing:
- net Net-(J3-Pin_1): track 14.0 -> 15.4 mm
Other:
- outline, holes or cut-outs redrawn
- board text added: "BAT"
- board text added: "LED"
- board text removed: "OUT"
- board text removed: "PWR"

Commit message: .
Parts:
- added G***: LOGO, LOGO, B.Cu at (121.4, 114.4)
Other:
- outline, holes or cut-outs redrawn

Commit message: .
Parts:
- moved LED1 10.9 mm to (125.4, 117.2), turned to 0 degrees
- moved R9 1.31 mm to (131.5, 121.7), turned to -90 degrees
- moved R8 0.94 mm to (117.5, 121.7), turned to -90 degrees
- moved J4 0.67 mm to (124.6, 126.8)
- moved U2 0.60 mm to (116.0, 115.0)
Routing:
- net Net-(C2-Pad1): track 47.8 -> 45.7 mm

Commit message: .
Parts:
- moved R5 1.19 mm to (131.6, 116.0)
- moved LED1 1.16 mm to (125.2, 116.0), turned to -90 degrees
Connections:
- LED1 pad 3: unconnected-(LED1-GRN-Pad3) -> /3V3
Changed lines of the file:
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@@
 	(net 9 "Net-(J3-Pin_1)")
 	(net 10 "Net-(J4-CC2)")
-	(net 11 "unconnected-(LED1-GRN-Pad3)")
-	(net 12 "/3V3")
-	(net 13 "Net-(LED1-GND-Pad1)")
-	(net 14 "VCC")
+	(net 11 "/3V3")
+	(net 12 "Net-(LED1-GND-Pad1)")
+	(net 13 "VCC")
 	(footprint "Package_TO_SOT_SMD:SOT-223-3_TabPin2"
 		(layer "F.Cu")
@@
 			(layers "F.Cu" "F.Paste" "F.Mask")
 			(roundrect_rratio 0.25)
-			(net 12 "/3V3")
+			(net 11 "/3V3")
 			(pinfunction "VO")
 			(pintype "power_out")
@@
 			(layers "*.Cu" "*.Mask")
 			(remove_unused_layers no)
-			(net 14 "VCC")
+			(net 13 "VCC")
 			(pinfunction "R")
 			(pintype "input")
@@
 			(layers "*.Cu" "*.Mask")
 			(remove_unused_layers no)
-			(net 14 "VCC")
+			(net 13 "VCC")
 			(pinfunction "VCC")
 			(pintype "power_in")
@@
 	(footprint "Resistor_SMD:R_1206_3216Metric_Pad1.30x1.75mm_HandSolder"
 		(layer "F.Cu")
-		(at 132.750001 115.6502 -90)
+		(at 131.6 115.95 -90)
 		(descr "Resistor SMD 1206 (3216 Metric), square (rectangular) end terminal, IPC_7351 nominal with elongated pad for handsoldering. (Body size source: IPC-SM-782 page 72, https://www.pcb-3d.com/wordpress/wp-content/uploads/ipc-sm-782a_amendment_1_and_2.pdf), generated with kicad-footprint-generator")
 		(tags "resistor handsolder")
@@
 			(layers "F.Cu" "F.Paste" "F.Mask")
 			(roundrect_rratio 0.192308)
-			(net 13 "Net-(LED1-GND-Pad1)")
+			(net 12 "Net-(LED1-GND-Pad1)")
 			(pintype "passive")
 		)
@@
 	(footprint "Alexander Footprint Library:B1552_HVK-M"
 		(layer "F.Cu")
-		(at 125.3998 117.150001)
+		(at 125.249999 116.0002 -90)
 		(tags "B1552USUG20D000113U1930 ")
 		(property "Reference" "LED1"
-			(at 0 0 0)
+			(at 0 0 -90)
 			(unlocked yes)
 			(layer "F.SilkS")
@@
 		)
 		(property "Value" "LED-RED-GREEN-B1552USUG20D"
-			(at 0 0 0)
+			(at 0 0 -90)
 			(unlocked yes)
 			(layer "F.Fab")
@@
 		)
 		(property "Footprint" "Alexander Footprint Library:B1552_HVK-M"
-			(at 0 0 360)
+			(at 0 0 90)
 			(layer "F.Fab")
 			(hide yes)
@@
 		)
 		(property "Datasheet" "B1552USUG20D000113U1930"
-			(at 0 0 360)
+			(at 0 0 90)
 			(layer "F.Fab")
 			(hide yes)
@@
 		)
 		(property "Description" ""
-			(at 0 0 360)
+			(at 0 0 90)
 			(layer "F.Fab")
 			(hide yes)
@@
 		(attr smd)
 		(fp_line
-			(start -0.777373 -1.4732)
-			(end 0.777373 -1.4732)
+			(start -0.777373 1.4732)
+			(end 0.777373 1.4732)
 			(stroke
 				(width 0.1524)
@@
 		)
 		(fp_line
-			(start -0.777373 1.4732)
-			(end 0.777373 1.4732)
+			(start -0.777373 -1.4732)
+			(end 0.777373 -1.4732)
 			(stroke
 				(width 0.1524)
@@
 		)
 		(fp_line
-			(start -2.667 -1.7787)
-			(end -2.1082 -1.7787)
+			(start -2.1082 1.8542)
+			(end -2.1082 1.7787)
 			(stroke
 				(width 0.1524)
@@
 		)
 		(fp_line
-			(start -2.667 1.7787)
-			(end -2.667 -1.7787)
+			(start 2.1082 1.8542)
+			(end -2.1082 1.8542)
 			(stroke
 				(width 0.1524)
@@
 		)
 		(fp_line
-			(start -2.1082 -1.8542)
-			(end 2.1082 -1.8542)
+			(start -2.667 1.7787)
+			(end -2.667 -1.7787)
 			(stroke
 				(width 0.1524)
@@
 		)
 		(fp_line
-			(start -2.1082 -1.7787)
-			(end -2.1082 -1.8542)
+			(start 2.1082 1.7787)
+			(end 2.1082 1.8542)
 			(stroke
 				(width 0.1524)
@@
 		)
 		(fp_line
-			(start -2.1082 1.8542)
-			(end -2.1082 1.7787)
+			(start 2.667 1.7787)
+			(end 2.1082 1.7787)
 			(stroke
 				(width 0.1524)
@@
 		)
 		(fp_line
-			(start 2.1082 -1.8542)
-			(end 2.1082 -1.7787)
+			(start -2.667 -1.7787)
+			(end -2.1082 -1.7787)
 			(stroke
 				(width 0.1524)
@@
 		)
 		(fp_line
-			(start 2.1082 1.7787)
-			(end 2.1082 1.8542)
+			(start -2.1082 -1.7787)
+			(end -2.1082 -1.8542)
 			(stroke
 				(width 0.1524)
@@
 		)
 		(fp_line
-			(start 2.1082 1.8542)
-			(end -2.1082 1.8542)
+			(start 2.667 -1.7787)
+			(end 2.667 1.7787)
 			(stroke
 				(width 0.1524)
@@
 		)
 		(fp_line
-			(start 2.667 -1.7787)
-			(end 2.667 1.7787)
+			(start -2.1082 -1.8542)
+			(end 2.1082 -1.8542)
 			(stroke
 				(width 0.1524)
@@
 		)
 		(fp_line
-			(start 2.667 1.7787)
-			(end 2.1082 1.7787)
+			(start 2.1082 -1.8542)
+			(end 2.1082 -1.7787)
 			(stroke
 				(width 0.1524)
@@
 		)
 		(fp_line
-			(start -1.6002 -1.3462)
-			(end 1.6002 -1.3462)
+			(start -1.6002 1.3462)
+			(end 1.6002 1.3462)
 			(stroke
 				(width 0.0254)
@@
 		)
 		(fp_line
-			(start -1.6002 -1.0548)
-			(end -1.6002 -1.3462)
+			(start -1.6002 1.0548)
+			(end -1.6002 1.3462)
 			(stroke
 				(width 0.0254)
@@
 		)
 		(fp_line
-			(start -1.6002 -0.445201)
-			(end -1.6002 0.445201)
+			(start 1.6002 1.0548)
+			(end 1.6002 1.3462)
 			(stroke
 				(width 0.0254)
@@
 		)
 		(fp_line
-			(start -1.6002 1.0548)
-			(end -1.6002 1.3462)
+			(start -1.6002 -0.445201)
+			(end -1.6002 0.445201)
 			(stroke
 				(width 0.0254)
@@
 		)
 		(fp_line
-			(start -1.6002 1.3462)
-			(end 1.6002 1.3462)
+			(start 1.6002 -0.445201)
+			(end 1.6002 0.445201)
 			(stroke
 				(width 0.0254)
@@
 		)
 		(fp_line
-			(start -1.3462 -1.3462)
-			(end -1.6002 -1.0922)
+			(start -1.6002 -1.0548)
+			(end -1.6002 -1.3462)
 			(stroke
 				(width 0.0254)
@@
 		)
 		(fp_line
-			(start 1.6002 -0.445201)
-			(end 1.6002 0.445201)
+			(start -1.6002 -1.3462)
+			(end 1.6002 -1.3462)
 			(stroke
 				(width 0.0254)
@@
 		)
 		(fp_line
-			(start 1.6002 1.0548)
-			(end 1.6002 1.3462)
+			(start -1.3462 -1.3462)
+			(end -1.6002 -1.0922)
 			(stroke
 				(width 0.0254)
@@
 		)
 		(fp_arc
-			(start -1.6002 -1.054801)
-			(mid -1.2954 -0.750001)
-			(end -1.6002 -0.445201)
+			(start 1.6002 1.054801)
+			(mid 1.295399 0.75)
+			(end 1.6002 0.445201)
 			(stroke
 				(width 0.0254)
@@
 		)
 		(fp_arc
-			(start 1.6002 1.054801)
-			(mid 1.295399 0.75)
-			(end 1.6002 0.445201)
+			(start -1.6002 -1.054801)
+			(mid -1.2954 -0.750001)
+			(end -1.6002 -0.445201)
 			(stroke
 				(width 0.0254)
@@
 		)
 		(fp_text user "*"
-			(at -2.2352 -1.8041 0)
+			(at -2.2352 -1.8041 -90)
 			(unlocked yes)
 			(layer "F.SilkS")
@@
 		)
 		(fp_text user "*"
-			(at -2.2352 -1.8041 360)
+			(at -2.2352 -1.8041 90)
 			(layer "F.SilkS")
 			(effects
@@
 		)
 		(fp_text user "${REFERENCE}"
-			(at 0 0 0)
+			(at 0 0 -90)
 			(unlocked yes)
 			(layer "F.Fab")
@@
 		)
 		(fp_text user "*"
-			(at -0.9652 -1.1691 0)
+			(at -0.9652 -1.1691 -90)
 			(unlocked yes)
 			(layer "F.Fab")
@@
 		)
 		(fp_text user "*"
-			(at -0.9652 -1.1691 360)
+			(at -0.9652 -1.1691 90)
 			(layer "F.Fab")
 			(effects
@@
 		)
 		(pad "1" smd rect
-			(at -1.6002 -0.750001)
+			(at -1.6002 -0.750001 270)
 			(size 1.1176 1.0414)
 			(layers "F.Cu" "F.Paste" "F.Mask")
-			(net 13 "Net-(LED1-GND-Pad1)")
+			(net 12 "Net-(LED1-GND-Pad1)")
 			(pinfunction "GND")
 			(pintype "power_in")
 		)
 		(pad "2" smd rect
-			(at -1.6002 0.750001)
+			(at -1.6002 0.750001 270)
 			(size 1.1176 1.0414)
 			(layers "F.Cu" "F.Paste" "F.Mask")
-			(net 14 "VCC")
+			(net 13 "VCC")
 			(pinfunction "RED")
 			(pintype "power_out")
 		)
 		(pad "3" smd rect
-			(at 1.6002 0.750001)
+			(at 1.6002 0.750001 270)
 			(size 1.1176 1.0414)
 			(layers "F.Cu" "F.Paste" "F.Mask")
-			(net 11 "unconnected-(LED1-GRN-Pad3)")
+			(net 11 "/3V3")
 			(pinfunction "GRN")
 			(pintype "power_in")
 		)
 		(pad "4" smd rect
-			(at 1.6002 -0.750001)
+			(at 1.6002 -0.750001 270)
 			(size 1.1176 1.0414)
 			(layers "F.Cu" "F.Paste" "F.Mask")
-			(net 13 "Net-(LED1-GND-Pad1)")
+			(net 12 "Net-(LED1-GND-Pad1)")
 			(pinfunction "GND")
 			(pintype "power_out")
@@
 			(layers "*.Cu" "*.Mask")
 			(remove_unused_layers no)
-			(net 14 "VCC")
+			(net 13 "VCC")
 			(pinfunction "B")
 			(pintype "passive")
@@
 			(layers "*.Cu" "*.Mask")
 			(remove_unused_layers no)
-			(net 12 "/3V3")
+			(net 11 "/3V3")
 			(pinfunction "C")
 			(pintype "passive")
@@
 			(layers "*.Cu" "*.Mask")
 			(remove_unused_layers no)
-			(net 14 "VCC")
+			(net 13 "VCC")
 			(pintype "passive")
 		)
@@
 			(layers "*.Cu" "*.Mask")
 			(remove_unused_layers no)
-			(net 14 "VCC")
+			(net 13 "VCC")
 			(pintype "passive")
 		)
@@
 		(tags "tact sw push 6mm")
 		(property "Reference" "SW1"
-			(at 3.25 -2.43 0)
+			(at 3.25 2.3 0)
 			(layer "F.SilkS")
 			(effects
@@
 	)
 	(gr_text "ON / OFF"
-		(at 121.8 114.6 0)
+		(at 121.8 104.6 0)
 		(layer "F.SilkS" knockout)
 		(effects
@@
 		(width 0.5)
 		(layer "F.Cu")
-		(net 14)
+		(net 13)
 	)
 	(segment
@@
 		(width 0.5)
 		(layer "F.Cu")
-		(net 14)
+		(net 13)
 	)
 	(segment
@@
 		(width 0.5)
 		(layer "B.Cu")
-		(net 14)
+		(net 13)
 	)
 	(segment
@@
 		(width 0.5)
 		(layer "B.Cu")
-		(net 14)
+		(net 13)
 	)
 	(segment
@@
 		(width 0.5)
 		(layer "B.Cu")
-		(net 14)
+		(net 13)
 	)
 	(segment
@@
 		(width 0.5)
 		(layer "B.Cu")
-		(net 14)
+		(net 13)
 	)
 	(segment
@@
 		(width 0.5)
 		(layer "B.Cu")
-		(net 14)
+		(net 13)
 	)
 	(zone

Commit message: .
Parts:
- added R6: 5k1, Resistor_SMD:R_1206_3216Metric_Pad1.30x1.75mm_HandSolder, F.Cu at (134.4, 114.6)
- moved R5 3.20 mm to (134.4, 117.4), turned to 0 degrees
Connections:
- LED1 pad 4: Net-(LED1-GND-Pad1) -> Net-(LED1-GND-Pad4)
- R5 pad 1: GND -> Net-(LED1-GND-Pad4)
- R5 pad 2: Net-(LED1-GND-Pad1) -> GND

Commit message: .
Parts:
- moved LED1 0.75 mm to (125.2, 115.3), turned to 180 degrees
Routing:
- net /VUSB: track 0.00 -> 11.0 mm
- net Net-(J4-CC1): track 0.00 -> 8.61 mm
- net Net-(J4-CC2): track 0.00 -> 8.45 mm
Changed lines of the file:
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@@
 		(tags "resistor handsolder")
 		(property "Reference" "R5"
-			(at 0 -1.82 360)
+			(at 0 -1.82 0)
 			(layer "F.SilkS")
 			(effects
@@
 		)
 		(property "Value" "5k1"
-			(at 0 1.82 360)
+			(at 0 1.82 0)
 			(layer "F.Fab")
 			(effects
@@
 		)
 		(fp_text user "${REFERENCE}"
-			(at 0 0 360)
+			(at 0 0 0)
 			(layer "F.Fab")
 			(effects
@@
 	(footprint "Alexander Footprint Library:B1552_HVK-M"
 		(layer "F.Cu")
-		(at 125.249999 116.0002 -90)
+		(at 125.249999 115.250001 180)
 		(tags "B1552USUG20D000113U1930 ")
 		(property "Reference" "LED1"
-			(at 0 0 -90)
+			(at 0 0 180)
 			(unlocked yes)
 			(layer "F.SilkS")
@@
 		)
 		(property "Value" "LED-RED-GREEN-B1552USUG20D"
-			(at 0 0 -90)
+			(at 0 0 180)
 			(unlocked yes)
 			(layer "F.Fab")
@@
 		)
 		(property "Footprint" "Alexander Footprint Library:B1552_HVK-M"
-			(at 0 0 90)
+			(at 0 0 0)
 			(layer "F.Fab")
 			(hide yes)
@@
 		)
 		(property "Datasheet" "B1552USUG20D000113U1930"
-			(at 0 0 90)
+			(at 0 0 0)
 			(layer "F.Fab")
 			(hide yes)
@@
 		)
 		(property "Description" ""
-			(at 0 0 90)
+			(at 0 0 0)
 			(layer "F.Fab")
 			(hide yes)
@@
 		)
 		(fp_line
-			(start -2.1082 1.8542)
-			(end -2.1082 1.7787)
+			(start 2.667 1.7787)
+			(end 2.1082 1.7787)
 			(stroke
 				(width 0.1524)
@@
 		)
 		(fp_line
-			(start 2.1082 1.8542)
-			(end -2.1082 1.8542)
+			(start 2.667 -1.7787)
+			(end 2.667 1.7787)
 			(stroke
 				(width 0.1524)
@@
 		)
 		(fp_line
-			(start -2.667 1.7787)
-			(end -2.1082 1.7787)
+			(start 2.667 -1.7787)
+			(end 2.1082 -1.7787)
 			(stroke
 				(width 0.1524)
@@
 		)
 		(fp_line
-			(start -2.667 1.7787)
-			(end -2.667 -1.7787)
+			(start 2.1082 1.8542)
+			(end -2.1082 1.8542)
 			(stroke
 				(width 0.1524)
@@
 		)
 		(fp_line
-			(start 2.667 1.7787)
-			(end 2.1082 1.7787)
+			(start 2.1082 -1.8542)
+			(end 2.1082 -1.7787)
 			(stroke
 				(width 0.1524)
@@
 		)
 		(fp_line
-			(start -2.667 -1.7787)
-			(end -2.1082 -1.7787)
+			(start -2.1082 1.8542)
+			(end -2.1082 1.7787)
 			(stroke
 				(width 0.1524)
@@
 		)
 		(fp_line
-			(start 2.667 -1.7787)
-			(end 2.667 1.7787)
+			(start -2.1082 -1.8542)
+			(end 2.1082 -1.8542)
 			(stroke
 				(width 0.1524)
@@
 		)
 		(fp_line
-			(start 2.667 -1.7787)
-			(end 2.1082 -1.7787)
+			(start -2.667 1.7787)
+			(end -2.1082 1.7787)
 			(stroke
 				(width 0.1524)
@@
 		)
 		(fp_line
-			(start -2.1082 -1.8542)
-			(end 2.1082 -1.8542)
+			(start -2.667 1.7787)
+			(end -2.667 -1.7787)
 			(stroke
 				(width 0.1524)
@@
 		)
 		(fp_line
-			(start 2.1082 -1.8542)
-			(end 2.1082 -1.7787)
+			(start -2.667 -1.7787)
+			(end -2.1082 -1.7787)
 			(stroke
 				(width 0.1524)
@@
 		)
 		(fp_line
-			(start -1.6002 1.3462)
+			(start 1.6002 1.0548)
 			(end 1.6002 1.3462)
 			(stroke
@@
 		)
 		(fp_line
-			(start -1.6002 1.0548)
-			(end -1.6002 1.3462)
+			(start 1.6002 -0.445201)
+			(end 1.6002 0.445201)
 			(stroke
 				(width 0.0254)
@@
 		)
 		(fp_line
-			(start 1.6002 1.0548)
-			(end 1.6002 1.3462)
+			(start 1.6002 -1.0548)
+			(end 1.6002 -1.3462)
 			(stroke
 				(width 0.0254)
@@
 		)
 		(fp_line
-			(start -1.6002 -0.445201)
-			(end -1.6002 0.445201)
+			(start -1.3462 -1.3462)
+			(end -1.6002 -1.0922)
 			(stroke
 				(width 0.0254)
@@
 		)
 		(fp_line
-			(start 1.6002 -0.445201)
-			(end 1.6002 0.445201)
+			(start -1.6002 1.3462)
+			(end 1.6002 1.3462)
 			(stroke
 				(width 0.0254)
@@
 		)
 		(fp_line
-			(start -1.6002 -1.0548)
-			(end -1.6002 -1.3462)
+			(start -1.6002 1.0548)
+			(end -1.6002 1.3462)
 			(stroke
 				(width 0.0254)
@@
 		)
 		(fp_line
-			(start 1.6002 -1.0548)
-			(end 1.6002 -1.3462)
+			(start -1.6002 -0.445201)
+			(end -1.6002 0.445201)
 			(stroke
 				(width 0.0254)
@@
 		)
 		(fp_line
-			(start -1.6002 -1.3462)
-			(end 1.6002 -1.3462)
+			(start -1.6002 -1.0548)
+			(end -1.6002 -1.3462)
 			(stroke
 				(width 0.0254)
@@
 		)
 		(fp_line
-			(start -1.3462 -1.3462)
-			(end -1.6002 -1.0922)
+			(start -1.6002 -1.3462)
+			(end 1.6002 -1.3462)
 			(stroke
 				(width 0.0254)
@@
 		)
 		(fp_arc
-			(start -1.6002 0.445201)
-			(mid -1.2954 0.750001)
-			(end -1.6002 1.054801)
+			(start 1.6002 -0.445201)
+			(mid 1.295401 -0.75)
+			(end 1.6002 -1.054801)
 			(stroke
 				(width 0.0254)
@@
 		)
 		(fp_arc
-			(start 1.6002 -0.445201)
-			(mid 1.295401 -0.75)
-			(end 1.6002 -1.054801)
+			(start -1.6002 0.445201)
+			(mid -1.2954 0.750001)
+			(end -1.6002 1.054801)
 			(stroke
 				(width 0.0254)
@@
 		)
 		(fp_text user "*"
-			(at -2.2352 -1.8041 -90)
+			(at -2.2352 -1.8041 180)
 			(unlocked yes)
 			(layer "F.SilkS")
@@
 		)
 		(fp_text user "*"
-			(at -2.2352 -1.8041 90)
+			(at -2.2352 -1.8041 0)
 			(layer "F.SilkS")
 			(effects
@@
 		)
 		(fp_text user "${REFERENCE}"
-			(at 0 0 -90)
+			(at 0 0 180)
 			(unlocked yes)
 			(layer "F.Fab")
@@
 		)
 		(fp_text user "*"
-			(at -0.9652 -1.1691 -90)
+			(at -0.9652 -1.1691 180)
 			(unlocked yes)
 			(layer "F.Fab")
@@
 		)
 		(fp_text user "*"
-			(at -0.9652 -1.1691 90)
+			(at -0.9652 -1.1691 0)
 			(layer "F.Fab")
 			(effects
@@
 		)
 		(pad "1" smd rect
-			(at -1.6002 -0.750001 270)
+			(at -1.6002 -0.750001 180)
 			(size 1.1176 1.0414)
 			(layers "F.Cu" "F.Paste" "F.Mask")
@@
 		)
 		(pad "2" smd rect
-			(at -1.6002 0.750001 270)
+			(at -1.6002 0.750001 180)
 			(size 1.1176 1.0414)
 			(layers "F.Cu" "F.Paste" "F.Mask")
@@
 		)
 		(pad "3" smd rect
-			(at 1.6002 0.750001 270)
+			(at 1.6002 0.750001 180)
 			(size 1.1176 1.0414)
 			(layers "F.Cu" "F.Paste" "F.Mask")
@@
 		)
 		(pad "4" smd rect
-			(at 1.6002 -0.750001 270)
+			(at 1.6002 -0.750001 180)
 			(size 1.1176 1.0414)
 			(layers "F.Cu" "F.Paste" "F.Mask")
@@
 	)
 	(segment
+		(start 124.105 121.695)
+		(end 124.105 120.32)
+		(width 0.2)
+		(layer "F.Cu")
+		(net 7)
+	)
+	(segment
+		(start 123.6 122.2)
+		(end 124.105 121.695)
+		(width 0.2)
+		(layer "F.Cu")
+		(net 7)
+	)
+	(segment
+		(start 117.525 123.27)
+		(end 117.83 123.27)
+		(width 0.2)
+		(layer "F.Cu")
+		(net 7)
+	)
+	(segment
+		(start 118.9 122.2)
+		(end 123.6 122.2)
+		(width 0.2)
+		(layer "F.Cu")
+		(net 7)
+	)
+	(segment
+		(start 117.83 123.27)
+		(end 118.9 122.2)
+		(width 0.2)
+		(layer "F.Cu")
+		(net 7)
+	)
+	(segment
+		(start 126.125 120.32)
+		(end 126.125 118.925)
+		(width 0.5)
+		(layer "F.Cu")
+		(net 8)
+	)
+	(segment
+		(start 120.7 117.3)
+		(end 121.9 118.5)
+		(width 0.5)
+		(layer "F.Cu")
+		(net 8)
+	)
+	(segment
+		(start 123.1 119.3)
+		(end 123.085 119.315)
+		(width 0.5)
+		(layer "F.Cu")
+		(net 8)
+	)
+	(segment
+		(start 126.125 118.925)
+		(end 125.7 118.5)
+		(width 0.5)
+		(layer "F.Cu")
+		(net 8)
+	)
+	(segment
+		(start 123.085 119.315)
+		(end 123.085 120.32)
+		(width 0.5)
+		(layer "F.Cu")
+		(net 8)
+	)
+	(segment
+		(start 123.1 118.9)
+		(end 123.1 119.3)
+		(width 0.5)
+		(layer "F.Cu")
+		(net 8)
+	)
+	(segment
+		(start 125.7 118.5)
+		(end 123.5 118.5)
+		(width 0.5)
+		(layer "F.Cu")
+		(net 8)
+	)
+	(segment
+		(start 121.9 118.5)
+		(end 123.5 118.5)
+		(width 0.5)
+		(layer "F.Cu")
+		(net 8)
+	)
+	(segment
+		(start 123.5 118.5)
+		(end 123.1 118.9)
+		(width 0.5)
+		(layer "F.Cu")
+		(net 8)
+	)
+	(segment
+		(start 119.15 117.3)
+		(end 120.7 117.3)
+		(width 0.5)
+		(layer "F.Cu")
+		(net 8)
+	)
+	(segment
 		(start 119.6 98.1)
 		(end 119.6 90.6)
@@
 	)
 	(segment
+		(start 125.105 121.705)
+		(end 125.6 122.2)
+		(width 0.2)
+		(layer "F.Cu")
+		(net 10)
+	)
+	(segment
+		(start 131.27 123.27)
+		(end 131.525 123.27)
+		(width 0.2)
+		(layer "F.Cu")
+		(net 10)
+	)
+	(segment
+		(start 125.6 122.2)
+		(end 130.2 122.2)
+		(width 0.2)
+		(layer "F.Cu")
+		(net 10)
+	)
+	(segment
+		(start 125.105 120.32)
+		(end 125.105 121.705)
+		(width 0.2)
+		(layer "F.Cu")
+		(net 10)
+	)
+	(segment
+		(start 130.2 122.2)
+		(end 131.27 123.27)
+		(width 0.2)
+		(layer "F.Cu")
+		(net 10)
+	)
+	(segment
