File: 555_toggle-switch_v2.0/555_toggle-switch_v2.kicad_pcb (KiCad board)
At the start: 2 copper layers, 29.8 x 39.8 mm, 19 parts, among them J1 3V3, J3 OUT, J4 USB-C_Receptacle_PowerOnly_6P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, SW1 SW_Push, SW2 SW_SPDT, SW3 SW_Reed, U1 NE555D, U2 AMS1117-3V3

Commit message: .
Parts:
- moved LED1 0.35 mm to (125.2, 115.6), turned to -90 degrees
Routing:
- net VCC: track 23.9 -> 32.7 mm
- net /3V3: track 0.00 -> 8.37 mm
- net /VBAT: track 0.00 -> 4.19 mm
Changed lines of the file:
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@@
 	(footprint "Alexander Footprint Library:B1552_HVK-M"
 		(layer "F.Cu")
-		(at 125.249999 115.250001 180)
+		(at 125.249999 115.6002 -90)
 		(tags "B1552USUG20D000113U1930 ")
 		(property "Reference" "LED1"
-			(at 0 0 180)
+			(at 0 0 -90)
 			(unlocked yes)
 			(layer "F.SilkS")
@@
 		)
 		(property "Value" "LED-RED-GREEN-B1552USUG20D"
-			(at 0 0 180)
+			(at 0 0 -90)
 			(unlocked yes)
 			(layer "F.Fab")
@@
 		)
 		(property "Footprint" "Alexander Footprint Library:B1552_HVK-M"
-			(at 0 0 0)
+			(at 0 0 90)
 			(layer "F.Fab")
 			(hide yes)
@@
 		)
 		(property "Datasheet" "B1552USUG20D000113U1930"
-			(at 0 0 0)
+			(at 0 0 90)
 			(layer "F.Fab")
 			(hide yes)
@@
 		)
 		(property "Description" ""
-			(at 0 0 0)
+			(at 0 0 90)
 			(layer "F.Fab")
 			(hide yes)
@@
 		)
 		(fp_line
-			(start 2.667 1.7787)
-			(end 2.1082 1.7787)
+			(start -2.1082 1.8542)
+			(end -2.1082 1.7787)
 			(stroke
 				(width 0.1524)
@@
 		)
 		(fp_line
-			(start 2.667 -1.7787)
-			(end 2.667 1.7787)
+			(start 2.1082 1.8542)
+			(end -2.1082 1.8542)
 			(stroke
 				(width 0.1524)
@@
 		)
 		(fp_line
-			(start 2.667 -1.7787)
-			(end 2.1082 -1.7787)
+			(start -2.667 1.7787)
+			(end -2.1082 1.7787)
 			(stroke
 				(width 0.1524)
@@
 		)
 		(fp_line
-			(start 2.1082 1.8542)
-			(end -2.1082 1.8542)
+			(start -2.667 1.7787)
+			(end -2.667 -1.7787)
 			(stroke
 				(width 0.1524)
@@
 		)
 		(fp_line
-			(start 2.1082 -1.8542)
-			(end 2.1082 -1.7787)
+			(start 2.667 1.7787)
+			(end 2.1082 1.7787)
 			(stroke
 				(width 0.1524)
@@
 		)
 		(fp_line
-			(start -2.1082 1.8542)
-			(end -2.1082 1.7787)
+			(start -2.667 -1.7787)
+			(end -2.1082 -1.7787)
 			(stroke
 				(width 0.1524)
@@
 		)
 		(fp_line
-			(start -2.1082 -1.8542)
-			(end 2.1082 -1.8542)
+			(start 2.667 -1.7787)
+			(end 2.667 1.7787)
 			(stroke
 				(width 0.1524)
@@
 		)
 		(fp_line
-			(start -2.667 1.7787)
-			(end -2.1082 1.7787)
+			(start 2.667 -1.7787)
+			(end 2.1082 -1.7787)
 			(stroke
 				(width 0.1524)
@@
 		)
 		(fp_line
-			(start -2.667 1.7787)
-			(end -2.667 -1.7787)
+			(start -2.1082 -1.8542)
+			(end 2.1082 -1.8542)
 			(stroke
 				(width 0.1524)
@@
 		)
 		(fp_line
-			(start -2.667 -1.7787)
-			(end -2.1082 -1.7787)
+			(start 2.1082 -1.8542)
+			(end 2.1082 -1.7787)
 			(stroke
 				(width 0.1524)
@@
 		)
 		(fp_line
-			(start 1.6002 1.0548)
+			(start -1.6002 1.3462)
 			(end 1.6002 1.3462)
 			(stroke
@@
 		)
 		(fp_line
-			(start 1.6002 -0.445201)
-			(end 1.6002 0.445201)
+			(start -1.6002 1.0548)
+			(end -1.6002 1.3462)
 			(stroke
 				(width 0.0254)
@@
 		)
 		(fp_line
-			(start 1.6002 -1.0548)
-			(end 1.6002 -1.3462)
+			(start 1.6002 1.0548)
+			(end 1.6002 1.3462)
 			(stroke
 				(width 0.0254)
@@
 		)
 		(fp_line
-			(start -1.3462 -1.3462)
-			(end -1.6002 -1.0922)
+			(start -1.6002 -0.445201)
+			(end -1.6002 0.445201)
 			(stroke
 				(width 0.0254)
@@
 		)
 		(fp_line
-			(start -1.6002 1.3462)
-			(end 1.6002 1.3462)
+			(start 1.6002 -0.445201)
+			(end 1.6002 0.445201)
 			(stroke
 				(width 0.0254)
@@
 		)
 		(fp_line
-			(start -1.6002 1.0548)
-			(end -1.6002 1.3462)
+			(start -1.6002 -1.0548)
+			(end -1.6002 -1.3462)
 			(stroke
 				(width 0.0254)
@@
 		)
 		(fp_line
-			(start -1.6002 -0.445201)
-			(end -1.6002 0.445201)
+			(start 1.6002 -1.0548)
+			(end 1.6002 -1.3462)
 			(stroke
 				(width 0.0254)
@@
 		)
 		(fp_line
-			(start -1.6002 -1.0548)
-			(end -1.6002 -1.3462)
+			(start -1.6002 -1.3462)
+			(end 1.6002 -1.3462)
 			(stroke
 				(width 0.0254)
@@
 		)
 		(fp_line
-			(start -1.6002 -1.3462)
-			(end 1.6002 -1.3462)
+			(start -1.3462 -1.3462)
+			(end -1.6002 -1.0922)
 			(stroke
 				(width 0.0254)
@@
 		)
 		(fp_arc
-			(start 1.6002 -0.445201)
-			(mid 1.295401 -0.75)
-			(end 1.6002 -1.054801)
+			(start -1.6002 0.445201)
+			(mid -1.2954 0.750001)
+			(end -1.6002 1.054801)
 			(stroke
 				(width 0.0254)
@@
 		)
 		(fp_arc
-			(start -1.6002 0.445201)
-			(mid -1.2954 0.750001)
-			(end -1.6002 1.054801)
+			(start 1.6002 -0.445201)
+			(mid 1.295401 -0.75)
+			(end 1.6002 -1.054801)
 			(stroke
 				(width 0.0254)
@@
 		)
 		(fp_text user "*"
-			(at -2.2352 -1.8041 180)
+			(at -2.2352 -1.8041 -90)
 			(unlocked yes)
 			(layer "F.SilkS")
@@
 		)
 		(fp_text user "*"
-			(at -2.2352 -1.8041 0)
+			(at -2.2352 -1.8041 90)
 			(layer "F.SilkS")
 			(effects
@@
 		)
 		(fp_text user "${REFERENCE}"
-			(at 0 0 180)
+			(at 0 0 -90)
 			(unlocked yes)
 			(layer "F.Fab")
@@
 		)
 		(fp_text user "*"
-			(at -0.9652 -1.1691 180)
+			(at -0.9652 -1.1691 -90)
 			(unlocked yes)
 			(layer "F.Fab")
@@
 		)
 		(fp_text user "*"
-			(at -0.9652 -1.1691 0)
+			(at -0.9652 -1.1691 90)
 			(layer "F.Fab")
 			(effects
@@
 		)
 		(pad "1" smd rect
-			(at -1.6002 -0.750001 180)
+			(at -1.6002 -0.750001 270)
 			(size 1.1176 1.0414)
 			(layers "F.Cu" "F.Paste" "F.Mask")
@@
 		)
 		(pad "2" smd rect
-			(at -1.6002 0.750001 180)
+			(at -1.6002 0.750001 270)
 			(size 1.1176 1.0414)
 			(layers "F.Cu" "F.Paste" "F.Mask")
@@
 		)
 		(pad "3" smd rect
-			(at 1.6002 0.750001 180)
+			(at 1.6002 0.750001 270)
 			(size 1.1176 1.0414)
 			(layers "F.Cu" "F.Paste" "F.Mask")
@@
 		)
 		(pad "4" smd rect
-			(at 1.6002 -0.750001 180)
+			(at 1.6002 -0.750001 270)
 			(size 1.1176 1.0414)
 			(layers "F.Cu" "F.Paste" "F.Mask")
@@
 	)
 	(segment
+		(start 113.4 100.075)
+		(end 113.4 104.26)
+		(width 0.5)
+		(layer "B.Cu")
+		(net 4)
+	)
+	(segment
 		(start 129.54 96.52)
 		(end 134.62 96.52)
@@
 	)
 	(segment
+		(start 113.4 109.34)
+		(end 115.34 109.34)
+		(width 0.5)
+		(layer "F.Cu")
+		(net 12)
+	)
+	(segment
+		(start 116 110)
+		(end 116 112.1)
+		(width 0.5)
+		(layer "F.Cu")
+		(net 12)
+	)
+	(segment
+		(start 116.6 112.7)
+		(end 119.15 112.7)
+		(width 0.5)
+		(layer "F.Cu")
+		(net 12)
+	)
+	(segment
+		(start 115.34 109.34)
+		(end 116 110)
+		(width 0.5)
+		(layer "F.Cu")
+		(net 12)
+	)
+	(segment
+		(start 116 112.1)
+		(end 116.6 112.7)
+		(width 0.5)
+		(layer "F.Cu")
+		(net 12)
+	)
+	(segment
 		(start 129.54 93.98)
 		(end 134.62 93.98)
@@
 	)
 	(segment
-		(start 118 101.6)
-		(end 121.92 101.6)
+		(start 115.4 106.8)
+		(end 116.1 106.1)
 		(width 0.5)
-		(layer "F.Cu")
+		(layer "B.Cu")
+		(net 14)
+	)
+	(segment
+		(start 113.4 106.8)
+		(end 115.4 106.8)
+		(width 0.5)
+		(layer "B.Cu")
 		(net 14)
 	)
@@
 	)
 	(segment
+		(start 117 101.6)
+		(end 118 101.6)
+		(width 0.5)
+		(layer "B.Cu")
+		(net 14)
+	)
+	(segment
 		(start 125.75 101.25)
 		(end 125.75 94.25)
@@
 	)
 	(segment
+		(start 116.1 102.5)
+		(end 117 101.6)
+		(width 0.5)
+		(layer "B.Cu")
+		(net 14)
+	)
+	(segment
 		(start 121.92 101.6)
 		(end 125.4 101.6)
@@
 	)
 	(segment
+		(start 121.85 101.6)
+		(end 118 101.6)
+		(width 0.5)
+		(layer "B.Cu")
+		(net 14)
+	)
+	(segment
 		(start 126.02 93.98)
 		(end 129.54 93.98)
 		(width 0.5)
 		(layer "B.Cu")
+		(net 14)
+	)
+	(segment
+		(start 116.1 106.1)
+		(end 116.1 102.5)
+		(width 0.5)
+		(layer "B.Cu")

Commit message: .
Routing:
- net VCC: track 32.7 -> 17.8 mm
- net Net-(U1-DIS): track 10.6 -> 15.8 mm
Changed lines of the file:
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@@
 		(end 118 104.14)
 		(width 0.5)
-		(layer "F.Cu")
+		(layer "B.Cu")
+		(net 3)
+	)
+	(segment
+		(start 125.1 106.7)
+		(end 122.4 106.7)
+		(width 0.5)
+		(layer "B.Cu")
+		(net 3)
+	)
+	(segment
+		(start 125.8 97.1)
+		(end 125.8 99.7)
+		(width 0.5)
+		(layer "B.Cu")
+		(net 3)
+	)
+	(segment
+		(start 125.8 106)
+		(end 125.1 106.7)
+		(width 0.5)
+		(layer "B.Cu")
+		(net 3)
+	)
+	(segment
+		(start 131.16 99.06)
+		(end 131.78 99.68)
+		(width 0.5)
+		(layer "B.Cu")
+		(net 3)
+	)
+	(segment
+		(start 129.47 99.06)
+		(end 131.16 99.06)
+		(width 0.5)
+		(layer "B.Cu")
+		(net 3)
+	)
+	(segment
+		(start 125.22 96.52)
+		(end 125.8 97.1)
+		(width 0.5)
+		(layer "B.Cu")
+		(net 3)
+	)
+	(segment
+		(start 134.235 106.7)
+		(end 128.9 106.7)
+		(width 0.5)
+		(layer "B.Cu")
+		(net 3)
+	)
+	(segment
+		(start 122.4 106.7)
+		(end 118.8 106.7)
+		(width 0.5)
+		(layer "B.Cu")
 		(net 3)
 	)
 	(segment
 		(start 128.9 106.7)
-		(end 134.235 106.7)
-		(width 0.5)
-		(layer "F.Cu")
-		(net 3)
-	)
-	(segment
-		(start 125.8 99.8)
-		(end 125.8 106.08)
-		(width 0.5)
-		(layer "F.Cu")
-		(net 3)
-	)
-	(segment
-		(start 125.8 97)
-		(end 125.8 99.8)
-		(width 0.5)
-		(layer "F.Cu")
-		(net 3)
-	)
-	(segment
-		(start 129.54 99.06)
-		(end 126.54 99.06)
-		(width 0.5)
-		(layer "F.Cu")
-		(net 3)
-	)
-	(segment
-		(start 125.8 106.08)
-		(end 125.2 106.68)
-		(width 0.5)
-		(layer "F.Cu")
-		(net 3)
-	)
-	(segment
-		(start 118.78 106.68)
+		(end 125.1 106.7)
+		(width 0.5)
+		(layer "B.Cu")
+		(net 3)
+	)
+	(segment
+		(start 126.44 99.06)
+		(end 125.8 99.7)
+		(width 0.5)
+		(layer "B.Cu")
+		(net 3)
+	)
+	(segment
+		(start 125.8 99.7)
+		(end 125.8 106)
+		(width 0.5)
+		(layer "B.Cu")
+		(net 3)
+	)
+	(segment
+		(start 121.85 96.52)
+		(end 125.22 96.52)
+		(width 0.5)
+		(layer "B.Cu")
+		(net 3)
+	)
+	(segment
+		(start 118.8 106.7)
 		(end 118 105.9)
 		(width 0.5)
-		(layer "F.Cu")
-		(net 3)
-	)
-	(segment
-		(start 131.88 99.68)
+		(layer "B.Cu")
+		(net 3)
+	)
+	(segment
+		(start 131.78 99.68)
 		(end 133.7 99.68)
 		(width 0.5)
-		(layer "F.Cu")
-		(net 3)
-	)
-	(segment
-		(start 129.54 99.06)
-		(end 131.26 99.06)
-		(width 0.5)
-		(layer "F.Cu")
-		(net 3)
-	)
-	(segment
-		(start 127.29 106.68)
-		(end 127.31 106.7)
-		(width 0.5)
-		(layer "F.Cu")
-		(net 3)
-	)
-	(segment
-		(start 127.31 106.7)
-		(end 128.9 106.7)
-		(width 0.5)
-		(layer "F.Cu")
-		(net 3)
-	)
-	(segment
-		(start 125.32 96.52)
-		(end 125.8 97)
-		(width 0.5)
-		(layer "F.Cu")
-		(net 3)
-	)
-	(segment
-		(start 125.2 106.68)
-		(end 118.78 106.68)
-		(width 0.5)
-		(layer "F.Cu")
-		(net 3)
-	)
-	(segment
-		(start 121.92 96.52)
-		(end 125.32 96.52)
-		(width 0.5)
-		(layer "F.Cu")
-		(net 3)
-	)
-	(segment
-		(start 125.2 106.68)
-		(end 127.29 106.68)
-		(width 0.5)
-		(layer "F.Cu")
-		(net 3)
-	)
-	(segment
-		(start 131.26 99.06)
-		(end 131.88 99.68)
-		(width 0.5)
-		(layer "F.Cu")
-		(net 3)
-	)
-	(segment
-		(start 126.54 99.06)
-		(end 125.8 99.8)
-		(width 0.5)
-		(layer "F.Cu")
+		(layer "B.Cu")
+		(net 3)
+	)
+	(segment
+		(start 129.47 99.06)
+		(end 126.44 99.06)
+		(width 0.5)
+		(layer "B.Cu")
 		(net 3)
 	)
@@
 	)
 	(segment
+		(start 129.47 96.52)
+		(end 134.62 96.52)
+		(width 0.5)
+		(layer "B.Cu")
+		(net 5)
+	)
+	(segment
 		(start 124.105 121.695)
 		(end 124.105 120.32)
@@
 	)
 	(segment
-		(start 125.75 94.25)
-		(end 126.02 93.98)
-		(width 0.5)
-		(layer "B.Cu")
-		(net 14)
-	)
-	(segment
-		(start 125.4 101.6)
-		(end 125.75 101.25)
-		(width 0.5)
-		(layer "B.Cu")
-		(net 14)
-	)
-	(segment
 		(start 117 101.6)
 		(end 118 101.6)
@@
 	)
 	(segment
-		(start 125.75 101.25)
-		(end 125.75 94.25)
-		(width 0.5)
-		(layer "B.Cu")
-		(net 14)
-	)
-	(segment
 		(start 116.1 102.5)
 		(end 117 101.6)
@@
 	)
 	(segment
-		(start 121.92 101.6)
-		(end 125.4 101.6)
-		(width 0.5)
-		(layer "B.Cu")
-		(net 14)
-	)
-	(segment
 		(start 121.85 101.6)
 		(end 118 101.6)
 		(width 0.5)
 		(layer "B.Cu")
-		(net 14)
-	)
-	(segment
-		(start 126.02 93.98)
-		(end 129.54 93.98)
-		(width 0.5)
-		(layer "B.Cu")
