File: prod_esp32-c3-wroom-socket-USB/esp32-c3-wroom-socket.kicad_pcb (KiCad board)
At the start: 2 copper layers, 30.5 x 25.4 mm, 14 parts, among them J4 USB-C_Receptacle_Data_16P_GCT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, SW1 SW_Push_SMD_6x3.5, SW2 SW_Push_SMD_6x3.5, U1 ESP32-C3-WROOM-02-N4, U2 AMS1117-3V3

Commit message: .
Parts:
- R7: moved to B.Cu
- moved G*** 20.6 mm to (180.0, 83.0)
- moved U2 13.5 mm to (161.9, 77.0)
- moved R7 8.88 mm to (147.2, 70.1)
- moved R4 3.52 mm to (163.8, 59.3), turned to 180 degrees
Routing:
- net USB_D+: track 27.2 -> 7.63 mm
- net USB_D-: track 53.3 -> 35.1 mm
- net GPIO8: track 20.9 -> 10.0 mm
- net GPIO9: track 19.1 -> 10.9 mm
- net 3V3: track 46.2 -> 49.4 mm
- net VBUS: track 10.4 -> 12.8 mm, vias 1 -> 0
- net Net-(LED1-GND-Pad1): track 9.15 -> 7.47 mm
- net GND: track 0.00 -> 1.35 mm, vias 13 -> 11

Commit message: .
Parts:
- moved R5 6.95 mm to (143.4, 86.1)
- moved R6 2.63 mm to (163.4, 86.3)
Routing:
- net USB_D+: track 7.63 -> 29.4 mm, vias 0 -> 1
- net USB_D-: track 35.1 -> 29.0 mm
- net VBUS: track 12.8 -> 9.80 mm
Changed lines of the file:
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@@
 	(footprint "Resistor_SMD:R_1206_3216Metric_Pad1.30x1.75mm_HandSolder"
 		(layer "B.Cu")
-		(at 137.9 81.85 -90)
+		(at 143.4 86.1 -90)
 		(descr "Resistor SMD 1206 (3216 Metric), square (rectangular) end terminal, IPC_7351 nominal with elongated pad for handsoldering. (Body size source: IPC-SM-782 page 72, https://www.pcb-3d.com/wordpress/wp-content/uploads/ipc-sm-782a_amendment_1_and_2.pdf), generated with kicad-footprint-generator")
 		(tags "resistor handsolder")
@@
 	(footprint "Resistor_SMD:R_1206_3216Metric_Pad1.30x1.75mm_HandSolder"
 		(layer "B.Cu")
-		(at 166 85.95 -90)
+		(at 163.4 86.35 -90)
 		(descr "Resistor SMD 1206 (3216 Metric), square (rectangular) end terminal, IPC_7351 nominal with elongated pad for handsoldering. (Body size source: IPC-SM-782 page 72, https://www.pcb-3d.com/wordpress/wp-content/uploads/ipc-sm-782a_amendment_1_and_2.pdf), generated with kicad-footprint-generator")
 		(tags "resistor handsolder")
@@
 	)
 	(via
-		(at 157.8 68.6)
+		(at 157.3 67.6)
 		(size 0.6)
 		(drill 0.3)
@@
 	)
 	(via
-		(at 159.4 68.6)
+		(at 158.9 67.6)
 		(size 0.6)
 		(drill 0.3)
@@
 	)
 	(via
-		(at 158.6 68.6)
+		(at 158.1 67.6)
 		(size 0.6)
 		(drill 0.3)
@@
 	)
 	(via
-		(at 160.2 68.6)
+		(at 159.7 67.6)
 		(size 0.6)
 		(drill 0.3)
@@
 	)
 	(segment
-		(start 150.1 64.2)
-		(end 150.1 66.3)
-		(width 0.25)
-		(layer "B.Cu")
-		(net 7)
-	)
-	(segment
-		(start 150.1 66.3)
-		(end 149.450016 66.949984)
-		(width 0.25)
-		(layer "B.Cu")
-		(net 7)
-	)
-	(segment
 		(start 159.6 73.85)
 		(end 154.35 73.85)
@@
 	)
 	(segment
+		(start 157.4 71.575)
+		(end 163.8 65.175)
+		(width 0.25)
+		(layer "F.Cu")
+		(net 9)
+	)
+	(segment
+		(start 163.8 64.7)
+		(end 164.3 64.2)
+		(width 0.25)
+		(layer "F.Cu")
+		(net 9)
+	)
+	(segment
+		(start 164.3 64.2)
+		(end 165.69 64.2)
+		(width 0.25)
+		(layer "F.Cu")
+		(net 9)
+	)
+	(segment
 		(start 166.8 64.2)
 		(end 167.4 64.8)
@@
 	)
 	(segment
+		(start 163.8 65.175)
+		(end 163.8 64.7)
+		(width 0.25)
+		(layer "F.Cu")
+		(net 9)
+	)
+	(segment
 		(start 167.4 64.8)
 		(end 167.4 65.655686)
@@
 	)
 	(segment
+		(start 152.000016 76.708408)
+		(end 152.000016 76.785)
+		(width 0.25)
+		(layer "F.Cu")
+		(net 9)
+	)
+	(segment
 		(start 167.8 68.03)
 		(end 169.41 69.64)
@@
 	)
 	(segment
-		(start 167 69.71)
-		(end 167 70.901372)
-		(width 0.2)
-		(layer "F.Cu")
-		(net 10)
-	)
-	(segment
-		(start 167.6 71.501372)
-		(end 167.6 75.45)
-		(width 0.2)
-		(layer "F.Cu")
-		(net 10)
-	)
-	(segment
-		(start 165.99 68.7)
-		(end 167 69.71)
-		(width 0.2)
-		(layer "F.Cu")
-		(net 10)
-	)
-	(segment
-		(start 165.69 68.7)
-		(end 165.99 68.7)
-		(width 0.2)
-		(layer "F.Cu")
-		(net 10)
-	)
-	(segment
-		(start 167 70.901372)
-		(end 167.6 71.501372)
-		(width 0.2)
-		(layer "F.Cu")
-		(net 10)
-	)
-	(segment
-		(start 167.6 75.45)
-		(end 169.41 77.26)
-		(width 0.2)
-		(layer "F.Cu")
-		(net 10)
-	)
-	(segment
-		(start 162.6 67.2)
-		(end 164.1 65.7)
-		(width 0.25)
-		(layer "F.Cu")
-		(net 11)
-	)
-	(segment
-		(start 164.1 65.7)
-		(end 165.69 65.7)
-		(width 0.25)
-		(layer "F.Cu")
-		(net 11)
-	)
-	(segment
-		(start 166.5 65.7)
-		(end 167.4 66.6)
-		(width 0.2)
-		(layer "F.Cu")
-		(net 11)
-	)
-	(segment
-		(start 167.4 68.195686)
-		(end 167.8 68.595686)
-		(width 0.2)
-		(layer "F.Cu")
-		(net 11)
-	)
-	(segment
-		(start 167.8 70.57)
-		(end 169.41 72.18)
-		(width 0.2)
-		(layer "F.Cu")
-		(net 11)
-	)
-	(segment
-		(start 167.8 68.595686)
-		(end 167.8 70.57)
-		(width 0.2)
-		(layer "F.Cu")
-		(net 11)
-	)
-	(segment
-		(start 167.4 66.6)
-		(end 167.4 68.195686)
-		(width 0.2)
-		(layer "F.Cu")
-		(net 11)
-	)
-	(segment
-		(start 157.4 67.2)
-		(end 162.6 67.2)
-		(width 0.25)
-		(layer "F.Cu")
-		(net 11)
-	)
-	(segment
-		(start 165.69 65.7)
-		(end 166.5 65.7)
-		(width 0.2)
-		(layer "F.Cu")
-		(net 11)
+		(start 151.150015 75.858407)
+		(end 152.000016 76.708408)
+		(width 0.25)
+		(layer "F.Cu")
+		(net 9)
+	)
+	(segment
+		(start 151.150015 75.435)
+		(end 151.150015 75.858407)
+		(width 0.25)
+		(layer "F.Cu")
+		(net 9)
 	)
 	(via
-		(at 157.4 67.2)
+		(at 157.4 71.575)
 		(size 0.6)
 		(drill 0.3)
 		(layers "F.Cu" "B.Cu")
+		(net 9)
+	)
+	(segment
+		(start 157.275 71.575)
+		(end 156.3 72.55)
+		(width 0.25)
+		(layer "B.Cu")
+		(net 9)
+	)
+	(segment
+		(start 157.4 71.575)
+		(end 157.275 71.575)
+		(width 0.25)
+		(layer "B.Cu")
+		(net 9)
+	)
+	(segment
+		(start 156.3 72.55)
+		(end 153.013604 72.55)
+		(width 0.25)
+		(layer "B.Cu")
+		(net 9)
+	)
+	(segment
+		(start 153.013604 72.55)
+		(end 151.150015 74.413589)
+		(width 0.25)
+		(layer "B.Cu")
+		(net 9)
+	)
+	(segment
+		(start 151.150015 74.413589)
+		(end 151.150015 75.435)
+		(width 0.25)
+		(layer "B.Cu")
+		(net 9)
+	)
+	(segment
+		(start 167 69.71)
+		(end 167 70.901372)
+		(width 0.2)
+		(layer "F.Cu")
+		(net 10)
+	)
+	(segment
+		(start 167.6 71.501372)
+		(end 167.6 75.45)
+		(width 0.2)
+		(layer "F.Cu")
+		(net 10)
+	)
+	(segment
+		(start 165.99 68.7)
+		(end 167 69.71)
+		(width 0.2)
+		(layer "F.Cu")
+		(net 10)
+	)
+	(segment
+		(start 165.69 68.7)
+		(end 165.99 68.7)
+		(width 0.2)
+		(layer "F.Cu")
+		(net 10)
+	)
+	(segment
+		(start 167 70.901372)
+		(end 167.6 71.501372)
+		(width 0.2)
+		(layer "F.Cu")
+		(net 10)
+	)
+	(segment
+		(start 167.6 75.45)
+		(end 169.41 77.26)
+		(width 0.2)
+		(layer "F.Cu")
+		(net 10)
+	)
+	(segment
+		(start 163.911396 65.7)
+		(end 165.69 65.7)
+		(width 0.25)
+		(layer "F.Cu")
+		(net 11)
+	)
+	(segment
+		(start 166.5 65.7)
+		(end 167.4 66.6)
+		(width 0.2)
+		(layer "F.Cu")
+		(net 11)
+	)
+	(segment
+		(start 167.4 68.195686)
+		(end 167.8 68.595686)
+		(width 0.2)
+		(layer "F.Cu")
+		(net 11)
+	)
+	(segment
+		(start 167.8 70.57)
+		(end 169.41 72.18)
+		(width 0.2)
+		(layer "F.Cu")
+		(net 11)
+	)
+	(segment
+		(start 167.8 68.595686)
+		(end 167.8 70.57)
+		(width 0.2)
+		(layer "F.Cu")
+		(net 11)
+	)
+	(segment
+		(start 167.4 66.6)
+		(end 167.4 68.195686)
+		(width 0.2)
+		(layer "F.Cu")
+		(net 11)
+	)
+	(segment
+		(start 158.1 71.511396)
+		(end 163.911396 65.7)
+		(width 0.25)
+		(layer "F.Cu")
+		(net 11)
+	)
+	(segment
+		(start 158.1 72.2)
+		(end 158.1 71.511396)
+		(width 0.25)
+		(layer "F.Cu")
+		(net 11)
+	)
+	(segment
+		(start 165.69 65.7)
+		(end 166.5 65.7)
+		(width 0.2)
+		(layer "F.Cu")
+		(net 11)
+	)
+	(via
+		(at 158.1 72.2)
+		(size 0.6)
+		(drill 0.3)
+		(layers "F.Cu" "B.Cu")
+		(net 11)
+	)
+	(segment
+		(start 152.000016 74.199984)
+		(end 152.000016 75.435)
+		(width 0.25)
+		(layer "B.Cu")
 		(net 11)
 	)
@@
 	)
 	(segment
-		(start 149.9 68.2)
-		(end 149.9 72.868011)
-		(width 0.25)
-		(layer "B.Cu")
-		(net 11)
-	)
-	(segment
-		(start 157.4 67.2)
-		(end 150.9 67.2)
-		(width 0.25)
-		(layer "B.Cu")
-		(net 11)
-	)
-	(segment
-		(start 149.9 72.868011)
-		(end 152.000016 74.968027)
-		(width 0.25)
-		(layer "B.Cu")
-		(net 11)
-	)
-	(segment
-		(start 152.000016 74.968027)
-		(end 152.000016 75.435)
+		(start 158.1 72.2)
+		(end 157.3 73)
 		(width 0.25)
 		(layer "B.Cu")
@@
 	)
 	(segment
-		(start 150.9 67.2)
-		(end 149.9 68.2)
-		(width 0.25)
-		(layer "B.Cu")
+		(start 153.2 73)
+		(end 152.000016 74.199984)
+		(width 0.25)
+		(layer "B.Cu")
+		(net 11)
+	)
+	(segment
+		(start 157.3 73)
+		(end 153.2 73)
+		(width 0.25)
+		(layer "B.Cu")

Commit message: .
Parts:
- removed R5, R6: 5k1, Resistor_SMD:R_1206_3216Metric_Pad1.30x1.75mm_HandSolder
- added R10: 5k1, Resistor_SMD:R_1206_3216Metric_Pad1.30x1.75mm_HandSolder, F.Cu at (152.8, 89.9)
- added R9: 5k1, Resistor_SMD:R_1206_3216Metric_Pad1.30x1.75mm_HandSolder, F.Cu at (152.8, 86.6)
- moved R8 5.30 mm to (152.5, 65.0)
- moved R7 5.18 mm to (148.1, 65.0)
Routing:
- net GPIO9: track 10.9 -> 17.0 mm, vias 0 -> 1
- net GPIO8: track 10.0 -> 14.1 mm, vias 0 -> 1
- net 3V3: track 49.4 -> 50.8 mm

Commit message: .
Parts:
- R10, R9: moved to B.Cu
- moved R10 19.8 mm to (148.1, 70.7), turned to -90 degrees
- moved R9 7.18 mm to (151.3, 79.6)
- moved SW2 5.43 mm to (164.9, 80.0), turned to 90 degrees
- moved SW1 5.38 mm to (160.1, 80.0), turned to 90 degrees
- moved U2 1.00 mm to (162.9, 77.0)
Routing:
- net 3V3: track 50.8 -> 40.1 mm
- net EN: track 32.1 -> 24.5 mm
- net VBUS: track 9.80 -> 17.0 mm
- net Net-(J4-CC1): track 0.00 -> 5.12 mm
- net Net-(J4-CC2): track 0.00 -> 2.82 mm
- net GND: vias 11 -> 12

Commit message: .
Routing:
- net 3V3: track 40.1 -> 57.4 mm, vias 2 -> 1
- net GPIO9: track 17.0 -> 30.5 mm
- net EN: track 24.5 -> 36.0 mm

Commit message: .
Parts:
- moved G*** 26.9 mm to (158.3, 67.1)
Routing:
- net GND: track 1.35 -> 2.70 mm
Changed lines of the file:
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@@
 	(footprint "LOGO"
 		(layer "B.Cu")
-		(at 180 83 180)
+		(at 158.3 67.1 180)
 		(property "Reference" "G***"
 			(at 0 0 0)
@@
 	)
 	(via
-		(at 156.9 67.1)
+		(at 156.3 61.9)
 		(size 0.6)
 		(drill 0.3)
@@
 	)
 	(via
-		(at 160.6 64.6)
+		(at 160.7 61.7)
 		(size 0.6)
 		(drill 0.3)
@@
 	)
 	(via
-		(at 158.5 67.1)
+		(at 157.9 61.9)
 		(size 0.6)
 		(drill 0.3)
@@
 	)
 	(via
-		(at 157.7 67.1)
+		(at 157.1 61.9)
 		(size 0.6)
 		(drill 0.3)
@@
 	)
 	(via
-		(at 160.6 65.4)
+		(at 160.7 62.5)
 		(size 0.6)
 		(drill 0.3)
@@
 	)
 	(via
-		(at 159.3 67.1)
+		(at 158.7 61.9)
 		(size 0.6)
 		(drill 0.3)
@@
 	)
 	(via
-		(at 160.6 66.2)
+		(at 160.7 63.3)
 		(size 0.6)
 		(drill 0.3)
@@
 	)
 	(segment
-		(start 154.550016 76.785)
-		(end 154.550016 75.435)
-		(width 0.25)
+		(start 148.600015 75.435)
+		(end 148.600015 76.785)
+		(width 0.5)
+		(layer "B.Cu")
+		(net 2)
+	)
+	(segment
+		(start 154.550016 75.435)
+		(end 154.550016 76.785)
+		(width 0.5)
 		(layer "B.Cu")
 		(net 2)
@@
 	)
 	(segment
-		(start 159.963756 68.763756)
-		(end 160.211244 68.763756)
+		(start 163.8 65.175)
+		(end 163.8 64.7)
 		(width 0.25)
 		(layer "F.Cu")
@@
 	)
 	(segment
+		(start 164.3 64.2)
+		(end 165.69 64.2)
+		(width 0.25)
+		(layer "F.Cu")
+		(net 9)
+	)
+	(segment
 		(start 166.8 64.2)
 		(end 167.4 64.8)
@@
 		(end 167.4 65.655686)
 		(width 0.2)
-		(layer "F.Cu")
-		(net 9)
-	)
-	(segment
-		(start 160.211244 68.763756)
-		(end 163.8 65.175)
-		(width 0.25)
 		(layer "F.Cu")
 		(net 9)
@@
 	)
 	(segment
-		(start 164.3 64.2)
-		(end 165.69 64.2)
-		(width 0.25)
-		(layer "F.Cu")
-		(net 9)
-	)
-	(segment
 		(start 151.150015 75.858407)
 		(end 152.000016 76.708408)
@@
 	)
 	(segment
-		(start 163.8 65.175)
-		(end 163.8 64.7)
+		(start 160 68.975)
+		(end 163.8 65.175)
 		(width 0.25)
 		(layer "F.Cu")
 		(net 9)
 	)
+	(segment
+		(start 159.875 68.975)
+		(end 160 68.975)
+		(width 0.25)
+		(layer "F.Cu")
+		(net 9)
+	)
 	(via
-		(at 159.963756 68.763756)
+		(at 159.875 68.975)
 		(size 0.6)
 		(drill 0.3)
@@
 	)
 	(segment
-		(start 159.963756 68.886244)
+		(start 159.875 68.975)
 		(end 156.3 72.55)
+		(width 0.25)
+		(layer "B.Cu")
+		(net 9)
+	)
+	(segment
+		(start 153.013604 72.55)
+		(end 151.150015 74.413589)
 		(width 0.25)
 		(layer "B.Cu")
@@
 	)
 	(segment
-		(start 153.013604 72.55)
-		(end 151.150015 74.413589)
-		(width 0.25)
-		(layer "B.Cu")
-		(net 9)
-	)
-	(segment
-		(start 159.963756 68.763756)
-		(end 159.963756 68.886244)
-		(width 0.25)
-		(layer "B.Cu")
-		(net 9)
-	)
-	(segment
 		(start 156.3 72.55)
 		(end 153.013604 72.55)
@@
 	)
 	(segment
-		(start 166.5 65.7)
-		(end 167.4 66.6)
-		(width 0.2)
-		(layer "F.Cu")
-		(net 11)
-	)
-	(segment
-		(start 167.4 68.195686)
-		(end 167.8 68.595686)
-		(width 0.2)
-		(layer "F.Cu")
-		(net 11)
-	)
-	(segment
-		(start 167.8 70.57)
-		(end 169.41 72.18)
-		(width 0.2)
-		(layer "F.Cu")
-		(net 11)
-	)
-	(segment
-		(start 167.8 68.595686)
-		(end 167.8 70.57)
-		(width 0.2)
-		(layer "F.Cu")
-		(net 11)
-	)
-	(segment
-		(start 161.079442 68.531954)
-		(end 163.911396 65.7)
-		(width 0.25)
-		(layer "F.Cu")
-		(net 11)
-	)
-	(segment
-		(start 167.4 66.6)
-		(end 167.4 68.195686)
-		(width 0.2)
-		(layer "F.Cu")
-		(net 11)
-	)
-	(segment
 		(start 163.911396 65.7)
 		(end 165.69 65.7)
@@
 	)
 	(segment
-		(start 161.079442 68.779442)
-		(end 161.079442 68.531954)
+		(start 166.5 65.7)
+		(end 167.4 66.6)
+		(width 0.2)
+		(layer "F.Cu")
+		(net 11)
+	)
+	(segment
+		(start 167.4 68.195686)
+		(end 167.8 68.595686)
+		(width 0.2)
+		(layer "F.Cu")
+		(net 11)
+	)
+	(segment
+		(start 167.8 70.57)
+		(end 169.41 72.18)
+		(width 0.2)
+		(layer "F.Cu")
+		(net 11)
+	)
+	(segment
+		(start 162.3 67.311396)
+		(end 163.911396 65.7)
 		(width 0.25)
+		(layer "F.Cu")
+		(net 11)
+	)
+	(segment
+		(start 167.8 68.595686)
+		(end 167.8 70.57)
+		(width 0.2)
+		(layer "F.Cu")
+		(net 11)
+	)
+	(segment
+		(start 162.3 68.5)
+		(end 162.3 67.311396)
+		(width 0.25)
+		(layer "F.Cu")
+		(net 11)
+	)
+	(segment
+		(start 167.4 66.6)
+		(end 167.4 68.195686)
+		(width 0.2)
 		(layer "F.Cu")
 		(net 11)
@@
 	)
 	(via
-		(at 161.079442 68.779442)
+		(at 162.3 68.5)
 		(size 0.6)
 		(drill 0.3)
 		(layers "F.Cu" "B.Cu")
+		(net 11)
+	)
+	(segment
+		(start 161.358884 68.5)
+		(end 156.658884 73.2)
+		(width 0.25)
+		(layer "B.Cu")
 		(net 11)
 	)
@@
 	)
 	(segment
-		(start 152.000016 74.199984)
-		(end 152.000016 75.435)
+		(start 153.3 73.2)
+		(end 152.000016 74.499984)
 		(width 0.25)
 		(layer "B.Cu")
@@
 	)
 	(segment
-		(start 156.858884 73)
-		(end 153.2 73)
+		(start 156.658884 73.2)
+		(end 153.3 73.2)
 		(width 0.25)
 		(layer "B.Cu")
@@
 	)
 	(segment
-		(start 153.2 73)
-		(end 152.000016 74.199984)
-		(width 0.25)
-		(layer "B.Cu")
-		(net 11)
-	)
-	(segment
-		(start 161.079442 68.779442)
-		(end 156.858884 73)
+		(start 152.000016 74.499984)
+		(end 152.000016 75.435)
 		(width 0.25)
 		(layer "B.Cu")
@@
 		(width 0.25)
 		(layer "B.Cu")
+		(net 11)
+	)
+	(segment
+		(start 162.3 68.5)
+		(end 161.358884 68.5)
+		(width 0.25)
+		(layer "B.Cu")

Commit message: .
Routing:
- net GND: vias 12 -> 11
Changed lines of the file:
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@@
-		)
-	)
-	(gr_text "ESP32-C3"
-		(at 176.1 55.3 0)
-		(layer "B.SilkS" knockout)
-		(effects
-			(font
-				(size 1 1)
-				(thickness 0.25)
-				(bold yes)
-			)
-			(justify left bottom mirror)
 		)
 	)
 	(gr_text "by:\nAlexander B."
-		(at 180.7 68.4 0)
+		(at 153.8 72.8 0)
 		(layer "B.SilkS")
 		(effects
@@
 	)
 	(gr_text "Aug 2024"
-		(at 174.3 61.5 90)
+		(at 165.9 61.7 0)
 		(layer "B.SilkS")
 		(effects
@@
 			)
 			(justify left bottom mirror)
+		)
+	)
+	(gr_text "ESP32-C3"
+		(at 149.8 73.3 0)
+		(layer "F.SilkS" knockout)
+		(effects
+			(font
+				(size 1 1)
+				(thickness 0.25)
+				(bold yes)
+			)
+			(justify left bottom)
 		)
 	)
@@
 	)
 	(via
-		(at 162.8 77)
+		(at 163.7 77)
 		(size 0.6)
 		(drill 0.3)
@@
 	)
 	(via
-		(at 161.2 77)
+		(at 162.1 77)
 		(size 0.6)
 		(drill 0.3)
@@
 	)
 	(via
-		(at 147.7 73.9)
-		(size 0.6)
-		(drill 0.3)
-		(layers "F.Cu" "B.Cu")
-		(free yes)
-		(net 2)
-	)
-	(via
 		(at 157.1 61.9)
 		(size 0.6)
@@
 	)
 	(via
-		(at 162 77)
+		(at 162.9 77)
 		(size 0.6)
 		(drill 0.3)

Commit message: .
Changed lines of the file:
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@@
 			(at 0 1.82 0)
 			(layer "B.SilkS")
+			(hide yes)
 			(effects
 				(font
@@
 			(at 0 1.82 90)
 			(layer "B.SilkS")
+			(hide yes)
 			(effects
 				(font
@@
 	)
 	(segment
-		(start 163.8 65.175)
-		(end 163.8 64.7)
-		(width 0.25)
-		(layer "F.Cu")
-		(net 9)
-	)
-	(segment
 		(start 167.4 65.655686)
 		(end 167.8 66.055686)
@@
 	)
 	(segment
-		(start 164.3 64.2)
-		(end 165.69 64.2)
+		(start 159.875 68.325)
+		(end 164 64.2)
 		(width 0.25)
 		(layer "F.Cu")
@@
 	)
 	(segment
-		(start 163.8 64.7)
-		(end 164.3 64.2)
+		(start 159.875 68.975)
+		(end 159.875 68.325)
 		(width 0.25)
 		(layer "F.Cu")
@@
 	)
 	(segment
-		(start 160 68.975)
-		(end 163.8 65.175)
+		(start 164 64.2)
+		(end 165.69 64.2)
 		(width 0.25)
 		(layer "F.Cu")
-		(net 9)
-	)
-	(segment
-		(start 159.875 68.975)
-		(end 160 68.975)
-		(width 0.25)
-		(layer "F.Cu")
