File: esp32-wroom-adapter-2-ePaper/esp32-wroom-adapter-epaper.kicad_sch (KiCad schematic)
At the start: 20 parts, among them J1 PWR, J2 I2C, J3 I2C, J4 e-Paper, J5 USB-C, J6 UART, U2 MAX1726EUK50, U3 MAX1726EUK33

Commit message: .
Parts:
- removed U2: MAX1726EUK50, Package_TO_SOT_SMD:SOT-223-3_TabPin2, symbol Regulator_Linear:LM78M05_TO220
- removed U3: MAX1726EUK33, Package_TO_SOT_SMD:SOT-223-3_TabPin2, symbol Regulator_Linear:LM78M05_TO220
- added U1: AMS1117-5.0, Package_TO_SOT_SMD:SOT-223-3_TabPin2, symbol Regulator_Linear:AMS1117-5.0
- added U2: AMS1117-3.3, Package_TO_SOT_SMD:SOT-223-3_TabPin2, symbol Regulator_Linear:AMS1117-3.3
Connections:
- net +3V3: now also U2.2 (VO)
- net +5V: now also U1.2 (VO)
- net GND: now also U1.1 (GND), U2.1 (GND)
- net VBUS: now also U1.3 (VI), U2.3 (VI)
Changed lines of the file:
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@@
 	)
 	(symbol
-		(lib_id "Regulator_Linear:LM78M05_TO220")
+		(lib_id "Regulator_Linear:AMS1117-3.3")
 		(at 49.53 64.77 0)
 		(unit 1)
@@
 		(on_board yes)
 		(dnp no)
-		(property "Reference" "U3"
+		(fields_autoplaced yes)
+		(property "Reference" "U2"
 			(at 49.53 58.42 0)
 			(effects
@@
 			)
 		)
-		(property "Value" "MAX1726EUK33"
+		(property "Value" "AMS1117-3.3"
 			(at 49.53 60.96 0)
 			(effects
@@
 		)
 		(property "Footprint" "Package_TO_SOT_SMD:SOT-223-3_TabPin2"
-			(at 49.53 59.055 0)
-			(effects
-				(font
-					(size 1.27 1.27)
-					(italic yes)
-				)
-				(hide yes)
-			)
-		)
-		(property "Datasheet" "https://www.onsemi.com/pub/Collateral/MC78M00-D.PDF"
-			(at 49.53 66.04 0)
-			(effects
-				(font
-					(size 1.27 1.27)
-				)
-				(hide yes)
-			)
-		)
-		(property "Description" ""
+			(at 49.53 59.69 0)
+			(effects
+				(font
+					(size 1.27 1.27)
+				)
+				(hide yes)
+			)
+		)
+		(property "Datasheet" "http://www.advanced-monolithic.com/pdf/ds1117.pdf"
+			(at 52.07 71.12 0)
+			(effects
+				(font
+					(size 1.27 1.27)
+				)
+				(hide yes)
+			)
+		)
+		(property "Description" "1A Low Dropout regulator, positive, 3.3V fixed output, SOT-223"
 			(at 49.53 64.77 0)
 			(effects
@@
 		(pin "1"
 		)
+		(pin "3"
+		)
 		(pin "2"
 		)
-		(pin "3"
-		)
-		(instances
-			(project "esp32-wroom-adapter-2"
-				(path "/4a90ead8-6e51-429d-a467-47fbf8655e89"
-					(reference "U3")
+		(instances
+			(project ""
+				(path "/4a90ead8-6e51-429d-a467-47fbf8655e89"
+					(reference "U2")
 					(unit 1)
 				)
@@
 	)
 	(symbol
+		(lib_id "Regulator_Linear:AMS1117-5.0")
+		(at 49.53 85.09 0)
+		(mirror x)
+		(unit 1)
+		(exclude_from_sim no)
+		(in_bom yes)
+		(on_board yes)
+		(dnp no)
+		(property "Reference" "U1"
+			(at 49.53 88.9 0)
+			(effects
+				(font
+					(size 1.27 1.27)
+				)
+			)
+		)
+		(property "Value" "AMS1117-5.0"
+			(at 49.53 91.44 0)
+			(effects
+				(font
+					(size 1.27 1.27)
+				)
+			)
+		)
+		(property "Footprint" "Package_TO_SOT_SMD:SOT-223-3_TabPin2"
+			(at 49.53 90.17 0)
+			(effects
+				(font
+					(size 1.27 1.27)
+				)
+				(hide yes)
+			)
+		)
+		(property "Datasheet" "http://www.advanced-monolithic.com/pdf/ds1117.pdf"
+			(at 52.07 78.74 0)
+			(effects
+				(font
+					(size 1.27 1.27)
+				)
+				(hide yes)
+			)
+		)
+		(property "Description" "1A Low Dropout regulator, positive, 5.0V fixed output, SOT-223"
+			(at 49.53 85.09 0)
+			(effects
+				(font
+					(size 1.27 1.27)
+				)
+				(hide yes)
+			)
+		)
+		(pin "1"
+		)
+		(pin "2"
+		)
+		(pin "3"
+		)
+		(instances
+			(project ""
+				(path "/4a90ead8-6e51-429d-a467-47fbf8655e89"
+					(reference "U1")
+					(unit 1)
+				)
+			)
+		)
+	)
+	(symbol
 		(lib_id "power:+5V")
 		(at 69.85 85.09 270)
@@
 					(unit 1)
 				)
-			)
-		)
-	)
-	(symbol
-		(lib_id "Regulator_Linear:LM78M05_TO220")
-		(at 49.53 85.09 0)
-		(mirror x)
-		(unit 1)
-		(exclude_from_sim no)
-		(in_bom yes)
-		(on_board yes)
-		(dnp no)
-		(fields_autoplaced yes)
-		(property "Reference" "U2"
-			(at 49.53 88.9 0)
-			(effects
-				(font
-					(size 1.27 1.27)
-				)
-			)
-		)
-		(property "Value" "MAX1726EUK50"
-			(at 49.53 91.44 0)
-			(effects
-				(font
-					(size 1.27 1.27)
-				)
-			)
-		)
-		(property "Footprint" "Package_TO_SOT_SMD:SOT-223-3_TabPin2"
-			(at 49.53 90.805 0)
-			(effects
-				(font
-					(size 1.27 1.27)
-					(italic yes)
-				)
-				(hide yes)
-			)
-		)
-		(property "Datasheet" "https://www.onsemi.com/pub/Collateral/MC78M00-D.PDF"
-			(at 49.53 83.82 0)
-			(effects
-				(font
-					(size 1.27 1.27)
-				)
-				(hide yes)
-			)
-		)
-		(property "Description" ""
-			(at 49.53 85.09 0)
-			(effects
-				(font
-					(size 1.27 1.27)
-				)
-				(hide yes)
-			)
-		)
-		(pin "3"
-		)
-		(pin "1"
-		)
-		(pin "2"
-		)
-		(instances
-			(project "esp32-wroom-adapter-2"
-				(path "/4a90ead8-6e51-429d-a467-47fbf8655e89"
-					(reference "U2")
-					(unit 1)
-				)

Commit message: .
Parts:
- added D1: LED_Dual_AAKK, symbol Device:LED_Dual_AAKK
- added Q1, Q2: NMOS, symbol Simulation_SPICE:NMOS
- added Q3: PMOS, symbol Simulation_SPICE:PMOS
- added R4, R5, R6, R7: 3k3, Resistor_SMD:R_1206_3216Metric_Pad1.30x1.75mm_HandSolder, symbol Device:R
Connections:
- net +3V3: now also R4.2
- net GND: now also D1.4 (K2), Q1.3 (S), Q2.3 (S)
- net OUTPUT_1: now reaches J8.16 (IO13)
- new net: D1.1 (A1), R4.1
- new net: D1.2 (A2), R5.1
- new net: Q2.1 (D), R6.2
- new net: Q3.2 (G), R6.1, R7.2
- new net OUTPUT_1/LED: D1.3 (K1), R5.2
- new net OUTPUT_1/SOURCE: Q1.2 (G)
- new net OUTPUT_2: Q2.2 (G)
- new net OUT_1: Q3.3 (S)
- new net SOURCE_1: Q1.1 (D)
- new net V+: Q3.1 (D), R7.1

Commit message: .
Parts:
- removed Q1: NMOS, symbol Simulation_SPICE:NMOS
- added Q4: MOSFET-N-2CH-DMT3020, Alexander Footprint Library:MOSFET-N-2CH-DMT3020-SO-8, symbol Alexander Symbol Library:MOSFET-N-2CH-DMT3020
Connections:
- net GND: now also Q4.1 (S1)
- net OUTPUT_1/SOURCE: now also Q4.2 (G1)
- net SOURCE_1: now also Q4.7 (D1), Q4.8 (D1)
- new net: Q4.5 (D2), Q4.6 (D2)
Changed lines of the file:
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@@
 	(wire
 		(pts
-			(xy 153.67 92.71) (xy 161.29 92.71)
-		)
-		(stroke
-			(width 0)
-			(type default)
-		)
-	)
-	(wire
-		(pts
-			(xy 168.91 97.79) (xy 168.91 101.6)
-		)
-		(stroke
-			(width 0)
-			(type default)
-		)
-	)
-	(wire
-		(pts
 			(xy 125.73 68.58) (xy 130.81 68.58)
 		)
@@
 	(wire
 		(pts
+			(xy 165.1 88.9) (xy 165.1 91.44)
+		)
+		(stroke
+			(width 0)
+			(type default)
+		)
+	)
+	(wire
+		(pts
 			(xy 224.79 123.19) (xy 218.44 123.19)
 		)
@@
 	(wire
 		(pts
+			(xy 165.1 74.93) (xy 165.1 78.74)
+		)
+		(stroke
+			(width 0)
+			(type default)
+		)
+	)
+	(wire
+		(pts
 			(xy 218.44 120.65) (xy 224.79 120.65)
 		)
@@
 	(wire
 		(pts
-			(xy 168.91 81.28) (xy 168.91 87.63)
-		)
-		(stroke
-			(width 0)
-			(type default)
-		)
-	)
-	(wire
-		(pts
 			(xy 57.15 64.77) (xy 59.69 64.77)
 		)
@@
 	(wire
 		(pts
+			(xy 157.48 83.82) (xy 156.21 83.82)
+		)
+		(stroke
+			(width 0)
+			(type default)
+		)
+	)
+	(wire
+		(pts
 			(xy 73.66 184.15) (xy 81.28 184.15)
 		)
@@
 		)
 	)
-	(global_label "OUT_1"
+	(global_label "SOURCE_1"
 		(shape input)
-		(at 102.87 152.4 0)
+		(at 165.1 74.93 90)
 		(fields_autoplaced yes)
 		(effects
@@
 		)
 		(property "Intersheetrefs" "${INTERSHEET_REFS}"
-			(at 111.6609 152.4 0)
+			(at 165.1 62.2082 90)
 			(effects
 				(font
@@
 		)
 	)
-	(global_label "SOURCE_1"
+	(global_label "OUT_1"
 		(shape input)
-		(at 168.91 81.28 90)
+		(at 102.87 152.4 0)
 		(fields_autoplaced yes)
 		(effects
@@
 		)
 		(property "Intersheetrefs" "${INTERSHEET_REFS}"
-			(at 168.91 68.5582 90)
+			(at 111.6609 152.4 0)
 			(effects
 				(font
@@
 		)
 	)
-	(hierarchical_label "OUTPUT_1{slash}LED"
+	(hierarchical_label "OUTPUT_1{slash}SOURCE"
 		(shape input)
-		(at 140.97 144.78 180)
+		(at 156.21 83.82 180)
 		(fields_autoplaced yes)
 		(effects
@@
 		)
 	)
-	(hierarchical_label "OUTPUT_1{slash}SOURCE"
+	(hierarchical_label "OUTPUT_1{slash}LED"
 		(shape input)
-		(at 153.67 92.71 180)
+		(at 140.97 144.78 180)
 		(fields_autoplaced yes)
 		(effects
@@
 	)
 	(symbol
-		(lib_id "Simulation_SPICE:NMOS")
-		(at 166.37 92.71 0)
-		(unit 1)
-		(exclude_from_sim no)
-		(in_bom yes)
-		(on_board yes)
-		(dnp no)
-		(fields_autoplaced yes)
-		(property "Reference" "Q1"
-			(at 172.72 91.4399 0)
-			(effects
-				(font
-					(size 1.27 1.27)
-				)
-				(justify left)
-			)
-		)
-		(property "Value" "NMOS"
-			(at 172.72 93.9799 0)
-			(effects
-				(font
-					(size 1.27 1.27)
-				)
-				(justify left)
-			)
-		)
-		(property "Footprint" ""
-			(at 171.45 90.17 0)
-			(effects
-				(font
-					(size 1.27 1.27)
-				)
-				(hide yes)
-			)
-		)
-		(property "Datasheet" "https://ngspice.sourceforge.io/docs/ngspice-html-manual/manual.xhtml#cha_MOSFETs"
-			(at 166.37 105.41 0)
-			(effects
-				(font
-					(size 1.27 1.27)
-				)
-				(hide yes)
-			)
-		)
-		(property "Description" "N-MOSFET transistor, drain/source/gate"
-			(at 166.37 92.71 0)
-			(effects
-				(font
-					(size 1.27 1.27)
-				)
-				(hide yes)
-			)
-		)
-		(property "Sim.Device" "NMOS"
-			(at 166.37 109.855 0)
-			(effects
-				(font
-					(size 1.27 1.27)
-				)
-				(hide yes)
-			)
-		)
-		(property "Sim.Type" "VDMOS"
-			(at 166.37 111.76 0)
-			(effects
-				(font
-					(size 1.27 1.27)
-				)
-				(hide yes)
-			)
-		)
-		(property "Sim.Pins" "1=D 2=G 3=S"
-			(at 166.37 107.95 0)
-			(effects
-				(font
-					(size 1.27 1.27)
-				)
-				(hide yes)
-			)
-		)
-		(pin "3"
-		)
-		(pin "1"
-		)
-		(pin "2"
-		)
-		(instances
-			(project ""
-				(path "/4a90ead8-6e51-429d-a467-47fbf8655e89"
-					(reference "Q1")
-					(unit 1)
-				)
-			)
-		)
-	)
-	(symbol
 		(lib_id "power:+3V3")
 		(at 218.44 93.98 90)
@@
 		(lib_name "GND_6")
 		(lib_id "power:GND")
-		(at 168.91 101.6 0)
+		(at 165.1 91.44 0)
 		(unit 1)
 		(exclude_from_sim no)
@@
 		(fields_autoplaced yes)
 		(property "Reference" "#PWR021"
-			(at 168.91 107.95 0)
+			(at 165.1 97.79 0)
 			(effects
 				(font
@@
 		)
 		(property "Value" "GND"
-			(at 168.91 106.68 0)
+			(at 165.1 96.52 0)
 			(effects
 				(font
@@
 		)
 		(property "Footprint" ""
-			(at 168.91 101.6 0)
+			(at 165.1 91.44 0)
 			(effects
 				(font
@@
 		)
 		(property "Datasheet" ""
-			(at 168.91 101.6 0)
+			(at 165.1 91.44 0)
 			(effects
 				(font
@@
 		)
 		(property "Description" "Power symbol creates a global label with name \"GND\" , ground"
-			(at 168.91 101.6 0)
+			(at 165.1 91.44 0)
 			(effects
 				(font
@@
 					(unit 1)
 				)
+			)
+		)
+	)
+	(symbol
+		(lib_id "Alexander Symbol Library:MOSFET-N-2CH-DMT3020")
+		(at 162.56 83.82 0)
+		(unit 1)
+		(exclude_from_sim no)
+		(in_bom yes)
+		(on_board yes)
+		(dnp no)
+		(fields_autoplaced yes)
+		(property "Reference" "Q4"
+			(at 194.31 82.5499 0)
+			(effects
+				(font
+					(size 1.27 1.27)
+				)
+				(justify left)
+			)
+		)
+		(property "Value" "MOSFET-N-2CH-DMT3020"
+			(at 194.31 85.0899 0)
+			(effects
+				(font
+					(size 1.27 1.27)
+				)
+				(justify left)
+			)
+		)
+		(property "Footprint" "Alexander Footprint Library:MOSFET-N-2CH-DMT3020-SO-8"
+			(at 167.64 81.28 0)
+			(effects
+				(font
+					(size 1.27 1.27)
+				)
+				(hide yes)
+			)
+		)
+		(property "Datasheet" ""
+			(at 162.56 96.52 0)
+			(effects
+				(font
+					(size 1.27 1.27)
+				)
+				(hide yes)
+			)
+		)
+		(property "Description" "N-MOSFET transistor, drain/source/gate"
+			(at 165.1 68.834 0)
+			(effects
+				(font
+					(size 1.27 1.27)
+				)
+				(hide yes)
+			)
+		)
+		(property "Sim.Device" "NMOS"
+			(at 162.56 100.965 0)
+			(effects
+				(font
+					(size 1.27 1.27)
+				)
+				(hide yes)
+			)
+		)
+		(property "Sim.Type" "VDMOS"
+			(at 162.56 102.87 0)
+			(effects
+				(font
+					(size 1.27 1.27)
+				)
+				(hide yes)
+			)
+		)
+		(property "Sim.Pins" "1=D 2=G 3=S"
+			(at 162.56 99.06 0)
+			(effects
+				(font
+					(size 1.27 1.27)
+				)
+				(hide yes)
+			)
+		)
+		(pin "5"
+		)
+		(pin "3"
+		)
+		(pin "7"
+		)
+		(pin "2"
+		)
+		(pin "8"
+		)
+		(pin "6"
+		)
+		(pin "1"
+		)
+		(pin "4"
+		)
+		(instances
+			(project ""
+				(path "/4a90ead8-6e51-429d-a467-47fbf8655e89"
+					(reference "Q4")
+					(unit 1)
+				)

Commit message: .
Connections:
- net OUTPUT_1/SOURCE is gone; now on net OUTPUT_1: Q4.2 (G1)
Changed lines of the file:
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@@
 	(wire
 		(pts
-			(xy 157.48 83.82) (xy 156.21 83.82)
+			(xy 157.48 83.82) (xy 153.67 83.82)
 		)
 		(stroke
@@
 		)
 	)
+	(global_label "OUTPUT_1"
+		(shape input)
+		(at 153.67 83.82 180)
+		(fields_autoplaced yes)
+		(effects
+			(font
+				(size 1.27 1.27)
+			)
+			(justify right)
+		)
+		(property "Intersheetrefs" "${INTERSHEET_REFS}"
+			(at 141.311 83.82 0)
+			(effects
+				(font
+					(size 1.27 1.27)
+				)
+				(justify right)
+				(hide yes)
+			)
+		)
+	)
 	(global_label "SOURCE_1"
 		(shape input)
@@
 		)
 	)
-	(hierarchical_label "OUTPUT_1{slash}SOURCE"
-		(shape input)
-		(at 156.21 83.82 180)
-		(fields_autoplaced yes)
-		(effects
-			(font
-				(size 1.27 1.27)
-			)
-			(justify right)
-		)
-	)

Commit message: .
Parts:
- removed D1: LED_Dual_AAKK, symbol Device:LED_Dual_AAKK
- added LED1: LED-RED-GREEN-B1552USUG20D, Alexander Footprint Library:B1552_HVK-M, symbol Alexander_Library_Symbols:LED-RED-GREEN-B1552USUG20D
Connections:
- net OUTPUT_1/LED is gone; now on net OUTPUT_1: R5.2
- net GND: now also LED1.4 (GND)
- net OUTPUT_1: now also LED1.1 (GND)
- net at R4.1: now also LED1.2 (RED)
- net at R5.1: now also LED1.3 (GRN)
Other:
- moved on the sheet: R4, R5

Commit message: .
Connections:
- net GND: now also Q4.3 (S2)
- net OUTPUT_1: no longer J8.16 (IO13)
- net OUTPUT_2: now also Q4.4 (G2)
- net SOURCE_2: now reaches Q4.5 (D2), Q4.6 (D2)
Changed lines of the file:
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@@
 	(wire
 		(pts
+			(xy 177.8 74.93) (xy 177.8 83.82)
+		)
+		(stroke
+			(width 0)
+			(type default)
+		)
+	)
+	(wire
+		(pts
 			(xy 57.15 85.09) (xy 59.69 85.09)
 		)
@@
 	(wire
 		(pts
+			(xy 177.8 83.82) (xy 182.88 83.82)
+		)
+		(stroke
+			(width 0)
+			(type default)
+		)
+	)
+	(wire
+		(pts
 			(xy 49.53 74.93) (xy 59.69 74.93)
 		)
@@
 	(wire
 		(pts
-			(xy 181.61 135.89) (xy 187.96 135.89)
+			(xy 154.94 83.82) (xy 157.48 83.82)
 		)
 		(stroke
@@
 	(wire
 		(pts
-			(xy 165.1 88.9) (xy 165.1 91.44)
+			(xy 181.61 135.89) (xy 187.96 135.89)
 		)
 		(stroke
@@
 	(wire
 		(pts
-			(xy 224.79 123.19) (xy 218.44 123.19)
+			(xy 165.1 88.9) (xy 165.1 91.44)
 		)
 		(stroke
@@
 	(wire
 		(pts
-			(xy 125.73 55.88) (xy 130.81 55.88)
+			(xy 224.79 123.19) (xy 218.44 123.19)
 		)
 		(stroke
@@
 	(wire
 		(pts
+			(xy 190.5 88.9) (xy 190.5 91.44)
+		)
+		(stroke
+			(width 0)
+			(type default)
+		)
+	)
+	(wire
+		(pts
 			(xy 93.98 152.4) (xy 102.87 152.4)
 		)
@@
 	(wire
 		(pts
+			(xy 190.5 74.93) (xy 190.5 78.74)
+		)
+		(stroke
+			(width 0)
+			(type default)
+		)
+	)
+	(wire
+		(pts
 			(xy 41.91 85.09) (xy 35.56 85.09)
 		)
@@
 	(wire
 		(pts
+			(xy 154.94 74.93) (xy 154.94 83.82)
+		)
+		(stroke
+			(width 0)
+			(type default)
+		)
+	)
+	(wire
+		(pts
 			(xy 218.44 99.06) (xy 224.79 99.06)
 		)
@@
 	(wire
 		(pts
-			(xy 157.48 83.82) (xy 153.67 83.82)
-		)
-		(stroke
-			(width 0)
-			(type default)
-		)
-	)
-	(wire
-		(pts
 			(xy 73.66 184.15) (xy 81.28 184.15)
 		)
@@
 		)
 	)
+	(global_label "V+"
+		(shape input)
+		(at 72.39 152.4 180)
+		(fields_autoplaced yes)
+		(effects
+			(font
+				(size 1.27 1.27)
+			)
+			(justify right)
+		)
+		(property "Intersheetrefs" "${INTERSHEET_REFS}"
+			(at 66.7438 152.4 0)
+			(effects
+				(font
+					(size 1.27 1.27)
+				)
+				(justify right)
+				(hide yes)
+			)
+		)
+	)
 	(global_label "OUTPUT_1"
 		(shape input)
-		(at 130.81 55.88 0)
+		(at 154.94 74.93 90)
 		(fields_autoplaced yes)
 		(effects
@@
 		)
 		(property "Intersheetrefs" "${INTERSHEET_REFS}"
-			(at 143.169 55.88 0)
+			(at 154.94 62.571 90)
 			(effects
 				(font
@@
 		)
 	)
-	(global_label "V+"
+	(global_label "SOURCE_1"
 		(shape input)
-		(at 72.39 152.4 180)
+		(at 165.1 74.93 90)
 		(fields_autoplaced yes)
 		(effects
@@
 				(size 1.27 1.27)
 			)
-			(justify right)
+			(justify left)
 		)
 		(property "Intersheetrefs" "${INTERSHEET_REFS}"
-			(at 66.7438 152.4 0)
+			(at 165.1 62.2082 90)
 			(effects
 				(font
 					(size 1.27 1.27)
 				)
-				(justify right)
+				(justify left)
 				(hide yes)
 			)
 		)
 	)
-	(global_label "OUTPUT_1"
+	(global_label "OUTPUT_2"
 		(shape input)
-		(at 153.67 83.82 180)
+		(at 177.8 74.93 90)
 		(fields_autoplaced yes)
 		(effects
@@
 				(size 1.27 1.27)
 			)
-			(justify right)
+			(justify left)
 		)
 		(property "Intersheetrefs" "${INTERSHEET_REFS}"
-			(at 141.311 83.82 0)
+			(at 177.8 62.571 90)
 			(effects
 				(font
 					(size 1.27 1.27)
 				)
-				(justify right)
+				(justify left)
 				(hide yes)
 			)
 		)
 	)
-	(global_label "SOURCE_1"
+	(global_label "SOURCE_2"
 		(shape input)
-		(at 165.1 74.93 90)
+		(at 190.5 74.93 90)
 		(fields_autoplaced yes)
 		(effects
@@
 		)
 		(property "Intersheetrefs" "${INTERSHEET_REFS}"
-			(at 165.1 62.2082 90)
+			(at 190.5 62.2082 90)
 			(effects
 				(font
@@
 					(unit 1)
 				)
+			)
+		)
+	)
+	(symbol
+		(lib_name "GND_7")
+		(lib_id "power:GND")
+		(at 190.5 91.44 0)
+		(unit 1)
+		(exclude_from_sim no)
+		(in_bom yes)
+		(on_board yes)
+		(dnp no)
+		(fields_autoplaced yes)
+		(property "Reference" "#PWR023"
+			(at 190.5 97.79 0)
+			(effects
+				(font
+					(size 1.27 1.27)
+				)
+				(hide yes)
+			)
+		)
+		(property "Value" "GND"
+			(at 190.5 96.52 0)
+			(effects
+				(font
+					(size 1.27 1.27)
+				)
+			)
+		)
+		(property "Footprint" ""
+			(at 190.5 91.44 0)
+			(effects
+				(font
+					(size 1.27 1.27)
+				)
+				(hide yes)
+			)
+		)
+		(property "Datasheet" ""
+			(at 190.5 91.44 0)
+			(effects
+				(font
+					(size 1.27 1.27)
+				)
+				(hide yes)
+			)
+		)
+		(property "Description" "Power symbol creates a global label with name \"GND\" , ground"
+			(at 190.5 91.44 0)
+			(effects
+				(font
+					(size 1.27 1.27)
+				)
+				(hide yes)
+			)
+		)
+		(pin "1"
+		)
+		(instances
+			(project ""
+				(path "/4a90ead8-6e51-429d-a467-47fbf8655e89"
+					(reference "#PWR023")
+					(unit 1)
+				)

Commit message: ,
Parts:
- removed LED1: LED-RED-GREEN-B1552USUG20D, Alexander Footprint Library:B1552_HVK-M, symbol Alexander_Library_Symbols:LED-RED-GREEN-B1552USUG20D
- removed Q4: MOSFET-N-2CH-DMT3020, Alexander Footprint Library:MOSFET-N-2CH-DMT3020-SO-8, symbol Alexander Symbol Library:MOSFET-N-2CH-DMT3020
- removed R4, R5: 3k3, Resistor_SMD:R_1206_3216Metric_Pad1.30x1.75mm_HandSolder, symbol Device:R
Other:
- added sheet Interfaces (interfaces.kicad_sch)

Commit message: .
Parts:
- removed C1, C2, C3: 1uF, Capacitor_THT:CP_Radial_D4.0mm_P2.00mm, symbol Device:C_Polarized_Small
- removed J1: PWR, Connector_PinHeader_2.54mm:PinHeader_1x02_P2.54mm_Vertical, symbol Connector:Conn_01x02_Pin
- removed J5: USB-C, Alexander Footprint Library:USB-C MOLEX 2171750001, symbol Alexander_Library_Symbols:USB-C RCP USB2.0 6POS (B)
- removed Q2: NMOS, symbol Simulation_SPICE:NMOS
- removed Q3: PMOS, symbol Simulation_SPICE:PMOS
- removed R2, R3: 5k1, Resistor_SMD:R_1206_3216Metric_Pad1.30x1.75mm_HandSolder, symbol Device:R
- removed R6, R7: 3k3, Resistor_SMD:R_1206_3216Metric_Pad1.30x1.75mm_HandSolder, symbol Device:R
- removed TP1: TP1, Alexander Footprints Library:TestPoint_D2.5mm, symbol Connector:TestPoint
- removed TP2: GND, Alexander Footprints Library:TestPoint_D2.5mm, symbol Connector:TestPoint
- removed U1: AMS1117-5.0, Package_TO_SOT_SMD:SOT-223-3_TabPin2, symbol Regulator_Linear:AMS1117-5.0
- removed U2: AMS1117-3.3, Package_TO_SOT_SMD:SOT-223-3_TabPin2, symbol Regulator_Linear:AMS1117-3.3
- R1: footprint Alexander Footprints Library:STA_RMCF1206_STP-L -> Resistor_SMD:R_1206_3216Metric_Pad1.30x1.75mm_HandSolder
Other:
- added sheet Power Supply (power-supply.kicad_sch)
