File: Production/prod_esp32-node-box-40x65_telemetry-002/esp32-node-board-40x65_telemetry/schematics-snips.kicad_sch (KiCad schematic)
At the start: 15 parts, among them J11 Conn_01x06_Socket, J12 Conn_01x02_Socket, J13 Conn_01x02_Socket, Q1 NPN, Q2 NPN, Q3 2N3904, U2 4N35, U6 PC817

Commit message: .
Parts:
- renumbered D3 to D7, J11 to J13, J12 to J14, J13 to J15, Q3 to Q2, Q2 to Q3, R4 to R10, R5 to R6, R2 to R7, R6 to R8, R3 to R9, U6 to U5, U2 to U6
Changed lines of the file:
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@@
 		(dnp no)
 		(fields_autoplaced yes)
-		(property "Reference" "U6"
+		(property "Reference" "U5"
 			(at 46.99 82.55 0)
 			(effects
@@
 			(project "esp32-node-board-40x65_telemetry"
 				(path "/5f5eb0ac-ab9b-41ab-8d2f-875870c41abc/4d11314b-2f19-4ab5-8867-985fed32d05b"
-					(reference "U6")
+					(reference "U5")
 					(unit 1)
 				)
@@
 		(dnp no)
 		(fields_autoplaced yes)
-		(property "Reference" "R5"
+		(property "Reference" "R6"
 			(at 33.02 82.55 90)
 			(effects
@@
 			(project "esp32-node-board-40x65_telemetry"
 				(path "/5f5eb0ac-ab9b-41ab-8d2f-875870c41abc/4d11314b-2f19-4ab5-8867-985fed32d05b"
-					(reference "R5")
+					(reference "R6")
 					(unit 1)
 				)
@@
 		(dnp no)
 		(fields_autoplaced yes)
-		(property "Reference" "Q3"
+		(property "Reference" "Q2"
 			(at 76.2 92.7099 0)
 			(effects
@@
 			(project "esp32-node-board-40x65_telemetry"
 				(path "/5f5eb0ac-ab9b-41ab-8d2f-875870c41abc/4d11314b-2f19-4ab5-8867-985fed32d05b"
-					(reference "Q3")
+					(reference "Q2")
 					(unit 1)
 				)
@@
 		(dnp no)
 		(fields_autoplaced yes)
-		(property "Reference" "#PWR020"
+		(property "Reference" "#PWR027"
 			(at 73.66 109.22 0)
 			(effects
@@
 			(project "esp32-node-board-40x65_telemetry"
 				(path "/5f5eb0ac-ab9b-41ab-8d2f-875870c41abc/4d11314b-2f19-4ab5-8867-985fed32d05b"
-					(reference "#PWR020")
+					(reference "#PWR027")
 					(unit 1)
 				)
@@
 		(dnp no)
 		(fields_autoplaced yes)
-		(property "Reference" "R3"
+		(property "Reference" "R9"
 			(at 73.66 22.86 90)
 			(effects
@@
 			(project "esp32-node-board-40x65_telemetry"
 				(path "/5f5eb0ac-ab9b-41ab-8d2f-875870c41abc/4d11314b-2f19-4ab5-8867-985fed32d05b"
-					(reference "R3")
+					(reference "R9")
 					(unit 1)
 				)
@@
 		(on_board no)
 		(dnp no)
-		(property "Reference" "J11"
+		(property "Reference" "J13"
 			(at 39.37 44.4499 0)
 			(effects
@@
 			(project "esp32-node-board-40x65_telemetry"
 				(path "/5f5eb0ac-ab9b-41ab-8d2f-875870c41abc/4d11314b-2f19-4ab5-8867-985fed32d05b"
-					(reference "J11")
+					(reference "J13")
 					(unit 1)
 				)
@@
 		(dnp no)
 		(fields_autoplaced yes)
-		(property "Reference" "Q2"
+		(property "Reference" "Q3"
 			(at 91.44 27.9399 0)
 			(effects
@@
 			(project "esp32-node-board-40x65_telemetry"
 				(path "/5f5eb0ac-ab9b-41ab-8d2f-875870c41abc/4d11314b-2f19-4ab5-8867-985fed32d05b"
-					(reference "Q2")
+					(reference "Q3")
 					(unit 1)
 				)
@@
 		(dnp no)
 		(fields_autoplaced yes)
-		(property "Reference" "R6"
+		(property "Reference" "R8"
 			(at 60.96 87.63 90)
 			(effects
@@
 			(project "esp32-node-board-40x65_telemetry"
 				(path "/5f5eb0ac-ab9b-41ab-8d2f-875870c41abc/4d11314b-2f19-4ab5-8867-985fed32d05b"
-					(reference "R6")
+					(reference "R8")
 					(unit 1)
 				)
@@
 		(dnp no)
 		(fields_autoplaced yes)
-		(property "Reference" "R2"
+		(property "Reference" "R7"
 			(at 35.56 118.11 90)
 			(effects
@@
 			(project "esp32-node-board-40x65_telemetry"
 				(path "/5f5eb0ac-ab9b-41ab-8d2f-875870c41abc/4d11314b-2f19-4ab5-8867-985fed32d05b"
-					(reference "R2")
+					(reference "R7")
 					(unit 1)
 				)
@@
 		(dnp no)
 		(fields_autoplaced yes)
-		(property "Reference" "J12"
+		(property "Reference" "J14"
 			(at 76.2 126.9999 0)
 			(effects
@@
 			(project "esp32-node-board-40x65_telemetry"
 				(path "/5f5eb0ac-ab9b-41ab-8d2f-875870c41abc/4d11314b-2f19-4ab5-8867-985fed32d05b"
-					(reference "J12")
+					(reference "J14")
 					(unit 1)
 				)
@@
 		(dnp no)
 		(fields_autoplaced yes)
-		(property "Reference" "#PWR011"
+		(property "Reference" "#PWR025"
 			(at 40.64 140.97 0)
 			(effects
@@
 			(project "esp32-node-board-40x65_telemetry"
 				(path "/5f5eb0ac-ab9b-41ab-8d2f-875870c41abc/4d11314b-2f19-4ab5-8867-985fed32d05b"
-					(reference "#PWR011")
+					(reference "#PWR025")
 					(unit 1)
 				)
@@
 		(dnp no)
 		(fields_autoplaced yes)
-		(property "Reference" "#PWR018"
+		(property "Reference" "#PWR024"
 			(at 34.29 109.22 0)
 			(effects
@@
 			(project "esp32-node-board-40x65_telemetry"
 				(path "/5f5eb0ac-ab9b-41ab-8d2f-875870c41abc/4d11314b-2f19-4ab5-8867-985fed32d05b"
-					(reference "#PWR018")
+					(reference "#PWR024")
 					(unit 1)
 				)
@@
 		(dnp no)
 		(fields_autoplaced yes)
-		(property "Reference" "D3"
+		(property "Reference" "D7"
 			(at 76.2 81.2799 90)
 			(effects
@@
 			(project "esp32-node-board-40x65_telemetry"
 				(path "/5f5eb0ac-ab9b-41ab-8d2f-875870c41abc/4d11314b-2f19-4ab5-8867-985fed32d05b"
-					(reference "D3")
+					(reference "D7")
 					(unit 1)
 				)
@@
 		(dnp no)
 		(fields_autoplaced yes)
-		(property "Reference" "J13"
+		(property "Reference" "J15"
 			(at 91.44 81.2799 0)
 			(effects
@@
 			(project "esp32-node-board-40x65_telemetry"
 				(path "/5f5eb0ac-ab9b-41ab-8d2f-875870c41abc/4d11314b-2f19-4ab5-8867-985fed32d05b"
-					(reference "J13")
+					(reference "J15")
 					(unit 1)
 				)
@@
 		(dnp no)
 		(fields_autoplaced yes)
-		(property "Reference" "#PWR019"
+		(property "Reference" "#PWR026"
 			(at 57.15 77.47 0)
 			(effects
@@
 			(project "esp32-node-board-40x65_telemetry"
 				(path "/5f5eb0ac-ab9b-41ab-8d2f-875870c41abc/4d11314b-2f19-4ab5-8867-985fed32d05b"
-					(reference "#PWR019")
+					(reference "#PWR026")
 					(unit 1)
 				)
@@
 		(dnp no)
 		(fields_autoplaced yes)
-		(property "Reference" "R4"
+		(property "Reference" "R10"
 			(at 77.47 35.56 90)
 			(effects
@@
 			(project "esp32-node-board-40x65_telemetry"
 				(path "/5f5eb0ac-ab9b-41ab-8d2f-875870c41abc/4d11314b-2f19-4ab5-8867-985fed32d05b"
-					(reference "R4")
+					(reference "R10")
 					(unit 1)
 				)
@@
 		(dnp no)
 		(fields_autoplaced yes)
-		(property "Reference" "U2"
+		(property "Reference" "U6"
 			(at 50.8 118.11 0)
 			(effects
@@
 			(project "esp32-node-board-40x65_telemetry"
 				(path "/5f5eb0ac-ab9b-41ab-8d2f-875870c41abc/4d11314b-2f19-4ab5-8867-985fed32d05b"
-					(reference "U2")
-					(unit 1)
-				)
+					(reference "U6")
+					(unit 1)
+				)
