File: ESP32-C3-BreadBoardAdapter/ESP32-C3-BreadBoardAdapter/ESP32-C3-BreadBoardAdapter.kicad_sch (KiCad schematic)
At the start: 2 parts, among them U1 ESP32-C3-WROOM-02-N4

Commit message: .
Connections:
- net EN: now also BRD1.1 (A1), U1.2 (EN)
- net IO0: now also BRD1.15 (B7), U1.18 (IO0)
- net IO1: now also BRD1.16 (B8), U1.17 (IO1)
- net IO10: now also U1.10 (IO10)
- net IO13: now also U1.13 (IO18)
- net IO19: now also U1.14 (IO19)
- net IO2: now also U1.16 (IO2)
- net IO3: now also U1.15 (IO3)
- net IO4: now also BRD1.2 (A2), U1.3 (IO4)
- net IO5: now also BRD1.3 (A3), U1.4 (IO5)
- net IO6: now also BRD1.4 (A4), U1.5 (IO6)
- net IO7: now also BRD1.6 (A6), U1.6 (IO7)
- net IO8: now also BRD1.5 (A5), U1.7 (IO8)
- net IO9: now also BRD1.7 (A7), U1.8 (IO9)
- net RXD: now also U1.11 (RXD)
- net TXD: now also U1.12 (TXD)

Commit message: .
Connections:
- net IO13: now also BRD1.12 (B4)
- net IO2: now also BRD1.13 (B5)
- net IO3: now also BRD1.14 (B6)
Changed lines of the file:
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@@
+	(wire
+		(pts
+			(xy 154.94 60.96) (xy 160.02 60.96)
+		)
+		(stroke
+			(width 0)
+			(type default)
+		)
+	)
 	(wire
 		(pts
@@
 	(wire
 		(pts
+			(xy 154.94 66.04) (xy 160.02 66.04)
+		)
+		(stroke
+			(width 0)
+			(type default)
+		)
+	)
+	(wire
+		(pts
 			(xy 116.84 63.5) (xy 121.92 63.5)
 		)
@@
 		(pts
 			(xy 215.9 64.77) (xy 218.44 64.77)
+		)
+		(stroke
+			(width 0)
+			(type default)
+		)
+	)
+	(wire
+		(pts
+			(xy 154.94 63.5) (xy 160.02 63.5)
 		)
 		(stroke
@@
 	)
 	(label "IO2"
-		(at 162.56 78.74 0)
+		(at 160.02 63.5 0)
 		(fields_autoplaced yes)
 		(effects
@@
 	)
 	(label "IO19"
-		(at 160.02 63.5 0)
-		(fields_autoplaced yes)
-		(effects
+		(at 170.18 46.99 0)
+		(fields_autoplaced yes)
+		(effects

Commit message: .
Connections:
- net IO10: now also BRD1.7 (A7)
- net IO13: now also BRD1.11 (B3); no longer BRD1.12 (B4)
- net IO19: now also BRD1.12 (B4)
- net IO9: now also BRD1.8 (A8); no longer BRD1.7 (A7)
- net RXD: now also BRD1.9 (B1)
- net TXD: now also BRD1.10 (B2)
Changed lines of the file:
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@@
+	(wire
+		(pts
+			(xy 137.16 81.28) (xy 138.43 81.28)
+		)
+		(stroke
+			(width 0)
+			(type default)
+		)
+	)
+	(wire
+		(pts
+			(xy 215.9 85.09) (xy 224.79 85.09)
+		)
+		(stroke
+			(width 0)
+			(type default)
+		)
+	)
+	(wire
+		(pts
+			(xy 223.52 52.07) (xy 215.9 52.07)
+		)
+		(stroke
+			(width 0)
+			(type default)
+		)
+	)
+	(wire
+		(pts
+			(xy 215.9 72.39) (xy 218.44 72.39)
+		)
+		(stroke
+			(width 0)
+			(type default)
+		)
+	)
+	(wire
+		(pts
+			(xy 215.9 69.85) (xy 218.44 69.85)
+		)
+		(stroke
+			(width 0)
+			(type default)
+		)
+	)
+	(wire
+		(pts
+			(xy 175.26 72.39) (xy 180.34 72.39)
+		)
+		(stroke
+			(width 0)
+			(type default)
+		)
+	)
+	(wire
+		(pts
+			(xy 154.94 58.42) (xy 160.02 58.42)
+		)
+		(stroke
+			(width 0)
+			(type default)
+		)
+	)
+	(wire
+		(pts
+			(xy 116.84 68.58) (xy 121.92 68.58)
+		)
+		(stroke
+			(width 0)
+			(type default)
+		)
+	)
+	(wire
+		(pts
+			(xy 137.16 77.47) (xy 137.16 81.28)
+		)
+		(stroke
+			(width 0)
+			(type default)
+		)
+	)
+	(wire
+		(pts
+			(xy 116.84 71.12) (xy 121.92 71.12)
+		)
+		(stroke
+			(width 0)
+			(type default)
+		)
+	)
+	(wire
+		(pts
+			(xy 154.94 66.04) (xy 160.02 66.04)
+		)
+		(stroke
+			(width 0)
+			(type default)
+		)
+	)
 	(wire
 		(pts
@@
 	(wire
 		(pts
-			(xy 137.16 81.28) (xy 138.43 81.28)
-		)
-		(stroke
-			(width 0)
-			(type default)
-		)
-	)
-	(wire
-		(pts
-			(xy 215.9 85.09) (xy 224.79 85.09)
-		)
-		(stroke
-			(width 0)
-			(type default)
-		)
-	)
-	(wire
-		(pts
-			(xy 116.84 68.58) (xy 121.92 68.58)
-		)
-		(stroke
-			(width 0)
-			(type default)
-		)
-	)
-	(wire
-		(pts
-			(xy 223.52 52.07) (xy 215.9 52.07)
-		)
-		(stroke
-			(width 0)
-			(type default)
-		)
-	)
-	(wire
-		(pts
-			(xy 215.9 72.39) (xy 218.44 72.39)
-		)
-		(stroke
-			(width 0)
-			(type default)
-		)
-	)
-	(wire
-		(pts
-			(xy 215.9 69.85) (xy 218.44 69.85)
-		)
-		(stroke
-			(width 0)
-			(type default)
-		)
-	)
-	(wire
-		(pts
-			(xy 175.26 72.39) (xy 180.34 72.39)
-		)
-		(stroke
-			(width 0)
-			(type default)
-		)
-	)
-	(wire
-		(pts
-			(xy 137.16 77.47) (xy 137.16 81.28)
-		)
-		(stroke
-			(width 0)
-			(type default)
-		)
-	)
-	(wire
-		(pts
-			(xy 154.94 66.04) (xy 160.02 66.04)
-		)
-		(stroke
-			(width 0)
-			(type default)
-		)
-	)
-	(wire
-		(pts
 			(xy 116.84 63.5) (xy 121.92 63.5)
 		)
@@
 	(wire
 		(pts
+			(xy 154.94 55.88) (xy 160.02 55.88)
+		)
+		(stroke
+			(width 0)
+			(type default)
+		)
+	)
+	(wire
+		(pts
 			(xy 175.26 69.85) (xy 180.34 69.85)
 		)
@@
 		(pts
 			(xy 223.52 46.99) (xy 223.52 52.07)
+		)
+		(stroke
+			(width 0)
+			(type default)
+		)
+	)
+	(wire
+		(pts
+			(xy 154.94 53.34) (xy 160.02 53.34)
 		)
 		(stroke
@@
 	)
 	(label "RXD"
-		(at 160.02 55.88 0)
+		(at 160.02 53.34 0)
 		(fields_autoplaced yes)
 		(effects
@@
 	)
 	(label "IO13"
-		(at 160.02 60.96 0)
+		(at 160.02 58.42 0)
 		(fields_autoplaced yes)
 		(effects
@@
 	)
 	(label "TXD"
-		(at 160.02 58.42 0)
+		(at 160.02 55.88 0)
 		(fields_autoplaced yes)
 		(effects
@@
 	)
 	(label "IO10"
-		(at 160.02 53.34 0)
+		(at 116.84 68.58 0)
 		(fields_autoplaced yes)
 		(effects
@@
 	)
 	(label "IO19"
-		(at 170.18 46.99 0)
+		(at 160.02 60.96 0)
 		(fields_autoplaced yes)
 		(effects
@@
 	)
 	(label "IO9"
-		(at 116.84 68.58 0)
-		(fields_autoplaced yes)
-		(effects
+		(at 116.84 71.12 0)
+		(fields_autoplaced yes)
+		(effects

Commit message: .
Parts:
- added C1, C2, C3: 1uF, Capacitor_THT:CP_Radial_D4.0mm_P2.00mm, symbol Device:C_Polarized_Small
- added C4: 10uF, Capacitor_SMD:CP_Elec_3x5.3, symbol Device:C_Polarized_Small
- added C5: 0.1uF, Capacitor_SMD:CP_Elec_3x5.3, symbol Device:C_Polarized_Small
- added D1: D, Diode_SMD:D_1210_3225Metric, symbol Device:D
- added J1: PWR, Connector_PinSocket_2.54mm:PinSocket_1x02_P2.54mm_Vertical, symbol Connector:Conn_01x02_Socket
- added J2: USB-C_Receptacle_Data_16P_GCT-USB4085, Alexander Footprint Library:USB-C_GCT CONN16_USB4085-GF-A, symbol Alexander Symbol Library:USB-C_Receptacle_Data_16P_GCT-USB4085
- added R1, R2: 5k1, Resistor_SMD:R_1206_3216Metric_Pad1.30x1.75mm_HandSolder, symbol Device:R
- added TP1: VIN, TestPoint:TestPoint_Pad_D1.5mm, symbol Connector:TestPoint
- added TP2: GND, TestPoint:TestPoint_Pad_D1.5mm, symbol Connector:TestPoint
- added TP3: 3V3, TestPoint:TestPoint_Pad_D1.5mm, symbol Connector:TestPoint
- added TP4: 5V, TestPoint:TestPoint_Pad_D1.5mm, symbol Connector:TestPoint
- added U2: MAX1726EUK33, Package_TO_SOT_SMD:SOT-223-3_TabPin2, symbol Regulator_Linear:LM78M05_TO220
- added U3: L7805, Alexander Footprint Library:LD1117, symbol Regulator_Linear:L7805
Connections:
- net +3V3: now also C2.1, C4.1, C5.1, TP3.1, U2.3 (VO)
- net GND: now also C1.2, C2.2, C3.2, C4.2, C5.2, J1.1 (Pin_1), J2.A1 (GND), J2.A12 (GND), J2.B1 (GND), J2.B12 (GND), J2.S1 (SHIELD), J2.S2 (SHIELD), J2.S3 (SHIELD), J2.S4 (SHIELD), R1.1, R2.1, TP2.1, U2.2 (GND), U3.2 (GND)
- new net: J2.A5 (CC1), R2.2
- new net: J2.B5 (CC2), R1.2
- new net +5V: C3.1, TP4.1, U3.3 (OUT)
- new net USB_D+: J2.A6 (D+), J2.B6 (D+)
- new net USB_D-: J2.A7 (D-), J2.B7 (D-)
- new net VBUS: J2.A4 (VBUS), J2.A9 (VBUS), J2.B4 (VBUS), J2.B9 (VBUS)
- new net VDC: D1.2 (A), J1.2 (Pin_2)
- new net VIN: C1.1, D1.1 (K), TP1.1, U2.1 (VI), U3.1 (IN)
Other:
- note added: "Voltage Regulators"

Commit message: .
Parts:
- removed U2: MAX1726EUK33, Package_TO_SOT_SMD:SOT-223-3_TabPin2, symbol Regulator_Linear:LM78M05_TO220
- added U2: AMS1117-3V3, Alexander Footprint Library:AMS1117 SOT-223, symbol Alexander KiCad Libraries:AMS1117-3V3
Connections:
- net +3V3: now also U2.2 (VO)
- net GND: now also U2.1 (ADJ)
- net VIN: now also U2.3 (VI)
Changed lines of the file:
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@@
-	)
-	(symbol
-		(lib_id "Regulator_Linear:LM78M05_TO220")
-		(at 64.77 100.33 0)
-		(unit 1)
-		(exclude_from_sim no)
-		(in_bom yes)
-		(on_board yes)
-		(dnp no)
-		(property "Reference" "U2"
-			(at 64.77 93.98 0)
-			(effects
-				(font
-					(size 1.27 1.27)
-				)
-			)
-		)
-		(property "Value" "MAX1726EUK33"
-			(at 64.77 96.52 0)
-			(effects
-				(font
-					(size 1.27 1.27)
-				)
-			)
-		)
-		(property "Footprint" "Package_TO_SOT_SMD:SOT-223-3_TabPin2"
-			(at 64.77 94.615 0)
-			(effects
-				(font
-					(size 1.27 1.27)
-					(italic yes)
-				)
-				(hide yes)
-			)
-		)
-		(property "Datasheet" "https://www.onsemi.com/pub/Collateral/MC78M00-D.PDF"
-			(at 64.77 101.6 0)
-			(effects
-				(font
-					(size 1.27 1.27)
-				)
-				(hide yes)
-			)
-		)
-		(property "Description" ""
-			(at 64.77 100.33 0)
-			(effects
-				(font
-					(size 1.27 1.27)
-				)
-				(hide yes)
-			)
-		)
-		(pin "1"
-		)
-		(pin "2"
-		)
-		(pin "3"
-		)
-		(instances
-			(project "ESP32-C3-BreadBoardAdapter"
-				(path "/7ebe7346-feca-4308-bb7e-1ef2e739e742"
-					(reference "U2")
-					(unit 1)
-				)
-			)
-		)
 	)
 	(symbol
@@
 					(unit 1)
 				)
+			)
+		)
+	)
+	(symbol
+		(lib_id "Alexander KiCad Libraries:AMS1117-3V3")
+		(at 64.77 96.52 0)
+		(unit 1)
+		(exclude_from_sim yes)
+		(in_bom yes)
+		(on_board yes)
+		(dnp no)
+		(fields_autoplaced yes)
+		(property "Reference" "U2"
+			(at 64.77 93.98 0)
+			(effects
+				(font
+					(size 1.27 1.27)
+				)
+			)
+		)
+		(property "Value" "AMS1117-3V3"
+			(at 64.77 96.52 0)
+			(effects
+				(font
+					(size 1.27 1.27)
+				)
+			)
+		)
+		(property "Footprint" "Alexander Footprint Library:AMS1117 SOT-223"
+			(at 64.77 92.202 0)
+			(effects
+				(font
+					(size 1.27 1.27)
+				)
+				(hide yes)
+			)
+		)
+		(property "Datasheet" ""
+			(at 64.77 96.52 0)
+			(effects
+				(font
+					(size 1.27 1.27)
+				)
+				(hide yes)
+			)
+		)
+		(property "Description" "AMS1117"
+			(at 64.77 92.71 0)
+			(effects
+				(font
+					(size 1.27 1.27)
+				)
+				(hide yes)
+			)
+		)
+		(pin "2"
+		)
+		(pin "1"
+		)
+		(pin "3"
+		)
+		(instances
+			(project ""
+				(path "/7ebe7346-feca-4308-bb7e-1ef2e739e742"
+					(reference "U2")
+					(unit 1)
+				)

Commit message: .
Parts:
- removed C2: 1uF, Capacitor_THT:CP_Radial_D4.0mm_P2.00mm, symbol Device:C_Polarized_Small
Connections:
- net GNDD is gone; now on net GND: BRD1.G1 (GND1), BRD1.G2 (GND2), U1.19 (GND__1), U1.20 (GND__2), U1.21 (GND__3), U1.22 (GND__4), U1.23 (GND__5), U1.24 (GND__6), U1.25 (GND__7), U1.26 (GND__8), U1.27 (GND__9), U1.28 (GND__10), U1.29 (GND__11), U1.30 (GND__12), U1.31 (GND__13), U1.32 (GND__14), U1.33 (GND__15), U1.34 (GND__16), U1.35 (GND__17), U1.36 (GND__18), U1.37 (GND__19), U1.38 (GND__20), U1.39 (GND__21), U1.9 (GND)
- net VBUS: now also C1.1, TP1.1, U2.3 (VI), U3.1 (IN)
- removed net VIN: C1.1, D1.1 (K), TP1.1, U2.3 (VI), U3.1 (IN)

Commit message: .
Connections:
- net IO13 is gone; now on net USB_D-: BRD1.11 (B3), U1.13 (IO18)
- net IO19 is gone; now on net USB_D+: BRD1.12 (B4), U1.14 (IO19)
Changed lines of the file:
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@@
 	(wire
 		(pts
-			(xy 215.9 72.39) (xy 218.44 72.39)
-		)
-		(stroke
-			(width 0)
-			(type default)
-		)
-	)
-	(wire
-		(pts
-			(xy 215.9 69.85) (xy 218.44 69.85)
+			(xy 215.9 72.39) (xy 228.6 72.39)
+		)
+		(stroke
+			(width 0)
+			(type default)
+		)
+	)
+	(wire
+		(pts
+			(xy 215.9 69.85) (xy 228.6 69.85)
 		)
 		(stroke
@@
 		)
 	)
-	(label "IO13"
+	(label "IO18"
 		(at 160.02 58.42 0)
 		(fields_autoplaced yes)
@@
 		)
 	)
-	(label "IO13"
+	(label "IO18"
 		(at 218.44 69.85 0)
 		(fields_autoplaced yes)
@@
 			)
 			(justify left bottom)
+		)
+	)
+	(global_label "USB_D+"
+		(shape input)
+		(at 228.6 72.39 0)
+		(fields_autoplaced yes)
+		(effects
+			(font
+				(size 1.27 1.27)
+			)
+			(justify left)
+		)
+		(property "Intersheetrefs" "${INTERSHEET_REFS}"
+			(at 239.2052 72.39 0)
+			(effects
+				(font
+					(size 1.27 1.27)
+				)
+				(justify left)
+				(hide yes)
+			)
 		)
 	)
@@
 			(effects
 				(font
+					(size 1.27 1.27)
+				)
+				(justify left)
+				(hide yes)
+			)
+		)
+	)
+	(global_label "USB_D-"
+		(shape input)
+		(at 228.6 69.85 0)
+		(fields_autoplaced yes)
+		(effects
+			(font
+				(size 1.27 1.27)
+			)
+			(justify left)
+		)
+		(property "Intersheetrefs" "${INTERSHEET_REFS}"
+			(at 239.2052 69.85 0)
+			(effects
+				(font

Commit message: .
Parts:
- U3: footprint Alexander Footprint Library:LD1117 -> Package_TO_SOT_SMD:TO-252-2
Connections:
- net IO0: now also BRD1.16 (B8); no longer BRD1.15 (B7)
- net IO1: now also BRD1.15 (B7); no longer BRD1.16 (B8)
- net IO2: now also BRD1.14 (B6); no longer BRD1.13 (B5)
- net IO3: now also BRD1.13 (B5); no longer BRD1.14 (B6)
- net RXD: now also BRD1.10 (B2); no longer BRD1.9 (B1)
- net TXD: now also BRD1.12 (B4); no longer BRD1.10 (B2)
- net USB_D+: now also BRD1.9 (B1); no longer BRD1.12 (B4)
Changed lines of the file:
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@@
 	(wire
 		(pts
-			(xy 154.94 66.04) (xy 160.02 66.04)
-		)
-		(stroke
-			(width 0)
-			(type default)
-		)
-	)
-	(wire
-		(pts
 			(xy 57.15 120.65) (xy 54.61 120.65)
 		)
@@
 	(wire
 		(pts
-			(xy 154.94 60.96) (xy 160.02 60.96)
+			(xy 44.45 100.33) (xy 44.45 102.87)
 		)
 		(stroke
@@
 	(wire
 		(pts
-			(xy 44.45 100.33) (xy 44.45 102.87)
+			(xy 116.84 63.5) (xy 121.92 63.5)
 		)
 		(stroke
@@
 	(wire
 		(pts
-			(xy 116.84 63.5) (xy 121.92 63.5)
+			(xy 60.96 49.53) (xy 62.23 49.53)
 		)
 		(stroke
@@
 	(wire
 		(pts
-			(xy 154.94 55.88) (xy 160.02 55.88)
+			(xy 175.26 69.85) (xy 180.34 69.85)
 		)
 		(stroke
@@
 	(wire
 		(pts
-			(xy 60.96 49.53) (xy 62.23 49.53)
+			(xy 29.21 110.49) (xy 44.45 110.49)
 		)
 		(stroke
@@
 	(wire
 		(pts
-			(xy 175.26 69.85) (xy 180.34 69.85)
+			(xy 78.74 100.33) (xy 90.17 100.33)
 		)
 		(stroke
@@
 	(wire
 		(pts
-			(xy 29.21 110.49) (xy 44.45 110.49)
+			(xy 102.87 110.49) (xy 109.22 110.49)
 		)
 		(stroke
@@
 	(wire
 		(pts
-			(xy 78.74 100.33) (xy 90.17 100.33)
+			(xy 83.82 46.99) (xy 83.82 49.53)
 		)
 		(stroke
@@
 	(wire
 		(pts
-			(xy 102.87 110.49) (xy 109.22 110.49)
+			(xy 116.84 60.96) (xy 121.92 60.96)
 		)
 		(stroke
@@
 	(wire
 		(pts
-			(xy 83.82 46.99) (xy 83.82 49.53)
+			(xy 76.2 46.99) (xy 76.2 49.53)
 		)
 		(stroke
@@
 	(wire
 		(pts
-			(xy 116.84 60.96) (xy 121.92 60.96)
+			(xy 154.94 53.34) (xy 160.02 53.34)
 		)
 		(stroke
@@
 	(wire
 		(pts
-			(xy 76.2 46.99) (xy 76.2 49.53)
+			(xy 154.94 68.58) (xy 160.02 68.58)
 		)
 		(stroke
@@
 	(wire
 		(pts
+			(xy 154.94 60.96) (xy 160.02 60.96)
+		)
+		(stroke
+			(width 0)
+			(type default)
+		)
+	)
+	(wire
+		(pts
 			(xy 54.61 100.33) (xy 54.61 120.65)
 		)
@@
 	(wire
 		(pts
-			(xy 154.94 71.12) (xy 160.02 71.12)
+			(xy 102.87 107.95) (xy 102.87 110.49)
 		)
 		(stroke
@@
 	(wire
 		(pts
-			(xy 102.87 107.95) (xy 102.87 110.49)
+			(xy 132.08 77.47) (xy 132.08 81.28)
 		)
 		(stroke
@@
 	(wire
 		(pts
-			(xy 132.08 77.47) (xy 132.08 81.28)
+			(xy 154.94 55.88) (xy 160.02 55.88)
 		)
 		(stroke
@@
 	(wire
 		(pts
-			(xy 139.7 81.28) (xy 138.43 81.28)
+			(xy 154.94 71.12) (xy 160.02 71.12)
 		)
 		(stroke
@@
 	(wire
 		(pts
-			(xy 116.84 66.04) (xy 121.92 66.04)
+			(xy 139.7 81.28) (xy 138.43 81.28)
 		)
 		(stroke
@@
 	(wire
 		(pts
-			(xy 44.45 97.79) (xy 44.45 100.33)
+			(xy 116.84 66.04) (xy 121.92 66.04)
 		)
 		(stroke
@@
 	(wire
 		(pts
-			(xy 78.74 110.49) (xy 78.74 113.03)
+			(xy 44.45 97.79) (xy 44.45 100.33)
 		)
 		(stroke
@@
 	(wire
 		(pts
-			(xy 154.94 68.58) (xy 160.02 68.58)
+			(xy 78.74 110.49) (xy 78.74 113.03)
 		)
 		(stroke
@@
 	(wire
 		(pts
+			(xy 154.94 66.04) (xy 160.02 66.04)
+		)
+		(stroke
+			(width 0)
+			(type default)
+		)
+	)
+	(wire
+		(pts
 			(xy 59.69 36.83) (xy 76.2 36.83)
 		)
@@
 	(wire
 		(pts
-			(xy 154.94 53.34) (xy 160.02 53.34)
-		)
-		(stroke
-			(width 0)
-			(type default)
-		)
-	)
-	(wire
-		(pts
 			(xy 78.74 120.65) (xy 85.09 120.65)
 		)
@@
 	(wire
 		(pts
-			(xy 116.84 58.42) (xy 121.92 58.42)
+			(xy 154.94 63.5) (xy 160.02 63.5)
 		)
 		(stroke
@@
 	(wire
 		(pts
-			(xy 59.69 44.45) (xy 60.96 44.45)
+			(xy 116.84 58.42) (xy 121.92 58.42)
 		)
 		(stroke
@@
 	(wire
 		(pts
-			(xy 116.84 55.88) (xy 121.92 55.88)
+			(xy 59.69 44.45) (xy 60.96 44.45)
 		)
 		(stroke
@@
 	(wire
 		(pts
-			(xy 59.69 49.53) (xy 60.96 49.53)
+			(xy 116.84 55.88) (xy 121.92 55.88)
 		)
 		(stroke
@@
 	(wire
 		(pts
-			(xy 215.9 64.77) (xy 218.44 64.77)
+			(xy 59.69 49.53) (xy 60.96 49.53)
 		)
 		(stroke
@@
 	(wire
 		(pts
-			(xy 83.82 34.29) (xy 83.82 39.37)
+			(xy 215.9 64.77) (xy 218.44 64.77)
 		)
 		(stroke
@@
 	(wire
 		(pts
-			(xy 154.94 63.5) (xy 160.02 63.5)
+			(xy 83.82 34.29) (xy 83.82 39.37)
 		)
 		(stroke
@@
 	)
 	(label "RXD"
-		(at 160.02 53.34 0)
+		(at 160.02 55.88 0)
 		(fields_autoplaced yes)
 		(effects
@@
 	)
 	(label "IO2"
-		(at 160.02 63.5 0)
+		(at 160.02 66.04 0)
 		(fields_autoplaced yes)
 		(effects
@@
 	)
 	(label "IO1"
-		(at 160.02 71.12 0)
+		(at 160.02 68.58 0)
 		(fields_autoplaced yes)
 		(effects
@@
 	)
 	(label "TXD"
-		(at 160.02 55.88 0)
+		(at 160.02 60.96 0)
 		(fields_autoplaced yes)
 		(effects
@@
 	)
 	(label "IO3"
-		(at 160.02 66.04 0)
+		(at 160.02 63.5 0)
 		(fields_autoplaced yes)
 		(effects
@@
 	)
 	(label "IO0"
-		(at 160.02 68.58 0)
+		(at 160.02 71.12 0)
 		(fields_autoplaced yes)
 		(effects
@@
 	)
 	(label "IO19"
-		(at 160.02 60.96 0)
+		(at 160.02 53.34 0)
 		(fields_autoplaced yes)
 		(effects
@@
 			)
 		)
-		(property "Footprint" "Alexander Footprint Library:LD1117"
+		(property "Footprint" "Package_TO_SOT_SMD:TO-252-2"
 			(at 65.405 124.46 0)
 			(effects
