File: ESP32-C3-BreadBoardAdapter/ESP32-C3-BreadBoardAdapter/ESP32-C3-BreadBoardAdapter.kicad_pcb (KiCad board)
At the start: 2 copper layers, 50.8 x 39.4 mm, 17 parts, among them J1 PWR, J2 USB-C_Receptacle_Data_16P_GCT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, J3 PWR_JMP, J4 PWR_JMP, U1 ESP32-C3-WROOM-02-N4, U2 AMS1117-3V3, U3 L7805

Commit message: .
Parts:
- added R3: 10k, Resistor_SMD:R_1206_3216Metric_Pad1.30x1.75mm_HandSolder, F.Cu at (122.3, 68.4)
- added SW1: SW_Push, Alexander Footprint Library:SW_SPST_6x3, F.Cu at (121.1, 78.0)
- moved C3 39.1 mm to (175.5, 78.8), turned to 180 degrees
Connections:
- net +3V3 renamed 3V3
- net /EN renamed EN
Routing:
- net EN: track 34.9 -> 44.5 mm
- net 3V3: track 81.6 -> 83.7 mm, vias 1 -> 2

Commit message: .
Parts:
- removed R3: 10k, Resistor_SMD:R_1206_3216Metric_Pad1.30x1.75mm_HandSolder
- removed SW1: SW_Push, Alexander Footprint Library:SW_SPST_6x3
- added R4: 10k, Resistor_SMD:R_1206_3216Metric_Pad1.30x1.75mm_HandSolder, F.Cu at (122.1, 69.0)
- added R5: 2K2, Resistor_SMD:R_1206_3216Metric_Pad1.30x1.75mm_HandSolder, F.Cu at (135.7, 73.8)
- added R6: 2K2, Resistor_SMD:R_1206_3216Metric_Pad1.30x1.75mm_HandSolder, F.Cu at (137.0, 66.0)
- added SW2: SW_Push_SMD_6x3.5, Alexander Footprint Library:SW_PUSH_6x3.5mm, F.Cu at (130.6, 79.4)
- added SW3: SW_Push_SMD_6x3.5, Alexander Footprint Library:SW_PUSH_6x3.5mm, F.Cu at (124.2, 73.8)
Routing:
- net EN: track 44.5 -> 38.1 mm

Commit message: .
Parts:
- moved SW3 6.33 mm to (130.5, 74.4), turned to 180 degrees
- moved TP2 1.61 mm to (114.5, 64.2)
- moved R5 0.63 mm to (135.5, 74.4)
Connections:
- R5 pad 2: /GPIO9 -> /IO9
- R6 pad 2: /GPIO8 -> /IO8
- SW3 pad 1: GND -> /IO9
- SW3 pad 2: /GPIO9 -> GND
Routing:
- net /IO9: track 31.4 -> 43.5 mm
- net VBUS: track 64.7 -> 74.1 mm, vias 0 -> 1
- net /VDC: track 0.00 -> 4.80 mm
Changed lines of the file:
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@@
 	(net 26 "unconnected-(J2-SBU1-PadA8)")
 	(net 27 "/VCC2")
-	(net 28 "/GPIO9")
-	(net 29 "/GPIO8")
 	(footprint "Resistor_SMD:R_1206_3216Metric_Pad1.30x1.75mm_HandSolder"
 		(layer "F.Cu")
-		(at 135.74 73.8 180)
+		(at 135.54 74.4 180)
 		(descr "Resistor SMD 1206 (3216 Metric), square (rectangular) end terminal, IPC_7351 nominal with elongated pad for handsoldering. (Body size source: IPC-SM-782 page 72, https://www.pcb-3d.com/wordpress/wp-content/uploads/ipc-sm-782a_amendment_1_and_2.pdf), generated with kicad-footprint-generator")
 		(tags "resistor handsolder")
@@
 			(layers "F.Cu" "F.Paste" "F.Mask")
 			(roundrect_rratio 0.192308)
-			(net 28 "/GPIO9")
+			(net 8 "/IO9")
 			(pintype "passive")
 		)
@@
 	(footprint "TestPoint:TestPoint_Pad_D1.5mm"
 		(layer "F.Cu")
-		(at 115.8 65.2)
+		(at 114.54 64.2)
 		(descr "SMD pad as test Point, diameter 1.5mm")
 		(tags "test point SMD pad")
@@
 			(layers "F.Cu" "F.Paste" "F.Mask")
 			(roundrect_rratio 0.192308)
-			(net 29 "/GPIO8")
+			(net 7 "/IO8")
 			(pintype "passive")
 		)
@@
 	(footprint "Alexander Footprint Library:SW_PUSH_6x3.5mm"
 		(layer "F.Cu")
-		(at 124.24 73.8)
+		(at 130.54 74.4 180)
 		(descr "tactile push button, 6x3.5mm, https://www.apem.com/idec-apem/en_US/PCB-switches/Tactile-Switches/MJTP-6mm-through-hole/c/MJTP_6mm_through%20hole?page=1")
 		(tags "PHAP3362 6mm tact sw THT")
@@
 		)
 		(property "Footprint" "Alexander Footprint Library:SW_PUSH_6x3.5mm"
-			(at 0 0 0)
+			(at 0 0 180)
 			(unlocked yes)
 			(layer "F.Fab")
@@
 		)
 		(property "Datasheet" ""
-			(at 0 0 0)
+			(at 0 0 180)
 			(unlocked yes)
 			(layer "F.Fab")
@@
 		)
 		(property "Description" ""
-			(at 0 0 0)
+			(at 0 0 180)
 			(unlocked yes)
 			(layer "F.Fab")
@@
 		(attr through_hole)
 		(fp_line
-			(start 0.15 -1.85)
-			(end 0.15 -1.39)
+			(start 6.35 1.39)
+			(end 6.35 1.85)
 			(stroke
 				(width 0.12)
-				(type default)
+				(type solid)
 			)
 			(layer "F.SilkS")
 		)
 		(fp_line
-			(start 0.15 -1.39)
-			(end -0.85 -1.39)
+			(start 6.35 -1.85)
+			(end 6.35 -1.39)
 			(stroke
 				(width 0.12)
-				(type default)
+				(type solid)
 			)
 			(layer "F.SilkS")
 		)
 		(fp_line
-			(start 0.15 1.39)
-			(end 0.15 1.85)
+			(start 6.35 -1.85)
+			(end 0.15 -1.85)
 			(stroke
 				(width 0.12)
@@
 		)
 		(fp_line
-			(start 6.35 -1.85)
-			(end 0.15 -1.85)
+			(start 0.15 1.39)
+			(end 0.15 1.85)
 			(stroke
 				(width 0.12)
@@
 		)
 		(fp_line
-			(start 6.35 -1.85)
-			(end 6.35 -1.39)
+			(start 0.15 -1.39)
+			(end -0.85 -1.39)
 			(stroke
 				(width 0.12)
-				(type solid)
+				(type default)
 			)
 			(layer "F.SilkS")
 		)
 		(fp_line
-			(start 6.35 1.39)
-			(end 6.35 1.85)
+			(start 0.15 -1.85)
+			(end 0.15 -1.39)
 			(stroke
 				(width 0.12)
-				(type solid)
+				(type default)
 			)
 			(layer "F.SilkS")
@@
 		)
 		(fp_line
-			(start -1.38 -1.38)
-			(end 0 -1.38)
+			(start 6.5 2)
+			(end 0 2)
 			(stroke
 				(width 0.05)
-				(type default)
+				(type solid)
 			)
 			(layer "F.CrtYd")
 		)
 		(fp_line
-			(start -1.38 1.38)
-			(end -1.38 -1.38)
+			(start 6.5 1.38)
+			(end 6.5 2)
 			(stroke
 				(width 0.05)
-				(type solid)
+				(type default)
 			)
 			(layer "F.CrtYd")
 		)
 		(fp_line
-			(start -1.38 1.38)
-			(end 0 1.38)
+			(start 6.5 -2)
+			(end 6.5 -1.38)
 			(stroke
 				(width 0.05)
@@
 		)
 		(fp_line
-			(start 0 -2)
-			(end 0 -1.38)
+			(start 0 1.38)
+			(end 0 2)
 			(stroke
 				(width 0.05)
@@
 		)
 		(fp_line
-			(start 0 1.38)
-			(end 0 2)
+			(start 0 -2)
+			(end 0 -1.38)
 			(stroke
 				(width 0.05)
@@
 		)
 		(fp_line
-			(start 6.5 -2)
-			(end 6.5 -1.38)
+			(start -1.38 1.38)
+			(end 0 1.38)
 			(stroke
 				(width 0.05)
@@
 		)
 		(fp_line
-			(start 6.5 1.38)
-			(end 6.5 2)
+			(start -1.38 1.38)
+			(end -1.38 -1.38)
 			(stroke
 				(width 0.05)
-				(type default)
+				(type solid)
 			)
 			(layer "F.CrtYd")
 		)
 		(fp_line
-			(start 6.5 2)
-			(end 0 2)
+			(start -1.38 -1.38)
+			(end 0 -1.38)
 			(stroke
 				(width 0.05)
-				(type solid)
+				(type default)
 			)
 			(layer "F.CrtYd")
@@
 		)
 		(fp_line
-			(start 0.25 1.75)
-			(end 0.25 -1.35)
+			(start 6.25 1.75)
+			(end 0.25 1.75)
 			(stroke
 				(width 0.1)
@@
 		)
 		(fp_line
-			(start 0.65 -1.75)
-			(end 0.25 -1.35)
+			(start 6.25 -1.75)
+			(end 6.25 1.75)
 			(stroke
 				(width 0.1)
-				(type default)
+				(type solid)
 			)
 			(layer "F.Fab")
@@
 		)
 		(fp_line
-			(start 6.25 -1.75)
-			(end 6.25 1.75)
+			(start 0.65 -1.75)
+			(end 0.25 -1.35)
 			(stroke
 				(width 0.1)
-				(type solid)
+				(type default)
 			)
 			(layer "F.Fab")
 		)
 		(fp_line
-			(start 6.25 1.75)
-			(end 0.25 1.75)
+			(start 0.25 1.75)
+			(end 0.25 -1.35)
 			(stroke
 				(width 0.1)
@@
 		)
 		(pad "1" smd rect
-			(at 0 0 90)
+			(at 0 0 270)
 			(size 2.25 2.25)
 			(layers "F.Cu" "F.Paste" "F.Mask")
-			(net 2 "GND")
+			(net 8 "/IO9")
 			(pinfunction "1")
 			(pintype "passive")
 		)
 		(pad "2" smd oval
-			(at 6.5 0 90)
+			(at 6.5 0 270)
 			(size 2.25 2.25)
 			(layers "F.Cu" "F.Paste" "F.Mask")
-			(net 28 "/GPIO9")
+			(net 2 "GND")
 			(pinfunction "2")
 			(pintype "passive")
@@
 	)
 	(segment
+		(start 115.6 76.6)
+		(end 115.6 71.8)
+		(width 0.5)
+		(layer "F.Cu")
+		(net 4)
+	)
+	(segment
 		(start 160.164445 67.585555)
 		(end 160.25 67.5)
@@
 	)
 	(segment
+		(start 130.54 74.4)
+		(end 133.99 74.4)
+		(width 0.2)
+		(layer "F.Cu")
+		(net 8)
+	)
+	(segment
+		(start 133.99 69.05)
+		(end 133.99 74.4)
+		(width 0.2)
+		(layer "F.Cu")
+		(net 8)
+	)
+	(segment
 		(start 128.5 87.437256)
 		(end 130.962744 89.9)
@@
 	)
 	(segment
+		(start 133.54 68.6)
+		(end 133.99 69.05)
+		(width 0.2)
+		(layer "F.Cu")
+		(net 8)
+	)
+	(segment
+		(start 130.89 68.6)
+		(end 133.54 68.6)
+		(width 0.2)
+		(layer "F.Cu")
+		(net 8)
+	)
+	(segment
 		(start 134 90.6)
 		(end 134 92.4)
@@
 	)
 	(segment
+		(start 115.6 65.94)
+		(end 115.6 69)
+		(width 0.5)
+		(layer "F.Cu")
+		(net 23)
+	)
+	(segment
 		(start 155.582435 66.735557)
 		(end 156.932435 66.735557)
@@
 		(net 23)
 	)
+	(via
+		(at 115.6 65.94)
+		(size 0.6)
+		(drill 0.3)
+		(layers "F.Cu" "B.Cu")
+		(net 23)
+	)
 	(segment
 		(start 153 59.25)
@@
 	)
 	(segment
+		(start 117.09 64.45)
+		(end 121.35 64.45)
+		(width 0.5)
+		(layer "B.Cu")
+		(net 23)
+	)
+	(segment
 		(start 121.35 59.4)
 		(end 121.35 64.45)
@@
 		(width 0.5)
 		(layer "B.Cu")
+		(net 23)
+	)
+	(segment
+		(start 115.6 65.94)
+		(end 117.09 64.45)
+		(width 0.5)
+		(layer "B.Cu")

Commit message: .
Parts:
- added LED1: LED-RED-GREEN-B1552USUG20D, Alexander Footprint Library:LED_B1552_HVK-M, F.Cu at (136.1, 81.8)
- added LED2: LED-RED-GREEN-B1552USUG20D, Alexander Footprint Library:LED_B1552_HVK-M, F.Cu at (120.0, 75.2)
- added R3: 5k1, Resistor_SMD:R_1206_3216Metric_Pad1.30x1.75mm_HandSolder, F.Cu at (137.7, 75.2)
- added R7: 5k1, Resistor_SMD:R_1206_3216Metric_Pad1.30x1.75mm_HandSolder, F.Cu at (134.5, 75.2)
- added R8: 2K2, Resistor_SMD:R_1206_3216Metric_Pad1.30x1.75mm_HandSolder, F.Cu at (143.7, 75.2)
- added SW1: SW_Push_SMD_6x3.5, Alexander Footprint Library:SW_PUSH_6x3.5mm, F.Cu at (143.7, 80.2)
- R5, R6: moved to B.Cu
- moved C3 55.1 mm to (120.5, 82.6)
- moved R5 12.1 mm to (136.7, 62.4), turned to -90 degrees
- moved R6 4.85 mm to (133.7, 62.4)
Connections:
- R4 pad 2: EN -> Net-(LED2-GRN)
- SW2 pad 2: EN -> Net-(LED2-GRN)
Routing:
- net Net-(LED2-GRN): track 0.00 -> 18.0 mm
- net /IO3: track 32.1 -> 45.8 mm
- net 3V3: track 83.9 -> 97.2 mm, vias 2 -> 4
- net /IO10: track 32.3 -> 41.9 mm
- net /IO8: track 29.2 -> 34.9 mm, vias 0 -> 1
- net Net-(LED1-GND-Pad4): track 0.00 -> 4.30 mm
- net Net-(LED1-GND-Pad1): track 0.00 -> 4.30 mm
- net +5V: track 52.3 -> 56.2 mm
- net Net-(R8-Pad2): track 0.00 -> 3.40 mm
- net EN: track 38.1 -> 40.6 mm
- net /IO9: track 43.5 -> 43.7 mm, vias 0 -> 1

Commit message: .
Parts:
- removed TP2: GND, TestPoint:TestPoint_Pad_D1.5mm
- added J5: Debug_GND, Connector_PinHeader_2.54mm:PinHeader_1x02_P2.54mm_Vertical, F.Cu at (115.4, 65.0)
- added J6: Debug_3V3, Connector_PinHeader_2.54mm:PinHeader_1x02_P2.54mm_Vertical, F.Cu at (105.6, 76.3)
- D1: moved to B.Cu
- moved D1 1.51 mm to (115.4, 71.9)
- turned R4 to 180 degrees
Routing:
- net VBUS: track 74.1 -> 64.7 mm, vias 1 -> 0
- net /VDC: track 4.80 -> 0.00 mm
- net 3V3: track 97.2 -> 99.3 mm, vias 4 -> 3

Commit message: .
Parts:
- added TP2: GND, TestPoint:TestPoint_Pad_D1.5mm, F.Cu at (100.0, 74.8)
- J5, J6: footprint Connector_PinHeader_2.54mm:PinHeader_1x02_P2.54mm_Vertical -> Alexander Footprint Library:Conn_Debug_1x02_P2.54mm
- moved TP3 24.6 mm to (102.3, 59.0)
- moved J6 13.4 mm to (117.4, 69.8), turned to -90 degrees
- moved D1 7.94 mm to (120.1, 78.3)
- moved C4 3.31 mm to (125.4, 61.1), turned to -90 degrees
- moved C5 3.22 mm to (121.1, 61.1), turned to -90 degrees
- moved U2 3.20 mm to (126.4, 64.2), turned to 90 degrees
- moved J1 2.02 mm to (115.4, 77.1), turned to 0 degrees
- moved R4 1.74 mm to (123.2, 67.7), turned to -90 degrees
- moved C1 1.14 mm to (154.1, 60.1)
- moved J5 0.65 mm to (114.9, 64.7), turned to 90 degrees
Routing:
- net VBUS: track 64.7 -> 83.2 mm, vias 0 -> 1
- net 3V3: track 99.3 -> 107.1 mm
- net /VDC: track 0.00 -> 4.71 mm
- net /TXD: track 33.3 -> 32.5 mm
- net /RXD: track 33.0 -> 32.3 mm

Commit message: .
Routing:
- net VBUS: track 83.2 -> 90.0 mm, vias 1 -> 2
Changed lines of the file:
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@@
-	)
-	(segment
-		(start 153.64 63.8)
-		(end 152.64 62.8)
-		(width 0.5)
-		(layer "F.Cu")
-		(net 23)
 	)
 	(segment
@@
 	)
 	(segment
-		(start 154.514444 70.985556)
-		(end 152.7 72.8)
-		(width 0.5)
-		(layer "F.Cu")
-		(net 23)
-	)
-	(segment
-		(start 155.582435 66.735557)
-		(end 154.275557 66.735557)
-		(width 0.5)
-		(layer "F.Cu")
-		(net 23)
-	)
-	(segment
-		(start 155.582435 70.985556)
-		(end 154.514444 70.985556)
-		(width 0.5)
-		(layer "F.Cu")
-		(net 23)
-	)
-	(segment
 		(start 158.235557 66.735557)
 		(end 158.5 67)
-		(width 0.5)
-		(layer "F.Cu")
-		(net 23)
-	)
-	(segment
-		(start 152.64 62.8)
-		(end 152.64 60.1)
 		(width 0.5)
 		(layer "F.Cu")
@@
 	)
 	(segment
-		(start 152.7 72.8)
-		(end 152.7 76.6225)
-		(width 0.5)
-		(layer "F.Cu")
-		(net 23)
-	)
-	(segment
 		(start 155.582435 66.735557)
 		(end 156.932435 66.735557)
@@
 	)
 	(segment
-		(start 153.64 66.1)
-		(end 153.64 63.8)
-		(width 0.5)
-		(layer "F.Cu")
-		(net 23)
-	)
-	(segment
-		(start 154.275557 66.735557)
-		(end 153.64 66.1)
+		(start 152.7 74.56)
+		(end 152.34 74.2)
 		(width 0.5)
 		(layer "F.Cu")
@@
 		(net 23)
 	)
+	(segment
+		(start 152.7 76.6225)
+		(end 152.7 74.56)
+		(width 0.5)
+		(layer "F.Cu")
+		(net 23)
+	)
+	(via
+		(at 152.34 74.2)
+		(size 0.6)
+		(drill 0.3)
+		(layers "F.Cu" "B.Cu")
+		(net 23)
+	)
 	(via
 		(at 151.75 58)
@@
 	)
 	(segment
+		(start 152.34 74.2)
+		(end 148.94 74.2)
+		(width 0.5)
+		(layer "B.Cu")
+		(net 23)
+	)
+	(segment
 		(start 120.14 68.5)
 		(end 121.29 67.35)
+		(width 0.5)
+		(layer "B.Cu")
+		(net 23)
+	)
+	(segment
+		(start 147.94 73.2)
+		(end 147.94 58.7)
+		(width 0.5)
+		(layer "B.Cu")
+		(net 23)
+	)
+	(segment
+		(start 147.94 58.7)
+		(end 147.24 58)
+		(width 0.5)
+		(layer "B.Cu")
+		(net 23)
+	)
+	(segment
+		(start 151.75 58)
+		(end 148.14 58)
+		(width 0.5)
+		(layer "B.Cu")
+		(net 23)
+	)
+	(segment
+		(start 148.94 74.2)
+		(end 147.94 73.2)
 		(width 0.5)
 		(layer "B.Cu")
@@
 	)
 	(segment
-		(start 151.75 58)
+		(start 148.14 58)
 		(end 122.75 58)
 		(width 0.5)

Commit message: .
Parts:
- removed TP2: GND, TestPoint:TestPoint_Pad_D1.5mm
- removed TP3: 3V3, TestPoint:TestPoint_Pad_D1.5mm
- added D2: D, Diode_SMD:D_1210_3225Metric, B.Cu at (152.3, 61.1)
Connections:
- C1 pad 1: VBUS -> Net-(D1-K)
- D1 pad 1: VBUS -> Net-(D1-K)
- J2 pad A4: VBUS -> VUSB
- J2 pad A9: VBUS -> VUSB
- J2 pad B4: VBUS -> VUSB
- J2 pad B9: VBUS -> VUSB
- U2 pad 3: VBUS -> Net-(D1-K)
- U3 pad 1: VBUS -> Net-(D1-K)
Routing:
- net VBUS: track 90.0 -> 0.00 mm, vias 2 -> 0
- net Net-(D1-K): track 0.00 -> 84.0 mm, vias 0 -> 2
- net VUSB: track 0.00 -> 16.5 mm
