File: ESP32-C3-BreadBoardAdapter/ESP32-C3-BreadBoardAdapter/usb-c_interface.kicad_sch (KiCad schematic)
At the start: 4 parts, among them J2 USB-C_Receptacle_Data_16P_GCT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

Commit message: .
Changed lines of the file:
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@@
 		)
 	)
-	(global_label "VUSB"
-		(shape passive)
-		(at 88.9 45.72 0)
+	(hierarchical_label "USB_D-"
+		(shape output)
+		(at 76.2 58.42 0)
 		(fields_autoplaced yes)
 		(effects
@@
 			(justify left)
 		)
-		(property "Intersheetrefs" "${INTERSHEET_REFS}"
-			(at 95.6725 45.72 0)
-			(effects
-				(font
-					(size 1.27 1.27)
-				)
-				(justify left)
-				(hide yes)
-			)
-		)
 	)
-	(hierarchical_label "USB_D-"
-		(shape output)
-		(at 76.2 58.42 0)
+	(hierarchical_label "VUSB"
+		(shape passive)
+		(at 88.9 45.72 0)
 		(fields_autoplaced yes)
 		(effects

Commit message: ,
Connections:
- net VUSB renamed VUSB_OUT
Other:
- title: (none) -> ESP32-C3 Breadboard Adapter.
Changed lines of the file:
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@@
 	(generator_version "8.0")
 	(paper "USLetter")
+	(title_block
+		(title "ESP32-C3 Breadboard Adapter.")
+	)
 	(junction
 		(at 72.39 66.04)
@@
 		)
 	)
-	(hierarchical_label "VUSB"
+	(hierarchical_label "VUSB_OUT"
 		(shape passive)
 		(at 88.9 45.72 0)
