File: ESP32-C3-BreadBoardAdapter_v2/ESP32-C3-BreadBoardAdapter_v2/ESP32-C3-BreadBoardAdapter.kicad_pcb (KiCad board)
At the start: 2 copper layers, 50.8 x 39.4 mm, 33 parts, among them J1 PWR, J2 USB-C_Receptacle_Data_16P_GCT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, J3 PWR_JMP, J4 PWR_JMP, J6 Debug_3V3, J7 Debug_VIN, SW1 SW_Push_SMD_6x3.5, SW2 SW_Push_SMD_6x3.5, SW3 SW_Push_SMD_6x3.5, U1 ESP32-C3-WROOM-02-N4, U2 AMS1117-3V3, U3 L7805

Commit message: .
Parts:
- R5: value 2K2 -> 10k
- renumbered ESP32-C3 to BRD1
Changed lines of the file:
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@@
 		(descr "Universal Power Adapter for Bread Board")
 		(tags "Power Adapter Bread Board")
-		(property "Reference" "ESP32-C3"
+		(property "Reference" "BRD1"
 			(at 1.67 -10.4 0)
 			(unlocked yes)
@@
 			)
 		)
-		(property "Value" "2K2"
+		(property "Value" "10k"
 			(at 0 -1.82 90)
 			(layer "B.Fab")
