File: ESP32-C3-WROOM-Node-Temperature/ESP32-C3-WROOM-Node-Temperature.kicad_pcb (KiCad board)
At the start: 2 copper layers, 65 x 40 mm, 27 parts, among them J1 PWR, J2 Conn_01x02_Socket, J3 Conn_01x02_Socket, J4 I2C, K1 Relay_DPDT_HK19F_HUI, Q1 NPN, SW1 SW_SPDT, U2 AMS1117-3V3, U4 L7805, U5 ESP32-C3 SuperMini

Commit message: .
Parts:
- moved U5 27.4 mm to (150.4, 69.7), turned to -90 degrees
- moved R1 6.10 mm to (156.9, 75.5), turned to 45 degrees
Routing:
- net Net-(D1-AG): track 25.3 -> 11.0 mm
- net /GPIO10: track 8.92 -> 0.00 mm
- net /SCL: track 23.9 -> 15.4 mm
- net /SDA: track 27.3 -> 18.9 mm
- net /ADC1: track 10.8 -> 3.26 mm
- net +5V: track 67.5 -> 60.5 mm
- net +3V3: track 167.4 -> 164.4 mm
Changed lines of the file:
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@@
 	(footprint "Alexander Footprint Library:ESP32-C3_SuperMini"
 		(layer "F.Cu")
-		(at 173.14 84.94 90)
+		(at 150.42 69.7 -90)
 		(descr "ESP32 C3 Super Mini")
 		(tags "ESP32 C3")
 		(property "Reference" "U5"
-			(at 0 -0.5 90)
+			(at 0 -0.5 -90)
 			(unlocked yes)
 			(layer "F.SilkS")
@@
 		)
 		(property "Value" "ESP32-C3 SuperMini"
-			(at 0 1 90)
+			(at 0 1 -90)
 			(unlocked yes)
 			(layer "F.Fab")
@@
 		)
 		(property "Footprint" "Alexander Footprint Library:ESP32-C3_SuperMini"
-			(at 0 0 90)
+			(at 0 0 -90)
 			(unlocked yes)
 			(layer "F.Fab")
@@
 		)
 		(property "Datasheet" ""
-			(at 0 0 90)
+			(at 0 0 -90)
 			(unlocked yes)
 			(layer "F.Fab")
@@
 		)
 		(property "Description" ""
-			(at 0 0 90)
+			(at 0 0 -90)
 			(unlocked yes)
 			(layer "F.Fab")
@@
 		(attr through_hole)
 		(fp_text user "${REFERENCE}"
-			(at 0 2.5 90)
+			(at 0 2.5 -90)
 			(unlocked yes)
 			(layer "F.Fab")
@@
 		)
 		(pad "1" thru_hole roundrect
-			(at 0 -20.32 90)
+			(at 0 -20.32 270)
 			(size 1.7 1.7)
 			(drill 1)
@@
 		)
 		(pad "2" thru_hole oval
-			(at 0 -17.78 90)
+			(at 0 -17.78 270)
 			(size 1.7 1.7)
 			(drill 1)
@@
 		)
 		(pad "3" thru_hole oval
-			(at 0 -15.24 90)
+			(at 0 -15.24 270)
 			(size 1.7 1.7)
 			(drill 1)
@@
 		)
 		(pad "4" thru_hole oval
-			(at 0 -12.7 90)
+			(at 0 -12.7 270)
 			(size 1.7 1.7)
 			(drill 1)
@@
 		)
 		(pad "5" thru_hole oval
-			(at 0 -10.16 90)
+			(at 0 -10.16 270)
 			(size 1.7 1.7)
 			(drill 1)
@@
 		)
 		(pad "6" thru_hole oval
-			(at 0 -7.62 90)
+			(at 0 -7.62 270)
 			(size 1.7 1.7)
 			(drill 1)
@@
 		)
 		(pad "7" thru_hole oval
-			(at 0 -5.08 90)
+			(at 0 -5.08 270)
 			(size 1.7 1.7)
 			(drill 1)
@@
 		)
 		(pad "8" thru_hole oval
-			(at 0 -2.54 90)
+			(at 0 -2.54 270)
 			(size 1.7 1.7)
 			(drill 1)
@@
 		)
 		(pad "9" thru_hole oval
-			(at 15.24 -2.54 90)
+			(at 15.24 -2.54 270)
 			(size 1.7 1.7)
 			(drill 1)
@@
 		)
 		(pad "10" thru_hole oval
-			(at 15.24 -5.08 90)
+			(at 15.24 -5.08 270)
 			(size 1.7 1.7)
 			(drill 1)
@@
 		)
 		(pad "11" thru_hole oval
-			(at 15.24 -7.62 90)
+			(at 15.24 -7.62 270)
 			(size 1.7 1.7)
 			(drill 1)
@@
 		)
 		(pad "12" thru_hole oval
-			(at 15.24 -10.16 90)
+			(at 15.24 -10.16 270)
 			(size 1.7 1.7)
 			(drill 1)
@@
 		)
 		(pad "13" thru_hole oval
-			(at 15.24 -12.7 90)
+			(at 15.24 -12.7 270)
 			(size 1.7 1.7)
 			(drill 1)
@@
 		)
 		(pad "14" thru_hole oval
-			(at 15.24 -15.24 90)
+			(at 15.24 -15.24 270)
 			(size 1.7 1.7)
 			(drill 1)
@@
 		)
 		(pad "15" thru_hole rect
-			(at 15.24 -17.78 90)
+			(at 15.24 -17.78 270)
 			(size 1.7 1.7)
 			(drill 1)
@@
 		)
 		(pad "16" thru_hole oval
-			(at 15.24 -20.32 90)
+			(at 15.24 -20.32 270)
 			(size 1.7 1.7)
 			(drill 1)
@@
 	(footprint "Resistor_SMD:R_1206_3216Metric_Pad1.30x1.75mm_HandSolder"
 		(layer "B.Cu")
-		(at 163 75.5 -45)
+		(at 156.9 75.5 45)
 		(descr "Resistor SMD 1206 (3216 Metric), square (rectangular) end terminal, IPC_7351 nominal with elongated pad for handsoldering. (Body size source: IPC-SM-782 page 72, https://www.pcb-3d.com/wordpress/wp-content/uploads/ipc-sm-782a_amendment_1_and_2.pdf), generated with kicad-footprint-generator")
 		(tags "resistor handsolder")
 		(property "Reference" "R1"
-			(at 0.070711 -2.192031 135)
+			(at 0.070711 -2.192031 45)
 			(layer "B.SilkS")
 			(effects
@@
 		)
 		(property "Value" "10K"
-			(at 0 -1.82 135)
+			(at 0 -1.82 45)
 			(layer "B.Fab")
 			(effects
@@
 		)
 		(property "Footprint" "Resistor_SMD:R_1206_3216Metric_Pad1.30x1.75mm_HandSolder"
-			(at 0 0 135)
+			(at 0 0 -135)
 			(unlocked yes)
 			(layer "B.Fab")
@@
 		)
 		(property "Datasheet" ""
-			(at 0 0 135)
+			(at 0 0 -135)
 			(unlocked yes)
 			(layer "B.Fab")
@@
 		)
 		(property "Description" "Resistor"
-			(at 0 0 135)
+			(at 0 0 -135)
 			(unlocked yes)
 			(layer "B.Fab")
@@
 		(attr smd)
 		(fp_line
+			(start 0.727064 -0.91)
+			(end -0.727064 -0.91)
+			(stroke
+				(width 0.12)
+				(type solid)
+			)
+			(layer "B.SilkS")
+		)
+		(fp_line
 			(start 0.727064 0.91)
 			(end -0.727064 0.91)
@@
 		)
 		(fp_line
-			(start 0.727064 -0.91)
-			(end -0.727064 -0.91)
-			(stroke
-				(width 0.12)
-				(type solid)
-			)
-			(layer "B.SilkS")
+			(start -2.45 -1.12)
+			(end 2.45 -1.12)
+			(stroke
+				(width 0.05)
+				(type solid)
+			)
+			(layer "B.CrtYd")
 		)
 		(fp_line
@@
 		)
 		(fp_line
-			(start -2.45 -1.12)
-			(end 2.45 -1.12)
+			(start 2.45 -1.12)
+			(end 2.45 1.12)
 			(stroke
 				(width 0.05)
@@
 		)
 		(fp_line
-			(start 2.45 -1.12)
-			(end 2.45 1.12)
-			(stroke
-				(width 0.05)
-				(type solid)
-			)
-			(layer "B.CrtYd")
+			(start -1.6 -0.8)
+			(end 1.6 -0.8)
+			(stroke
+				(width 0.1)
+				(type solid)
+			)
+			(layer "B.Fab")
 		)
 		(fp_line
@@
 		)
 		(fp_line
-			(start -1.6 -0.8)
-			(end 1.6 -0.8)
+			(start 1.6 -0.8)
+			(end 1.6 0.8)
 			(stroke
 				(width 0.1)
@@
 			(layer "B.Fab")
 		)
-		(fp_line
-			(start 1.6 -0.8)
-			(end 1.6 0.8)
-			(stroke
-				(width 0.1)
-				(type solid)
-			)
-			(layer "B.Fab")
-		)
 		(fp_text user "${REFERENCE}"
-			(at 0 0 135)
+			(at 0 0 45)
 			(layer "B.Fab")
 			(effects
@@
 		)
 		(pad "1" smd roundrect
-			(at -1.550001 0 315)
+			(at -1.550001 0 45)
 			(size 1.3 1.75)
 			(layers "B.Cu" "B.Paste" "B.Mask")
@@
 		)
 		(pad "2" smd roundrect
-			(at 1.550001 0 315)
+			(at 1.550001 0 45)
 			(size 1.3 1.75)
 			(layers "B.Cu" "B.Paste" "B.Mask")
@@
 	)
 	(segment
-		(start 155.38 69.68)
-		(end 155.4 69.7)
-		(width 0.5)
-		(layer "B.Cu")
-		(net 1)
-	)
-	(segment
 		(start 160.58 96.58)
 		(end 159 95)
@@
 	)
 	(segment
-		(start 155.38 86.58)
-		(end 155.38 84.92)
-		(width 0.2)
-		(layer "F.Cu")
-		(net 2)
-	)
-	(segment
 		(start 159 90.2)
 		(end 155.38 86.58)
@@
 	)
 	(segment
-		(start 155.38 91.72)
-		(end 155.38 84.92)
-		(width 0.2)
-		(layer "B.Cu")
-		(net 2)
-	)
-	(segment
 		(start 152.68 94.42)
 		(end 155.38 91.72)
@@
 	)
 	(segment
-		(start 157.92 88.52)
-		(end 157.92 84.92)
-		(width 0.2)
-		(layer "F.Cu")
-		(net 3)
-	)
-	(segment
 		(start 160.24 94.04)
 		(end 159.4 93.2)
@@
 	)
 	(segment
-		(start 157.92 89.88)
-		(end 157.92 84.92)
-		(width 0.2)
-		(layer "B.Cu")
-		(net 3)
-	)
-	(segment
 		(start 155.22 92.58)
 		(end 157.92 89.88)
@@
 	)
 	(segment
-		(start 165.54 82.74)
-		(end 165.54 84.92)
-		(width 0.2)
-		(layer "B.Cu")
-		(net 5)
-	)
-	(segment
-		(start 164.096016 76.596016)
-		(end 164.096016 81.296016)
-		(width 0.2)
-		(layer "B.Cu")
-		(net 5)
-	)
-	(segment
-		(start 164.096016 81.296016)
-		(end 165.54 82.74)
-		(width 0.2)
-		(layer "B.Cu")
-		(net 5)
-	)
-	(segment
 		(start 168.08 66.55)
 		(end 165.8 64.27)
@@
 	)
 	(segment
-		(start 168.08 69.68)
-		(end 168.08 66.55)
-		(width 0.2)
-		(layer "F.Cu")
-		(net 6)
-	)
-	(segment
-		(start 168.08 69.68)
-		(end 168.08 74.08)
-		(width 0.2)
-		(layer "B.Cu")
-		(net 6)
-	)
-	(segment
 		(start 168.08 74.08)
 		(end 168.103984 74.103984)
@@
 		(start 157.92 66.68)
 		(end 158.5 66.1)
-		(width 0.25)
-		(layer "F.Cu")
-		(net 7)
-	)
-	(segment
-		(start 157.92 69.68)
-		(end 157.92 66.68)
 		(width 0.25)
 		(layer "F.Cu")
@@
 	)
 	(segment
-		(start 152.82 69.7)
-		(end 152.82 67.28)
-		(width 0.25)
-		(layer "F.Cu")
-		(net 9)
-	)
-	(segment
 		(start 129.9 73.1)
 		(end 129.445 72.645)
@@
 	)
 	(segment
-		(start 152.82 69.7)
-		(end 152.82 71.98)
-		(width 0.5)
-		(layer "F.Cu")
-		(net 9)
-	)
-	(segment
 		(start 151.6 73.2)
 		(end 130 73.2)
-		(width 0.5)
-		(layer "B.Cu")
-		(net 9)
-	)
-	(segment
-		(start 152.82 69.7)
-		(end 152.82 71.98)
 		(width 0.5)
 		(layer "B.Cu")
@@
 		(net 15)
 	)
-	(segment
-		(start 157.698098 74.403984)
-		(end 155.402082 76.7)
-		(width 0.2)
-		(layer "B.Cu")
-		(net 15)
-	)
-	(segment
-		(start 155.402082 76.7)
-		(end 148.5 76.7)
-		(width 0.2)
-		(layer "B.Cu")
-		(net 15)
-	)
-	(segment
-		(start 161.903984 74.403984)
-		(end 157.698098 74.403984)
-		(width 0.2)
-		(layer "B.Cu")
-		(net 15)
-	)

Commit message: .
Parts:
- moved 5V 33.2 mm to (187.6, 68.8)
Routing:
- net +5V: track 60.5 -> 25.7 mm
- net /SDA: track 18.9 -> 0.00 mm
- net /SCL: track 15.4 -> 0.00 mm
- net +3V3: track 164.4 -> 156.6 mm
- net /ADC1: track 3.26 -> 0.03 mm
Changed lines of the file:
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@@
 	(footprint "TestPoint:TestPoint_Pad_D1.5mm"
 		(layer "F.Cu")
-		(at 155 62.4)
+		(at 187.6 68.8)
 		(descr "SMD pad as test Point, diameter 1.5mm")
 		(tags "test point SMD pad")
@@
 	)
 	(segment
-		(start 160.58 96.58)
-		(end 159 95)
-		(width 0.2)
-		(layer "F.Cu")
-		(net 2)
-	)
-	(segment
-		(start 159 95)
-		(end 159 90.2)
-		(width 0.2)
-		(layer "F.Cu")
-		(net 2)
-	)
-	(segment
-		(start 162.1 96.58)
-		(end 160.58 96.58)
-		(width 0.2)
-		(layer "F.Cu")
-		(net 2)
-	)
-	(segment
-		(start 159 90.2)
-		(end 155.38 86.58)
-		(width 0.2)
-		(layer "F.Cu")
-		(net 2)
-	)
-	(segment
-		(start 152.68 95.8)
-		(end 152.68 94.42)
-		(width 0.2)
-		(layer "B.Cu")
-		(net 2)
-	)
-	(segment
-		(start 152.68 94.42)
-		(end 155.38 91.72)
-		(width 0.2)
-		(layer "B.Cu")
-		(net 2)
-	)
-	(segment
-		(start 160.24 94.04)
-		(end 159.4 93.2)
-		(width 0.2)
-		(layer "F.Cu")
-		(net 3)
-	)
-	(segment
-		(start 159.4 90)
-		(end 157.92 88.52)
-		(width 0.2)
-		(layer "F.Cu")
-		(net 3)
-	)
-	(segment
-		(start 162.1 94.04)
-		(end 160.24 94.04)
-		(width 0.2)
-		(layer "F.Cu")
-		(net 3)
-	)
-	(segment
-		(start 159.4 93.2)
-		(end 159.4 90)
-		(width 0.2)
-		(layer "F.Cu")
-		(net 3)
-	)
-	(segment
-		(start 155.22 92.58)
-		(end 157.92 89.88)
-		(width 0.2)
-		(layer "B.Cu")
-		(net 3)
-	)
-	(segment
-		(start 155.22 95.8)
-		(end 155.22 92.58)
-		(width 0.2)
-		(layer "B.Cu")
-		(net 3)
-	)
-	(segment
 		(start 145.76 79.3)
 		(end 145.83 79.37)
@@
 	)
 	(segment
-		(start 168.08 66.55)
-		(end 165.8 64.27)
-		(width 0.2)
-		(layer "F.Cu")
-		(net 6)
-	)
-	(segment
 		(start 168.08 74.08)
 		(end 168.103984 74.103984)
@@
 	)
 	(segment
-		(start 157.92 66.68)
-		(end 158.5 66.1)
-		(width 0.25)
-		(layer "F.Cu")
-		(net 7)
-	)
-	(segment
 		(start 152.2 76.849999)
 		(end 152.180001 76.83)
@@
 		(net 7)
 	)
-	(segment
-		(start 158.5 66.1)
-		(end 158.5 62.4)
-		(width 0.25)
-		(layer "F.Cu")
-		(net 7)
-	)
 	(via
 		(at 136 65.1)
@@
 	)
 	(segment
-		(start 152.44 98.1)
-		(end 150.14 95.8)
-		(width 0.5)
-		(layer "B.Cu")
-		(net 7)
-	)
-	(segment
 		(start 159 65.1)
 		(end 160.2 66.3)
@@
 	)
 	(segment
-		(start 152.82 71.98)
-		(end 151.7 73.1)
-		(width 0.5)
-		(layer "F.Cu")
-		(net 9)
-	)
-	(segment
 		(start 129.9 73.1)
 		(end 129.445 72.645)
@@
 	)
 	(segment
-		(start 152.82 67.28)
-		(end 155 65.1)
-		(width 0.25)
-		(layer "F.Cu")
-		(net 9)
-	)
-	(segment
-		(start 155 65.1)
-		(end 155 62.4)
-		(width 0.25)
-		(layer "F.Cu")
-		(net 9)
-	)
-	(segment
 		(start 151.7 73.1)
 		(end 129.9 73.1)
@@
 		(net 9)
 	)
-	(segment
-		(start 151.6 73.2)
-		(end 130 73.2)
-		(width 0.5)
-		(layer "B.Cu")
-		(net 9)
-	)
-	(segment
-		(start 129.445 72.645)
-		(end 126.14 72.645)
-		(width 0.5)
-		(layer "B.Cu")
-		(net 9)
-	)
-	(segment
-		(start 130 73.2)
-		(end 129.445 72.645)
-		(width 0.5)
-		(layer "B.Cu")
-		(net 9)
-	)
-	(segment
-		(start 152.82 71.98)
-		(end 151.6 73.2)
-		(width 0.5)
-		(layer "B.Cu")
-		(net 9)
-	)

Commit message: .
Parts:
- moved J4 43.8 mm to (180.9, 80.2)
- moved U3 24.8 mm to (185.6, 87.6)
Routing:
- net +3V3: track 156.6 -> 20.6 mm
- net Net-(D1-AG): track 11.0 -> 9.00 mm
Changed lines of the file:
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@@
 	(footprint "Alexander Footprint Library:Conn_I2C"
 		(layer "F.Cu")
-		(at 139.98 95.8 90)
+		(at 180.9 80.2 90)
 		(property "Reference" "J4"
 			(at 0 -0.5 90)
@@
 	(footprint "Alexander Footprint Library:BME280_BMP280_I2C"
 		(layer "F.Cu")
-		(at 160.8 87.74)
+		(at 185.6 87.6)
 		(descr "Temperature, Humidity and Pressure sensor")
 		(tags "BME BMP 280 sensor")
@@
 	)
 	(segment
-		(start 168.1 94.3)
-		(end 168.1 96.6)
-		(width 0.5)
-		(layer "B.Cu")
-		(net 7)
-	)
-	(segment
-		(start 142.8 77.6)
-		(end 142.8 95.8)
-		(width 0.5)
-		(layer "B.Cu")
-		(net 7)
-	)
-	(segment
-		(start 173.7 91.1)
-		(end 172.7 92.1)
-		(width 0.5)
-		(layer "B.Cu")
-		(net 7)
-	)
-	(segment
-		(start 170.296016 76.296016)
-		(end 171.5 77.5)
-		(width 0.25)
-		(layer "B.Cu")
-		(net 7)
-	)
-	(segment
-		(start 171.5 66.3)
-		(end 173.7 68.5)
-		(width 0.5)
-		(layer "B.Cu")
-		(net 7)
-	)
-	(segment
-		(start 173.7 87.6)
-		(end 173.7 79)
-		(width 0.5)
-		(layer "B.Cu")
-		(net 7)
-	)
-	(segment
-		(start 166.6 98.1)
-		(end 152.44 98.1)
-		(width 0.5)
-		(layer "B.Cu")
-		(net 7)
-	)
-	(segment
-		(start 145.1 98.1)
-		(end 152.44 98.1)
-		(width 0.5)
-		(layer "B.Cu")
-		(net 7)
-	)
-	(segment
-		(start 170.3 92.1)
-		(end 168.1 94.3)
-		(width 0.5)
-		(layer "B.Cu")
-		(net 7)
-	)
-	(segment
-		(start 136 65.1)
-		(end 159 65.1)
-		(width 0.5)
-		(layer "B.Cu")
-		(net 7)
-	)
-	(segment
-		(start 142.8 95.8)
-		(end 145.1 98.1)
-		(width 0.5)
-		(layer "B.Cu")
-		(net 7)
-	)
-	(segment
-		(start 145.83 76.83)
-		(end 143.57 76.83)
-		(width 0.5)
-		(layer "B.Cu")
-		(net 7)
-	)
-	(segment
-		(start 143.57 76.83)
-		(end 142.8 77.6)
-		(width 0.5)
-		(layer "B.Cu")
-		(net 7)
-	)
-	(segment
-		(start 172.2 77.5)
-		(end 173.7 79)
-		(width 0.25)
-		(layer "B.Cu")
-		(net 7)
-	)
-	(segment
-		(start 160.2 66.3)
-		(end 171.5 66.3)
-		(width 0.5)
-		(layer "B.Cu")
-		(net 7)
-	)
-	(segment
-		(start 172.7 92.1)
-		(end 170.3 92.1)
-		(width 0.5)
-		(layer "B.Cu")
-		(net 7)
-	)
-	(segment
-		(start 171.5 77.5)
-		(end 172.2 77.5)
-		(width 0.25)
-		(layer "B.Cu")
-		(net 7)
-	)
-	(segment
-		(start 173.7 87.6)
-		(end 173.7 91.1)
-		(width 0.5)
-		(layer "B.Cu")
-		(net 7)
-	)
-	(segment
-		(start 173.7 68.5)
-		(end 173.7 79)
-		(width 0.5)
-		(layer "B.Cu")
-		(net 7)
-	)
-	(segment
 		(start 136 65.1)
 		(end 132.05 65.1)
@@
 	)
 	(segment
-		(start 172.34 88.96)
-		(end 173.7 87.6)
-		(width 0.5)
-		(layer "B.Cu")
-		(net 7)
-	)
-	(segment
-		(start 162.1 88.96)
-		(end 172.34 88.96)
-		(width 0.5)
-		(layer "B.Cu")
-		(net 7)
-	)
-	(segment
-		(start 159 65.1)
-		(end 160.2 66.3)
-		(width 0.5)
-		(layer "B.Cu")
-		(net 7)
-	)
-	(segment
-		(start 168.1 96.6)
-		(end 166.6 98.1)
-		(width 0.5)
-		(layer "B.Cu")
-		(net 7)
-	)
-	(segment
 		(start 121.06 70.86)
 		(end 121.06 72.645)
@@
 		(net 15)
 	)
-	(segment
-		(start 148.5 76.7)
-		(end 147.1 78.1)
-		(width 0.2)
-		(layer "B.Cu")
-		(net 15)
-	)

Commit message: .
Parts:
- moved R3 8.14 mm to (170.0, 83.3)
- moved R4 6.10 mm to (152.4, 84.5)
- moved U5 6.00 mm to (150.4, 75.7)
- moved R1 5.40 mm to (156.9, 80.9)
Routing:
- net +5V: track 25.7 -> 3.30 mm
- net +3V3: track 20.6 -> 14.2 mm
- net Net-(D1-AB): track 13.8 -> 8.31 mm
Changed lines of the file:
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@@
 	(footprint "Resistor_SMD:R_1206_3216Metric_Pad1.30x1.75mm_HandSolder"
 		(layer "F.Cu")
-		(at 152.2 78.4 -90)
+		(at 152.4 84.5 -90)
 		(descr "Resistor SMD 1206 (3216 Metric), square (rectangular) end terminal, IPC_7351 nominal with elongated pad for handsoldering. (Body size source: IPC-SM-782 page 72, https://www.pcb-3d.com/wordpress/wp-content/uploads/ipc-sm-782a_amendment_1_and_2.pdf), generated with kicad-footprint-generator")
 		(tags "resistor handsolder")
@@
 	(footprint "Alexander Footprint Library:ESP32-C3_SuperMini"
 		(layer "F.Cu")
-		(at 150.42 69.7 -90)
+		(at 150.44 75.7 -90)
 		(descr "ESP32 C3 Super Mini")
 		(tags "ESP32 C3")
@@
 	(footprint "Resistor_SMD:R_1206_3216Metric_Pad1.30x1.75mm_HandSolder"
 		(layer "B.Cu")
-		(at 156.9 75.5 45)
+		(at 156.9 80.9 45)
 		(descr "Resistor SMD 1206 (3216 Metric), square (rectangular) end terminal, IPC_7351 nominal with elongated pad for handsoldering. (Body size source: IPC-SM-782 page 72, https://www.pcb-3d.com/wordpress/wp-content/uploads/ipc-sm-782a_amendment_1_and_2.pdf), generated with kicad-footprint-generator")
 		(tags "resistor handsolder")
@@
 	(footprint "Resistor_SMD:R_1206_3216Metric_Pad1.30x1.75mm_HandSolder"
 		(layer "B.Cu")
-		(at 169.2 75.2 135)
+		(at 170 83.3 135)
 		(descr "Resistor SMD 1206 (3216 Metric), square (rectangular) end terminal, IPC_7351 nominal with elongated pad for handsoldering. (Body size source: IPC-SM-782 page 72, https://www.pcb-3d.com/wordpress/wp-content/uploads/ipc-sm-782a_amendment_1_and_2.pdf), generated with kicad-footprint-generator")
 		(tags "resistor handsolder")
@@
 	)
 	(segment
-		(start 168.08 74.08)
-		(end 168.103984 74.103984)
-		(width 0.2)
-		(layer "B.Cu")
-		(net 6)
-	)
-	(segment
-		(start 152.180001 76.83)
-		(end 145.83 76.83)
-		(width 0.2)
-		(layer "F.Cu")
-		(net 7)
-	)
-	(segment
 		(start 136 65.1)
 		(end 135 66.1)
@@
 		(net 7)
 	)
-	(segment
-		(start 152.2 76.849999)
-		(end 152.180001 76.83)
-		(width 0.2)
-		(layer "F.Cu")
-		(net 7)
-	)
 	(via
 		(at 136 65.1)
@@
 	)
 	(segment
-		(start 129.9 73.1)
-		(end 129.445 72.645)
-		(width 0.5)
-		(layer "F.Cu")
-		(net 9)
-	)
-	(segment
-		(start 151.7 73.1)
-		(end 129.9 73.1)
-		(width 0.5)
-		(layer "F.Cu")
-		(net 9)
-	)
-	(segment
 		(start 113.8 76.22)
 		(end 113.8 72.1)
@@
 	)
 	(segment
-		(start 152.2 81.4)
-		(end 152.2 79.950001)
-		(width 0.2)
-		(layer "F.Cu")
-		(net 16)
-	)
-	(segment
-		(start 150.2 83.4)
-		(end 150.2 87.4)
-		(width 0.2)
-		(layer "F.Cu")
-		(net 16)
-	)
-	(segment
-		(start 150.2 87.4)
-		(end 149.6 88)
-		(width 0.2)
-		(layer "F.Cu")
-		(net 16)
-	)
-	(segment
-		(start 150.2 83.4)
-		(end 152.2 81.4)
+		(start 150.450001 88)
+		(end 144.9 88)
 		(width 0.2)
 		(layer "F.Cu")
@@
 	)
 	(segment
-		(start 149.6 88)
-		(end 144.9 88)
+		(start 152.4 86.050001)
+		(end 150.450001 88)
 		(width 0.2)
 		(layer "F.Cu")

Commit message: .
Parts:
- moved R3 15.1 mm to (164.8, 69.1), turned to 45 degrees
- moved R1 1.57 mm to (157.6, 82.3), turned to -45 degrees
- moved C3 0.22 mm to (136.1, 71.2)
- moved C6 0.22 mm to (141.9, 71.2)
Routing:
- net +5V: track 3.30 -> 74.7 mm
- net +3V3: track 14.2 -> 72.7 mm

Commit message: .
Parts:
- moved R4 9.94 mm to (146.5, 92.5), turned to 180 degrees
- moved D1 0.10 mm to (146.5, 85.6)
Routing:
- net Net-(D1-AB): track 8.31 -> 0.00 mm
Changed lines of the file:
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@@
 	(footprint "Resistor_SMD:R_1206_3216Metric_Pad1.30x1.75mm_HandSolder"
 		(layer "F.Cu")
-		(at 152.4 84.5 -90)
+		(at 146.5 92.5 180)
 		(descr "Resistor SMD 1206 (3216 Metric), square (rectangular) end terminal, IPC_7351 nominal with elongated pad for handsoldering. (Body size source: IPC-SM-782 page 72, https://www.pcb-3d.com/wordpress/wp-content/uploads/ipc-sm-782a_amendment_1_and_2.pdf), generated with kicad-footprint-generator")
 		(tags "resistor handsolder")
 		(property "Reference" "R4"
-			(at 0 -1.82 90)
+			(at 0 -1.82 0)
 			(layer "F.SilkS")
 			(effects
@@
 		)
 		(property "Value" "10K"
-			(at 0 1.82 90)
+			(at 0 1.82 0)
 			(layer "F.Fab")
 			(effects
@@
 		)
 		(property "Footprint" "Resistor_SMD:R_1206_3216Metric_Pad1.30x1.75mm_HandSolder"
-			(at 0 0 -90)
+			(at 0 0 180)
 			(unlocked yes)
 			(layer "F.Fab")
@@
 		)
 		(property "Datasheet" ""
-			(at 0 0 -90)
+			(at 0 0 180)
 			(unlocked yes)
 			(layer "F.Fab")
@@
 		)
 		(property "Description" "Resistor"
-			(at 0 0 -90)
+			(at 0 0 180)
 			(unlocked yes)
 			(layer "F.Fab")
@@
 		)
 		(fp_line
-			(start -2.45 1.12)
-			(end -2.45 -1.12)
+			(start 2.45 1.12)
+			(end -2.45 1.12)
 			(stroke
 				(width 0.05)
@@
 		)
 		(fp_line
-			(start 2.45 1.12)
-			(end -2.45 1.12)
+			(start 2.45 -1.12)
+			(end 2.45 1.12)
 			(stroke
 				(width 0.05)
@@
 		)
 		(fp_line
-			(start -2.45 -1.12)
-			(end 2.45 -1.12)
+			(start -2.45 1.12)
+			(end -2.45 -1.12)
 			(stroke
 				(width 0.05)
@@
 		)
 		(fp_line
-			(start 2.45 -1.12)
-			(end 2.45 1.12)
+			(start -2.45 -1.12)
+			(end 2.45 -1.12)
 			(stroke
 				(width 0.05)
@@
 		)
 		(fp_line
-			(start -1.6 0.8)
-			(end -1.6 -0.8)
+			(start 1.6 0.8)
+			(end -1.6 0.8)
 			(stroke
 				(width 0.1)
@@
 		)
 		(fp_line
-			(start 1.6 0.8)
-			(end -1.6 0.8)
+			(start 1.6 -0.8)
+			(end 1.6 0.8)
 			(stroke
 				(width 0.1)
@@
 		)
 		(fp_line
-			(start -1.6 -0.8)
-			(end 1.6 -0.8)
+			(start -1.6 0.8)
+			(end -1.6 -0.8)
 			(stroke
 				(width 0.1)
@@
 		)
 		(fp_line
-			(start 1.6 -0.8)
-			(end 1.6 0.8)
+			(start -1.6 -0.8)
+			(end 1.6 -0.8)
 			(stroke
 				(width 0.1)
@@
 		)
 		(fp_text user "${REFERENCE}"
-			(at 0 0 90)
+			(at 0 0 0)
 			(layer "F.Fab")
 			(effects
@@
 		)
 		(pad "1" smd roundrect
-			(at -1.550001 0 270)
+			(at -1.550001 0 180)
 			(size 1.3 1.75)
 			(layers "F.Cu" "F.Paste" "F.Mask")
@@
 		)
 		(pad "2" smd roundrect
-			(at 1.550001 0 270)
+			(at 1.550001 0 180)
 			(size 1.3 1.75)
 			(layers "F.Cu" "F.Paste" "F.Mask")
@@
 	(footprint "Alexander Footprint Library:LED_5050-6"
 		(layer "F.Cu")
-		(at 146.6 85.6 90)
+		(at 146.5 85.6 90)
 		(descr "http://cdn.sparkfun.com/datasheets/Components/LED/5060BRG4.pdf")
 		(tags "RGB LED 5050-6")
@@
 		(net 15)
 	)
-	(segment
-		(start 150.450001 88)
-		(end 144.9 88)
-		(width 0.2)
-		(layer "F.Cu")
-		(net 16)
-	)
-	(segment
-		(start 152.4 86.050001)
-		(end 150.450001 88)
-		(width 0.2)
-		(layer "F.Cu")
-		(net 16)
-	)
 	(zone
