File: amplifier/amplifier.kicad_pcb (KiCad board)
At the start: 2 copper layers, 3 parts

Commit message: .
Parts:
- moved DZ1 15.1 mm to (221.6, 61.2)
Changed lines of the file:
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@@
 	(footprint "PCM_Diode_SMD_AKL:D_SOD-123"
 		(layer "F.Cu")
-		(at 206.93 64.725)
+		(at 221.6 61.2)
 		(descr "SOD-123, Alternate KiCad Library")
 		(tags "SOD-123")

Commit message: .
Parts:
- added HS1: Heatsink_Pad, Heatsink:Heatsink_AAVID_573300D00010G_TO-263, F.Cu at (75.6, 75.5)
- added HS2: Heatsink_Pad, Heatsink:Heatsink_AAVID_573300D00010G_TO-263, F.Cu at (75.6, 90.9)
- added HS3: Heatsink_Pad, Heatsink:Heatsink_AAVID_573300D00010G_TO-263, F.Cu at (75.6, 106.3)
- added HS4: Heatsink_Pad, Heatsink:Heatsink_AAVID_573300D00010G_TO-263, F.Cu at (75.6, 121.8)

Commit message: .
Parts:
- added RV1: 10k, PCM_Potentiometer_THT_AKL_Double:Potentiometer_Alps_RK163_Dual_Horizontal, F.Cu at (125.5, 57.0)

Commit message: .
Parts:
- moved DZ1 251.9 mm to (473.4, 66.1)
- moved C4 251.9 mm to (444.9, 76.7)
- moved C9 251.9 mm to (444.9, 94.8)
- moved HS1 251.9 mm to (327.4, 80.3)
- moved HS2 251.9 mm to (327.4, 95.8)
- moved HS3 251.9 mm to (327.4, 111.2)
- moved HS4 251.9 mm to (327.4, 126.7)
- moved RV1 251.9 mm to (377.3, 61.9)
Other:
- board outline added: 65 x 30 mm
Changed lines of the file:
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@@
 	(footprint "Heatsink:Heatsink_AAVID_573300D00010G_TO-263"
 		(layer "F.Cu")
-		(at 75.58 75.45)
+		(at 327.4 80.35)
 		(descr "Heatsink, 12.70mm x 26.16mm x 10.16, SMD, 18K/W, TO-263, D2 Pak, https://www.shopaavid.com/Product/573300D00000G")
 		(tags "Heatsink AAVID TO-263 D2 Pak")
@@
 	(footprint "PCM_Potentiometer_THT_AKL_Double:Potentiometer_Alps_RK163_Dual_Horizontal"
 		(layer "F.Cu")
-		(at 125.45 57)
+		(at 377.27 61.9)
 		(descr "Potentiometer, horizontal, Alps RK163 Dual, http://www.alps.com/prod/info/E/HTML/Potentiometer/RotaryPotentiometers/RK16/RK16_list.html")
 		(tags "Potentiometer horizontal Alps RK163 Dual")
@@
 	(footprint "Heatsink:Heatsink_AAVID_573300D00010G_TO-263"
 		(layer "F.Cu")
-		(at 75.58 90.9)
+		(at 327.4 95.8)
 		(descr "Heatsink, 12.70mm x 26.16mm x 10.16, SMD, 18K/W, TO-263, D2 Pak, https://www.shopaavid.com/Product/573300D00000G")
 		(tags "Heatsink AAVID TO-263 D2 Pak")
@@
 	(footprint "Capacitor_SMD:CP_Elec_16x17.5"
 		(layer "F.Cu")
-		(at 193.05 71.75)
+		(at 444.87 76.65)
 		(descr "SMD capacitor, aluminum electrolytic, Vishay 1616, 16.0x17.5mm, http://www.vishay.com/docs/28395/150crz.pdf")
 		(tags "capacitor electrolytic")
@@
 	(footprint "PCM_Diode_SMD_AKL:D_SOD-123"
 		(layer "F.Cu")
-		(at 221.6 61.2)
+		(at 473.42 66.1)
 		(descr "SOD-123, Alternate KiCad Library")
 		(tags "SOD-123")
@@
 	(footprint "Capacitor_SMD:CP_Elec_16x17.5"
 		(layer "F.Cu")
-		(at 193.05 89.9)
+		(at 444.87 94.8)
 		(descr "SMD capacitor, aluminum electrolytic, Vishay 1616, 16.0x17.5mm, http://www.vishay.com/docs/28395/150crz.pdf")
 		(tags "capacitor electrolytic")
@@
 	(footprint "Heatsink:Heatsink_AAVID_573300D00010G_TO-263"
 		(layer "F.Cu")
-		(at 75.58 106.35)
+		(at 327.4 111.25)
 		(descr "Heatsink, 12.70mm x 26.16mm x 10.16, SMD, 18K/W, TO-263, D2 Pak, https://www.shopaavid.com/Product/573300D00000G")
 		(tags "Heatsink AAVID TO-263 D2 Pak")
@@
 	(footprint "Heatsink:Heatsink_AAVID_573300D00010G_TO-263"
 		(layer "F.Cu")
-		(at 75.58 121.8)
+		(at 327.4 126.7)
 		(descr "Heatsink, 12.70mm x 26.16mm x 10.16, SMD, 18K/W, TO-263, D2 Pak, https://www.shopaavid.com/Product/573300D00000G")
 		(tags "Heatsink AAVID TO-263 D2 Pak")
@@
 		)
 	)
+	(gr_rect
+		(start 50 50)
+		(end 115 80)
+		(stroke
+			(width 0.05)
+			(type default)
+		)
+		(fill none)
+		(layer "Edge.Cuts")
+	)
 )

Commit message: .
Parts:
- added H5: MountingHole_M3_3.2mm_Pad, PCM_SL_Mechanical:MountingHole_3.2mm_Pad, F.Cu at (53.5, 53.5)
- added H6: MountingHole_M3_3.2mm_Pad, PCM_SL_Mechanical:MountingHole_3.2mm_Pad, F.Cu at (111.5, 53.5)
- added H7: MountingHole_M3_3.2mm_Pad, PCM_SL_Mechanical:MountingHole_3.2mm_Pad, F.Cu at (53.5, 76.5)
- added H8: MountingHole_M3_3.2mm_Pad, PCM_SL_Mechanical:MountingHole_3.2mm_Pad, F.Cu at (111.5, 76.5)
Other:
- outline, holes or cut-outs redrawn
