File: RaspberryPiZero2W_Header/RPi-zero2W_Header/RPi-zero2W_Header.kicad_pcb (KiCad board)
At the start: 2 copper layers, 65 x 30 mm, 1 part

Commit message: .
Parts:
- added H1: MountingHole_M3_3.2mm_Pad, PCM_SL_Mechanical:MountingHole_3.2mm_Pad, F.Cu at (82.6, 97.1)
- moved RaspberryPi-Zero2W1 71.5 mm to (160.6, 135.2)
Connections:
- RaspberryPi-Zero2W1 pad 17: (no net) -> unconnected-(RaspberryPi-Zero2W1-3V3-Pad17)
- RaspberryPi-Zero2W1 pad 28: (no net) -> unconnected-(RaspberryPi-Zero2W1-ID_SC-Pad28)
