File: ESP32-C3-BreadBoardAdapter_2025-06/ESP32-C3-BreadBoardAdapter_2025-06.kicad_pcb (KiCad board)
At the start: 2 copper layers, 52.1 x 40.6 mm, 32 parts, among them J1 PWR, J2 USB-C_Receptacle_Data_16P_GCT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, J3 PWR_JMP, J4 PWR_JMP, J6 Debug_3V3, SW1 SW_Push_SMD_6x3.5, SW2 SW_Push_SMD_6x3.5, SW3 SW_Push_SMD_6x3.5, U1 ESP32-C3-WROOM-02-N4, U2 AMS1117-3V3, U3 L7805

Commit message: .
Routing:
- net EN: track 50.4 -> 42.0 mm
Changed lines of the file:
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@@
-	)
-	(segment
-		(start 125.5102 76.8002)
-		(end 126.1 77.39)
-		(width 0.2)
-		(layer "F.Cu")
-		(net 6)
 	)
 	(segment
@@
 		(start 128.5 62.468628)
 		(end 128.234314 62.734314)
-		(width 0.2)
-		(layer "F.Cu")
-		(net 6)
-	)
-	(segment
-		(start 124.09 77.4002)
-		(end 123.49 76.8002)
 		(width 0.2)
 		(layer "F.Cu")
@@
 		(start 126.1 66.237254)
 		(end 126.1 77.39)
-		(width 0.2)
-		(layer "F.Cu")
-		(net 6)
-	)
-	(segment
-		(start 120.74 76.8002)
-		(end 123.49 76.8002)
 		(width 0.2)
 		(layer "F.Cu")
@@
 		(width 0.2)
 		(layer "F.Cu")
-		(net 6)
-	)
-	(segment
-		(start 124.09 79.4)
-		(end 124.09 77.4002)
-		(width 0.2)
-		(layer "F.Cu")
-		(net 6)
-	)
-	(segment
-		(start 123.49 76.8002)
-		(end 125.5102 76.8002)
-		(width 0.2)
-		(layer "F.Cu")

Commit message: .
Routing:
- net /IO9: track 31.1 -> 31.6 mm

Commit message: .
Routing:
- net /IO8: track 30.4 -> 34.8 mm, vias 0 -> 1
Changed lines of the file:
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@@
+	)
+	(segment
+		(start 130.89 67.1)
+		(end 131.84 67.1)
+		(width 0.2)
+		(layer "F.Cu")
+		(net 7)
 	)
 	(segment
@@
 		(start 128.599 92.451)
 		(end 127.64 91.492)
+		(width 0.2)
+		(layer "F.Cu")
+		(net 7)
+	)
+	(segment
+		(start 131.84 67.1)
+		(end 132.94 66)
 		(width 0.2)
 		(layer "F.Cu")
@@
 		(net 7)
 	)
+	(via
+		(at 132.94 66)
+		(size 0.6)
+		(drill 0.3)
+		(layers "F.Cu" "B.Cu")
+		(net 7)
+	)
+	(segment
+		(start 132.94 66)
+		(end 132.94 64.1)
+		(width 0.2)
+		(layer "B.Cu")
+		(net 7)
+	)

Commit message: .
Routing:
- net /IO9: track 31.6 -> 36.0 mm, vias 0 -> 1
Changed lines of the file:
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@@
+	)
+	(segment
+		(start 128.243 69.457)
+		(end 128.72 68.98)
+		(width 0.2)
+		(layer "F.Cu")
+		(net 8)
 	)
 	(segment
@@
 	)
 	(segment
-		(start 128.243 69.457)
+		(start 128.72 68.98)
 		(end 129.1 68.6)
 		(width 0.2)
@@
 		(net 8)
 	)
+	(via
+		(at 128.72 68.98)
+		(size 0.6)
+		(drill 0.3)
+		(layers "F.Cu" "B.Cu")
+		(net 8)
+	)
+	(segment
+		(start 129.1 68.6)
+		(end 128.72 68.98)
+		(width 0.2)
+		(layer "B.Cu")
+		(net 8)
+	)
+	(segment
+		(start 132.94 68.6)
+		(end 129.1 68.6)
+		(width 0.2)
+		(layer "B.Cu")
+		(net 8)
+	)

Commit message: .
Routing:
- net /IO5: track 36.3 -> 37.0 mm
Changed lines of the file:
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@@
 	)
 	(segment
-		(start 128.234314 62.734314)
-		(end 128.234314 63.368628)
+		(start 127.7 61.44)
+		(end 127.7 64.637254)
 		(width 0.2)
 		(layer "F.Cu")
@@
 	)
 	(segment
+		(start 129.54 59.6)
+		(end 127.7 61.44)
+		(width 0.2)
+		(layer "F.Cu")
+		(net 6)
+	)
+	(segment
+		(start 127.7 64.637254)
+		(end 125.760358 66.576896)
+		(width 0.2)
+		(layer "F.Cu")
+		(net 6)
+	)
+	(segment
 		(start 130.89 59.6)
-		(end 129.2 59.6)
+		(end 129.54 59.6)
+		(width 0.2)
+		(layer "F.Cu")
+		(net 6)
+	)
+	(segment
+		(start 125.760358 81.536585)
+		(end 115.899 91.397943)
+		(width 0.2)
+		(layer "F.Cu")
+		(net 6)
+	)
+	(segment
+		(start 115.899 91.397943)
+		(end 115.899 94.365)
 		(width 0.2)
 		(layer "F.Cu")
@@
 		(start 125.760358 66.576896)
 		(end 125.760358 81.536585)
-		(width 0.2)
-		(layer "F.Cu")
-		(net 6)
-	)
-	(segment
-		(start 125.760358 81.536585)
-		(end 115.899 91.397943)
-		(width 0.2)
-		(layer "F.Cu")
-		(net 6)
-	)
-	(segment
-		(start 128.234314 63.368628)
-		(end 127.7 63.902942)
-		(width 0.2)
-		(layer "F.Cu")
-		(net 6)
-	)
-	(segment
-		(start 128.9 59.9)
-		(end 128.9 60.834314)
-		(width 0.2)
-		(layer "F.Cu")
-		(net 6)
-	)
-	(segment
-		(start 115.899 91.397943)
-		(end 115.899 94.365)
-		(width 0.2)
-		(layer "F.Cu")
-		(net 6)
-	)
-	(segment
-		(start 128.5 62.468628)
-		(end 128.234314 62.734314)
-		(width 0.2)
-		(layer "F.Cu")
-		(net 6)
-	)
-	(segment
-		(start 128.9 60.834314)
-		(end 128.5 61.234314)
-		(width 0.2)
-		(layer "F.Cu")
-		(net 6)
-	)
-	(segment
-		(start 128.5 61.234314)
-		(end 128.5 62.468628)
-		(width 0.2)
-		(layer "F.Cu")
-		(net 6)
-	)
-	(segment
-		(start 127.7 64.637254)
-		(end 125.760358 66.576896)
-		(width 0.2)
-		(layer "F.Cu")
-		(net 6)
-	)
-	(segment
-		(start 129.2 59.6)
-		(end 128.9 59.9)
-		(width 0.2)
-		(layer "F.Cu")
-		(net 6)
-	)
-	(segment
-		(start 127.7 63.902942)
-		(end 127.7 64.637254)
 		(width 0.2)
 		(layer "F.Cu")
@@
 	)
 	(segment
-		(start 128.9 62.634314)
-		(end 128.9 61.54)
+		(start 118.439 94.365)
+		(end 118.439 89.423628)
 		(width 0.2)
 		(layer "F.Cu")
@@
 	)
 	(segment
-		(start 128.634314 63.534314)
-		(end 128.634314 62.9)
+		(start 118.439 89.423628)
+		(end 126.24 81.622628)
 		(width 0.2)
 		(layer "F.Cu")
@@
 	(segment
 		(start 128.100001 65.039998)
-		(end 128.100001 64.068628)
+		(end 128.100001 62.339999)
+		(width 0.2)
+		(layer "F.Cu")
+		(net 12)
+	)
+	(segment
+		(start 126.24 66.899999)
+		(end 128.100001 65.039998)
 		(width 0.2)
 		(layer "F.Cu")
@@
 	)
 	(segment
-		(start 128.100001 64.068628)
-		(end 128.634314 63.534314)
-		(width 0.2)
-		(layer "F.Cu")
-		(net 12)
-	)
-	(segment
-		(start 128.9 61.54)
+		(start 128.100001 62.339999)
 		(end 129.34 61.1)
-		(width 0.2)
-		(layer "F.Cu")
-		(net 12)
-	)
-	(segment
-		(start 128.634314 62.9)
-		(end 128.9 62.634314)
-		(width 0.2)
-		(layer "F.Cu")
-		(net 12)
-	)
-	(segment
-		(start 118.439 89.423628)
-		(end 126.24 81.622628)
-		(width 0.2)
-		(layer "F.Cu")
-		(net 12)
-	)
-	(segment
-		(start 126.24 66.899999)
-		(end 128.100001 65.039998)
-		(width 0.2)
-		(layer "F.Cu")
-		(net 12)
-	)
-	(segment
-		(start 118.439 94.365)
-		(end 118.439 89.423628)
 		(width 0.2)
 		(layer "F.Cu")
@@
 	)
 	(segment
-		(start 130.59 62.6)
+		(start 128.5 63.14)
+		(end 129.04 62.6)
+		(width 0.2)
+		(layer "F.Cu")
+		(net 19)
+	)
+	(segment
+		(start 129.04 62.6)
 		(end 130.89 62.6)
+		(width 0.2)
+		(layer "F.Cu")
+		(net 19)
+	)
+	(segment
+		(start 126.64 67.233126)
+		(end 128.5 65.373126)
+		(width 0.2)
+		(layer "F.Cu")
+		(net 19)
+	)
+	(segment
+		(start 126.64 81.788314)
+		(end 126.64 67.233126)
 		(width 0.2)
 		(layer "F.Cu")
@@
 	)
 	(segment
-		(start 129.49 63.7)
-		(end 130.59 62.6)
+		(start 128.5 65.373126)
+		(end 128.5 63.14)
 		(width 0.2)
 		(layer "F.Cu")
@@
 		(width 0.2)
 		(layer "F.Cu")
-		(net 19)
-	)
-	(segment
-		(start 128.5 64.234314)
-		(end 129.034315 63.7)
-		(width 0.2)
-		(layer "F.Cu")
-		(net 19)
-	)
-	(segment
-		(start 128.5 65.373126)
-		(end 128.5 64.234314)
-		(width 0.2)
-		(layer "F.Cu")
-		(net 19)
-	)
-	(segment
-		(start 129.034315 63.7)
-		(end 129.49 63.7)
-		(width 0.2)
-		(layer "F.Cu")
-		(net 19)
-	)
-	(segment
-		(start 126.64 67.233126)
-		(end 128.5 65.373126)
-		(width 0.2)
-		(layer "F.Cu")
-		(net 19)
-	)
-	(segment
-		(start 126.64 81.788314)
-		(end 126.64 67.233126)
-		(width 0.2)
-		(layer "F.Cu")

Commit message: .
Routing:
- net EN: track 41.8 -> 47.8 mm, vias 0 -> 1
Changed lines of the file:
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@@
+		(net 6)
+	)
+	(via
+		(at 127.7 61.44)
+		(size 0.6)
+		(drill 0.3)
+		(layers "F.Cu" "B.Cu")
+		(net 6)
+	)
+	(segment
+		(start 129.54 59.6)
+		(end 127.7 61.44)
+		(width 0.2)
+		(layer "B.Cu")
+		(net 6)
+	)
+	(segment
+		(start 132.94 59.6)
+		(end 129.54 59.6)
+		(width 0.2)
+		(layer "B.Cu")
 		(net 6)
 	)

Commit message: .
Routing:
- net 3V3: track 41.8 -> 22.0 mm, vias 1 -> 0
Changed lines of the file:
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@@
-	)
-	(segment
-		(start 136.14 67.3)
-		(end 136.24 67.4)
-		(width 0.5)
-		(layer "F.Cu")
-		(net 14)
-	)
-	(segment
-		(start 136.24 67.4)
-		(end 141.44 67.4)
-		(width 0.5)
-		(layer "F.Cu")
-		(net 14)
-	)
-	(segment
-		(start 135.14 66.3)
-		(end 136.14 67.3)
-		(width 0.5)
-		(layer "F.Cu")
-		(net 14)
-	)
-	(segment
-		(start 141.44 67.4)
-		(end 141.84 67.4)
-		(width 0.5)
-		(layer "F.Cu")
-		(net 14)
-	)
-	(segment
-		(start 134.34 58.1)
-		(end 135.14 58.9)
-		(width 0.5)
-		(layer "F.Cu")
-		(net 14)
-	)
-	(segment
-		(start 132.64 58.1)
-		(end 134.34 58.1)
-		(width 0.5)
-		(layer "F.Cu")
-		(net 14)
-	)
-	(segment
-		(start 135.14 58.9)
-		(end 135.14 66.3)
-		(width 0.5)
-		(layer "F.Cu")
-		(net 14)
-	)
-	(segment
-		(start 130.89 58.1)
-		(end 132.64 58.1)
-		(width 0.5)
-		(layer "F.Cu")
-		(net 14)
-	)
-	(via
-		(at 141.84 67.4)
-		(size 0.6)
-		(drill 0.3)
-		(layers "F.Cu" "B.Cu")
-		(net 14)
 	)
 	(segment
@@
 		(width 0.5)
 		(layer "B.Cu")
-		(net 14)
-	)
-	(segment
-		(start 141.84 67.4)
-		(end 142.44 67.4)
-		(width 0.5)
-		(layer "B.Cu")

Commit message: .
Parts:
- moved R2 3.65 mm to (153.0, 74.7)
- moved U2 1.38 mm to (144.8, 73.6)
Routing:
- net 3V3: track 22.0 -> 3.60 mm
- net VUSB: track 13.8 -> 0.00 mm
- net Net-(J2-CC1): track 4.64 -> 0.04 mm
Changed lines of the file:
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@@
 	(footprint "Resistor_SMD:R_1206_3216Metric_Pad1.30x1.75mm_HandSolder"
 		(layer "B.Cu")
-		(at 150.951 71.658 90)
+		(at 153.04 74.65 90)
 		(descr "Resistor SMD 1206 (3216 Metric), square (rectangular) end terminal, IPC_7351 nominal with elongated pad for handsoldering. (Body size source: IPC-SM-782 page 72, https://www.pcb-3d.com/wordpress/wp-content/uploads/ipc-sm-782a_amendment_1_and_2.pdf), generated with kicad-footprint-generator")
 		(tags "resistor handsolder")
@@
 	(footprint "Alexander Footprint Library:AMS1117 SOT-223"
 		(layer "B.Cu")
-		(at 143.458 73.562 -90)
+		(at 144.84 73.6 -90)
 		(descr "module CMS SOT223 4 pins")
 		(tags "CMS SOT")
@@
 	)
 	(segment
-		(start 143.458 70.412)
-		(end 143.458 72.718)
-		(width 0.5)
-		(layer "B.Cu")
-		(net 14)
-	)
-	(segment
-		(start 143.458 72.718)
-		(end 152.44 81.7)
-		(width 0.5)
-		(layer "B.Cu")
-		(net 14)
-	)
-	(segment
-		(start 143.458 68.418)
-		(end 143.458 70.412)
-		(width 0.5)
-		(layer "B.Cu")
-		(net 14)
-	)
-	(segment
 		(start 152.44 81.7)
 		(end 156.04 81.7)
@@
 	)
 	(segment
-		(start 142.44 67.4)
-		(end 143.458 68.418)
-		(width 0.5)
-		(layer "B.Cu")
-		(net 14)
-	)
-	(segment
 		(start 151.7 64.885785)
 		(end 150.5 63.685785)
@@
 	)
 	(segment
-		(start 155.582435 70.135558)
-		(end 150.978558 70.135558)
-		(width 0.2)
-		(layer "B.Cu")
-		(net 21)
-	)
-	(segment
 		(start 150.978558 70.135558)
 		(end 150.951 70.108)
@@
 	)
 	(segment
-		(start 146.778 61.2)
-		(end 150.94 61.2)
-		(width 0.5)
-		(layer "B.Cu")
-		(net 32)
-	)
-	(segment
-		(start 145.758 62.22)
-		(end 146.778 61.2)
-		(width 0.5)
-		(layer "B.Cu")
-		(net 32)
-	)
-	(segment
-		(start 145.758 70.412)
-		(end 145.758 62.22)
-		(width 0.5)
-		(layer "B.Cu")
-		(net 32)
-	)
-	(segment
