File: ESP32-C3_RC-2/esp32-c3_breadboard-adapter.kicad_sch (KiCad schematic)
At the start: 0 parts

Commit message: schematic
Parts:
- added BRD1: ESP32-C3 Breadboard Adapter, Alexander Footprint Library:ESP32-C3_Breadboard-Adapter, symbol Alexander Library:ESP32-C3-Breadboard-USB-C
Connections:
- new net +3V3: BRD1.3V3 (3.3V)
- new net +5VD: BRD1.5V
- new net +9V: BRD1.VIN
- new net GNDD: BRD1.GND
- new net MTR_FRONT_LEFT: BRD1.4 (GPIO6)
- new net MTR_FRONT_LEFT_REV: BRD1.2 (GPIO4_ADC1_CH4)
- new net MTR_FRONT_RIGHT: BRD1.3 (GPIO5_ADC2_CH0)
- new net MTR_FRONT_RIGHT_REV: BRD1.6 (GPIO7)
- new net PROJ_X: BRD1.15 (GPIO1_ADC1_CH1)
- new net PROJ_Y: BRD1.16 (GPIO0_ADC1_CH0)
- no-connect marks 0 -> 1
