File: ESP32-C3_RC-2/breadboard.kicad_sch (KiCad schematic)
At the start: 0 parts

Commit message: schematic
Parts:
- added U1: 74LS125, symbol 74xx:74LS125
Connections:
- new net GNDD: U1.1, U1.10, U1.13, U1.4
- new net LFT_FWD: U1.11
- new net LFT_REV: U1.8
- new net MTR_FRONT_LEFT: U1.12
- new net MTR_FRONT_LEFT_REV: U1.9
- new net MTR_FRONT_RIGHT: U1.2
- new net MTR_FRONT_RIGHT_REV: U1.5
- new net RGT_FWD: U1.3
- new net RGT_REV: U1.6
