File: ClassAB_StereoAmp_SMD/_autosave-Class AB Stereo Amp SMD.kicad_pcb (KiCad board)
At the start: 2 copper layers, 146.5 x 126.8 mm, 80 parts, among them J1 Screw_Terminal_01x02, J2 Barrel_Jack_Switch, J3 AudioJack3, J4 Screw_Terminal_01x04, J6 Conn_Coaxial_x2, Q1 NJVMJB42CT4G, Q2 NJVMJB41CT4G, Q3 NJVMJB42CT4G, Q4 NJVMJB41CT4G, Q5 DMP6180SK3, SW1 SW_SPDT, U1 NE5532, U2 NE5532, U3 NE5532

Commit message: amp
Parts:
- moved TP3 111.0 mm to (148.1, 193.8)
- moved J3 104.3 mm to (153.4, 184.3), turned to 90 degrees
- moved TP4 92.5 mm to (148.4, 174.2)
- moved C5 86.0 mm to (139.7, 173.1), turned to 0 degrees
- moved C7 80.2 mm to (134.9, 188.9), turned to 0 degrees
- moved R10 78.2 mm to (139.7, 168.8), turned to 180 degrees
- moved R9 76.6 mm to (140.2, 161.8)
- moved U3 56.7 mm to (104.3, 175.6), turned to 90 degrees
- moved R5 45.6 mm to (96.2, 187.1), turned to 0 degrees
- moved R6 39.6 mm to (96.3, 182.6), turned to 180 degrees
- moved R7 25.8 mm to (132.9, 162.3), turned to 0 degrees
- moved R3 22.3 mm to (95.5, 168.9)
- moved C4 18.2 mm to (127.5, 162.3), turned to 180 degrees
- moved U1 10.2 mm to (95.0, 175.6), turned to 90 degrees
- moved C6 9.70 mm to (129.2, 188.9)
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Connections:
- RV1 pad 2: Net-(U3A-+) -> Net-(U3B--)
- RV1 pad 5: Net-(U3B-+) -> Net-(U3A--)
- U3 pad 1: RIN2 -> LIN2
- U3 pad 2: RIN2 -> Net-(U3A--)
- U3 pad 3: Net-(U3A-+) -> LIN2
- U3 pad 5: Net-(U3B-+) -> RIN2
- U3 pad 6: LIN2 -> Net-(U3B--)
- U3 pad 7: LIN2 -> RIN2
