File: Production/ESP32-C3-WROOM-Node-Temperature/ESP32-C3-WROOM-Node-Temperature/ESP32-C3-WROOM-Node-Temperature.kicad_pcb (KiCad board)
At the start: 2 copper layers, 65 x 40 mm, 27 parts, among them J1 PWR, J2 Conn_01x02_Socket, J3 Conn_01x02_Socket, J4 I2C, K1 Relay_DPDT_HK19F_HUI, Q1 NPN, SW1 SW_SPDT, U2 AMS1117-3V3, U4 L7805, U5 ESP32-C3 SuperMini

Commit message: .
Parts:
- Q1: footprint Package_TO_SOT_THT:TO-92 -> Package_TO_SOT_THT:TO-92L_HandSolder
- R4: value 10K -> 100
- moved Q1 0.35 mm to (146.2, 76.8)
Routing:
- net /ADC1: track 10.8 -> 11.6 mm
