File: Production/ESP32-C3-WROOM-Node-Temperature/ESP32-C3-WROOM-Node-Temperature/ESP32-C3-WROOM-Node-Temperature.kicad_sch (KiCad schematic)
At the start: 13 parts, among them J2 Conn_01x02_Socket, J3 Conn_01x02_Socket, J4 I2C, K1 Relay_DPDT_HK19F_HUI, Q1 NPN, U5 ESP32-C3 SuperMini

Commit message: .
Parts:
- R4: value 10K -> 100
Changed lines of the file:
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@@
 			)
 		)
-		(property "Value" "10K"
+		(property "Value" "100"
 			(at 57.15 44.4499 0)
 			(effects

Commit message: .
Parts:
- Q1: footprint Package_TO_SOT_THT:TO-92 -> Package_TO_SOT_THT:TO-92L_HandSolder
