File: Audio-Amplifier_TDA2822/Audio-Amplifier_TDA2822.kicad_pcb (KiCad board)
At the start: 2 copper layers, 50 x 50 mm, 28 parts, among them J1 Conn_SPKR_L, J2 Conn_SPKR_L, J3 Conn_01x02_Socket, J4 Conn_01x02_Socket, U1 TDA2822M_2

Commit message: .
Parts:
- moved C1 5.55 mm to (211.5, 94.3)
- moved C7 5.55 mm to (209.5, 105.8)
- moved C8 5.55 mm to (218.0, 87.8)
- moved J1 5.55 mm to (204.5, 105.8)
- moved R1 5.55 mm to (216.5, 106.2)
- moved R3 5.55 mm to (208.0, 87.8)
- moved R4 5.55 mm to (208.0, 83.8)
- moved C3 5.55 mm to (218.5, 83.7)
Changed lines of the file:
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@@
 	(footprint "Capacitor_THT:CP_Radial_D5.0mm_P2.50mm"
 		(layer "F.Cu")
-		(at 212.5 87 -90)
+		(at 218 87.75 -90)
 		(descr "CP, Radial series, Radial, pin pitch=2.50mm, diameter=5mm, height=7mm, Electrolytic Capacitor")
 		(tags "CP Radial series Radial pin pitch 2.50mm diameter 5mm height 7mm Electrolytic Capacitor")
@@
 	(footprint "Capacitor_THT:CP_Radial_D5.0mm_P2.50mm"
 		(layer "F.Cu")
-		(at 213 83 90)
+		(at 218.5 83.705113 90)
 		(descr "CP, Radial series, Radial, pin pitch=2.50mm, diameter=5mm, height=7mm, Electrolytic Capacitor")
 		(tags "CP Radial series Radial pin pitch 2.50mm diameter 5mm height 7mm Electrolytic Capacitor")
@@
 	(footprint "Resistor_THT:R_Axial_DIN0204_L3.6mm_D1.6mm_P5.08mm_Vertical"
 		(layer "F.Cu")
-		(at 202.51 87)
+		(at 208.01 87.75)
 		(descr "Resistor, Axial_DIN0204 series, Axial, Vertical, pin pitch=5.08mm, 0.167W, length*diameter=3.6*1.6mm^2, http://cdn-reichelt.de/documents/datenblatt/B400/1_4W%23YAG.pdf")
 		(tags "Resistor Axial_DIN0204 series Axial Vertical pin pitch 5.08mm 0.167W length 3.6mm diameter 1.6mm")
@@
 	(footprint "Resistor_THT:R_Axial_DIN0204_L3.6mm_D1.6mm_P5.08mm_Vertical"
 		(layer "F.Cu")
-		(at 211 105.49 90)
+		(at 216.5 106.24 90)
 		(descr "Resistor, Axial_DIN0204 series, Axial, Vertical, pin pitch=5.08mm, 0.167W, length*diameter=3.6*1.6mm^2, http://cdn-reichelt.de/documents/datenblatt/B400/1_4W%23YAG.pdf")
 		(tags "Resistor Axial_DIN0204 series Axial Vertical pin pitch 5.08mm 0.167W length 3.6mm diameter 1.6mm")
@@
 	(footprint "Capacitor_THT:CP_Radial_D5.0mm_P2.50mm"
 		(layer "F.Cu")
-		(at 204 105)
+		(at 209.5 105.75)
 		(descr "CP, Radial series, Radial, pin pitch=2.50mm, diameter=5mm, height=7mm, Electrolytic Capacitor")
 		(tags "CP Radial series Radial pin pitch 2.50mm diameter 5mm height 7mm Electrolytic Capacitor")
@@
 	(footprint "Connector_PinHeader_2.54mm:PinHeader_1x02_P2.54mm_Vertical"
 		(layer "F.Cu")
-		(at 199 105 -90)
+		(at 204.5 105.75 -90)
 		(descr "Through hole straight pin header, 1x02, 2.54mm pitch, single row")
 		(tags "Through hole pin header THT 1x02 2.54mm single row")
@@
 	(footprint "Capacitor_THT:CP_Radial_D8.0mm_P5.00mm"
 		(layer "F.Cu")
-		(at 206 93.597349 -90)
+		(at 211.5 94.347349 -90)
 		(descr "CP, Radial series, Radial, pin pitch=5.00mm, diameter=8mm, height=16mm, Electrolytic Capacitor")
 		(tags "CP Radial series Radial pin pitch 5.00mm diameter 8mm height 16mm Electrolytic Capacitor")
@@
 	(footprint "Resistor_THT:R_Axial_DIN0204_L3.6mm_D1.6mm_P5.08mm_Vertical"
 		(layer "F.Cu")
-		(at 202.51 83)
+		(at 208.01 83.75)
 		(descr "Resistor, Axial_DIN0204 series, Axial, Vertical, pin pitch=5.08mm, 0.167W, length*diameter=3.6*1.6mm^2, http://cdn-reichelt.de/documents/datenblatt/B400/1_4W%23YAG.pdf")
 		(tags "Resistor Axial_DIN0204 series Axial Vertical pin pitch 5.08mm 0.167W length 3.6mm diameter 1.6mm")

Commit message: .
Parts:
- J1: value Conn_SPKR_L -> LFT_OUT
- J2: value Conn_SPKR_L -> RGT_OUT
- J3: value Conn_01x02_Socket -> SOUND_IN
- J4: value Conn_01x02_Socket -> PWR; footprint Connector_PinHeader_2.54mm:PinHeader_1x02_P2.54mm_Vertical -> TerminalBlock:TerminalBlock_Altech_AK300-2_P5.00mm
- moved J4 55.6 mm to (233.0, 74.8)

Commit message: .
Connections:
- C1 pad 2: Net-(J1-Pin_1) -> /LFT_OUT
- C12 pad 2: Net-(J2-Pin_1) -> /RGT_OUT
- C14 pad 1: Net-(J2-Pin_1) -> /RGT_OUT
- C7 pad 1: Net-(J1-Pin_1) -> /LFT_OUT
Changed lines of the file:
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@@
 	(net 21 "Net-(VR1-CCW_1)")
 	(net 22 "Net-(VR1-CCW_2)")
+	(net 23 "/LFT_OUT")
+	(net 24 "/RGT_OUT")
 	(footprint "Resistor_THT:R_Axial_DIN0204_L3.6mm_D1.6mm_P5.08mm_Vertical"
 		(layer "F.Cu")
@@
 			(remove_unused_layers no)
 			(roundrect_rratio 0.15625)
-			(net 11 "Net-(J2-Pin_1)")
+			(net 24 "/RGT_OUT")
 			(pintype "passive")
 		)
@@
 			(remove_unused_layers no)
 			(roundrect_rratio 0.15625)
-			(net 6 "Net-(J1-Pin_1)")
+			(net 23 "/LFT_OUT")
 			(pintype "passive")
 		)
@@
 			(layers "*.Cu" "*.Mask")
 			(remove_unused_layers no)
-			(net 6 "Net-(J1-Pin_1)")
+			(net 23 "/LFT_OUT")
 			(pintype "passive")
 		)
@@
 			(layers "*.Cu" "*.Mask")
 			(remove_unused_layers no)
-			(net 11 "Net-(J2-Pin_1)")
+			(net 24 "/RGT_OUT")
 			(pintype "passive")
 		)

Commit message: .
Parts:
- removed J1: LFT_OUT, Connector_PinHeader_2.54mm:PinHeader_1x02_P2.54mm_Vertical
- removed J2: RGT_OUT, Connector_PinHeader_2.54mm:PinHeader_1x02_P2.54mm_Vertical
- added J5: SOUND_OUT, TerminalBlock:TerminalBlock_Altech_AK300-4_P5.00mm, F.Cu at (191.0, 102.0)
- moved C15 19.1 mm to (207.0, 84.5), turned to -90 degrees
- moved C9 13.8 mm to (203.5, 84.5), turned to -90 degrees
- moved R11 9.01 mm to (186.0, 105.5)
- moved C7 7.99 mm to (217.0, 103.0), turned to -90 degrees
- moved C3 5.71 mm to (218.5, 78.0), turned to -90 degrees
- moved C1 5.55 mm to (217.0, 93.6)
- moved R1 5.55 mm to (211.0, 105.5)
- moved R4 5.15 mm to (213.0, 82.5), turned to 90 degrees
- moved R3 3.74 mm to (211.0, 85.5), turned to -90 degrees
- moved C14 3.61 mm to (181.0, 103.0), turned to -90 degrees
- moved C12 3.06 mm to (181.0, 93.6)
- moved C8 2.02 mm to (217.0, 86.0)

Commit message: .
Parts:
- removed J3: SOUND_IN, Connector_PinHeader_2.54mm:PinHeader_1x02_P2.54mm_Vertical
- added J1: AudioJack3, Connector_Audio:Jack_3.5mm_CUI_SJ1-3513N_Horizontal, F.Cu at (221.3, 67.0)
- moved R8 10.7 mm to (181.5, 76.0)
- moved R5 9.62 mm to (186.5, 76.0)
- moved J4 6.93 mm to (236.0, 81.0)
- moved R7 6.71 mm to (205.0, 74.0), turned to 90 degrees
- moved R6 5.66 mm to (205.0, 61.5), turned to -90 degrees
- moved C16 2.24 mm to (198.0, 70.0), turned to -90 degrees
- moved C2 2.24 mm to (198.0, 65.0), turned to 90 degrees

Commit message: .
Parts:
- moved C15 28.8 mm to (234.5, 93.0)
- moved C9 28.8 mm to (231.0, 93.0)
- moved R8 15.1 mm to (196.5, 78.0)
- moved R5 13.6 mm to (200.0, 78.0)
- moved R4 6.49 mm to (206.5, 82.5), turned to 0 degrees
- moved R3 4.73 mm to (206.5, 87.0), turned to 0 degrees
- moved C3 3.91 mm to (216.0, 81.0), turned to 0 degrees
- moved U1 3.19 mm to (194.4, 89.8)
- moved C10 2.24 mm to (180.0, 82.0), turned to 180 degrees
- moved C16 2.24 mm to (200.0, 71.0), turned to 180 degrees
- moved C2 2.24 mm to (200.0, 64.0), turned to 180 degrees
- moved R9 2.24 mm to (189.5, 82.0)
- moved C14 2.00 mm to (179.0, 103.0)
- moved R10 2.00 mm to (189.5, 87.0)
- moved C11 1.12 mm to (179.0, 86.5)
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
Commit message: .
Parts:
- moved C15 30.4 mm to (207.0, 80.0), turned to 180 degrees
- moved C9 29.1 mm to (207.0, 76.5), turned to 180 degrees
- moved C3 21.2 mm to (195.0, 78.0), turned to -90 degrees
- moved J4 19.0 mm to (217.0, 82.0)
- moved R8 15.1 mm to (181.5, 76.0)
- moved R5 10.1 mm to (190.1, 76.0), turned to 180 degrees
- moved R6 8.23 mm to (207.0, 69.5), turned to 90 degrees
- moved R4 6.59 mm to (200.0, 81.5), turned to 90 degrees
- moved R7 5.10 mm to (204.0, 69.5)
- moved U1 3.04 mm to (194.9, 92.8)
- moved J5 0.07 mm to (190.9, 102.0)

Commit message: .
Parts:
- moved C8 8.06 mm to (210.0, 91.0)
- moved R6 5.51 mm to (206.5, 64.0), turned to 180 degrees
- moved C11 5.22 mm to (184.0, 88.0), turned to 180 degrees
- moved R5 4.57 mm to (185.5, 76.0), turned to 0 degrees
- moved R7 2.91 mm to (206.5, 71.0), turned to 180 degrees
- moved C16 2.00 mm to (198.0, 71.0)
- moved C2 2.00 mm to (198.0, 64.0)
- moved C3 1.00 mm to (195.0, 77.0)
- moved R10 0.49 mm to (189.5, 86.5), turned to -90 degrees
Connections:
- R5 pad 1: LFT -> GND
- R5 pad 2: GND -> LFT
Other:
- outline, holes or cut-outs redrawn
