File: ESP32-C3-WROOM-Socket_VeloComputer/ESP32-C3-WROOM-Socket_VeloComputer.kicad_sch (KiCad schematic)
At the start: 29 parts, among them J1 I2C, J3 Reed_Speed_Socket, J4 USB-C_Receptacle_Data_16P_GCT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, J5 Conn_01x02_Socket, J6 Speed_01x02_Pin, J7 Cadense_01x02_Pin, SW1 SW_Push_SMD_6x3.5, SW2 ENABLE, SW3 SW_Reed_Speed, SW4 SW_Reed_Cadence, U1 ESP32-C3-WROOM-02-N4, U2 AMS1117-3V3, U3 74LS14

Commit message: velocomputer
Connections:
- net CADENCE: no longer U3.10
- net GPIO4: no longer U3.4
- net at C4.1, J3.1 (Pin_1), R2.2: no longer U3.1
- net at U3.3: no longer U3.2
- net at C5.1, J5.1 (Pin_1), R3.2: no longer U3.13
- net at U3.12: no longer U3.11

Commit message: velocomputer
Connections:
- net CADENCE: now also U3.10; no longer J2.4
- net GPIO4: no longer U1.3 (IO4)
- net at U3.3: now also C5.1, J5.1 (Pin_1), R3.2
- net at U3.4: now also U3.11
- net SPEED: now reaches U3.12
- net SPEED: now also U1.3 (IO4)
- net at U3.13: now also U3.2
- net at C4.1, J3.1 (Pin_1), R2.2: now also U3.1
- new net GPIO5: J2.4
Other:
- moved on the sheet: U3E, U3F
Changed lines of the file:
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@@
 		)
 	)
-	(label "GPIO5"
-		(at 252.73 138.43 180)
-		(effects
-			(font
-				(size 1.27 1.27)
-			)
-			(justify right bottom)
-		)
-	)
-	(label "GPIO4"
-		(at 175.26 138.43 180)
-		(effects
-			(font
-				(size 1.27 1.27)
-			)
-			(justify right bottom)
-		)
-	)
 	(label "3V3"
 		(at 46.99 90.17 0)
@@
 	(symbol
 		(lib_id "74xx:74LS14")
-		(at 171.45 125.73 0)
-		(unit 2)
-		(exclude_from_sim no)
-		(in_bom yes)
-		(on_board yes)
-		(dnp no)
-		(fields_autoplaced yes)
-		(property "Reference" "U3"
-			(at 171.45 116.84 0)
-			(effects
-				(font
-					(size 1.27 1.27)
-				)
-			)
-		)
-		(property "Value" "74LS14"
-			(at 171.45 119.38 0)
-			(effects
-				(font
-					(size 1.27 1.27)
-				)
-			)
-		)
-		(property "Footprint" "Package_SO:SOIC-14_3.9x8.7mm_P1.27mm"
-			(at 171.45 125.73 0)
-			(effects
-				(font
-					(size 1.27 1.27)
-				)
-				(hide yes)
-			)
-		)
-		(property "Datasheet" "http://www.ti.com/lit/gpn/sn74LS14"
-			(at 171.45 125.73 0)
-			(effects
-				(font
-					(size 1.27 1.27)
-				)
-				(hide yes)
-			)
-		)
-		(property "Description" "Hex inverter schmitt trigger"
-			(at 171.45 125.73 0)
-			(effects
-				(font
-					(size 1.27 1.27)
-				)
-				(hide yes)
-			)
-		)
-		(pin "11"
-		)
-		(pin "4"
-		)
-		(pin "3"
-		)
-		(pin "10"
-		)
-		(pin "13"
-		)
-		(pin "8"
-		)
-		(pin "5"
-		)
-		(pin "2"
-		)
-		(pin "1"
-		)
-		(pin "6"
-		)
-		(pin "9"
-		)
-		(pin "14"
-		)
-		(pin "7"
-		)
-		(pin "12"
-		)
-		(instances
-			(project "ESP32-C3-WROOM-Socket_VeloComputer"
-				(path "/1aed2ed1-0515-43a4-a546-c7b070175ea1"
-					(reference "U3")
-					(unit 2)
-				)
-			)
-		)
-	)
-	(symbol
-		(lib_id "74xx:74LS14")
-		(at 226.06 123.19 0)
+		(at 161.29 138.43 0)
 		(unit 6)
 		(exclude_from_sim no)
@@
 		(fields_autoplaced yes)
 		(property "Reference" "U3"
-			(at 226.06 114.3 0)
+			(at 161.29 129.54 0)
 			(effects
 				(font
@@
 		)
 		(property "Value" "74LS14"
-			(at 226.06 116.84 0)
+			(at 161.29 132.08 0)
 			(effects
 				(font
@@
 		)
 		(property "Footprint" "Package_SO:SOIC-14_3.9x8.7mm_P1.27mm"
-			(at 226.06 123.19 0)
+			(at 161.29 138.43 0)
 			(effects
 				(font
@@
 		)
 		(property "Datasheet" "http://www.ti.com/lit/gpn/sn74LS14"
-			(at 226.06 123.19 0)
+			(at 161.29 138.43 0)
 			(effects
 				(font
@@
 		)
 		(property "Description" "Hex inverter schmitt trigger"
-			(at 226.06 123.19 0)
+			(at 161.29 138.43 0)
 			(effects
 				(font
@@
 	)
 	(symbol
+		(lib_id "74xx:74LS14")
+		(at 146.05 138.43 0)
+		(unit 1)
+		(exclude_from_sim no)
+		(in_bom yes)
+		(on_board yes)
+		(dnp no)
+		(fields_autoplaced yes)
+		(property "Reference" "U3"
+			(at 146.05 129.54 0)
+			(effects
+				(font
+					(size 1.27 1.27)
+				)
+			)
+		)
+		(property "Value" "74LS14"
+			(at 146.05 132.08 0)
+			(effects
+				(font
+					(size 1.27 1.27)
+				)
+			)
+		)
+		(property "Footprint" "Package_SO:SOIC-14_3.9x8.7mm_P1.27mm"
+			(at 146.05 138.43 0)
+			(effects
+				(font
+					(size 1.27 1.27)
+				)
+				(hide yes)
+			)
+		)
+		(property "Datasheet" "http://www.ti.com/lit/gpn/sn74LS14"
+			(at 146.05 138.43 0)
+			(effects
+				(font
+					(size 1.27 1.27)
+				)
+				(hide yes)
+			)
+		)
+		(property "Description" "Hex inverter schmitt trigger"
+			(at 146.05 138.43 0)
+			(effects
+				(font
+					(size 1.27 1.27)
+				)
+				(hide yes)
+			)
+		)
+		(pin "11"
+		)
+		(pin "4"
+		)
+		(pin "3"
+		)
+		(pin "10"
+		)
+		(pin "13"
+		)
+		(pin "8"
+		)
+		(pin "5"
+		)
+		(pin "2"
+		)
+		(pin "1"
+		)
+		(pin "6"
+		)
+		(pin "9"
+		)
+		(pin "14"
+		)
+		(pin "7"
+		)
+		(pin "12"
+		)
+		(instances
+			(project "ESP32-C3-WROOM-Socket_VeloComputer"
+				(path "/1aed2ed1-0515-43a4-a546-c7b070175ea1"
+					(reference "U3")
+					(unit 1)
+				)
+			)
+		)
+	)
+	(symbol
 		(lib_id "Device:R")
 		(at 210.82 130.81 0)
@@
 	(symbol
 		(lib_id "74xx:74LS14")
-		(at 246.38 125.73 0)
+		(at 238.76 138.43 0)
 		(unit 5)
 		(exclude_from_sim no)
@@
 		(fields_autoplaced yes)
 		(property "Reference" "U3"
-			(at 246.38 116.84 0)
+			(at 238.76 129.54 0)
 			(effects
 				(font
@@
 		)
 		(property "Value" "74LS14"
-			(at 246.38 119.38 0)
+			(at 238.76 132.08 0)
 			(effects
 				(font
@@
 		)
 		(property "Footprint" "Package_SO:SOIC-14_3.9x8.7mm_P1.27mm"
-			(at 246.38 125.73 0)
+			(at 238.76 138.43 0)
 			(effects
 				(font
@@
 		)
 		(property "Datasheet" "http://www.ti.com/lit/gpn/sn74LS14"
-			(at 246.38 125.73 0)
+			(at 238.76 138.43 0)
 			(effects
 				(font
@@
 		)
 		(property "Description" "Hex inverter schmitt trigger"
-			(at 246.38 125.73 0)
+			(at 238.76 138.43 0)
 			(effects
 				(font
@@
 	)
 	(symbol
-		(lib_id "74xx:74LS14")
-		(at 148.59 123.19 0)
-		(unit 1)
-		(exclude_from_sim no)
-		(in_bom yes)
-		(on_board yes)
-		(dnp no)
-		(fields_autoplaced yes)
-		(property "Reference" "U3"
-			(at 148.59 114.3 0)
-			(effects
-				(font
-					(size 1.27 1.27)
-				)
-			)
-		)
-		(property "Value" "74LS14"
-			(at 148.59 116.84 0)
-			(effects
-				(font
-					(size 1.27 1.27)
-				)
-			)
-		)
-		(property "Footprint" "Package_SO:SOIC-14_3.9x8.7mm_P1.27mm"
-			(at 148.59 123.19 0)
-			(effects
-				(font
-					(size 1.27 1.27)
-				)
-				(hide yes)
-			)
-		)
-		(property "Datasheet" "http://www.ti.com/lit/gpn/sn74LS14"
-			(at 148.59 123.19 0)
-			(effects
-				(font
-					(size 1.27 1.27)
-				)
-				(hide yes)
-			)
-		)
-		(property "Description" "Hex inverter schmitt trigger"
-			(at 148.59 123.19 0)
-			(effects
-				(font
-					(size 1.27 1.27)
-				)
-				(hide yes)
-			)
-		)
-		(pin "11"
-		)
-		(pin "4"
-		)
-		(pin "3"
-		)
-		(pin "10"
-		)
-		(pin "13"
-		)
-		(pin "8"
-		)
-		(pin "5"
-		)
-		(pin "2"
-		)
-		(pin "1"
-		)
-		(pin "6"
-		)
-		(pin "9"
-		)
-		(pin "14"
-		)
-		(pin "7"
-		)
-		(pin "12"
-		)
-		(instances
-			(project "ESP32-C3-WROOM-Socket_VeloComputer"
-				(path "/1aed2ed1-0515-43a4-a546-c7b070175ea1"
-					(reference "U3")
-					(unit 1)
-				)
-			)
-		)
-	)
-	(symbol
 		(lib_id "power:GND")
 		(at 133.35 149.86 0)
@@
 				)
 			)
+		)
+	)
+	(symbol
+		(lib_id "74xx:74LS14")
+		(at 223.52 138.43 0)
+		(unit 2)
+		(exclude_from_sim no)
+		(in_bom yes)
+		(on_board yes)
+		(dnp no)
+		(fields_autoplaced yes)
+		(property "Reference" "U3"
+			(at 223.52 129.54 0)
+			(effects
+				(font
+					(size 1.27 1.27)
+				)
+			)
+		)
+		(property "Value" "74LS14"
+			(at 223.52 132.08 0)
+			(effects
+				(font
+					(size 1.27 1.27)
+				)
+			)
+		)
+		(property "Footprint" "Package_SO:SOIC-14_3.9x8.7mm_P1.27mm"
+			(at 223.52 138.43 0)
+			(effects
+				(font
+					(size 1.27 1.27)
+				)
+				(hide yes)
+			)
+		)
+		(property "Datasheet" "http://www.ti.com/lit/gpn/sn74LS14"
+			(at 223.52 138.43 0)
+			(effects
+				(font
+					(size 1.27 1.27)
+				)
+				(hide yes)
+			)
+		)
+		(property "Description" "Hex inverter schmitt trigger"
+			(at 223.52 138.43 0)
+			(effects
+				(font
+					(size 1.27 1.27)
+				)
+				(hide yes)
+			)
+		)
+		(pin "11"
+		)
+		(pin "4"
+		)
+		(pin "3"
+		)
+		(pin "10"
+		)
+		(pin "13"
+		)
+		(pin "8"
+		)
+		(pin "5"
+		)
+		(pin "2"
+		)
+		(pin "1"
+		)
+		(pin "6"
+		)
+		(pin "9"
+		)
+		(pin "14"
+		)
+		(pin "7"
+		)
+		(pin "12"
+		)
+		(instances
+			(project "ESP32-C3-WROOM-Socket_VeloComputer"
+				(path "/1aed2ed1-0515-43a4-a546-c7b070175ea1"
+					(reference "U3")
+					(unit 2)
+				)
+			)

Commit message: velocomputer
Parts:
- C2, R8, SW1: now not fitted; now left out of the parts list
Changed lines of the file:
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@@
 		(unit 1)
 		(exclude_from_sim no)
-		(in_bom yes)
+		(in_bom no)
 		(on_board no)
-		(dnp no)
+		(dnp yes)
 		(fields_autoplaced yes)
 		(property "Reference" "C2"
@@
 		(unit 1)
 		(exclude_from_sim no)
-		(in_bom yes)
-		(on_board yes)
-		(dnp no)
+		(in_bom no)
+		(on_board no)
+		(dnp yes)
 		(fields_autoplaced yes)
 		(property "Reference" "R8"
@@
 		(unit 1)
 		(exclude_from_sim no)
-		(in_bom yes)
-		(on_board yes)
-		(dnp no)
+		(in_bom no)
+		(on_board no)
+		(dnp yes)
 		(property "Reference" "SW1"
 			(at 127.762 49.022 0)

Commit message: velocomputer
Connections:
- net CADENCE: now also U3.2; no longer U3.10
- net SPEED: now also U3.4; no longer U3.12
- net at U3.13: no longer U3.2
- net at C5.1, J5.1 (Pin_1), R3.2: no longer U3.3
- net at C4.1, J3.1 (Pin_1), R2.2: no longer U3.1
- net at U3.11: no longer U3.4

Commit message: velocomputer
Connections:
- net CADENCE: now also U3.4; no longer U3.2
- net SPEED: now also U3.6; no longer U3.4
- net at U3.5: now also U3.8
- net at U3.9: now also C4.1, J3.1 (Pin_1), R2.2
- net at C5.1, J5.1 (Pin_1), R3.2: now also U3.11
- net at U3.10: now also U3.3
Other:
- moved on the sheet: U3C, U3D, U3E

Commit message: velocomputer
Parts:
- J2: now in the parts list
- U1: now not fitted; now left out of the parts list
Connections:
- net GPIO4 is gone; now on net SPEED: J2.3
- net GPIO5 is gone; now on net CADENCE: J2.4
- net CADENCE: no longer U1.4 (IO5)
- net SPEED: no longer U1.3 (IO4)
Changed lines of the file:
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@@
 	(wire
 		(pts
-			(xy 222.25 91.44) (xy 223.52 91.44)
+			(xy 205.74 91.44) (xy 223.52 91.44)
 		)
 		(stroke
@@
 	(wire
 		(pts
-			(xy 222.25 93.98) (xy 223.52 93.98)
+			(xy 205.74 93.98) (xy 223.52 93.98)
 		)
 		(stroke
@@
 		)
 	)
+	(label "GPIO4"
+		(at 209.55 91.44 0)
+		(effects
+			(font
+				(size 1.27 1.27)
+			)
+			(justify left bottom)
+		)
+	)
+	(label "GPIO5"
+		(at 209.55 93.98 0)
+		(effects
+			(font
+				(size 1.27 1.27)
+			)
+			(justify left bottom)
+		)
+	)
 	(label "3V3"
 		(at 46.99 90.17 0)
@@
 		)
 	)
-	(global_label "SPEED"
-		(shape input)
-		(at 203.2 48.26 180)
-		(fields_autoplaced yes)
-		(effects
-			(font
-				(size 1.27 1.27)
-			)
-			(justify right)
-		)
-		(property "Intersheetrefs" "${INTERSHEET_REFS}"
-			(at 194.1673 48.26 0)
-			(effects
-				(font
-					(size 1.27 1.27)
-				)
-				(justify right)
-				(hide yes)
-			)
-		)
-	)
 	(global_label "CADENCE"
 		(shape output)
@@
 		)
 	)
-	(global_label "GPIO5"
+	(global_label "UART-RX"
 		(shape input)
-		(at 222.25 93.98 180)
+		(at 203.2 60.96 180)
 		(fields_autoplaced yes)
 		(effects
@@
 		)
 		(property "Intersheetrefs" "${INTERSHEET_REFS}"
-			(at 213.58 93.98 0)
+			(at 191.5062 60.96 0)
 			(effects
 				(font
@@
 		)
 	)
-	(global_label "UART-RX"
+	(global_label "SPEED"
 		(shape input)
-		(at 203.2 60.96 180)
+		(at 205.74 91.44 180)
 		(fields_autoplaced yes)
 		(effects
@@
 		)
 		(property "Intersheetrefs" "${INTERSHEET_REFS}"
-			(at 191.5062 60.96 0)
+			(at 196.7073 91.44 0)
 			(effects
 				(font
@@
 		)
 	)
-	(global_label "CADENCE"
-		(shape input)
-		(at 203.2 50.8 180)
-		(fields_autoplaced yes)
-		(effects
-			(font
-				(size 1.27 1.27)
-			)
-			(justify right)
-		)
-		(property "Intersheetrefs" "${INTERSHEET_REFS}"
-			(at 191.6877 50.8 0)
-			(effects
-				(font
-					(size 1.27 1.27)
-				)
-				(justify right)
-				(hide yes)
-			)
-		)
-	)
 	(global_label "USB_D-"
 		(shape bidirectional)
@@
 		)
 	)
+	(global_label "CADENCE"
+		(shape input)
+		(at 205.74 93.98 180)
+		(fields_autoplaced yes)
+		(effects
+			(font
+				(size 1.27 1.27)
+			)
+			(justify right)
+		)
+		(property "Intersheetrefs" "${INTERSHEET_REFS}"
+			(at 194.2277 93.98 0)
+			(effects
+				(font
+					(size 1.27 1.27)
+				)
+				(justify right)
+				(hide yes)
+			)
+		)
+	)
 	(global_label "3V3"
 		(shape input)
@@
 		)
 	)
-	(global_label "GPIO4"
-		(shape input)
-		(at 222.25 91.44 180)
-		(fields_autoplaced yes)
-		(effects
-			(font
-				(size 1.27 1.27)
-			)
-			(justify right)
-		)
-		(property "Intersheetrefs" "${INTERSHEET_REFS}"
-			(at 213.58 91.44 0)
-			(effects
-				(font
-					(size 1.27 1.27)
-				)
-				(justify right)
-				(hide yes)
-			)
-		)
-	)
 	(global_label "GND"
 		(shape input)
@@
 		(unit 1)
 		(exclude_from_sim no)
-		(in_bom no)
-		(on_board no)
+		(in_bom yes)
+		(on_board yes)
 		(dnp no)
 		(fields_autoplaced yes)
@@
 		(unit 1)
 		(exclude_from_sim no)
-		(in_bom yes)
-		(on_board yes)
-		(dnp no)
+		(in_bom no)
+		(on_board no)
+		(dnp yes)
 		(fields_autoplaced yes)
 		(property "Reference" "U1"

Commit message: velocomputer
Parts:
- J2: footprint Alexander Footprint Library:Conn_ESP32-C3-WROOM-02 -> Alexander Footprints:ESP32-C3-WROOM-02-Socket-board
- R1, R7, SW2: now not fitted; now left out of the parts list
Connections:
- net SPEED: now also U3.2; no longer U3.6
- net at U3.5: no longer U3.8
- net at C4.1, J3.1 (Pin_1), R2.2: now also U3.13; no longer U3.9
- net at U3.1: now also U3.12
Other:
- moved on the sheet: U3A, U3F

Commit message: velocomputer
Connections:
- net CADENCE: now also U3.6; no longer U3.4
- net SPEED: now also U3.4; no longer U3.2
- net at U3.12: now also U3.3; no longer U3.1
- net at U3.5: now also U3.10
Other:
- moved on the sheet: U3C
Changed lines of the file:
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@@
+	)
+	(symbol
+		(lib_id "Switch:SW_Reed")
+		(at 233.68 157.48 0)
+		(unit 1)
+		(exclude_from_sim no)
+		(in_bom no)
+		(on_board no)
+		(dnp no)
+		(fields_autoplaced yes)
+		(property "Reference" "SW4"
+			(at 233.68 151.13 0)
+			(effects
+				(font
+					(size 1.27 1.27)
+				)
+			)
+		)
+		(property "Value" "SW_Reed_Cadence"
+			(at 233.68 153.67 0)
+			(effects
+				(font
+					(size 1.27 1.27)
+				)
+			)
+		)
+		(property "Footprint" "Connector_PinSocket_2.54mm:PinSocket_1x02_P2.54mm_Vertical"
+			(at 233.68 157.48 0)
+			(effects
+				(font
+					(size 1.27 1.27)
+				)
+				(hide yes)
+			)
+		)
+		(property "Datasheet" "~"
+			(at 233.68 157.48 0)
+			(effects
+				(font
+					(size 1.27 1.27)
+				)
+				(hide yes)
+			)
+		)
+		(property "Description" "reed switch"
+			(at 233.68 157.48 0)
+			(effects
+				(font
+					(size 1.27 1.27)
+				)
+				(hide yes)
+			)
+		)
+		(pin "1"
+		)
+		(pin "2"
+		)
+		(instances
+			(project "ESP32-C3-WROOM-Socket_VeloComputer"
+				(path "/1aed2ed1-0515-43a4-a546-c7b070175ea1"
+					(reference "SW4")
+					(unit 1)
+				)
+			)
+		)
 	)
 	(symbol
 		(lib_id "74xx:74LS14")
 		(at 161.29 138.43 0)
-		(unit 1)
+		(unit 2)
 		(exclude_from_sim no)
 		(in_bom yes)
@@
 				(path "/1aed2ed1-0515-43a4-a546-c7b070175ea1"
 					(reference "U3")
-					(unit 1)
-				)
-			)
-		)
-	)
-	(symbol
-		(lib_id "Switch:SW_Reed")
-		(at 233.68 157.48 0)
-		(unit 1)
-		(exclude_from_sim no)
-		(in_bom no)
-		(on_board no)
-		(dnp no)
-		(fields_autoplaced yes)
-		(property "Reference" "SW4"
-			(at 233.68 151.13 0)
-			(effects
-				(font
-					(size 1.27 1.27)
-				)
-			)
-		)
-		(property "Value" "SW_Reed_Cadence"
-			(at 233.68 153.67 0)
-			(effects
-				(font
-					(size 1.27 1.27)
-				)
-			)
-		)
-		(property "Footprint" "Connector_PinSocket_2.54mm:PinSocket_1x02_P2.54mm_Vertical"
-			(at 233.68 157.48 0)
-			(effects
-				(font
-					(size 1.27 1.27)
-				)
-				(hide yes)
-			)
-		)
-		(property "Datasheet" "~"
-			(at 233.68 157.48 0)
-			(effects
-				(font
-					(size 1.27 1.27)
-				)
-				(hide yes)
-			)
-		)
-		(property "Description" "reed switch"
-			(at 233.68 157.48 0)
-			(effects
-				(font
-					(size 1.27 1.27)
-				)
-				(hide yes)
-			)
-		)
-		(pin "1"
-		)
-		(pin "2"
-		)
-		(instances
-			(project "ESP32-C3-WROOM-Socket_VeloComputer"
-				(path "/1aed2ed1-0515-43a4-a546-c7b070175ea1"
-					(reference "SW4")
-					(unit 1)
+					(unit 2)
 				)
 			)
@@
 	(symbol
 		(lib_id "74xx:74LS14")
-		(at 335.28 143.51 0)
+		(at 238.76 138.43 0)
 		(unit 3)
 		(exclude_from_sim no)
@@
 		(fields_autoplaced yes)
 		(property "Reference" "U3"
-			(at 335.28 134.62 0)
+			(at 238.76 129.54 0)
 			(effects
 				(font
@@
 		)
 		(property "Value" "74LS14"
-			(at 335.28 137.16 0)
+			(at 238.76 132.08 0)
 			(effects
 				(font
@@
 		)
 		(property "Footprint" "Package_SO:SOIC-14_3.9x8.7mm_P1.27mm"
-			(at 335.28 143.51 0)
+			(at 238.76 138.43 0)
 			(effects
 				(font
@@
 		)
 		(property "Datasheet" "http://www.ti.com/lit/gpn/sn74LS14"
-			(at 335.28 143.51 0)
+			(at 238.76 138.43 0)
 			(effects
 				(font
@@
 		)
 		(property "Description" "Hex inverter schmitt trigger"
-			(at 335.28 143.51 0)
+			(at 238.76 138.43 0)
 			(effects
 				(font
@@
 					(reference "U3")
 					(unit 3)
-				)
-			)
-		)
-	)
-	(symbol
-		(lib_id "74xx:74LS14")
-		(at 238.76 138.43 0)
-		(unit 2)
-		(exclude_from_sim no)
-		(in_bom yes)
-		(on_board yes)
-		(dnp no)
-		(fields_autoplaced yes)
-		(property "Reference" "U3"
-			(at 238.76 129.54 0)
-			(effects
-				(font
-					(size 1.27 1.27)
-				)
-			)
-		)
-		(property "Value" "74LS14"
-			(at 238.76 132.08 0)
-			(effects
-				(font
-					(size 1.27 1.27)
-				)
-			)
-		)
-		(property "Footprint" "Package_SO:SOIC-14_3.9x8.7mm_P1.27mm"
-			(at 238.76 138.43 0)
-			(effects
-				(font
-					(size 1.27 1.27)
-				)
-				(hide yes)
-			)
-		)
-		(property "Datasheet" "http://www.ti.com/lit/gpn/sn74LS14"
-			(at 238.76 138.43 0)
-			(effects
-				(font
-					(size 1.27 1.27)
-				)
-				(hide yes)
-			)
-		)
-		(property "Description" "Hex inverter schmitt trigger"
-			(at 238.76 138.43 0)
-			(effects
-				(font
-					(size 1.27 1.27)
-				)
-				(hide yes)
-			)
-		)
-		(pin "11"
-		)
-		(pin "4"
-		)
-		(pin "3"
-		)
-		(pin "10"
-		)
-		(pin "13"
-		)
-		(pin "8"
-		)
-		(pin "5"
-		)
-		(pin "2"
-		)
-		(pin "1"
-		)
-		(pin "6"
-		)
-		(pin "9"
-		)
-		(pin "14"
-		)
-		(pin "7"
-		)
-		(pin "12"
-		)
-		(instances
-			(project "ESP32-C3-WROOM-Socket_VeloComputer"
-				(path "/1aed2ed1-0515-43a4-a546-c7b070175ea1"
-					(reference "U3")
-					(unit 2)
 				)
 			)
@@
 					(unit 1)
 				)
+			)
+		)
+	)
+	(symbol
+		(lib_id "74xx:74LS14")
+		(at 317.5 132.08 0)
+		(unit 1)
+		(exclude_from_sim no)
+		(in_bom yes)
+		(on_board yes)
+		(dnp no)
+		(fields_autoplaced yes)
+		(property "Reference" "U3"
+			(at 317.5 123.19 0)
+			(effects
+				(font
+					(size 1.27 1.27)
+				)
+			)
+		)
+		(property "Value" "74LS14"
+			(at 317.5 125.73 0)
+			(effects
+				(font
+					(size 1.27 1.27)
+				)
+			)
+		)
+		(property "Footprint" "Package_SO:SOIC-14_3.9x8.7mm_P1.27mm"
+			(at 317.5 132.08 0)
+			(effects
+				(font
+					(size 1.27 1.27)
+				)
+				(hide yes)
+			)
+		)
+		(property "Datasheet" "http://www.ti.com/lit/gpn/sn74LS14"
+			(at 317.5 132.08 0)
+			(effects
+				(font
+					(size 1.27 1.27)
+				)
+				(hide yes)
+			)
+		)
+		(property "Description" "Hex inverter schmitt trigger"
+			(at 317.5 132.08 0)
+			(effects
+				(font
+					(size 1.27 1.27)
+				)
+				(hide yes)
+			)
+		)
+		(pin "11"
+		)
+		(pin "4"
+		)
+		(pin "3"
+		)
+		(pin "10"
+		)
+		(pin "13"
+		)
+		(pin "8"
+		)
+		(pin "5"
+		)
+		(pin "2"
+		)
+		(pin "1"
+		)
+		(pin "6"
+		)
+		(pin "9"
+		)
+		(pin "14"
+		)
+		(pin "7"
+		)
+		(pin "12"
+		)
+		(instances
+			(project "ESP32-C3-WROOM-Socket_VeloComputer"
+				(path "/1aed2ed1-0515-43a4-a546-c7b070175ea1"
+					(reference "U3")
+					(unit 1)
+				)
